File: kicad/usb_emulator.sch (KiCad schematic (older format))
At the start: 48 parts, among them U202 TPD2E001DRLR, U204 TPS73033DBVR

Commit message: datasheets added, I'll remove usb interface completely
I've decided to remove the jtag and isolation interface completely
maybe next I'll add some rs485 isolation interfase for debug, but for
now, it's not neccesary 'cose I'd use a jtag isolated interface
exclusively for that
Parts:
- U201: value ~ -> 93LC46C
- U203: value ~ -> DS_FT2232H.
Connections:
- net labels added: EMU_GND, ~EMU_TRST~
- net labels removed: EMU_TRSTn, GND
Changed lines of the file:
@@
 $Descr B 17000 11000
 encoding utf-8
-Sheet 2 7
+Sheet 7 7
 Title "usb_emulator"
 Date "25 10 2019"
@@
 U 1 1 5DB39162
 P 5400 9100
-F 0 "#EMU_GND0201" H 5400 9240 20  0000 C CNN
-F 1 "GND" H 5400 9210 30  0000 C CNN
+F 0 "#EMU_GND0201" H 5405 8951 20  0000 C CNN
+F 1 "EMU_GND" H 5405 8899 30  0000 C CNN
 F 2 "" H 5400 9100 70  0000 C CNN
 F 3 "" H 5400 9100 70  0000 C CNN
@@
 U 1 1 5DB39161
 P 6800 9700
-F 0 "#EMU_GND_0208" H 6805 9835 20  0000 C CNN
-F 1 "GND" H 6805 9783 30  0000 C CNN
+F 0 "#EMU_GND_0208" H 6805 9551 20  0000 C CNN
+F 1 "EMU_GND" H 6805 9499 30  0000 C CNN
 F 2 "" H 6800 9700 70  0000 C CNN
 F 3 "" H 6800 9700 70  0000 C CNN
@@
 U 1 1 5DB39160
 P 7400 9700
-F 0 "#EMU_GND_0209" H 7323 9693 20  0000 R CNN
-F 1 "GND" H 7323 9641 30  0000 R CNN
+F 0 "#EMU_GND_0209" H 7405 9551 20  0000 C CNN
+F 1 "EMU_GND" H 7405 9499 30  0000 C CNN
 F 2 "" H 7400 9700 70  0000 C CNN
 F 3 "" H 7400 9700 70  0000 C CNN
@@
 U 1 1 5DB3915F
 P 9100 9700
-F 0 "#EMU_GND_0210" H 9188 9693 20  0000 L CNN
-F 1 "GND" H 9188 9641 30  0000 L CNN
+F 0 "#EMU_GND_0210" H 9105 9551 20  0000 C CNN
+F 1 "EMU_GND" H 9105 9499 30  0000 C CNN
 F 2 "" H 9100 9700 70  0000 C CNN
 F 3 "" H 9100 9700 70  0000 C CNN
@@
 P 3200 6300
 F 0 "#EMU_GND_0203" H 3123 6293 20  0000 R CNN
-F 1 "GND" H 3123 6241 30  0000 R CNN
+F 1 "EMU_GND" H 3123 6241 30  0000 R CNN
 F 2 "" H 3200 6300 70  0000 C CNN
 F 3 "" H 3200 6300 70  0000 C CNN
@@
 U 1 1 5DB39158
 P 2800 9400
-F 0 "#EMU_GND_0202" H 2800 9540 20  0000 C CNN
-F 1 "GND" H 2800 9510 30  0000 C CNN
+F 0 "#EMU_GND_0202" H 2805 9251 20  0000 C CNN
+F 1 "EMU_GND" H 2805 9199 30  0000 C CNN
 F 2 "" H 2800 9400 70  0000 C CNN
 F 3 "" H 2800 9400 70  0000 C CNN
@@
 P 1800 8800
 F 0 "#EMU_GND_0201" H 1805 8651 20  0000 C CNN
-F 1 "GND" H 1805 8599 30  0000 C CNN
+F 1 "EMU_GND" H 1805 8599 30  0000 C CNN
 F 2 "" H 1800 8800 70  0000 C CNN
 F 3 "" H 1800 8800 70  0000 C CNN
@@
 U 1 1 5DB3914F
 P 10500 1000
-F 0 "#EMU_5V0_0202" H 10588 1067 20  0000 L CNN
-F 1 "EMU_5V0" H 10588 1015 30  0000 L CNN
+F 0 "#EMU_5V0_0202" H 10515 1209 20  0000 C CNN
+F 1 "EMU_5V0" H 10515 1157 30  0000 C CNN
 F 2 "" H 10500 1000 70  0000 C CNN
 F 3 "" H 10500 1000 70  0000 C CNN
@@
 U 1 1 5DB3914D
 P 13300 2400
-F 0 "#EMU_GND_0216" H 13388 2393 20  0000 L CNN
-F 1 "GND" H 13388 2341 30  0000 L CNN
+F 0 "#EMU_GND_0216" H 13305 2251 20  0000 C CNN
+F 1 "EMU_GND" H 13305 2199 30  0000 C CNN
 F 2 "" H 13300 2400 70  0000 C CNN
 F 3 "" H 13300 2400 70  0000 C CNN
@@
 U 1 1 5DB3914C
 P 9200 4100
-F 0 "#EMU_GND_0211" H 9288 4093 20  0000 L CNN
-F 1 "GND" H 9288 4041 30  0000 L CNN
+F 0 "#EMU_GND_0211" H 9205 3951 20  0000 C CNN
+F 1 "EMU_GND" H 9205 3899 30  0000 C CNN
 F 2 "" H 9200 4100 70  0000 C CNN
 F 3 "" H 9200 4100 70  0000 C CNN
@@
 U 1 1 5DB3914B
 P 6600 8500
-F 0 "#EMU_GND_0207" H 6522 8493 20  0000 R CNN
-F 1 "GND" H 6522 8441 30  0000 R CNN
+F 0 "#EMU_GND_0207" H 6605 8351 20  0000 C CNN
+F 1 "EMU_GND" H 6605 8299 30  0000 C CNN
 F 2 "" H 6600 8500 70  0000 C CNN
 F 3 "" H 6600 8500 70  0000 C CNN
@@
 U 1 1 5DB39148
 P 10600 6200
-F 0 "#EMU_GND_0212" H 10688 6193 20  0000 L CNN
-F 1 "GND" H 10688 6141 30  0000 L CNN
+F 0 "#EMU_GND_0212" H 10605 6051 20  0000 C CNN
+F 1 "EMU_GND" H 10605 5999 30  0000 C CNN
 F 2 "" H 10600 6200 70  0000 C CNN
 F 3 "" H 10600 6200 70  0000 C CNN
@@
 U 1 1 5DB39147
 P 10800 8600
-F 0 "#EMU_GND_0214" H 10888 8593 20  0000 L CNN
-F 1 "GND" H 10888 8541 30  0000 L CNN
+F 0 "#EMU_GND_0214" H 10805 8451 20  0000 C CNN
+F 1 "EMU_GND" H 10805 8399 30  0000 C CNN
 F 2 "" H 10800 8600 70  0000 C CNN
 F 3 "" H 10800 8600 70  0000 C CNN
@@
 U 1 1 5DB39145
 P 4300 5000
-F 0 "#EMU_GND_0206" H 4222 4993 20  0000 R CNN
-F 1 "GND" H 4222 4941 30  0000 R CNN
+F 0 "#EMU_GND_0206" H 4305 4851 20  0000 C CNN
+F 1 "EMU_GND" H 4305 4799 30  0000 C CNN
 F 2 "" H 4300 5000 70  0000 C CNN
 F 3 "" H 4300 5000 70  0000 C CNN
@@
 U 1 1 5DB39144
 P 3400 4800
-F 0 "#EMU_GND_0204" H 3322 4793 20  0000 R CNN
-F 1 "GND" H 3322 4741 30  0000 R CNN
+F 0 "#EMU_GND_0204" H 3405 4651 20  0000 C CNN
+F 1 "EMU_GND" H 3405 4599 30  0000 C CNN
 F 2 "" H 3400 4800 70  0000 C CNN
 F 3 "" H 3400 4800 70  0000 C CNN
@@
 U 1 1 5DB39143
 P 4200 3000
-F 0 "#EMU_GND_0205" H 4122 2993 20  0000 R CNN
-F 1 "GND" H 4122 2941 30  0000 R CNN
+F 0 "#EMU_GND_0205" H 4205 2851 20  0000 C CNN
+F 1 "EMU_GND" H 4205 2799 30  0000 C CNN
 F 2 "" H 4200 3000 70  0000 C CNN
 F 3 "" H 4200 3000 70  0000 C CNN
@@
 U 1 1 5DB39142
 P 14200 2400
-F 0 "#EMU_GND_0217" H 14288 2393 20  0000 L CNN
-F 1 "GND" H 14288 2341 30  0000 L CNN
+F 0 "#EMU_GND_0217" H 14205 2251 20  0000 C CNN
+F 1 "EMU_GND" H 14205 2199 30  0000 C CNN
 F 2 "" H 14200 2400 70  0000 C CNN
 F 3 "" H 14200 2400 70  0000 C CNN
@@
 U 1 1 5DB39141
 P 11400 2400
-F 0 "#EMU_GND_0215" H 11488 2393 20  0000 L CNN
-F 1 "GND" H 11488 2341 30  0000 L CNN
+F 0 "#EMU_GND_0215" H 11405 2251 20  0000 C CNN
+F 1 "EMU_GND" H 11405 2199 30  0000 C CNN
 F 2 "" H 11400 2400 70  0000 C CNN
 F 3 "" H 11400 2400 70  0000 C CNN
@@
 U 1 1 5DB39140
 P 10700 2400
-F 0 "#EMU_GND_0213" H 10788 2393 20  0000 L CNN
-F 1 "GND" H 10788 2341 30  0000 L CNN
+F 0 "#EMU_GND_0213" H 10705 2251 20  0000 C CNN
+F 1 "EMU_GND" H 10705 2199 30  0000 C CNN
 F 2 "" H 10700 2400 70  0000 C CNN
 F 3 "" H 10700 2400 70  0000 C CNN
@@
 U 1 1 5DB3913F
 P 14800 2800
-F 0 "#EMU_GND_0218" H 14888 2793 20  0000 L CNN
-F 1 "GND" H 14888 2741 30  0000 L CNN
+F 0 "#EMU_GND_0218" H 14805 2651 20  0000 C CNN
+F 1 "EMU_GND" H 14805 2599 30  0000 C CNN
 F 2 "" H 14800 2800 70  0000 C CNN
 F 3 "" H 14800 2800 70  0000 C CNN
@@
 U 1 1 5DB3913E
 P 15900 1200
-F 0 "#EMU_GND_0219" H 15988 1193 20  0000 L CNN
-F 1 "GND" H 15988 1141 30  0000 L CNN
+F 0 "#EMU_GND_0219" H 15905 1051 20  0000 C CNN
+F 1 "EMU_GND" H 15905 999 30  0000 C CNN
 F 2 "" H 15900 1200 70  0000 C CNN
 F 3 "" H 15900 1200 70  0000 C CNN
@@
 Wire Wire Line
 	11000 5200 9000 5200
-Text Label 10600 4800 0    60   ~ 0
-EMU_TCK
-Text Label 10600 4900 0    60   ~ 0
-EMU_TDI
-Text Label 10600 5000 0    60   ~ 0
-EMU_TDO
-Text Label 10600 5100 0    60   ~ 0
-EMU_TMS
-Text Label 10600 5200 0    60   ~ 0
-EMU_TRSTn
 Text Label 9500 6600 0    60   ~ 0
 EMU_SCI-RX
@@
 U 1 1 5DB3913C
 P 8200 7200
-F 0 "U203" H 8200 9883 60  0000 C CNN
-F 1 "~" H 8200 7200 50  0001 C CNN
+F 0 "U203" H 8200 9973 60  0000 C CNN
+F 1 "DS_FT2232H." H 8200 9875 50  0000 C CNN
 F 2 "" H 8200 7200 50  0001 C CNN
-F 3 "" H 8200 7200 50  0001 C CNN
+F 3 "../doc/datasheets/DS_FT2232H.pdf" H 8200 7200 50  0001 C CNN
 	1    8200 7200
 	1    0    0    -1
@@
 F 1 "TPD2E001DRLR" H 4400 6600 60  0000 R TNN
 F 2 "" H 4400 6600 60  0000 C CNN
-F 3 "" H 4400 6600 60  0000 C CNN
+F 3 "../doc/datasheets/tpd2e001.pdf" H 4400 6600 60  0001 C CNN
 	1    4000 6200
 	-1   0    0    1
@@
 P 3500 8900
 F 0 "U201" H 3900 9300 60  0000 R BNN
-F 1 "~" H 3500 8900 50  0001 C CNN
+F 1 "93LC46C" H 3500 8900 50  0001 C CNN
 F 2 "" H 3500 8900 50  0001 C CNN
-F 3 "" H 3500 8900 50  0001 C CNN
+F 3 "../doc/datasheets/93LC46C.pdf" H 3500 8900 50  0001 C CNN
 	1    3500 8900
 	-1   0    0    -1
@@
 F 1 "TPS73033DBVR" H 12500 1983 60  0000 C CNN
 F 2 "" H 12000 1000 60  0000 C CNN
-F 3 "" H 12000 1000 60  0000 C CNN
+F 3 "../doc/datasheets/tps730.pdf" H 12000 1000 60  0001 C CNN
 	1    12500 1500
 	1    0    0    -1
@@
 P 10300 1000
 F 0 "#FLG0202" H 10300 1075 50  0001 C CNN
-F 1 "PWR_FLAG" H 10300 1174 50  0000 C CNN
+F 1 "PWR_FLAG" H 10150 1150 50  0000 C CNN
 F 2 "" H 10300 1000 50  0001 C CNN
 F 3 "~" H 10300 1000 50  0001 C CNN
@@
 P 13450 1000
 F 0 "#FLG0203" H 13450 1075 50  0001 C CNN
-F 1 "PWR_FLAG" H 13450 1174 50  0000 C CNN
+F 1 "PWR_FLAG" H 13350 1200 50  0000 C CNN
 F 2 "" H 13450 1000 50  0001 C CNN
 F 3 "~" H 13450 1000 50  0001 C CNN
@@
 U 1 1 5DB3914E
 P 13700 1000
-F 0 "#EMU_3V3_0209" H 13788 1067 20  0000 L CNN
-F 1 "EMU_3V3" H 13788 1015 30  0000 L CNN
+F 0 "#EMU_3V3_0209" H 13715 1209 20  0000 C CNN
+F 1 "EMU_3V3" H 13715 1157 30  0000 C CNN
 F 2 "" H 13700 1000 70  0000 C CNN
 F 3 "" H 13700 1000 70  0000 C CNN
@@
 	1    0    0    -1
 $EndComp
+Text HLabel 11000 4800 2    50   Input ~ 0
+EMU_TCK
+Text HLabel 11000 4900 2    50   Input ~ 0
+EMU_TDI
+Text HLabel 11000 5000 2    50   Input ~ 0
+EMU_TDO
+Text HLabel 11000 5100 2    50   Input ~ 0
+EMU_TMS
+Text HLabel 11000 5200 2    50   Input ~ 0
+~EMU_TRST~
+Text HLabel 12200 4800 2    50   Input ~ 0
+EMU_3V3
+Text HLabel 12200 4900 2    50   Input ~ 0
+EMU_5V0
+Text HLabel 12200 5000 2    50   Input ~ 0
+EMU_GND
+$Comp
+L servo:EMU_5V0 #EMU_5V0_?
+U 1 1 5DD6DA83
+P 12050 4900
+F 0 "#EMU_5V0_?" V 12095 5028 20  0000 L CNN
+F 1 "EMU_5V0" V 12043 5028 30  0000 L CNN
+F 2 "" H 12050 4900 70  0000 C CNN
+F 3 "" H 12050 4900 70  0000 C CNN
+	1    12050 4900
+	0    -1   -1   0
+$EndComp
+$Comp
+L servo:EMU_3V3 #EMU_3V3_?
+U 1 1 5DDA1F5E
+P 12050 4800
+F 0 "#EMU_3V3_?" V 12050 5050 20  0000 C CNN
+F 1 "EMU_3V3" V 12100 5050 30  0000 C CNN
+F 2 "" H 12050 4800 70  0000 C CNN
+F 3 "" H 12050 4800 70  0000 C CNN
+	1    12050 4800
+	0    -1   -1   0
+$EndComp
+$Comp
+L power:GND #EMU_GND_?
+U 1 1 5DDD6477
+P 12050 5000
+F 0 "#EMU_GND_?" V 12025 4872 20  0000 R CNN
+F 1 "EMU_GND" V 12077 4872 30  0000 R CNN
+F 2 "" H 12050 5000 70  0000 C CNN
+F 3 "" H 12050 5000 70  0000 C CNN
+	1    12050 5000
+	0    1    1    0
+$EndComp
 $EndSCHEMATC
