File: kicad/ac_input.sch (KiCad schematic (older format))
At the start: 25 parts

Commit message: ok, it's enough cleaned to mix with power interface
I think it's time to mix with power interfaces.. It's enough cleaned
Parts:
- added F?: Fuse, symbol Device:Fuse
- added FL?: EMI_Filter_CommonMode, symbol Device:EMI_Filter_CommonMode
- added J?: Conn_01x03, symbol Connector_Generic:Conn_01x03
- added TP? (x4): ~, symbol servo:CMP-0078143-2
Connections:
- net labels added: ACL, ACN, Earth, IN_1V2C, IN_3V3C
- net labels removed: 1V2C, 3V3C, VDD_1V2, VDD_3V3
- wire segments 69 -> 88
Other:
- moved on the sheet: C?, D?, R?
