File: kicad/iso_gipo.sch (KiCad schematic (older format))
At the start: 18 parts

Commit message: I've added LCD UI interfase, EQEP and finish ENDAT
I think I have almos all the interfases ready, I'm begining the
verigication process and then the part definig
Connections:
- net 15VH: now also R?.1, R?.1, R?.1, R?.1
- net GNDH: now reaches J?.1 (Pin_1), J?.2 (Pin_2), J?.3 (Pin_3), J?.4 (Pin_4), R?.1, R?.1, R?.1, R?.1, U?.5 (COM), U?.6 (COM)
- net GNDH: no longer R?.1, R?.1, R?.1, R?.1
- net at R?.2: now also J?.16 (Pin_16); no longer J?.9 (Pin_9)
- net at R?.2: now also J?.15 (Pin_15); no longer J?.10 (Pin_10)
- net at R?.2: now also J?.14 (Pin_14); no longer J?.11 (Pin_11)
- net at R?.2: now also J?.13 (Pin_13); no longer J?.12 (Pin_12)
- net at R?.2: now also J?.12 (Pin_12); no longer J?.13 (Pin_13)
- net at R?.2: now also J?.11 (Pin_11); no longer J?.14 (Pin_14)
- net at R?.2: now also J?.10 (Pin_10); no longer J?.15 (Pin_15)
- net at R?.2: now also J?.9 (Pin_9); no longer J?.16 (Pin_16)
- removed net MCU_GPIO??: U?.11 (B8), U?.12 (B7), U?.13 (B6), U?.14 (B5), U?.17 (B4), U?.18 (B3), U?.19 (B2), U?.20 (B1)
- new net ISO_GPI1: U?.20 (B1)
- new net ISO_GPI2: U?.19 (B2)
- new net ISO_GPI3: U?.18 (B3)
- new net ISO_GPI4: U?.17 (B4)
- new net ISO_GPI5: U?.14 (B5)
- new net ISO_GPI6: U?.13 (B6)
- new net ISO_GPI7: U?.12 (B7)
- new net ISO_GPI8: U?.11 (B8)
Other:
- note added: "4 Active Hi / to inyect\n4 Active LO / to source"
- note added: "active HI"
- note added: "active Low\n"
- note removed: "if the switch is active\n use these pairs and inyect\n power supply from switch\n in any polarity with respect COM"
- note removed: "if the switch is passive\n use these pairs"
- moved on the sheet: J?, R?, U?

Commit message: remove isolation GPIO's and replace it by free pins at IGBT
I remove completely the isolated inputs pins cause I've 8 pins free at
IGBT isolated interfase, so I leave 4 for outpus and 4 for inputs with
one isolated stage, the same as the previous isolated GPIO sheet..
I've improved the DBG sheet and some other details,. I'm ready to make
some electrical checks and fchoose the parts codes and footprints.. go
for it!
Changed lines of the file:
@@
 Sheet 15 19
 Title "clk"
-Date "25 10 2019"
+Date "2020-01-09"
 Rev "1.0"
 Comp "dci"
@@
 U 1 1 5E75F6F8
 P 8150 4050
-F 0 "#PWR?" H 8155 4257 20  0000 C CNN
+F 0 "#PWR?" H 8155 4257 20  0001 C CNN
 F 1 "3V3" H 8155 4207 28  0000 C CNN
 F 2 "" H 8150 4050 50  0001 C CNN
