File: kicad/sd_interface.sch (KiCad schematic (older format))
At the start: 4 parts

Commit message: remove isolation GPIO's and replace it by free pins at IGBT
I remove completely the isolated inputs pins cause I've 8 pins free at
IGBT isolated interfase, so I leave 4 for outpus and 4 for inputs with
one isolated stage, the same as the previous isolated GPIO sheet..
I've improved the DBG sheet and some other details,. I'm ready to make
some electrical checks and fchoose the parts codes and footprints.. go
for it!
Other:
- note added: "It's intended for power board circuitery to supply all the signals to\n control board. The control board will use the SD filter to aquire the\n data. All the power part will be at power board.\n\nPWM clk output to powerboard and then come back again to maintain\n delays with resect to SD data channels. On power board you have to\n respect traces length between clk and data"
- note removed: "It's intended for power board circuitery to supply all the signals to\n control board. The control board will use the SD filter to aquire the\n data. All the power part will be at power board."
- note removed: "PWM clk output to powerboard and then come back again to maintain\n delays with resect to SD data channels. On power board you have to\n respect traces length between clk and data"
Changed lines of the file:
@@
 $Descr A3 16535 11693
 encoding utf-8
-Sheet 19 19
+Sheet 19 18
 Title "Shunt Sigma Delta isolated"
-Date "25 10 2019"
+Date "2020-01-09"
 Rev "1.0"
 Comp "dci"
@@
 Comment4 ""
 $EndDescr
-Text Notes 5400 1700 0    197  ~ 39
+Text Notes 5450 1350 0    197  ~ 39
 Isolated sigma delta ADC
 Text GLabel 9800 2800 2    50   Input ~ 0
@@
 U 1 1 5ECC6BF2
 P 5000 2500
-F 0 "#PWR?" H 5005 2707 20  0000 C CNN
+F 0 "#PWR?" H 5005 2707 20  0001 C CNN
 F 1 "3V3" H 5005 2657 28  0000 C CNN
 F 2 "" H 5000 2500 50  0001 C CNN
@@
 U 1 1 5EEE31B5
 P 9750 2500
-F 0 "#PWR?" H 9755 2707 20  0000 C CNN
+F 0 "#PWR?" H 9755 2707 20  0001 C CNN
 F 1 "3V3" H 9755 2657 28  0000 C CNN
 F 2 "" H 9750 2500 50  0001 C CNN
@@
 Wire Wire Line
 	9650 3300 9800 3300
-Text Notes 6400 3950 0    39   ~ 0
-PWM clk output to powerboard and then come back again to maintain\n delays with resect to SD data channels. On power board you have to\n respect traces length between clk and data
 Text Notes 5450 2300 0    20   ~ 4
 Choose a package pin-to-pin compatible with\nTI ISO7761. But SIlabs cost halt the price as TI
 Text Notes 8600 2350 0    20   ~ 4
 Choose a package pin-to-pin compatible with\nTI ISO7761. But SIlabs cost halt the price as TI
-Text Notes 6200 2000 0    39   ~ 0
-It's intended for power board circuitery to supply all the signals to\n control board. The control board will use the SD filter to aquire the\n data. All the power part will be at power board.
+Text Notes 6400 1900 0    39   ~ 0
+It's intended for power board circuitery to supply all the signals to\n control board. The control board will use the SD filter to aquire the\n data. All the power part will be at power board.\n\nPWM clk output to powerboard and then come back again to maintain\n delays with resect to SD data channels. On power board you have to\n respect traces length between clk and data
 $EndSCHEMATC

Commit message: added 4 push buttons and more gpios on LCD connector
just to have more UI options. With those I'd manage graphics LCD plus 4
buttons, and charaveter LCD. or the embedded EVE graphic LCD
Parts:
- gave numbers to parts that had none: 4
Connections:
- net 3V3H renamed 5VH
Other:
- note added: "It's intended for power board circuitery to supply all the signals to\n control board. The control board will use the SD filter to aquire the\n data. All the power part will be at power board.\n\nPWM clk output to powerboard and then come back again to maintain\n delays with resect to SD data channels. On power board you have to\n respect traces length between clk and data\n\nI use 5VH on power s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"
- note removed: "It's intended for power board circuitery to supply all the signals to\n control board. The control board will use the SD filter to aquire the\n data. All the power part will be at power board.\n\nPWM clk output to powerboard and then come back again to maintain\n delays with resect to SD data channels. On power board you have to\n respect traces length between clk and data"
Changed lines of the file:
@@
 $Descr A3 16535 11693
 encoding utf-8
-Sheet 19 18
+Sheet 18 18
 Title "Shunt Sigma Delta isolated"
 Date "2020-01-09"
@@
 SD_A_CLK1
 $Comp
-L servo:GND #PWR?
+L servo:GND #PWR0299
 U 1 1 5E4779CD
 P 5050 3450
-F 0 "#PWR?" H 5050 3200 30  0001 C CNN
+F 0 "#PWR0299" H 5050 3200 30  0001 C CNN
 F 1 "GND" H 5050 3292 30  0000 C CNN
 F 2 "" H 5050 3450 50  0001 C CNN
@@
 SD_B_CLK1
 $Comp
-L servo:SI8661BD U?
+L servo:SI8661BD U1801
 U 1 1 5ECC54DD
 P 5800 3000
-F 0 "U?" H 5800 3589 60  0000 C CNN
+F 0 "U1801" H 5800 3589 60  0000 C CNN
 F 1 "SI8661BD" H 5800 3483 60  0000 C CNN
 F 2 "" H 5200 3300 60  0000 C CNN
@@
 	5050 3400 5050 3450
 $Comp
-L servo:3V3 #PWR?
+L servo:3V3 #PWR0300
 U 1 1 5ECC6BF2
 P 5000 2500
-F 0 "#PWR?" H 5005 2707 20  0001 C CNN
+F 0 "#PWR0300" H 5005 2707 20  0001 C CNN
 F 1 "3V3" H 5005 2657 28  0000 C CNN
 F 2 "" H 5000 2500 50  0001 C CNN
@@
 	5100 3100 4950 3100
 $Comp
-L servo:3V3H #PWR?
-U 1 1 5ECC7A5F
-P 6600 2550
-AR Path="/5DDE8C5E/5ECC7A5F" Ref="#PWR?"  Part="1"
-AR Path="/5EC40F3C/5ECC7A5F" Ref="#PWR?"  Part="1"
-F 0 "#PWR?" H 6600 2350 20  0001 C CNN
-F 1 "3V3H" H 6605 2707 28  0000 C CNN
-F 2 "" H 6600 2550 50  0001 C CNN
-F 3 "" H 6600 2550 50  0001 C CNN
-	1    6600 2550
-	1    0    0    -1
-$EndComp
-Wire Wire Line
-	6600 2550 6600 2700
-Wire Wire Line
-	6600 2700 6500 2700
-$Comp
 L servo:GNDH #PWR?
 U 1 1 5ECC8031
 P 6600 3450
 AR Path="/5DDE8C5E/5ECC8031" Ref="#PWR?"  Part="1"
-AR Path="/5EC40F3C/5ECC8031" Ref="#PWR?"  Part="1"
-F 0 "#PWR?" H 6600 3200 30  0001 C CNN
+AR Path="/5EC40F3C/5ECC8031" Ref="#PWR0302"  Part="1"
+F 0 "#PWR0302" H 6600 3200 30  0001 C CNN
 F 1 "GNDH" H 6600 3292 30  0000 C CNN
 F 2 "" H 6600 3450 50  0001 C CNN
@@
 	6900 2800 6500 2800
 $Comp
-L Connector:Screw_Terminal_01x06 J?
+L Connector:Screw_Terminal_01x06 J1801
 U 1 1 5EEE0A60
 P 7100 3000
-F 0 "J?" H 7180 2946 50  0000 L CNN
+F 0 "J1801" H 7180 2946 50  0000 L CNN
 F 1 "Screw_Terminal_01x06" H 7180 2901 50  0001 L CNN
 F 2 "" H 7100 3000 50  0001 C CNN
@@
 	6900 3300 6500 3300
 $Comp
-L servo:GND #PWR?
+L servo:GND #PWR0303
 U 1 1 5EEE31A4
 P 9700 3450
-F 0 "#PWR?" H 9700 3200 30  0001 C CNN
+F 0 "#PWR0303" H 9700 3200 30  0001 C CNN
 F 1 "GND" H 9700 3292 30  0000 C CNN
 F 2 "" H 9700 3450 50  0001 C CNN
@@
 PWM4SD_CLK
 $Comp
-L servo:SI8661BD U?
+L servo:SI8661BD U1802
 U 1 1 5EEE31AB
 P 8950 3000
-F 0 "U?" H 8950 3589 60  0000 C CNN
+F 0 "U1802" H 8950 3589 60  0000 C CNN
 F 1 "SI8661BD" H 8950 3483 60  0000 C CNN
 F 2 "" H 8350 3300 60  0000 C CNN
@@
 	9700 3400 9700 3450
 $Comp
-L servo:3V3 #PWR?
+L servo:3V3 #PWR0304
 U 1 1 5EEE31B5
 P 9750 2500
-F 0 "#PWR?" H 9755 2707 20  0001 C CNN
+F 0 "#PWR0304" H 9755 2707 20  0001 C CNN
 F 1 "3V3" H 9755 2657 28  0000 C CNN
 F 2 "" H 9750 2500 50  0001 C CNN
@@
 	9650 3100 9800 3100
 $Comp
-L servo:3V3H #PWR?
-U 1 1 5EEE31C6
-P 8150 2550
-AR Path="/5DDE8C5E/5EEE31C6" Ref="#PWR?"  Part="1"
-AR Path="/5EC40F3C/5EEE31C6" Ref="#PWR?"  Part="1"
-F 0 "#PWR?" H 8150 2350 20  0001 C CNN
-F 1 "3V3H" H 8155 2707 28  0000 C CNN
-F 2 "" H 8150 2550 50  0001 C CNN
-F 3 "" H 8150 2550 50  0001 C CNN
-	1    8150 2550
-	-1   0    0    -1
-$EndComp
-Wire Wire Line
-	8150 2550 8150 2700
-Wire Wire Line
-	8150 2700 8250 2700
-$Comp
 L servo:GNDH #PWR?
 U 1 1 5EEE31CE
 P 8150 3450
 AR Path="/5DDE8C5E/5EEE31CE" Ref="#PWR?"  Part="1"
-AR Path="/5EC40F3C/5EEE31CE" Ref="#PWR?"  Part="1"
-F 0 "#PWR?" H 8150 3200 30  0001 C CNN
+AR Path="/5EC40F3C/5EEE31CE" Ref="#PWR0306"  Part="1"
+F 0 "#PWR0306" H 8150 3200 30  0001 C CNN
 F 1 "GNDH" H 8150 3292 30  0000 C CNN
 F 2 "" H 8150 3450 50  0001 C CNN
@@
 	7850 2800 8250 2800
 $Comp
-L Connector:Screw_Terminal_01x06 J?
+L Connector:Screw_Terminal_01x06 J1802
 U 1 1 5EEE31D7
 P 7650 3000
-F 0 "J?" H 7570 3325 50  0000 C CNN
+F 0 "J1802" H 7570 3325 50  0000 C CNN
 F 1 "Screw_Terminal_01x06" H 7730 2901 50  0001 L CNN
 F 2 "" H 7650 3000 50  0001 C CNN
@@
 Text Notes 8600 2350 0    20   ~ 4
 Choose a package pin-to-pin compatible with\nTI ISO7761. But SIlabs cost halt the price as TI
-Text Notes 6400 1900 0    39   ~ 0
-It's intended for power board circuitery to supply all the signals to\n control board. The control board will use the SD filter to aquire the\n data. All the power part will be at power board.\n\nPWM clk output to powerboard and then come back again to maintain\n delays with resect to SD data channels. On power board you have to\n respect traces length between clk and data
+Text Notes 7050 1800 0    20   ~ 0
+It's intended for power board circuitery to supply all the signals to\n control board. The control board will use the SD filter to aquire the\n data. All the power part will be at power board.\n\nPWM clk output to powerboard and then come back again to maintain\n delays with resect to SD data channels. On power board you have to\n respect traces length between clk and data\n\nI use 5VH on power side to be less prone to noise error on the way on\n connection the two boards (and I've decided to not supply 3v3H too)\n\n
+$Comp
+L servo:5VH #PWR0235
+U 1 1 5EF378C8
+P 7350 2550
+F 0 "#PWR0235" H 7350 2350 20  0001 C CNN
+F 1 "5VH" H 7355 2707 28  0000 C CNN
+F 2 "" H 7350 2550 50  0001 C CNN
+F 3 "" H 7350 2550 50  0001 C CNN
+	1    7350 2550
+	1    0    0    -1
+$EndComp
+Wire Wire Line
+	6500 2700 7350 2700
+Wire Wire Line
+	7350 2550 7350 2700
+Connection ~ 7350 2700
+Wire Wire Line
+	7350 2700 8250 2700
 $EndSCHEMATC

Commit message: begin PCB!! it's amess but IT IS
Parts:
- J1801, J1802: footprint (none) -> Connector_PinHeader_2.54mm:PinHeader_1x06_P2.54mm_Vertical
- U1801, U1802: footprint (none) -> Package_SO:SOIC-16W_7.5x10.3mm_P1.27mm
Changed lines of the file:
@@
 Comment4 ""
 $EndDescr
-Text Notes 5450 1350 0    197  ~ 39
+Text Notes 5200 1500 0    197  ~ 39
 Isolated sigma delta ADC
 Text GLabel 9800 2800 2    50   Input ~ 0
@@
 F 0 "U1801" H 5800 3589 60  0000 C CNN
 F 1 "SI8661BD" H 5800 3483 60  0000 C CNN
-F 2 "" H 5200 3300 60  0000 C CNN
+F 2 "Package_SO:SOIC-16W_7.5x10.3mm_P1.27mm" H 5200 3300 60  0001 C CNN
 F 3 "../doc/datasheets/Si8660.pdf" H 5700 3600 60  0001 C CNN
 	1    5800 3000
@@
 F 0 "J1801" H 7180 2946 50  0000 L CNN
 F 1 "Screw_Terminal_01x06" H 7180 2901 50  0001 L CNN
-F 2 "" H 7100 3000 50  0001 C CNN
+F 2 "Connector_PinHeader_2.54mm:PinHeader_1x06_P2.54mm_Vertical" H 7100 3000 50  0001 C CNN
 F 3 "~" H 7100 3000 50  0001 C CNN
 	1    7100 3000
@@
 F 0 "U1802" H 8950 3589 60  0000 C CNN
 F 1 "SI8661BD" H 8950 3483 60  0000 C CNN
-F 2 "" H 8350 3300 60  0000 C CNN
+F 2 "Package_SO:SOIC-16W_7.5x10.3mm_P1.27mm" H 8350 3300 60  0001 C CNN
 F 3 "../doc/datasheets/Si8660.pdf" H 8850 3600 60  0001 C CNN
 	1    8950 3000
@@
 F 0 "J1802" H 7570 3325 50  0000 C CNN
 F 1 "Screw_Terminal_01x06" H 7730 2901 50  0001 L CNN
-F 2 "" H 7650 3000 50  0001 C CNN
+F 2 "Connector_PinHeader_2.54mm:PinHeader_1x06_P2.54mm_Vertical" H 7650 3000 50  0001 C CNN
 F 3 "~" H 7650 3000 50  0001 C CNN
 	1    7650 3000
@@
 Text Notes 8600 2350 0    20   ~ 4
 Choose a package pin-to-pin compatible with\nTI ISO7761. But SIlabs cost halt the price as TI
-Text Notes 7050 1800 0    20   ~ 0
+Text Notes 6800 1950 0    20   ~ 0
 It's intended for power board circuitery to supply all the signals to\n control board. The control board will use the SD filter to aquire the\n data. All the power part will be at power board.\n\nPWM clk output to powerboard and then come back again to maintain\n delays with resect to SD data channels. On power board you have to\n respect traces length between clk and data\n\nI use 5VH on power side to be less prone to noise error on the way on\n connection the two boards (and I've decided to not supply 3v3H too)\n\n
 $Comp
