File: kicad/_autosave-servo.kicad_pcb (KiCad board)
At the start: 2 copper layers, 600 parts, among them J1001 tblock, J1002 tblock, J1101 tblock, J1102 tblock, J1201 tblock, J1301 tblock, J1501 NHD-4.3-480272FT-CTXL-T, J1502 Conn_01x02, J1601 tblock, J1602 tblock, J1603 tblock, J1604 tblock, J1605 tblock, J1606 tblock, J1607 tblock, J1608 tblock, J1701 Screw_Terminal_01x03, J1702 Screw_Terminal_01x03, J1801 Conn_02x10_Odd_Even, J1802 Conn_02x10_Odd_Even, J1803 Conn_02x10_Odd_Even, J201 8P8C, J401 8P8C, J402 8P8C, J601 Conn_02x05_Counter_Clockwise, J602 Conn_01x02, J701 tBlock, J702 tBlock, J703 tBlock, SW1501 SW_Push, SW1502 SW_Push, SW1503 SW_Push, SW1504 SW_Push, U1001 ADM2483, U1002 ADM2483, U1003 ADM2483, U1004 ADM2483, U1101 SI8662BD, U1102 SI8662BD, U1201 ADM2483, U1301 ISO1050, U1501 PAM8301, U1601 LXS6-NPS, U1602 LXS6-NPS, U1603 LXS6-NPS, U1604 LXS6-NPS, U1605 LXS6-NPS, U1606 LXS6-NPS, U1607 LXS6-NPS, U1608 LXS6-NPS, U1701 AMC1311B, U1702 AMC1311B, U1703 RFM-0505S, U1704 RFM-0505S, U1901 SI8661BD, U1902 SI8661BD, U201 DP83822, U301 TMS320F28388DZWTS, U401 CAT24C16WI, U402 DP83822, U403 DP83822, U601 SN74ALVC244PW, U602 M25PX32-VMW, U701 R-78E5.0-1.0, U702 R-78E3.3-1.0, U703 R-78E5.0-1.0, U704 AP2114H-1.2TRG1, U705 AP2114H-1.2TRG1, U706 R-78E5.0-1.0, U801 SI8660BD, U802 SI8662BD, U803 SN74LVC2G17DBVR, U804 SN74LVC2G17DBVR, U805 SN74LVC2G17DBVR, U806 SN74LVC2G17DBVR, U807 SN74LVC2G17DBVR, U808 SN74LVC2G17DBVR, U809 SN74LVC2G17DBVR, U810 SN74LVC2G17DBVR, U811 SN74LVC2G17DBVR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

Commit message: passed all footprint, preliminarly.. and taken a pic
I've passed all 3d models, and make a pic of that, it's the first
impresion, but it need's more indeed reviews
Parts:
- removed D201, D403, D404, D405, D406: blue, servo:LED_0603_1608Metric
- added PS701: IRM-15-12, servo:Converter_ACDC_MeanWell_IRM-20-xx_THT, F.Cu at (257.2, 148.8)
- added PS702: IRM-15-12, servo:Converter_ACDC_MeanWell_IRM-20-xx_THT, F.Cu at (257.2, 176.8)
- C428, C429, C432, C433: value 0.1uF -> 1uF
- J1001, J1002: footprint TerminalBlock_RND:TerminalBlock_RND_205-00291_1x06_P5.08mm_Horizontal -> Connector_Phoenix_MSTB:PhoenixContact_MSTBA_2,5_6-G-5,08_1x06_P5.08mm_Horizontal
- J1101, J1102: footprint TerminalBlock_RND:TerminalBlock_RND_205-00293_1x08_P5.08mm_Horizontal -> Connector_Phoenix_MSTB:PhoenixContact_MSTBA_2,5_8-G-5,08_1x08_P5.08mm_Horizontal
- J1301: footprint TerminalBlock_RND:TerminalBlock_RND_205-00289_1x04_P5.08mm_Horizontal -> Connector_Phoenix_MSTB:PhoenixContact_MSTBA_2,5_4-G-5,08_1x04_P5.08mm_Horizontal
- J1701: footprint TerminalBlock_RND:TerminalBlock_RND_205-00288_1x03_P5.08mm_Horizontal -> Connector_Phoenix_MSTB:PhoenixContact_MSTBVA_2,5_3-G-5,08_1x03_P5.08mm_Vertical
- J1702: footprint TerminalBlock_RND:TerminalBlock_RND_205-00277_1x03_P5.00mm_Vertical -> Connector_Phoenix_MSTB:PhoenixContact_MSTBVA_2,5_3-G-5,08_1x03_P5.08mm_Vertical
- J1801, J1802, J1803: value Conn_02x10_Odd_Even -> NHD-4.3-480272FT-CTXL-T; footprint Connector_PinSocket_2.54mm:PinSocket_2x10_P2.54mm_Vertical_SMD -> Connector_IDC:IDC-Header_2x10_P2.54mm_Vertical
- J201, J401, J402: value 8P8C -> RJHSE-5384; footprint servo:RJ45_Amphenol_54602-x08_Horizontal -> Connector_RJ:RJ45_Amphenol_RJHSE538X
- R436, R439: value 2.2k -> 0e(dnp)
- R441, R443: value 470 -> 75e
- R445, R446: value 75e -> 470
- SW1501, SW1502, SW1503, SW1504: footprint Button_Switch_SMD:SW_SPST_B3S-1000 -> Button_Switch_SMD:SW_SPST_PTS645
- moved J1301 99.1 mm to (140.7, 101.3)
- moved J1605 59.1 mm to (100.0, 34.8)
- moved J1602 29.2 mm to (152.0, 32.0)
- moved J701 14.4 mm to (276.7, 75.6)
- moved J1607 10.2 mm to (139.7, 50.6)
Connections:
- R207 pad 2: Net-(D201-Pad1) -> Net-(J201-Pad11)
- R209 pad 2: Net-(D201-Pad2) -> Net-(J201-Pad12)
- R434 pad 1: Net-(R434-Pad1) -> 3V3
- R434 pad 2: 3V3 -> Net-(R434-Pad2)
- R439 pad 1: Net-(R434-Pad1) -> Net-(R434-Pad2)
- R441 pad 1: 3V3 -> Net-(R441-Pad1)
- R441 pad 2: Net-(D403-Pad2) -> Net-(C434-Pad2)
- R442 pad 1: 3V3 -> Net-(J402-Pad9)
- R442 pad 2: Net-(D404-Pad2) -> ECAT1_RJ_LED0
- R443 pad 1: 3V3 -> Net-(R443-Pad1)
- R443 pad 2: Net-(D405-Pad2) -> Net-(C434-Pad2)
- R444 pad 2: Net-(D406-Pad2) -> Net-(J401-Pad12)
- R445 pad 1: Net-(C434-Pad2) -> Net-(J401-Pad9)
- R445 pad 2: Net-(R445-Pad2) -> ECAT0_RJ_LED1
- R446 pad 1: Net-(C434-Pad2) -> 3V3
- R446 pad 2: Net-(R446-Pad2) -> Net-(J402-Pad12)
- R447 pad 1: Net-(C435-Pad2) -> Net-(R447-Pad1)
- R447 pad 2: Net-(R447-Pad2) -> Net-(C435-Pad2)
- R448 pad 1: Net-(C435-Pad2) -> Net-(R448-Pad1)
- R448 pad 2: Net-(R448-Pad2) -> Net-(C435-Pad2)
- TR401 pad 10: Net-(R445-Pad2) -> Net-(R441-Pad1)
- TR401 pad 15: Net-(R446-Pad2) -> Net-(R443-Pad1)
- TR402 pad 10: Net-(R447-Pad2) -> Net-(R447-Pad1)
- TR402 pad 15: Net-(R448-Pad2) -> Net-(R448-Pad1)
- U201 pad 17: Net-(D201-Pad1) -> Net-(J201-Pad11)
- U403 pad 17: Net-(R434-Pad1) -> Net-(R434-Pad2)
