File: kicad/can.sch (KiCad schematic (older format))
At the start: 6 parts, among them J1301 Screw_Terminal_01x05, U1301 ISO1050

Commit message: begin PCB!! it's amess but IT IS
Parts:
- C1301, C1302: footprint (none) -> Capacitor_SMD:C_0603_1608Metric
- R1301, R1302: footprint (none) -> Resistor_SMD:R_0603_1608Metric
Changed lines of the file:
@@
 F 0 "R1301" V 6353 2800 60  0000 R CNN
 F 1 "1k" V 6247 2800 60  0000 R CNN
-F 2 "" H 6300 2850 60  0000 C CNN
+F 2 "Resistor_SMD:R_0603_1608Metric" H 6300 2850 60  0000 C CNN
 F 3 "" H 6300 2850 60  0000 C CNN
 	1    6300 2850
@@
 F 0 "C1302" V 5847 2410 60  0000 L CNN
 F 1 "100nF" V 5953 2410 60  0000 L CNN
-F 2 "" H 5850 2300 60  0000 C CNN
+F 2 "Capacitor_SMD:C_0603_1608Metric" H 5850 2300 60  0000 C CNN
 F 3 "" H 5850 2300 60  0000 C CNN
 	1    5850 2300
@@
 F 0 "C1301" V 3847 2191 60  0000 R CNN
 F 1 "100nF" V 3953 2191 60  0000 R CNN
-F 2 "" H 3850 2300 60  0000 C CNN
+F 2 "Capacitor_SMD:C_0603_1608Metric" H 3850 2300 60  0000 C CNN
 F 3 "" H 3850 2300 60  0000 C CNN
 	1    3850 2300
@@
 F 0 "R1302" H 7350 2900 60  0000 C CNN
 F 1 "1e" H 7350 3000 60  0000 C CNN
-F 2 "" H 7350 3100 60  0000 C CNN
+F 2 "Resistor_SMD:R_0603_1608Metric" H 7350 3100 60  0000 C CNN
 F 3 "" H 7350 3100 60  0000 C CNN
 	1    7350 3100

Commit message: I've passed all footprin to layout BUT...
I've passed all, first glance... I need to confirm in details a lot of
things. The objetive for these is to have an aproximation of the size
I'll need to make the board.. then I choose the final detailed footprint
Parts:
- removed J1301: Screw_Terminal_01x05, symbol Connector:Screw_Terminal_01x05
- added J1301: tblock, TerminalBlock_RND:TerminalBlock_RND_205-00289_1x04_P5.08mm_Horizontal, symbol servo:Screw_Terminal_01x04
- added JP1301: jumper, Jumper:SolderJumper-3_P1.3mm_Open_RoundedPad1.0x1.5mm, symbol servo:Jumper_3_Bridged12
- added R1303: 1k, Resistor_SMD:R_0603_1608Metric, symbol servo:Resistor
- C1301, C1302: footprint Capacitor_SMD:C_0603_1608Metric -> servo:C_0603_1608Metric
- R1302: value 1e -> 1k
- U1301: footprint Package_SO:SOIC-16W_7.5x10.3mm_P1.27mm -> Package_SO:SSO-8_6.7x9.8mm_P2.54mm_Clearance8mm
Connections:
- net 15VH: now also JP1301.3 (B); no longer R1302.2
- net 5VH: now also R1302.1, JP1301.1 (A)
- net GNDH: now also J1301.4 (Pin_4), R1303.2
- net at U1301.6 (CANL): now also R1301.2, J1301.3 (Pin_3), R1303.1; no longer R1301.1
- net at U1301.7 (CANH): now also R1301.1, R1302.2, J1301.2 (Pin_2); no longer R1301.2
- new net: J1301.1 (Pin_1), JP1301.2 (C)
Other:
- note added: "A simple CAN driver. It also could be used as a RS485 driver in his \nspeed.. the minimum for CAN is 40kbos, so in RS485 at 9600 could be\n fine"
- note removed: "Could be used by isolated: \n485, 1-wire bus, general IO pin"
- note removed: "to use as a fuse \nor protection"
- moved on the sheet: C1301, C1302

Commit message: changing single row terminal block to double row
I've changed to double row all the connectors, RJ45 and terminal blocks,
I saves spaces and also make it more intuitive related to user
interface..lets go
Parts:
- J1301: footprint TerminalBlock_RND:TerminalBlock_RND_205-00289_1x04_P5.08mm_Horizontal -> Connector_Phoenix_MSTB:PhoenixContact_MSTBA_2,5_4-G-5,08_1x04_P5.08mm_Horizontal
Changed lines of the file:
@@
 F 0 "J1301" H 7280 2792 50  0000 L CNN
 F 1 "tblock" H 7280 2701 50  0000 L CNN
-F 2 "TerminalBlock_RND:TerminalBlock_RND_205-00289_1x04_P5.08mm_Horizontal" H 7200 2800 50  0001 C CNN
+F 2 "Connector_Phoenix_MSTB:PhoenixContact_MSTBA_2,5_4-G-5,08_1x04_P5.08mm_Horizontal" H 7200 2800 50  0001 C CNN
 F 3 "~" H 7200 2800 50  0001 C CNN
 	1    7200 2800
