File: kicad/servo.kicad_pcb (KiCad board)
At the start: 2 copper layers, 600 parts, among them J1001 tblock, J1002 tblock, J1101 tblock, J1102 tblock, J1201 tblock, J1301 tblock, J1501 NHD-4.3-480272FT-CTXL-T, J1502 Conn_01x02, J1601 tblock, J1602 tblock, J1603 tblock, J1604 tblock, J1605 tblock, J1606 tblock, J1607 tblock, J1608 tblock, J1701 Screw_Terminal_01x03, J1702 Screw_Terminal_01x03, J1801 Conn_02x10_Odd_Even, J1802 Conn_02x10_Odd_Even, J1803 Conn_02x10_Odd_Even, J201 8P8C, J401 8P8C, J402 8P8C, J601 Conn_02x05_Counter_Clockwise, J602 Conn_01x02, J701 tBlock, J702 tBlock, J703 tBlock, SW1501 SW_Push, SW1502 SW_Push, SW1503 SW_Push, SW1504 SW_Push, U1001 ADM2483, U1002 ADM2483, U1003 ADM2483, U1004 ADM2483, U1101 SI8662BD, U1102 SI8662BD, U1201 ADM2483, U1301 ISO1050, U1501 PAM8301, U1601 LXS6-NPS, U1602 LXS6-NPS, U1603 LXS6-NPS, U1604 LXS6-NPS, U1605 LXS6-NPS, U1606 LXS6-NPS, U1607 LXS6-NPS, U1608 LXS6-NPS, U1701 AMC1311B, U1702 AMC1311B, U1703 RFM-0505S, U1704 RFM-0505S, U1901 SI8661BD, U1902 SI8661BD, U201 DP83822, U301 TMS320F28388DZWTS, U401 CAT24C16WI, U402 DP83822, U403 DP83822, U601 SN74ALVC244PW, U602 M25PX32-VMW, U701 R-78E5.0-1.0, U702 R-78E3.3-1.0, U703 R-78E5.0-1.0, U704 AP2114H-1.2TRG1, U705 AP2114H-1.2TRG1, U706 R-78E5.0-1.0, U801 SI8660BD, U802 SI8662BD, U803 SN74LVC2G17DBVR, U804 SN74LVC2G17DBVR, U805 SN74LVC2G17DBVR, U806 SN74LVC2G17DBVR, U807 SN74LVC2G17DBVR, U808 SN74LVC2G17DBVR, U809 SN74LVC2G17DBVR, U810 SN74LVC2G17DBVR, U811 SN74LVC2G17DBVR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

Commit message: changing single row terminal block to double row
I've changed to double row all the connectors, RJ45 and terminal blocks,
I saves spaces and also make it more intuitive related to user
interface..lets go
Parts:
- removed C1301, C1302, C1618, C1622, C1623, C1624, C1701, C1702, C1703, C1704, C1707, C1708, C1709, C1710: 100nF, servo:C_0603_1608Metric
- removed C1611, C1612, C1613, C1614, C1615, C1616, C1617, C1619, C1620, C1621, C1901, C1902, C1903, C1904, C1905, C1906, C1907, C1908, C1909, C1910, C1911, C1912: 100pF, servo:C_0603_1608Metric
- removed C1705, C1706: 330p, servo:C_0603_1608Metric
- removed C217, C434, C435: 4700pF, servo:C_0603_1608Metric
- removed D1501, D1502: red@2mA, servo:LED_0603_1608Metric
- removed D201, D403, D404, D405, D406: blue, servo:LED_0603_1608Metric
- removed J1002: tblock, TerminalBlock_RND:TerminalBlock_RND_205-00291_1x06_P5.08mm_Horizontal
- removed J1102: tblock, TerminalBlock_RND:TerminalBlock_RND_205-00293_1x08_P5.08mm_Horizontal
- removed J1301: tblock, TerminalBlock_RND:TerminalBlock_RND_205-00289_1x04_P5.08mm_Horizontal
- removed J1603, J1604, J1605, J1606, J1607, J1608: tblock, Connector_Phoenix_MSTB:PhoenixContact_MSTBA_2,5_2-G-5,08_1x02_P5.08mm_Horizontal
- removed J1801, J1802, J1803: Conn_02x10_Odd_Even, Connector_PinSocket_2.54mm:PinSocket_2x10_P2.54mm_Vertical_SMD
- removed J201, J401, J402: 8P8C, servo:RJ45_Amphenol_54602-x08_Horizontal
- removed JP1301: jumper, Jumper:SolderJumper-3_P1.3mm_Open_RoundedPad1.0x1.5mm
- removed JP1601, JP1602, JP1603, JP1604, JP1605, JP1606, JP1607, JP1608, JP1609, JP1610, JP1611, JP1612, JP1613, JP1614, JP1615, JP1616, JP1617, JP1618, JP1619, JP1620, JP1621, JP1622, JP1623, JP1624, JP1625, JP1626, JP1627, JP1628, JP1629, JP1630, JP1631, JP1632, JP1633, JP1634, JP1635, JP1636, JP1637, JP1638, JP1639, JP1640, JP1641, JP1642, JP1643, JP1644, JP1645, JP1646, JP1647, JP1648: jumper, servo:SolderJumper-2_P1.3mm_Open_RoundedPad1.0x1.5mm
- removed L1701, L1702, L1703, L1704: L_Small, Inductor_SMD:L_0603_1608Metric
- removed R1301, R1302, R1303, R1707, R1708, R1709, R1710: 1k, Resistor_SMD:R_0603_1608Metric
- removed R1613, R1615: 5k, Resistor_SMD:R_0603_1608Metric
- removed R1614, R1616: 3.3k, Resistor_SMD:R_0603_1608Metric
- removed R1701, R1702, R1703, R1704, R1705, R1706: 12e, Resistor_SMD:R_0603_1608Metric
- removed R1711, R1712: 1M, Resistor_SMD:R_0603_1608Metric
- removed R1901, R1902, R1903, R1904, R1905, R1906, R1907, R1908, R1909, R1910, R1911, R1912: 10e, Resistor_SMD:R_0603_1608Metric
- removed R210: 49.9, Resistor_SMD:R_0603_1608Metric
- removed R211, R447, R448: 75e, Resistor_SMD:R_0603_1608Metric
- removed R443, R444: 470, Resistor_SMD:R_0603_1608Metric
- removed SW1501, SW1502, SW1503, SW1504: SW_Push, Button_Switch_SMD:SW_SPST_B3S-1000
- removed TR401, TR402: S558-5500-25-F, Transformer_SMD:Transformer_Ethernet_HALO_TG111-MSC13
- removed U1301: ISO1050, Package_SO:SSO-8_6.7x9.8mm_P2.54mm_Clearance8mm
- removed U1605, U1606, U1607, U1608: LXS6-NPS, servo:LEM_LTSR-NP
- removed U1701, U1702: AMC1311B, Package_SO:SSO-8_6.8x5.9mm_P1.27mm_Clearance8mm
- removed U1703, U1704: RFM-0505S, servo:rfm0505
- removed U1901, U1902: SI8661BD, Package_SO:SOIC-16W_7.5x10.3mm_P1.27mm
- added C1201: 100nF, servo:C_0603_1608Metric, F.Cu at (-284.9, 112.2)
- added C1202: 100nF, servo:C_0603_1608Metric, F.Cu at (-280.3, 109.4)
- added C1401: 1nF, servo:C_0603_1608Metric, F.Cu at (-227.2, 57.8)
- added C1402: 10u, servo:C_0603_1608Metric, F.Cu at (-230.2, 57.8)
- added C1403: 10u, servo:C_0603_1608Metric, F.Cu at (-233.2, 58.5)
- added C1404: 1uF, servo:C_0603_1608Metric, F.Cu at (-236.2, 58.5)
- added C1405: 10u, servo:C_0603_1608Metric, F.Cu at (-239.2, 57.0)
- added C1506: 100pF, servo:C_0603_1608Metric, F.Cu at (-307.5, 82.4)
- added C1507: 100pF, servo:C_0603_1608Metric, F.Cu at (-301.2, 81.4)
- added C1508: 100pF, servo:C_0603_1608Metric, F.Cu at (-305.9, 86.0)
- added C1509: 100pF, servo:C_0603_1608Metric, F.Cu at (-305.9, 84.4)
- added C1510: 100pF, servo:C_0603_1608Metric, F.Cu at (-304.2, 79.9)
- added C1511: 100pF, servo:C_0603_1608Metric, F.Cu at (-308.9, 85.0)
- added C1512: 100pF, servo:C_0603_1608Metric, F.Cu at (-262.7, 43.3)
- added C1513: 100pF, servo:C_0603_1608Metric, F.Cu at (-314.9, 85.0)
- added C1514: 100nF, servo:C_0603_1608Metric, F.Cu at (-317.9, 85.0)
- added C1515: 100pF, servo:C_0603_1608Metric, F.Cu at (-320.9, 85.0)
- added C1516: 100pF, servo:C_0603_1608Metric, F.Cu at (-300.8, 76.3)
- added C1517: 100nF, servo:C_0603_1608Metric, F.Cu at (-304.5, 82.9)
- added C1518: 100nF, servo:C_0603_1608Metric, F.Cu at (-297.8, 74.8)
- added C1801: 100pF, servo:C_0603_1608Metric, F.Cu at (-273.6, 93.8)
- added C1802: 100pF, servo:C_0603_1608Metric, F.Cu at (-284.2, 104.8)
- added C1803: 100pF, servo:C_0603_1608Metric, F.Cu at (-284.2, 101.8)
- added C1804: 100pF, servo:C_0603_1608Metric, F.Cu at (-281.2, 101.8)
- added C1805: 100pF, servo:C_0603_1608Metric, F.Cu at (-281.2, 103.3)
- added C1806: 100pF, servo:C_0603_1608Metric, F.Cu at (-284.2, 103.3)
- added C1807: 100pF, servo:C_0603_1608Metric, F.Cu at (-273.6, 95.3)
- added C1808: 100pF, servo:C_0603_1608Metric, F.Cu at (-281.2, 104.8)
- added C1809: 100pF, servo:C_0603_1608Metric, F.Cu at (-273.6, 96.8)
- added C1810: 100pF, servo:C_0603_1608Metric, F.Cu at (-278.2, 101.8)
- added C1811: 100pF, servo:C_0603_1608Metric, F.Cu at (-287.2, 104.8)
- added C1812: 100pF, servo:C_0603_1608Metric, F.Cu at (-296.3, 101.8)
- added D1401: red@2mA, servo:LED_0603_1608Metric, F.Cu at (-229.0, 56.3)
- added D1402: red@2mA, servo:LED_0603_1608Metric, F.Cu at (-248.9, 77.2)
- added J1401: NHD-4.3-480272FT-CTXL-T, Connector_IDC:IDC-Header_2x10_P2.54mm_Vertical, F.Cu at (-246.7, 48.2)
- added J1402: Conn_01x02, Connector_PinHeader_2.54mm:PinHeader_1x02_P2.54mm_Vertical_SMD_Pin1Left, F.Cu at (-227.1, 52.4)
- added J1503: tblock, Connector_Phoenix_MSTB:PhoenixContact_MSTBA_2,5_2-G-5,08_1x02_P5.08mm_Horizontal, F.Cu at (-282.9, 61.2)
- added J1504: tblock, Connector_Phoenix_MSTB:PhoenixContact_MSTBA_2,5_2-G-5,08_1x02_P5.08mm_Horizontal, F.Cu at (-282.9, 74.7)
- added J1505: tblock, Connector_Phoenix_MSTB:PhoenixContact_MSTBA_2,5_2-G-5,08_1x02_P5.08mm_Horizontal, F.Cu at (-269.7, 61.2)
- added J1506: tblock, Connector_Phoenix_MSTB:PhoenixContact_MSTBA_2,5_2-G-5,08_1x02_P5.08mm_Horizontal, F.Cu at (-269.7, 74.7)
- added J1703: NHD-4.3-480272FT-CTXL-T, Connector_IDC:IDC-Header_2x10_P2.54mm_Vertical, F.Cu at (-246.7, 86.7)
- added JP1202: Jumper_3_Bridged12, Jumper:SolderJumper-3_P1.3mm_Open_RoundedPad1.0x1.5mm, F.Cu at (-284.1, 109.9)
- added JP1501: jumper, servo:SolderJumper-2_P1.3mm_Open_RoundedPad1.0x1.5mm, F.Cu at (-327.5, 82.9)
- added JP1502: jumper, servo:SolderJumper-2_P1.3mm_Open_RoundedPad1.0x1.5mm, F.Cu at (-324.1, 82.9)
- added JP1503: jumper, servo:SolderJumper-2_P1.3mm_Open_RoundedPad1.0x1.5mm, F.Cu at (-320.8, 82.9)
- added JP1504: jumper, servo:SolderJumper-2_P1.3mm_Open_RoundedPad1.0x1.5mm, F.Cu at (-317.4, 82.9)
- added JP1505: jumper, servo:SolderJumper-2_P1.3mm_Open_RoundedPad1.0x1.5mm, F.Cu at (-314.1, 82.9)
- added JP1506: jumper, servo:SolderJumper-2_P1.3mm_Open_RoundedPad1.0x1.5mm, F.Cu at (-310.7, 77.8)
- added JP1507: jumper, servo:SolderJumper-2_P1.3mm_Open_RoundedPad1.0x1.5mm, F.Cu at (-314.1, 77.8)
- added JP1508: jumper, servo:SolderJumper-2_P1.3mm_Open_RoundedPad1.0x1.5mm, F.Cu at (-307.4, 75.3)
- added JP1509: jumper, servo:SolderJumper-2_P1.3mm_Open_RoundedPad1.0x1.5mm, F.Cu at (-324.1, 75.3)
- added JP1510: jumper, servo:SolderJumper-2_P1.3mm_Open_RoundedPad1.0x1.5mm, F.Cu at (-330.8, 77.8)
- added JP1511: jumper, servo:SolderJumper-2_P1.3mm_Open_RoundedPad1.0x1.5mm, F.Cu at (-327.5, 77.8)
- added JP1512: jumper, servo:SolderJumper-2_P1.3mm_Open_RoundedPad1.0x1.5mm, F.Cu at (-324.1, 77.8)
- added JP1513: jumper, servo:SolderJumper-2_P1.3mm_Open_RoundedPad1.0x1.5mm, F.Cu at (-314.1, 75.3)
- added JP1514: jumper, servo:SolderJumper-2_P1.3mm_Open_RoundedPad1.0x1.5mm, F.Cu at (-304.0, 75.3)
- added JP1515: jumper, servo:SolderJumper-2_P1.3mm_Open_RoundedPad1.0x1.5mm, F.Cu at (-324.1, 80.4)
- added JP1516: jumper, servo:SolderJumper-2_P1.3mm_Open_RoundedPad1.0x1.5mm, F.Cu at (-327.5, 75.3)
- added JP1517: jumper, servo:SolderJumper-2_P1.3mm_Open_RoundedPad1.0x1.5mm, F.Cu at (-330.8, 80.4)
- added JP1518: jumper, servo:SolderJumper-2_P1.3mm_Open_RoundedPad1.0x1.5mm, F.Cu at (-310.7, 75.3)
- added JP1519: jumper, servo:SolderJumper-2_P1.3mm_Open_RoundedPad1.0x1.5mm, F.Cu at (-317.4, 75.3)
- added JP1520: jumper, servo:SolderJumper-2_P1.3mm_Open_RoundedPad1.0x1.5mm, F.Cu at (-320.8, 77.8)
- added JP1521: jumper, servo:SolderJumper-2_P1.3mm_Open_RoundedPad1.0x1.5mm, F.Cu at (-330.8, 82.9)
- added JP1522: jumper, servo:SolderJumper-2_P1.3mm_Open_RoundedPad1.0x1.5mm, F.Cu at (-327.5, 80.4)
- added JP1523: jumper, servo:SolderJumper-2_P1.3mm_Open_RoundedPad1.0x1.5mm, F.Cu at (-330.8, 75.3)
- added JP1524: jumper, servo:SolderJumper-2_P1.3mm_Open_RoundedPad1.0x1.5mm, F.Cu at (-320.8, 75.3)
- added JP1525: jumper, servo:SolderJumper-2_P1.3mm_Open_RoundedPad1.0x1.5mm, F.Cu at (-317.4, 77.8)
- added JP1526: jumper, servo:SolderJumper-2_P1.3mm_Open_RoundedPad1.0x1.5mm, F.Cu at (-330.8, 85.5)
- added JP1527: jumper, servo:SolderJumper-2_P1.3mm_Open_RoundedPad1.0x1.5mm, F.Cu at (-304.0, 77.8)
- added JP1528: jumper, servo:SolderJumper-2_P1.3mm_Open_RoundedPad1.0x1.5mm, F.Cu at (-320.8, 80.4)
- added JP1529: jumper, servo:SolderJumper-2_P1.3mm_Open_RoundedPad1.0x1.5mm, F.Cu at (-317.4, 80.4)
- added JP1530: jumper, servo:SolderJumper-2_P1.3mm_Open_RoundedPad1.0x1.5mm, F.Cu at (-307.4, 77.8)
- added JP1531: jumper, servo:SolderJumper-2_P1.3mm_Open_RoundedPad1.0x1.5mm, F.Cu at (-310.7, 82.9)
- added JP1532: jumper, servo:SolderJumper-2_P1.3mm_Open_RoundedPad1.0x1.5mm, F.Cu at (-327.5, 85.5)
- added JP1533: jumper, servo:SolderJumper-2_P1.3mm_Open_RoundedPad1.0x1.5mm, F.Cu at (-307.4, 80.4)
- added JP1534: jumper, servo:SolderJumper-2_P1.3mm_Open_RoundedPad1.0x1.5mm, F.Cu at (-324.1, 85.5)
- added JP1535: jumper, servo:SolderJumper-2_P1.3mm_Open_RoundedPad1.0x1.5mm, F.Cu at (-314.1, 80.4)
- added JP1536: jumper, servo:SolderJumper-2_P1.3mm_Open_RoundedPad1.0x1.5mm, F.Cu at (-310.7, 80.4)
- added L1601: L_Small, Inductor_SMD:L_0603_1608Metric, F.Cu at (-306.7, 90.7)
- added L1602: L_Small, Inductor_SMD:L_0603_1608Metric, F.Cu at (-312.7, 93.8)
- added L1603: L_Small, Inductor_SMD:L_0603_1608Metric, F.Cu at (-312.7, 90.7)
- added L1604: L_Small, Inductor_SMD:L_0603_1608Metric, F.Cu at (-317.8, 100.8)
- added PS701: IRM-15-12, servo:Converter_ACDC_MeanWell_IRM-20-xx_THT, F.Cu at (50.0, -50.0)
- added PS702: IRM-15-12, servo:Converter_ACDC_MeanWell_IRM-20-xx_THT, F.Cu at (50.0, -20.0)
- added R1204: 10k, Resistor_SMD:R_0603_1608Metric, F.Cu at (-284.9, 115.2)
- added R1205: 120e, Resistor_SMD:R_0603_1608Metric, F.Cu at (-284.9, 113.7)
- added R1206: 10k, Resistor_SMD:R_0603_1608Metric, F.Cu at (-281.9, 112.2)
- added R1401: 680, Resistor_SMD:R_0603_1608Metric, F.Cu at (-230.2, 59.4)
- added R1402: 680, Resistor_SMD:R_0603_1608Metric, F.Cu at (-239.2, 58.5)
- added R1403: 680e, Resistor_SMD:R_0603_1608Metric, F.Cu at (-236.2, 57.0)
- added R1404: 220e, Resistor_SMD:R_0603_1608Metric, F.Cu at (-233.2, 57.0)
- added R1505: 5k, Resistor_SMD:R_0603_1608Metric, F.Cu at (-311.9, 85.0)
- added R1506: 3.3k, Resistor_SMD:R_0603_1608Metric, F.Cu at (-259.7, 43.3)
- added R1507: 5k, Resistor_SMD:R_0603_1608Metric, F.Cu at (-301.2, 79.9)
- added R1508: 3.3k, Resistor_SMD:R_0603_1608Metric, F.Cu at (-301.5, 82.9)
- added R1509: 5k, Resistor_SMD:R_0603_1608Metric, F.Cu at (-300.8, 74.8)
- added R1510: 3.3k, Resistor_SMD:R_0603_1608Metric, F.Cu at (-300.8, 77.8)
- added R1511: 5k, Resistor_SMD:R_0603_1608Metric, F.Cu at (-304.2, 81.4)
- added R1512: 3.3k, Resistor_SMD:R_0603_1608Metric, F.Cu at (-297.8, 76.3)
- added R1801: 10e, Resistor_SMD:R_0603_1608Metric, F.Cu at (-287.2, 103.3)
- added R1802: 10e, Resistor_SMD:R_0603_1608Metric, F.Cu at (-290.2, 104.8)
- added R1803: 10e, Resistor_SMD:R_0603_1608Metric, F.Cu at (-293.2, 104.8)
- added R1804: 10e, Resistor_SMD:R_0603_1608Metric, F.Cu at (-290.2, 103.3)
- added R1805: 10e, Resistor_SMD:R_0603_1608Metric, F.Cu at (-287.2, 101.8)
- added R1806: 10e, Resistor_SMD:R_0603_1608Metric, F.Cu at (-273.6, 90.7)
- added R1807: 10e, Resistor_SMD:R_0603_1608Metric, F.Cu at (-296.3, 103.3)
- added R1808: 10e, Resistor_SMD:R_0603_1608Metric, F.Cu at (-293.2, 101.8)
- added R1809: 10e, Resistor_SMD:R_0603_1608Metric, F.Cu at (-293.2, 103.3)
- added R1810: 10e, Resistor_SMD:R_0603_1608Metric, F.Cu at (-296.3, 104.8)
- added R1811: 10e, Resistor_SMD:R_0603_1608Metric, F.Cu at (-290.2, 101.8)
- added R1812: 10e, Resistor_SMD:R_0603_1608Metric, F.Cu at (-273.6, 92.3)
- added SW1401: SW_Push, Button_Switch_SMD:SW_SPST_PTS645, F.Cu at (-235.6, 52.8)
- added SW1402: SW_Push, Button_Switch_SMD:SW_SPST_PTS645, F.Cu at (-215.3, 45.9)
- added SW1403: SW_Push, Button_Switch_SMD:SW_SPST_PTS645, F.Cu at (-225.5, 45.9)
- added SW1404: SW_Push, Button_Switch_SMD:SW_SPST_PTS645, F.Cu at (-235.6, 45.9)
- added U1202: ADM2483, Package_SO:SOIC-16W_7.5x10.3mm_P1.27mm, F.Cu at (-292.1, 114.2)
- added U1401: PAM8301, Package_TO_SOT_SMD:SOT-23-6, F.Cu at (-221.7, 51.2)
- added U1502: LXS6-NPS, servo:LEM_LTSR-NP, F.Cu at (-322.8, 44.0)
- added U1503: LXS6-NPS, servo:LEM_LTSR-NP, F.Cu at (-322.8, 59.8)
- added U1504: LXS6-NPS, servo:LEM_LTSR-NP, F.Cu at (-277.3, 44.0)
- added U1505: LXS6-NPS, servo:LEM_LTSR-NP, F.Cu at (-300.0, 59.8)
- added U1506: LXS6-NPS, servo:LEM_LTSR-NP, F.Cu at (-300.0, 44.0)
- added U1801: SI8661BD, Package_SO:SOIC-16W_7.5x10.3mm_P1.27mm, F.Cu at (-280.7, 95.5)
- added U1802: SI8661BD, Package_SO:SOIC-16W_7.5x10.3mm_P1.27mm, F.Cu at (-292.1, 95.5)
- added U404: rj45x2, servo:rj45x2_0845-2G1T-H5, F.Cu at (118.6, 241.2)
- C1501, C908, C909: value 1nF -> 100nF
- C1502: value 1uF -> 100nF
- C1503, C1505: value 10u -> 100pF
- C1504: value 10u -> 100nF
- C1605, C1606: value 100pF -> 330p
- C1607, C1608, C1609, C1610: value 100pF -> 100nF
- C415: value 0.01uF -> 0.1uF
- C417: value 0.1uF -> 0.01uF
- C428, C429, C432, C433: value 0.1uF -> 1uF
- C702: value 22uF -> 220uF
- C705, C711: value 100nF -> 22uF
- C709, C713: value 22uF -> 100nF
- C712: value 220uF -> 22uF
- C902, C915: value 100nF -> 1nF
- D701: value red -> green
- D702: value green -> red
- D703: value blue -> red
- D706: value red -> blue
- J1001: footprint TerminalBlock_RND:TerminalBlock_RND_205-00291_1x06_P5.08mm_Horizontal -> servo:tblock02x06
- J1101: footprint TerminalBlock_RND:TerminalBlock_RND_205-00293_1x08_P5.08mm_Horizontal -> servo:tblock02x08
- J1201: footprint TerminalBlock_RND:TerminalBlock_RND_205-00289_1x04_P5.08mm_Horizontal -> servo:tblock02x04
- J1501: value NHD-4.3-480272FT-CTXL-T -> tblock; footprint Connector_IDC:IDC-Header_2x10_P2.54mm_Vertical -> Connector_Phoenix_MSTB:PhoenixContact_MSTBA_2,5_2-G-5,08_1x02_P5.08mm_Horizontal
- J1502: value Conn_01x02 -> tblock; footprint Connector_PinHeader_2.54mm:PinHeader_1x02_P2.54mm_Vertical_SMD_Pin1Left -> Connector_Phoenix_MSTB:PhoenixContact_MSTBA_2,5_2-G-5,08_1x02_P5.08mm_Horizontal
- J1601: value tblock -> Screw_Terminal_01x03; footprint Connector_Phoenix_MSTB:PhoenixContact_MSTBA_2,5_2-G-5,08_1x02_P5.08mm_Horizontal -> Connector_Phoenix_MSTB:PhoenixContact_MSTBVA_2,5_3-G-5,08_1x03_P5.08mm_Vertical; moved to B.Cu
- J1602: value tblock -> Screw_Terminal_01x03; footprint Connector_Phoenix_MSTB:PhoenixContact_MSTBA_2,5_2-G-5,08_1x02_P5.08mm_Horizontal -> Connector_Phoenix_MSTB:PhoenixContact_MSTBVA_2,5_3-G-5,08_1x03_P5.08mm_Vertical
- J1701: value Screw_Terminal_01x03 -> NHD-4.3-480272FT-CTXL-T; footprint TerminalBlock_RND:TerminalBlock_RND_205-00288_1x03_P5.08mm_Horizontal -> Connector_IDC:IDC-Header_2x10_P2.54mm_Vertical; moved to B.Cu
- J1702: value Screw_Terminal_01x03 -> NHD-4.3-480272FT-CTXL-T; footprint TerminalBlock_RND:TerminalBlock_RND_205-00277_1x03_P5.00mm_Vertical -> Connector_IDC:IDC-Header_2x10_P2.54mm_Vertical; moved to B.Cu
- J701: footprint TerminalBlock_RND:TerminalBlock_RND_205-00287_1x02_P5.08mm_Horizontal -> TerminalBlock_RND:TerminalBlock_RND_205-00288_1x03_P5.08mm_Horizontal; moved to B.Cu
- J702: moved to B.Cu
- J703: footprint TerminalBlock_RND:TerminalBlock_RND_205-00288_1x03_P5.08mm_Horizontal -> TerminalBlock_RND:TerminalBlock_RND_205-00287_1x02_P5.08mm_Horizontal; moved to B.Cu
- JP1201: value Jumper_3_Bridged12 -> jumper
- JP701: value Jumper_2_Bridged -> jumper; footprint Jumper:SolderJumper-2_P1.3mm_Open_RoundedPad1.0x1.5mm -> servo:SolderJumper-2_P1.3mm_Open_RoundedPad1.0x1.5mm
- JP703: value jumper -> Jumper_2_Bridged; footprint servo:SolderJumper-2_P1.3mm_Open_RoundedPad1.0x1.5mm -> Jumper:SolderJumper-2_P1.3mm_Open_RoundedPad1.0x1.5mm
- R1201, R1203: value 10k -> 1k
- R1202: value 120e -> 1k
- R1501: value 680 -> 5k
- R1502: value 680 -> 3.3k
- R1503: value 680e -> 5k
- R1504: value 220e -> 3.3k
- R1601, R1603, R1605: value 5k -> 12e
- R1602, R1604, R1606: value 3.3k -> 12e
- R1607, R1609: value 5k -> 1k
- R1608, R1610: value 3.3k -> 1k
- R1611: value 5k -> 1M
- R1612: value 3.3k -> 1M
- R207: value 2.2k -> 49.9
- R208: value 49.9 -> 2.2k
- R209: value 470 -> 49.9
- R212, R445, R446: value 75e -> 470
- R436, R439: value 2.2k -> 0e(dnp)
- R903: value 1k(dnp) -> 2k2
- R904, R907, R920: value 10k -> 2k2
- R905: value 2k2 -> 12e
- R906: value 120e NP -> 12e
- R908: value 12e -> 120e NP
- R909: value 12e -> 10k
- R912, R914: value 2k2 -> 1k(dnp)
- R913, R915: value 2k2 -> 10k
- R916: value 12e -> 1k(dnp)
- R917: value 1k(dnp) -> 10k
- R918: value 10k -> 12e
- R919: value 1k(dnp) -> 12e
- R921: value 12e -> 2k2
- TR201: value S558-5500-25-F -> RJ45x1_ARJM11D7-009-AB-ER2-T; footprint Transformer_SMD:Transformer_Ethernet_HALO_TG111-MSC13 -> servo:RJ45x1_RJM11D7-009-AB-ER2-T
- U1201: value ADM2483 -> ISO1050; footprint Package_SO:SOIC-16W_7.5x10.3mm_P1.27mm -> Package_SO:SSO-8_6.7x9.8mm_P2.54mm_Clearance8mm
- U1501: value PAM8301 -> LXS6-NPS; footprint Package_TO_SOT_SMD:SOT-23-6 -> servo:LEM_LTSR-NP
- U1601: value LXS6-NPS -> AMC1311B; footprint servo:LEM_LTSR-NP -> Package_SO:SSO-8_6.8x5.9mm_P1.27mm_Clearance8mm; moved to B.Cu
- U1602: value LXS6-NPS -> AMC1311B; footprint servo:LEM_LTSR-NP -> Package_SO:SSO-8_6.8x5.9mm_P1.27mm_Clearance8mm
- U1603, U1604: value LXS6-NPS -> RFM-0505S; footprint servo:LEM_LTSR-NP -> servo:rfm0505; moved to B.Cu
- U704: value AP2114H-1.2TRG1 -> R-78E5.0-1.0; footprint Package_TO_SOT_SMD:SOT-223 -> Converter_DCDC:Converter_DCDC_RECOM_R-78E-0.5_THT
- U706: value R-78E5.0-1.0 -> AP2114H-1.2TRG1; footprint Converter_DCDC:Converter_DCDC_RECOM_R-78E-0.5_THT -> Package_TO_SOT_SMD:SOT-223
- U901: value ADM2483 -> AMC1311B; footprint Package_SO:SOIC-16W_7.5x10.3mm_P1.27mm -> Package_SO:SSO-8_9.6x6.3mm_P1.27mm_Clearance10.5mm
- U903: value AMC1311B -> ADM2483; footprint Package_SO:SSO-8_9.6x6.3mm_P1.27mm_Clearance10.5mm -> Package_SO:SOIC-16W_7.5x10.3mm_P1.27mm
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Connections:
- C1501 pad 2: Net-(C1501-Pad2) -> 5VC
- C1502 pad 1: Net-(C1502-Pad1) -> GND
- C1502 pad 2: Net-(C1502-Pad2) -> 5VC
- C1503 pad 1: 5VC -> GND
- C1503 pad 2: GND -> LEM_A_V
- C1504 pad 1: 5VC -> GND
- C1504 pad 2: GND -> 5VC
- C1505 pad 1: 5VC -> GND
- C1505 pad 2: GND -> LEM_A_ALL
- C1601 pad 1: GND -> VBUS_A_N
- C1601 pad 2: 5VC -> VBUS_A_P
- C1602 pad 1: GND -> VBUS_B_N
- C1602 pad 2: 5VC -> VBUS_B_P
- C1603 pad 2: 5VC -> 3V3
- C1604 pad 2: 5VC -> 3V3
- C1605 pad 1: GND -> Net-(C1605-Pad1)
- C1605 pad 2: LEM_A_V -> Net-(C1605-Pad2)
- C1606 pad 1: GND -> Net-(C1606-Pad1)
- C1606 pad 2: LEM_A_W -> Net-(C1606-Pad2)
- C1607 pad 1: GND -> Net-(C1605-Pad1)
- C1607 pad 2: LEM_A_ALL -> Net-(C1607-Pad2)
- C1608 pad 1: GND -> Net-(C1606-Pad1)
- C1608 pad 2: LEM_A_U -> Net-(C1608-Pad2)
- C1609 pad 1: GND -> GNDH
- C1609 pad 2: LEM_A_V -> Net-(C1609-Pad2)
- C1610 pad 1: GND -> GNDH
- C1610 pad 2: LEM_A_W -> Net-(C1610-Pad2)
- C702 pad 1: GND -> GNDH
- C702 pad 2: Net-(C702-Pad2) -> 15VH
- C704 pad 2: 5VC -> Net-(C704-Pad2)
- C705 pad 2: Net-(C702-Pad2) -> 5VC
- C707 pad 2: 5VC -> Net-(C704-Pad2)
- C708 pad 1: GND -> GNDH
- C708 pad 2: 3V3 -> 5VH
- C709 pad 2: 1 -> 5VC
- C710 pad 1: GND -> GNDH
- C710 pad 2: 3V3 -> 5VH
- C711 pad 2: 1 -> 3V3
- C712 pad 1: GNDH -> GND
- C712 pad 2: 15VH -> 1
- C713 pad 1: GNDH -> GND
- C713 pad 2: 5VH -> 3V3
- C714 pad 1: GNDH -> GND
- C714 pad 2: 5VH -> 1
- C902 pad 1: GNDH -> NTCA2_N
- C902 pad 2: Net-(C902-Pad2) -> NTCA2_P
- C904 pad 1: GNDH -> GND
- C904 pad 2: 5VH -> 3V3
- C905 pad 2: Net-(C905-Pad2) -> 5VH
- C906 pad 1: GND -> GNDH
- C906 pad 2: 3V3 -> 5VH
- C907 pad 2: 5VH -> Net-(C907-Pad2)
- C908 pad 1: NTCB1_N -> GNDH
- C908 pad 2: NTCB1_P -> Net-(C908-Pad2)
- C909 pad 1: NTCA2_N -> GNDH
- C909 pad 2: NTCA2_P -> Net-(C909-Pad2)
- C910 pad 1: GND -> GNDH
- C910 pad 2: 3V3 -> Net-(C910-Pad2)
- C912 pad 2: Net-(C912-Pad2) -> 5VH
- C913 pad 1: GNDH -> GND
- C913 pad 2: Net-(C913-Pad2) -> 3V3
- C914 pad 1: GNDH -> GND
- C914 pad 2: 5VH -> 3V3
- C915 pad 1: GND -> NTCB1_N
- C915 pad 2: 3V3 -> NTCB1_P
- D702 pad 1: GND -> GNDH
- D706 pad 1: GNDH -> GND
- J1501 pad 1: 3V3 -> Net-(J1501-Pad1)
- J1501 pad 2: GND -> Net-(J1501-Pad2)
- J1601 pad 1: Net-(J1601-Pad1) -> Net-(C1607-Pad2)
- J1602 pad 1: Net-(J1602-Pad1) -> Net-(C1608-Pad2)
- J1701 pad 1: Net-(C1707-Pad2) -> 5VH
- J1701 pad 2: Net-(J1701-Pad2) -> 15VH
- J1701 pad 3: Net-(C1705-Pad1) -> SD_A1_H
- J1702 pad 1: Net-(C1708-Pad2) -> 5VH
- J1702 pad 2: Net-(J1702-Pad2) -> 15VH
- J1702 pad 3: Net-(C1706-Pad1) -> FREE_OUT_A1_H
- J701 pad 1: 15VH -> Net-(F701-Pad2)
- J701 pad 2: GNDH -> Net-(J701-Pad2)
- J702 pad 1: 15VC -> 15VH
- J702 pad 2: GND -> GNDH
- J703 pad 1: Net-(F701-Pad2) -> 15VC
- J703 pad 2: Net-(J703-Pad2) -> GND
- JP1001 pad 2: Net-(J1001-Pad1) -> Net-(J1001-Pad1a)
- JP1002 pad 2: Net-(J1002-Pad1) -> Net-(J1001-Pad1b)
- JP1101 pad 2: Net-(J1101-Pad1) -> Net-(J1101-Pad1a)
- JP1102 pad 2: Net-(J1102-Pad1) -> Net-(J1101-Pad1b)
- JP1201 pad 2: Net-(J1201-Pad1) -> Net-(J1201-Pad1a)
- JP701 pad 1: 5VC -> Net-(JP701-Pad1)
- JP701 pad 2: Net-(C702-Pad2) -> 15VC
- JP702 pad 2: 15VC -> 15VH
- JP703 pad 1: Net-(JP703-Pad1) -> 5VC
- JP703 pad 2: 15VH -> Net-(C703-Pad2)
- R1003 pad 2: Net-(J1001-Pad2) -> Net-(J1001-Pad2a)
- R1004 pad 1: Net-(J1001-Pad2) -> Net-(J1001-Pad2a)
- R1004 pad 2: Net-(J1001-Pad3) -> Net-(J1001-Pad3a)
- R1005 pad 1: Net-(J1001-Pad3) -> Net-(J1001-Pad3a)
- R1006 pad 2: Net-(J1001-Pad4) -> Net-(J1001-Pad4a)
- R1007 pad 1: Net-(J1001-Pad4) -> Net-(J1001-Pad4a)
- R1007 pad 2: Net-(J1001-Pad5) -> Net-(J1001-Pad5a)
- R1008 pad 1: Net-(J1001-Pad5) -> Net-(J1001-Pad5a)
- R1009 pad 2: Net-(J1002-Pad2) -> Net-(J1001-Pad2b)
- R1010 pad 1: Net-(J1002-Pad2) -> Net-(J1001-Pad2b)
- R1010 pad 2: Net-(J1002-Pad3) -> Net-(J1001-Pad3b)
- R1011 pad 1: Net-(J1002-Pad3) -> Net-(J1001-Pad3b)
- R1012 pad 2: Net-(J1002-Pad4) -> Net-(J1001-Pad4b)
- R1013 pad 1: Net-(J1002-Pad4) -> Net-(J1001-Pad4b)
- R1013 pad 2: Net-(J1002-Pad5) -> Net-(J1001-Pad5b)
- R1014 pad 1: Net-(J1002-Pad5) -> Net-(J1001-Pad5b)
- R1101 pad 2: Net-(J1101-Pad2) -> Net-(J1101-Pad2a)
- R1102 pad 2: Net-(J1101-Pad3) -> Net-(J1101-Pad3a)
- R1103 pad 2: Net-(J1101-Pad4) -> Net-(J1101-Pad4a)
- R1104 pad 2: Net-(J1101-Pad5) -> Net-(J1101-Pad5a)
- R1107 pad 2: Net-(J1102-Pad2) -> Net-(J1101-Pad2b)
- R1108 pad 2: Net-(J1102-Pad3) -> Net-(J1101-Pad3b)
- R1109 pad 2: Net-(J1102-Pad4) -> Net-(J1101-Pad4b)
- R1110 pad 2: Net-(J1102-Pad5) -> Net-(J1101-Pad5b)
- R1201 pad 2: Net-(J1201-Pad2) -> Net-(J1201-Pad2a)
- R1202 pad 1: Net-(J1201-Pad2) -> Net-(J1201-Pad2a)
- R1202 pad 2: Net-(J1201-Pad3) -> Net-(J1201-Pad3a)
- R1203 pad 1: Net-(J1201-Pad3) -> Net-(J1201-Pad3a)
- R1501 pad 1: 3V3 -> Net-(R1501-Pad1)
- R1501 pad 2: Net-(D1501-Pad2) -> LEM_A_V
- R1502 pad 1: 3V3 -> LEM_A_V
- R1502 pad 2: Net-(D1502-Pad2) -> GND
- R1503 pad 1: LCD_AUDIO -> Net-(R1503-Pad1)
- R1503 pad 2: Net-(C1501-Pad2) -> LEM_A_ALL
- R1504 pad 1: Net-(C1501-Pad2) -> LEM_A_ALL
- R1504 pad 2: Net-(C1502-Pad1) -> GND
- R1601 pad 1: Net-(R1601-Pad1) -> VBUS_A_P
- R1601 pad 2: LEM_A_V -> Net-(R1601-Pad2)
- R1602 pad 1: LEM_A_V -> VBUS_A_N
- R1602 pad 2: GND -> Net-(R1602-Pad2)
- R1603 pad 1: Net-(R1603-Pad1) -> VBUS_B_P
- R1603 pad 2: LEM_A_W -> Net-(R1603-Pad2)
- R1604 pad 1: LEM_A_W -> VBUS_B_N
- R1604 pad 2: GND -> Net-(R1604-Pad2)
- R1605 pad 1: Net-(R1605-Pad1) -> Net-(C1605-Pad2)
- R1605 pad 2: LEM_A_ALL -> Net-(R1605-Pad2)
- R1606 pad 1: LEM_A_ALL -> Net-(C1606-Pad2)
- R1606 pad 2: GND -> Net-(R1606-Pad2)
- R1607 pad 1: Net-(R1607-Pad1) -> Net-(C1607-Pad2)
- R1607 pad 2: LEM_A_U -> Net-(R1605-Pad2)
- R1608 pad 1: LEM_A_U -> Net-(R1605-Pad2)
- R1608 pad 2: GND -> Net-(C1605-Pad1)
- R1609 pad 1: Net-(R1609-Pad1) -> Net-(C1608-Pad2)
- R1609 pad 2: LEM_B_U -> Net-(R1606-Pad2)
- R1610 pad 1: LEM_B_U -> Net-(R1606-Pad2)
- R1610 pad 2: GND -> Net-(C1606-Pad1)
- R1611 pad 1: Net-(R1611-Pad1) -> Net-(R1605-Pad2)
- R1611 pad 2: LEM_B_W -> Net-(J1601-Pad2)
- R1612 pad 1: LEM_B_W -> Net-(R1606-Pad2)
- R1612 pad 2: GND -> Net-(J1602-Pad2)
- R205 pad 1: /ethernet/DIFFPAIR -> 3V3
- R206 pad 1: /ethernet/DIFFPAIR -> 3V3
- R207 pad 2: Net-(D201-Pad1) -> 3V3
- R208 pad 1: /ethernet/DIFFPAIR -> 3V3
- R208 pad 2: 3V3 -> Net-(R208-Pad2)
- R209 pad 2: Net-(D201-Pad2) -> 3V3
- R212 pad 1: Net-(C217-Pad2) -> 3V3
- R434 pad 1: Net-(R434-Pad1) -> 3V3
- R434 pad 2: 3V3 -> Net-(R434-Pad2)
- R439 pad 1: Net-(R434-Pad1) -> Net-(R434-Pad2)
- R445 pad 1: Net-(C434-Pad2) -> 3V3
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Other:
- copper layers 2 -> 6

Commit message: added some 3d models, elminating 15vc and 2 lems
I've elminated 15vc 'cause I don't use these voltage, so I'd change 20w
15v heating power to 10w 5v more efficiency voltage to drive 3.3 and
1.2v to the core and logic. I've also elminated 2 LEMS 'cause space..
even thought there remain 3 for each motor.. more than necesary...keep
going
Parts:
- removed C701: 220uF, servo:C_0603_1608Metric
- removed C705: 22uF, servo:C_0603_1608Metric
- removed C709: 100nF, servo:C_0603_1608Metric
- removed D703: red, servo:LED_0603_1608Metric
- removed J1506: tblock, Connector_Phoenix_MSTB:PhoenixContact_MSTBA_2,5_2-G-5,08_1x02_P5.08mm_Horizontal
- removed J1601, J1602: Screw_Terminal_01x03, Connector_Phoenix_MSTB:PhoenixContact_MSTBVA_2,5_3-G-5,08_1x03_P5.08mm_Vertical
- removed J702, J703: tBlock, TerminalBlock_RND:TerminalBlock_RND_205-00287_1x02_P5.08mm_Horizontal
- removed JP1501, JP1502, JP1503, JP1504, JP1505, JP1506, JP1507, JP1508, JP1509, JP1510, JP1511, JP1512, JP1513, JP1514, JP1515, JP1516, JP1517, JP1518, JP1519, JP1520, JP1521, JP1522, JP1523, JP1524, JP1525, JP1526, JP1527, JP1528, JP1529, JP1530, JP1531, JP1532, JP1533, JP1534, JP1535, JP1536: jumper, servo:SolderJumper-2_P1.3mm_Open_RoundedPad1.0x1.5mm
- removed JP703: Jumper_2_Bridged, Jumper:SolderJumper-2_P1.3mm_Open_RoundedPad1.0x1.5mm
- removed R703: 680, Resistor_SMD:R_0603_1608Metric
- removed SW1401, SW1402: SW_Push, Button_Switch_SMD:SW_SPST_PTS645
- removed U701, U703: R-78E5.0-1.0, Converter_DCDC:Converter_DCDC_RECOM_R-78E-0.5_THT
- added J1507: tblock, servo:tblock02x03, F.Cu at (84.2, 55.0)
- added R1613: 1M, Resistor_SMD:R_0603_1608Metric, F.Cu at (23.6, 302.3)
- added R1614: 1M, Resistor_SMD:R_0603_1608Metric, F.Cu at (383.2, 74.0)
- C1501, C1502, C1514, C1517, C1518: value 100nF -> 100pF
- C1505, C1508, C1510, C1511, C1512: value 100pF -> 100nF
- J1401: footprint Connector_IDC:IDC-Header_2x10_P2.54mm_Vertical -> servo:HD-4.3-480272
- J1501, J1502, J1503, J1504, J1505: footprint Connector_Phoenix_MSTB:PhoenixContact_MSTBA_2,5_2-G-5,08_1x02_P5.08mm_Horizontal -> servo:tblock02x03
- J1703, U1602, U705, U706: moved to B.Cu
- J701: value tBlock -> tblock; footprint TerminalBlock_RND:TerminalBlock_RND_205-00288_1x03_P5.08mm_Horizontal -> servo:tblock02x04; moved to F.Cu
- PS701: value IRM-15-12 -> IRM-10-5; footprint servo:Converter_ACDC_MeanWell_IRM-20-xx_THT -> servo:Converter_ACDC_MeanWell_IRM-10-xx_THT
- PS702: value IRM-15-12 -> irm-10-12; footprint servo:Converter_ACDC_MeanWell_IRM-20-xx_THT -> servo:Converter_ACDC_MeanWell_IRM-10-xx_THT
- moved C1506 631.4 mm to (312.6, 201.2)
- moved C1513 631.4 mm to (305.2, 203.8)
- moved C1517 631.4 mm to (315.6, 201.7)
- moved R1505 631.4 mm to (308.2, 203.8)
- moved C1507 631.4 mm to (319.0, 200.2)
- moved C1508 631.4 mm to (314.3, 204.8)
- moved C1509 631.4 mm to (314.3, 203.2)
- moved C1510 631.4 mm to (316.0, 198.7)
- moved C1511 631.4 mm to (311.2, 203.8)
- moved C1514 631.4 mm to (302.2, 203.8)
- moved C1515 631.4 mm to (299.2, 203.8)
- moved C1516 631.4 mm to (319.3, 195.1)
- moved C1518 631.4 mm to (322.3, 193.6)
- moved C1602 631.4 mm to (305.3, 219.7)
- moved C1606 631.4 mm to (310.5, 212.6)
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Connections:
- C1501 pad 2: 5VC -> LEM_A_V
- C1502 pad 2: 5VC -> LEM_A_ALL
- C1505 pad 2: LEM_A_ALL -> 5VC
- C1507 pad 2: LEM_A_V -> LEM_A_ALL
- C1508 pad 2: LEM_A_ALL -> 5VC
- C1510 pad 2: LEM_B_U -> 5VC
- C1511 pad 2: LEM_B_ALL -> 5VC
- C1512 pad 2: LEM_B_V -> 5VC
- C1514 pad 2: 5VC -> LEM_B_V
- C1516 pad 2: LEM_B_V -> LEM_B_U
- C1517 pad 2: 5VC -> LEM_B_V
- C1518 pad 2: 5VC -> LEM_B_ALL
- C1605 pad 1: Net-(C1605-Pad1) -> VBUS_A_N_H
- C1606 pad 1: Net-(C1606-Pad1) -> VBUS_B_N_H
- C1607 pad 1: Net-(C1605-Pad1) -> VBUS_A_N_H
- C1608 pad 1: Net-(C1606-Pad1) -> VBUS_B_N_H
- C214 pad 2: 3V3 -> /ethernet/DIFFPAIR
- C703 pad 2: Net-(C703-Pad2) -> 5VC
- C706 pad 2: Net-(C703-Pad2) -> 5VC
- F702 pad 2: Net-(F701-Pad2) -> Net-(F702-Pad2)
- JP701 pad 2: 15VC -> 5VC
- PS701 pad 2: Net-(J701-Pad3) -> Net-(J701-Pad1b)
- PS702 pad 2: Net-(J701-Pad3) -> Net-(J701-Pad4b)
- R1509 pad 2: LEM_B_ALL -> LEM_B_V
- R1510 pad 1: LEM_B_ALL -> LEM_B_V
- R1511 pad 2: LEM_B_V -> LEM_B_ALL
- R1512 pad 1: LEM_B_V -> LEM_B_ALL
- R1608 pad 2: Net-(C1605-Pad1) -> VBUS_A_N_H
- R1610 pad 2: Net-(C1606-Pad1) -> VBUS_B_N_H
- R205 pad 1: 3V3 -> /ethernet/DIFFPAIR
- R206 pad 1: 3V3 -> /ethernet/DIFFPAIR
- R207 pad 1: 3V3 -> /ethernet/DIFFPAIR
- R209 pad 1: 3V3 -> /ethernet/DIFFPAIR
- TR201 pad 1: 3V3 -> /ethernet/DIFFPAIR
- TR201 pad 2: 3V3 -> /ethernet/DIFFPAIR
- TR201 pad 3: 3V3 -> /ethernet/DIFFPAIR
- TR201 pad 6: 3V3 -> /ethernet/DIFFPAIR
- U1501 pad 1: Net-(J1501-Pad2) -> Net-(J1501-Pad1)
- U1501 pad 2: Net-(JP1502-Pad1) -> Net-(J1501-Pad2)
- U1501 pad 3: Net-(JP1507-Pad2) -> Net-(J1501-Pad3)
- U1501 pad 4: Net-(JP1501-Pad2) -> Net-(J1501-Pad4)
- U1501 pad 5: Net-(JP1507-Pad2) -> Net-(J1501-Pad5)
- U1501 pad 6: Net-(JP1502-Pad2) -> Net-(J1501-Pad6)
- U1502 pad 1: Net-(J1502-Pad2) -> Net-(J1502-Pad1)
- U1502 pad 2: Net-(JP1504-Pad1) -> Net-(J1502-Pad2)
- U1502 pad 3: Net-(JP1509-Pad2) -> Net-(J1502-Pad3)
- U1502 pad 4: Net-(JP1503-Pad2) -> Net-(J1502-Pad4)
- U1502 pad 5: Net-(JP1509-Pad2) -> Net-(J1502-Pad5)
- U1502 pad 6: Net-(JP1504-Pad2) -> Net-(J1502-Pad6)
- U1503 pad 1: Net-(J1503-Pad2) -> Net-(J1507-Pad1)
- U1503 pad 3: Net-(JP1511-Pad2) -> Net-(J1507-Pad3)
- U1503 pad 5: Net-(JP1511-Pad2) -> Net-(J1507-Pad5)
- U1504 pad 1: Net-(J1504-Pad2) -> Net-(J1503-Pad1)
- U1504 pad 2: Net-(JP1519-Pad2) -> Net-(J1503-Pad2)
- U1504 pad 3: Net-(JP1520-Pad2) -> Net-(J1503-Pad3)
- U1504 pad 4: Net-(JP1524-Pad2) -> Net-(J1503-Pad4)
- U1504 pad 5: Net-(JP1520-Pad2) -> Net-(J1503-Pad5)
- U1504 pad 6: Net-(JP1520-Pad1) -> Net-(J1503-Pad6)
- U1505 pad 1: Net-(J1505-Pad2) -> Net-(J1504-Pad1)
- U1505 pad 2: Net-(JP1521-Pad2) -> Net-(J1504-Pad2)
- U1505 pad 3: Net-(JP1522-Pad2) -> Net-(J1504-Pad3)
- U1505 pad 4: Net-(JP1528-Pad2) -> Net-(J1504-Pad4)
- U1505 pad 5: Net-(JP1522-Pad2) -> Net-(J1504-Pad5)
- U1505 pad 6: Net-(JP1522-Pad1) -> Net-(J1504-Pad6)
- U1506 pad 1: Net-(J1506-Pad2) -> Net-(J1505-Pad1)
- U1506 pad 2: Net-(JP1525-Pad2) -> Net-(J1505-Pad2)
- U1506 pad 3: Net-(JP1526-Pad2) -> Net-(J1505-Pad3)
- U1506 pad 4: Net-(JP1530-Pad2) -> Net-(J1505-Pad4)
- U1506 pad 5: Net-(JP1526-Pad2) -> Net-(J1505-Pad5)
- U1506 pad 6: Net-(JP1526-Pad1) -> Net-(J1505-Pad6)
- U1601 pad 3: Net-(C1605-Pad1) -> VBUS_A_N_H
- U1601 pad 4: Net-(C1605-Pad1) -> VBUS_A_N_H
- U1602 pad 3: Net-(C1606-Pad1) -> VBUS_B_N_H
- U1602 pad 4: Net-(C1606-Pad1) -> VBUS_B_N_H
- U1603 pad 3: Net-(C1605-Pad1) -> VBUS_A_N_H
- U1604 pad 3: Net-(C1606-Pad1) -> VBUS_B_N_H
- U201 pad 10: 3V3 -> /ethernet/DIFFPAIR
- U201 pad 11: 3V3 -> /ethernet/DIFFPAIR
- U201 pad 12: 3V3 -> /ethernet/DIFFPAIR
- U201 pad 9: 3V3 -> /ethernet/DIFFPAIR
- U404 pad 14: Net-(U404-Pad14) -> GND
- U404 pad 7: Net-(U404-Pad7) -> GND
- U702 pad 1: 15VC -> 5VC
- U705 pad 3: Net-(C703-Pad2) -> 5VC
Other:
- board outline added: 220 x 200 mm

Commit message: I've reducede the PCB size ADC TVS, USB host and IDC out
TVS for ADC protection, USB out 'cause it's almost free and IDC debug
out in an IDC. Better and thinner terminal block connector help in
reduce the board size.
Parts:
- removed J1507: tblock, servo:tblock02x03
- removed TR201: RJ45x1_ARJM11D7-009-AB-ER2-T, servo:RJ45x1_RJM11D7-009-AB-ER2-T
- added C217: 4n7, servo:C_0603_1608Metric, F.Cu at (291.5, 63.3)
- added C434: 4n7, servo:C_0603_1608Metric, F.Cu at (297.6, 63.3)
- added IC201: TPD4E001QDBV, Package_TO_SOT_SMD:SOT-23-6, B.Cu at (164.9, 149.2)
- added IC301: TPD4E001QDBV, Package_TO_SOT_SMD:SOT-23-6, B.Cu at (156.1, 149.2)
- added IC302: TPD4E001QDBV, Package_TO_SOT_SMD:SOT-23-6, B.Cu at (152.2, 145.6)
- added IC303: TPD4E001QDBV, Package_TO_SOT_SMD:SOT-23-6, B.Cu at (152.2, 149.2)
- added IC304: TPD4E001QDBV, Package_TO_SOT_SMD:SOT-23-6, B.Cu at (148.4, 145.6)
- added IC305: TPD4E001QDBV, Package_TO_SOT_SMD:SOT-23-6, B.Cu at (148.4, 149.2)
- added J1506: tblock2x3, servo:tblock02x03, F.Cu at (79.3, 55.5)
- added J201: 0821-1X1T-36-F, servo:BEL_0821-1X1T-36-F, B.Cu at (207.1, 199.9)
- added R210: 1oe, Resistor_SMD:R_0603_1608Metric, F.Cu at (62.5, 252.5)
- added R302: 10e, Resistor_SMD:R_0603_1608Metric, F.Cu at (-26.0, 263.3)
- added R303: 10e, Resistor_SMD:R_0603_1608Metric, F.Cu at (-26.0, 264.8)
- added R304: 10e, Resistor_SMD:R_0603_1608Metric, F.Cu at (-23.0, 263.3)
- added R305: 10e, Resistor_SMD:R_0603_1608Metric, F.Cu at (-26.0, 266.3)
- added R306: 10e, Resistor_SMD:R_0603_1608Metric, F.Cu at (-23.0, 264.8)
- added R307: 10e, Resistor_SMD:R_0603_1608Metric, F.Cu at (-20.0, 263.3)
- added R308: 10e, Resistor_SMD:R_0603_1608Metric, F.Cu at (-26.0, 267.8)
- added R309: 10e, Resistor_SMD:R_0603_1608Metric, F.Cu at (-23.0, 266.3)
- added R310: 10e, Resistor_SMD:R_0603_1608Metric, F.Cu at (-20.0, 264.8)
- added R311: 10e, Resistor_SMD:R_0603_1608Metric, F.Cu at (-26.0, 269.3)
- added R312: 10e, Resistor_SMD:R_0603_1608Metric, F.Cu at (-17.0, 263.3)
- added R313: 10e, Resistor_SMD:R_0603_1608Metric, F.Cu at (-23.0, 267.8)
- added R314: 10e, Resistor_SMD:R_0603_1608Metric, F.Cu at (-20.0, 266.3)
- added R315: 10e, Resistor_SMD:R_0603_1608Metric, F.Cu at (-17.0, 269.3)
- added R316: 10e, Resistor_SMD:R_0603_1608Metric, F.Cu at (-17.0, 267.8)
- added R317: 10e, Resistor_SMD:R_0603_1608Metric, F.Cu at (-17.0, 264.8)
- added R318: 10e, Resistor_SMD:R_0603_1608Metric, F.Cu at (-23.0, 269.3)
- added R319: 10e, Resistor_SMD:R_0603_1608Metric, F.Cu at (-20.0, 267.8)
- added R320: 10e, Resistor_SMD:R_0603_1608Metric, F.Cu at (-17.0, 266.3)
- added R321: 10e, Resistor_SMD:R_0603_1608Metric, F.Cu at (-20.0, 269.3)
- J1001: value tblock -> tblock2x6
- J1201: value tblock -> tblock2x4
- J1501, J1502, J1503, J1504, J1505: value tblock -> tblock2x3
- J601: footprint Connector_IDC:IDC-Header_2x05_P2.54mm_Vertical -> Connector_IDC:IDC-Header_2x05_P2.54mm_Horizontal
- U1603, U1604: moved to F.Cu
- moved U1603 196.6 mm to (226.0, 147.5)
- moved U1604 196.6 mm to (211.0, 147.5)
- moved U705 186.8 mm to (207.5, 112.5)
- moved U706 174.9 mm to (220.0, 113.2)
- moved U702 166.6 mm to (217.2, 131.5)
- moved U704 166.1 mm to (232.2, 131.5)
- moved F702 161.4 mm to (232.9, 63.0)
- moved F701 155.3 mm to (231.5, 58.5)
- moved J602 153.4 mm to (234.2, 176.3)
- moved U1601 140.8 mm to (209.1, 85.7)
- moved U1602 140.8 mm to (221.9, 85.7)
- moved TP601 89.3 mm to (285.0, 130.0)
- moved SW1404 81.5 mm to (304.0, 170.2), turned to 180 degrees
- moved J601 77.5 mm to (234.0, 199.5), turned to 270 degrees
- moved SW1403 67.1 mm to (305.0, 182.5), turned to 180 degrees
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Connections:
- C214 pad 2: /ethernet/DIFFPAIR -> /ethernet/P0_TD_N
- J701 pad 1b: Net-(J701-Pad1b) -> Net-(F701-Pad2)
- J701 pad 2b: Net-(F701-Pad2) -> Net-(F702-Pad2)
- J701 pad 3b: Net-(F702-Pad2) -> Net-(J701-Pad3b)
- J701 pad 4b: Net-(J701-Pad4b) -> Earth
- PS701 pad 2: Net-(J701-Pad1b) -> Net-(J701-Pad3b)
- PS702 pad 2: Net-(J701-Pad4b) -> Net-(J701-Pad3b)
- R205 pad 1: /ethernet/DIFFPAIR -> 3V3
- R205 pad 2: 3V3 -> /ethernet/P0_TD_P
- R206 pad 1: /ethernet/DIFFPAIR -> 3V3
- R206 pad 2: 3V3 -> /ethernet/P0_TD_N
- R207 pad 1: /ethernet/DIFFPAIR -> 3V3
- R207 pad 2: 3V3 -> /ethernet/P0_RD_P
- R209 pad 1: /ethernet/DIFFPAIR -> 3V3
- R209 pad 2: 3V3 -> /ethernet/P0_RD_N
- U1503 pad 1: Net-(J1507-Pad1) -> Net-(J1503-Pad1)
- U1503 pad 2: Net-(J1507-Pad2) -> Net-(J1503-Pad2)
- U1503 pad 3: Net-(J1507-Pad3) -> Net-(J1503-Pad3)
- U1503 pad 4: Net-(J1507-Pad4) -> Net-(J1503-Pad4)
- U1503 pad 5: Net-(J1507-Pad5) -> Net-(J1503-Pad5)
- U1503 pad 6: Net-(J1507-Pad6) -> Net-(J1503-Pad6)
- U1504 pad 1: Net-(J1503-Pad1) -> Net-(J1504-Pad3)
- U1504 pad 2: Net-(J1503-Pad2) -> Net-(J1504-Pad2)
- U1504 pad 3: Net-(J1503-Pad3) -> Net-(J1504-Pad1)
- U1504 pad 4: Net-(J1503-Pad4) -> Net-(J1504-Pad6)
- U1504 pad 5: Net-(J1503-Pad5) -> Net-(J1504-Pad5)
- U1504 pad 6: Net-(J1503-Pad6) -> Net-(J1504-Pad4)
- U1505 pad 1: Net-(J1504-Pad1) -> Net-(J1505-Pad3)
- U1505 pad 2: Net-(J1504-Pad2) -> Net-(J1505-Pad2)
- U1505 pad 3: Net-(J1504-Pad3) -> Net-(J1505-Pad1)
- U1505 pad 4: Net-(J1504-Pad4) -> Net-(J1505-Pad6)
- U1505 pad 5: Net-(J1504-Pad5) -> Net-(J1505-Pad5)
- U1505 pad 6: Net-(J1504-Pad6) -> Net-(J1505-Pad4)
- U1506 pad 1: Net-(J1505-Pad1) -> Net-(J1506-Pad3)
- U1506 pad 2: Net-(J1505-Pad2) -> Net-(J1506-Pad2)
- U1506 pad 3: Net-(J1505-Pad3) -> Net-(J1506-Pad1)
- U1506 pad 4: Net-(J1505-Pad4) -> Net-(J1506-Pad6)
- U1506 pad 5: Net-(J1505-Pad5) -> Net-(J1506-Pad5)
- U1506 pad 6: Net-(J1505-Pad6) -> Net-(J1506-Pad4)
- U201 pad 10: /ethernet/DIFFPAIR -> /ethernet/P0_RD_P
- U201 pad 11: /ethernet/DIFFPAIR -> /ethernet/P0_TD_N
- U201 pad 12: /ethernet/DIFFPAIR -> /ethernet/P0_TD_P
- U201 pad 9: /ethernet/DIFFPAIR -> /ethernet/P0_RD_N
- U301 pad C19: FREE_IN_A4 -> USB_D+
- U301 pad D19: FREE_IN_A3 -> USB_D-
- U301 pad E18: FREE_IN_B4 -> FREE_OUT_B2
- U301 pad E19: FREE_IN_B3 -> FREE_OUT_B1
- U301 pad K18: FREE_OUT_B1 -> FREE_IN_A3
- U301 pad K19: FREE_OUT_B2 -> FREE_IN_A4
- U301 pad N16: Net-(U301-PadN16) -> RS485_EN
- U301 pad P17: RS485_EN -> FREE_IN_B4
- U301 pad P3: NTCA2_N -> Net-(IC304-Pad6)
- U301 pad P4: NTCB2_N -> Net-(IC304-Pad3)
- U301 pad R16: Net-(U301-PadR16) -> FREE_IN_B3
- U301 pad R3: NTCA2_P -> Net-(IC303-Pad4)
- U301 pad R4: NTCB2_P -> Net-(IC304-Pad1)
- U301 pad T1: DACB_DBG_OUT -> Net-(IC301-Pad1)
- U301 pad T2: NTCA1_N -> Net-(IC301-Pad4)
- U301 pad T3: NTCB1_N -> Net-(IC302-Pad1)
- U301 pad T5: LEM_A_U -> Net-(IC304-Pad4)
- U301 pad T6: LEM_A_ALL -> Net-(IC305-Pad1)
- U301 pad T7: VBUS_A_P -> Net-(IC305-Pad3)
- U301 pad U1: LCD_AUDIO -> Net-(IC301-Pad6)
- U301 pad U2: NTCA1_P -> Net-(IC301-Pad3)
- U301 pad U3: NTCB1_P -> Net-(IC302-Pad6)
- U301 pad U5: LEM_A_V -> Net-(IC305-Pad6)
- U301 pad U7: VBUS_A_N -> Net-(IC305-Pad4)
- U301 pad V2: LEM_B_U -> Net-(IC302-Pad3)
- U301 pad V3: LEM_B_ALL -> Net-(IC303-Pad6)
- U301 pad V4: VBUS_B_P -> Net-(IC303-Pad1)
- U301 pad W2: LEM_B_V -> Net-(IC302-Pad4)
- U301 pad W4: VBUS_B_N -> Net-(IC303-Pad3)
- U404 pad 14: GND -> Earth
- U404 pad 7: GND -> Earth
Other:
- board size 220 x 200 mm -> 180 x 155 mm
