File: kicad/servo.kicad_pcb (KiCad board)
At the start: 6 copper layers, 180 x 155 mm, 536 parts, among them IC201 TPD4E001QDBV, IC301 TPD4E001QDBV, IC302 TPD4E001QDBV, IC303 TPD4E001QDBV, IC304 TPD4E001QDBV, IC305 TPD4E001QDBV, J1001 tblock2x6, J1101 tblock, J1201 tblock2x4, J1401 NHD-4.3-480272FT-CTXL-T, J1402 Conn_01x02, J1501 tblock2x3, J1502 tblock2x3, J1503 tblock2x3, J1504 tblock2x3, J1505 tblock2x3, J1506 tblock2x3, J1701 NHD-4.3-480272FT-CTXL-T, J1702 NHD-4.3-480272FT-CTXL-T, J1703 NHD-4.3-480272FT-CTXL-T, J201 0821-1X1T-36-F, J601 Conn_02x05_Counter_Clockwise, J602 Conn_01x02, J701 tblock, SW1403 SW_Push, SW1404 SW_Push, U1001 ADM2483, U1002 ADM2483, U1003 ADM2483, U1004 ADM2483, U1101 SI8662BD, U1102 SI8662BD, U1201 ISO1050, U1202 ADM2483, U1401 PAM8301, U1501 LXS6-NPS, U1502 LXS6-NPS, U1503 LXS6-NPS, U1504 LXS6-NPS, U1505 LXS6-NPS, U1506 LXS6-NPS, U1601 AMC1311B, U1602 AMC1311B, U1603 RFM-0505S, U1604 RFM-0505S, U1801 SI8661BD, U1802 SI8661BD, U201 DP83822, U301 TMS320F28388DZWTS, U401 CAT24C16WI, U402 DP83822, U403 DP83822, U404 rj45x2, U601 SN74ALVC244PW, U602 M25PX32-VMW, U702 R-78E3.3-1.0, U704 R-78E5.0-1.0, U705 AP2114H-1.2TRG1, U706 AP2114H-1.2TRG1, U801 SI8660BD, U802 SI8662BD, U803 SN74LVC2G17DBVR, U804 SN74LVC2G17DBVR, U805 SN74LVC2G17DBVR, U806 SN74LVC2G17DBVR, U807 SN74LVC2G17DBVR, U808 SN74LVC2G17DBVR, U809 SN74LVC2G17DBVR, U810 SN74LVC2G17DBVR, U811 SN74LVC2G17DBVR, U812 SN74LVC2G17DBVR, U813 SI8660BD, U814 SI8662BD, U901 AMC1311B, U902 AMC1311B, U903 ADM2483, U904 AMC1311B, U905 AMC1311B

Commit message: I forgot that QUEP was diferential!! all to back....
Parts:
- removed C1001, C1002, C1003, C1004, C1005, C1006, C1007, C1008: 100nF, servo:C_0603_1608Metric
- removed C1101, C1102, C1103, C1104, C1105, C1106, C1107, C1108, C1109, C1110, C1111, C1112: 1nF, servo:C_0603_1608Metric
- removed JP1002, JP1102: jumper, Jumper:SolderJumper-3_P1.3mm_Open_RoundedPad1.0x1.5mm
- removed R1013: 120e, Resistor_SMD:R_0603_1608Metric
- removed R1014: 100k, Resistor_SMD:R_0603_1608Metric
- removed R1015: 0e(dnp), Resistor_SMD:R_0603_1608Metric
- removed R1016: 0e, Resistor_SMD:R_0603_1608Metric
- removed R1801, R1812: 10e, Resistor_SMD:R_0603_1608Metric
- removed U1002, U1003, U1004: ADM2483, Package_SO:SOIC-16W_7.5x10.3mm_P1.27mm
- added C1901: 100nF, servo:C_0603_1608Metric, F.Cu at (127.2, 264.0)
- added C1904: 100nF, servo:C_0603_1608Metric, F.Cu at (164.4, 240.5)
- added C1905: 100nF, servo:C_0603_1608Metric, F.Cu at (122.5, 265.5)
- added C1910: 100nF, servo:C_0603_1608Metric, F.Cu at (119.5, 268.3)
- added C1913: 100nF, servo:C_0603_1608Metric, F.Cu at (124.2, 264.0)
- added C1914: 100nF, servo:C_0603_1608Metric, F.Cu at (116.5, 268.3)
- added J1901: tblock2x6, Connector_Phoenix_MC:PhoenixContact_MC_1,5_6-G-3.81_1x06_P3.81mm_Horizontal, F.Cu at (99.5, 199.3)
- added JP1901: jumper, Jumper:SolderJumper-3_P1.3mm_Open_RoundedPad1.0x1.5mm, F.Cu at (117.3, 264.5)
- added R1113: 10k, Resistor_SMD:R_0603_1608Metric, F.Cu at (190.6, 246.5)
- added R1114: 1k, Resistor_SMD:R_0603_1608Metric, F.Cu at (171.8, 251.6)
- added R1115: 10k, Resistor_SMD:R_0603_1608Metric, F.Cu at (186.2, 251.1)
- added R1116: 10k, Resistor_SMD:R_0603_1608Metric, F.Cu at (190.6, 245.0)
- added R1117: 1k, Resistor_SMD:R_0603_1608Metric, F.Cu at (190.6, 243.5)
- added R1118: 10k, Resistor_SMD:R_0603_1608Metric, F.Cu at (190.6, 242.0)
- added R1119: 10k, Resistor_SMD:R_0603_1608Metric, F.Cu at (177.8, 251.6)
- added R1120: 1k, Resistor_SMD:R_0603_1608Metric, F.Cu at (190.6, 240.5)
- added R1121: 10k, Resistor_SMD:R_0603_1608Metric, F.Cu at (174.8, 251.6)
- added R1122: 10k, Resistor_SMD:R_0603_1608Metric, F.Cu at (183.2, 251.1)
- added R1123: 1k, Resistor_SMD:R_0603_1608Metric, F.Cu at (190.6, 248.1)
- added R1124: 10k, Resistor_SMD:R_0603_1608Metric, F.Cu at (189.2, 251.1)
- added R1901: 0e, Resistor_SMD:R_0603_1608Metric, F.Cu at (134.6, 264.0)
- added R1902: 0e(dnp), Resistor_SMD:R_0603_1608Metric, F.Cu at (131.6, 264.0)
- added R1903: 10k, Resistor_SMD:R_0603_1608Metric, F.Cu at (125.5, 267.0)
- added R1904: 1k, Resistor_SMD:R_0603_1608Metric, F.Cu at (128.5, 267.0)
- added R1905: 10k, Resistor_SMD:R_0603_1608Metric, F.Cu at (134.6, 265.5)
- added R1906: 10k, Resistor_SMD:R_0603_1608Metric, F.Cu at (131.6, 265.5)
- added R1907: 1k, Resistor_SMD:R_0603_1608Metric, F.Cu at (137.6, 264.0)
- added R1908: 10k, Resistor_SMD:R_0603_1608Metric, F.Cu at (137.6, 265.5)
- added R1911: 10k, Resistor_SMD:R_0603_1608Metric, F.Cu at (128.5, 265.5)
- added R1912: 1k, Resistor_SMD:R_0603_1608Metric, F.Cu at (121.2, 264.0)
- added R1913: 10k, Resistor_SMD:R_0603_1608Metric, F.Cu at (122.5, 267.0)
- added R1914: 10k, Resistor_SMD:R_0603_1608Metric, F.Cu at (125.5, 265.5)
- added R1915: 1k, Resistor_SMD:R_0603_1608Metric, F.Cu at (161.4, 240.5)
- added R1916: 10k, Resistor_SMD:R_0603_1608Metric, F.Cu at (116.5, 266.8)
- added R1931: 0e(dnp), Resistor_SMD:R_0603_1608Metric, F.Cu at (161.4, 242.0)
- added R1932: 0e, Resistor_SMD:R_0603_1608Metric, F.Cu at (119.5, 266.8)
- added U1103: am26ls32a, Package_SO:SOIC-16_3.9x9.9mm_P1.27mm, F.Cu at (185.4, 245.0)
- added U1104: SI8660BD, Package_SO:SOIC-16W_7.5x10.3mm_P1.27mm, F.Cu at (176.0, 245.3)
- added U1803: SN74LVC2G17DBVR, servo:SOT-23-6, B.Cu at (87.7, 113.0)
- added U1804: SN74LVC2G17DBVR, servo:SOT-23-6, B.Cu at (83.8, 113.0)
- added U1901: SI8662BD, Package_SO:SOIC-16W_7.5x10.3mm_P1.27mm, F.Cu at (154.2, 256.3)
- added U1904: SN75C1167DBR, Package_SO:SSOP-16_5.3x6.2mm_P0.65mm, F.Cu at (161.5, 265.3)
- added U1905: SN75C1167DBR, Package_SO:SSOP-16_5.3x6.2mm_P0.65mm, F.Cu at (152.8, 265.3)
- added U1908: SI8662BD, Package_SO:SOIC-16W_7.5x10.3mm_P1.27mm, F.Cu at (154.2, 245.3)
- J1001: footprint servo:tblock02x06 -> Connector_Phoenix_MC:PhoenixContact_MC_1,5_6-G-3.81_1x06_P3.81mm_Horizontal
- J1101: footprint servo:tblock02x08 -> Connector_Phoenix_MC:PhoenixContact_MCV_1,5_10-G-3.81_1x10_P3.81mm_Vertical
- J1201: footprint servo:tblock02x04 -> Connector_Phoenix_MC:PhoenixContact_MC_1,5_4-G-3.81_1x04_P3.81mm_Horizontal
- R1001: value 0e -> 10k
- R1002: value 0e(dnp) -> 1k
- R1003, R1006, R1009, R1012: value 100k -> 10k
- R1004, R1007, R1010: value 120e -> 10k
- R1005, R1008, R1011: value 100k -> 1k
- R1101, R1103, R1104, R1106, R1107, R1109, R1110, R1112: value 100e -> 10k
- R1102, R1105, R1108, R1111: value 100e -> 1k
- U1001: value ADM2483 -> am26ls32a; footprint Package_SO:SOIC-16W_7.5x10.3mm_P1.27mm -> Package_SO:SOIC-16_3.9x9.9mm_P1.27mm
- U1101: value SI8662BD -> SI8660BD
- U1102: value SI8662BD -> am26ls32a; footprint Package_SO:SOIC-16W_7.5x10.3mm_P1.27mm -> Package_SO:SOIC-16_3.9x9.9mm_P1.27mm
- moved U1506 103.1 mm to (73.2, 84.3)
- moved U601 64.8 mm to (280.4, 150.3)
- moved J601 64.1 mm to (285.3, 161.1)
- moved U1503 62.1 mm to (135.1, 84.3)
- moved Y401 23.3 mm to (218.1, 162.2)
- moved U402 23.3 mm to (206.7, 166.9)
- moved J201 23.3 mm to (230.2, 196.6)
- moved U1101 23.3 mm to (166.2, 179.3)
- moved U1201 23.3 mm to (192.3, 179.0)
- moved U1202 23.3 mm to (179.4, 179.3)
- moved U201 23.3 mm to (231.9, 172.8)
- moved U403 23.3 mm to (218.2, 167.8)
- moved U404 23.3 mm to (210.4, 199.6)
- moved Y201 23.3 mm to (230.9, 167.3)
- moved Y402 23.3 mm to (206.0, 161.4)
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Connections:
- net FREE_IN_A3 renamed FAN_RPM1
- net FREE_IN_A3_H renamed FAN_RPM1_H
- net FREE_IN_A4 renamed IGBT_ALARM1
- net FREE_IN_A4_H renamed IGBT_ALARM1_H
- net FREE_IN_B3 renamed FAN_RPM2
- net FREE_IN_B3_H renamed FAN_RPM2_H
- net FREE_IN_B4 renamed IGBT_ALARM2
- net FREE_IN_B4_H renamed IGBT_ALARM2_H
- net Net-(J1501-Pad1) renamed /lem/LemAV_1
- net Net-(J1501-Pad2) renamed /lem/LemAV_2
- net Net-(J1501-Pad3) renamed /lem/LemAV_3
- net Net-(J1501-Pad4) renamed /lem/LemAV_4
- net Net-(J1501-Pad5) renamed /lem/LemAV_5
- net Net-(J1501-Pad6) renamed /lem/LemAV_6
- net Net-(J1502-Pad1) renamed /lem/LemA_All_1
- net Net-(J1502-Pad2) renamed /lem/LemA_All_2
- net Net-(J1502-Pad3) renamed /lem/LemA_All_3
- net Net-(J1502-Pad4) renamed /lem/LemA_All_4
- net Net-(J1502-Pad5) renamed /lem/LemA_All_5
- net Net-(J1502-Pad6) renamed /lem/LemA_All_6
- net Net-(J1503-Pad1) renamed /lem/LemAU_1
- net Net-(J1503-Pad2) renamed /lem/LemAU_2
- net Net-(J1503-Pad3) renamed /lem/LemAU_3
- net Net-(J1503-Pad4) renamed /lem/LemAU_4
- net Net-(J1503-Pad5) renamed /lem/LemAU_5
- net Net-(J1503-Pad6) renamed /lem/LemAU_6
- net Net-(J1504-Pad1) renamed /lem/LemBU_3
- net Net-(J1504-Pad2) renamed /lem/LemBU_2
- net Net-(J1504-Pad3) renamed /lem/LemBU_1
- net Net-(J1504-Pad4) renamed /lem/LemBU_6
- net Net-(J1504-Pad5) renamed /lem/LemBU_5
- net Net-(J1504-Pad6) renamed /lem/LemBU_4
- net Net-(J1505-Pad1) renamed /lem/LemBV_3
- net Net-(J1505-Pad2) renamed /lem/LemBV_2
- net Net-(J1505-Pad3) renamed /lem/LemBV_1
- net Net-(J1505-Pad4) renamed /lem/LemBV_6
- net Net-(J1505-Pad5) renamed /lem/LemBV_5
- net Net-(J1505-Pad6) renamed /lem/LemBV_4
- net Net-(J1506-Pad1) renamed /lem/LemB_All_3
- net Net-(J1506-Pad2) renamed /lem/LemB_All_2
- net Net-(J1506-Pad3) renamed /lem/LemB_All_1
- net Net-(J1506-Pad4) renamed /lem/LemB_All_6
- net Net-(J1506-Pad5) renamed /lem/LemB_All_5
- net Net-(J1506-Pad6) renamed /lem/LemB_All_4
- C214 pad 2: /ethernet/P0_TD_N -> 3V3
- J201 pad 11: 3V3 -> /ethernet/P0_RD_N
- J201 pad 12: /ethernet/P0_RD_N -> 3V3
- J201 pad 7: /ethernet/P0_TD_P -> 3V3
- J201 pad 8: 3V3 -> /ethernet/P0_TD_P
- R1001 pad 1: ENDAT1_CLK -> 5VH
- R1001 pad 2: ENDAT1_Y_SKEW_CLK -> /step_dir/QEP1_A+_H
- R1002 pad 1: ENDAT1_Y_SKEW_CLK -> /step_dir/QEP1_A+_H
- R1002 pad 2: ENDAT1_N_SKEW_CLK -> /step_dir/QEP1_A-_H
- R1003 pad 1: 5VH -> /step_dir/QEP1_A-_H
- R1003 pad 2: Net-(J1001-Pad2a) -> GNDH
- R1004 pad 1: Net-(J1001-Pad2a) -> 5VH
- R1004 pad 2: Net-(J1001-Pad3a) -> /step_dir/QEP1_B+_H
- R1005 pad 1: Net-(J1001-Pad3a) -> /step_dir/QEP1_B+_H
- R1005 pad 2: GNDH -> /step_dir/QEP1_B-_H
- R1006 pad 1: 5VH -> /step_dir/QEP1_B-_H
- R1006 pad 2: Net-(J1001-Pad4a) -> GNDH
- R1007 pad 1: Net-(J1001-Pad4a) -> 5VH
- R1007 pad 2: Net-(J1001-Pad5a) -> Net-(J1001-Pad4b)
- R1008 pad 1: Net-(J1001-Pad5a) -> Net-(J1001-Pad4b)
- R1008 pad 2: GNDH -> Net-(J1001-Pad5b)
- R1009 pad 1: 5VH -> Net-(J1001-Pad5b)
- R1009 pad 2: Net-(J1001-Pad2b) -> GNDH
- R1010 pad 1: Net-(J1001-Pad2b) -> 5VH
- R1010 pad 2: Net-(J1001-Pad3b) -> Net-(J1001-Pad2b)
- R1011 pad 1: Net-(J1001-Pad3b) -> Net-(J1001-Pad2b)
- R1011 pad 2: GNDH -> Net-(J1001-Pad3b)
- R1012 pad 1: 5VH -> Net-(J1001-Pad3b)
- R1012 pad 2: Net-(J1001-Pad4b) -> GNDH
- R1101 pad 1: Net-(C1101-Pad2) -> 5VH
- R1101 pad 2: Net-(J1101-Pad2a) -> /qep/QEP1_A+_H
- R1102 pad 1: Net-(C1102-Pad2) -> /qep/QEP1_A+_H
- R1102 pad 2: Net-(J1101-Pad3a) -> /qep/QEP1_A+_H
- R1103 pad 1: Net-(C1103-Pad2) -> /qep/QEP1_A+_H
- R1103 pad 2: Net-(J1101-Pad4a) -> GNDH
- R1104 pad 1: Net-(C1104-Pad2) -> 5VH
- R1104 pad 2: Net-(J1101-Pad5a) -> /qep/QEP1_B+_H
- R1105 pad 1: Net-(R1105-Pad1) -> /qep/QEP1_B+_H
- R1105 pad 2: Net-(C1105-Pad2) -> /qep/QEP1_B-_H
- R1106 pad 1: Net-(R1106-Pad1) -> /qep/QEP1_B-_H
- R1106 pad 2: Net-(C1106-Pad2) -> GNDH
- R1107 pad 1: Net-(C1112-Pad2) -> 5VH
- R1107 pad 2: Net-(J1101-Pad2b) -> /qep/QEP1_I+_H
- R1108 pad 1: Net-(C1111-Pad2) -> /qep/QEP1_I+_H
- R1108 pad 2: Net-(J1101-Pad3b) -> /qep/QEP1_I-_H
- R1109 pad 1: Net-(C1110-Pad2) -> /qep/QEP1_I-_H
- R1109 pad 2: Net-(J1101-Pad4b) -> GNDH
- R1110 pad 1: Net-(C1109-Pad2) -> 5VH
- R1110 pad 2: Net-(J1101-Pad5b) -> /qep/QEP1_S+_H
- R1111 pad 1: Net-(R1111-Pad1) -> /qep/QEP1_S+_H
- R1111 pad 2: Net-(C1108-Pad2) -> /qep/QEP1_S+_H
- R1112 pad 1: Net-(R1112-Pad1) -> /qep/QEP1_S+_H
- R1112 pad 2: Net-(C1107-Pad2) -> GNDH
- U1001 pad 1: 3V3 -> /step_dir/QEP1_A-_H
- U1001 pad 10: Net-(U1001-Pad10) -> Net-(J1001-Pad4b)
- U1001 pad 11: Net-(U1001-Pad11) -> DIR2_H
- U1001 pad 12: Net-(J1001-Pad2a) -> GNDH
- U1001 pad 13: Net-(J1001-Pad3a) -> STEP2_H
- U1001 pad 14: Net-(U1001-Pad14) -> Net-(J1001-Pad2b)
- U1001 pad 15: GNDH -> Net-(J1001-Pad3b)
- U1001 pad 2: GND -> /step_dir/QEP1_A+_H
- U1001 pad 3: ENDAT1_MISO -> STEP1_H
- U1001 pad 4: ENDAT1_CS -> 5VH
- U1001 pad 5: ENDAT1_CS -> DIR1_H
- U1001 pad 6: ENDAT1_MOSI -> /step_dir/QEP1_B+_H
- U1001 pad 7: 3V3 -> /step_dir/QEP1_B-_H
- U1001 pad 8: GND -> GNDH
- U1001 pad 9: GNDH -> Net-(J1001-Pad5b)
- U1101 pad 10: QEP1_OUT2 -> DIR1
- U1101 pad 11: QEP1_OUT1 -> STEP1
- U1101 pad 2: Net-(C1101-Pad2) -> Net-(U1101-Pad2)
- U1101 pad 3: Net-(C1102-Pad2) -> Net-(U1101-Pad3)
- U1101 pad 4: Net-(C1103-Pad2) -> Net-(U1101-Pad4)
- U1101 pad 5: Net-(C1104-Pad2) -> Net-(U1101-Pad5)
- U1101 pad 6: Net-(R1105-Pad1) -> STEP1_H
- U1101 pad 7: Net-(R1106-Pad1) -> DIR1_H
- U1102 pad 1: 5VH -> /qep/QEP1_A+_H
- U1102 pad 10: QEP2_OUT2 -> /qep/QEP1_I+_H
- U1102 pad 11: QEP2_OUT1 -> Net-(U1101-Pad4)
- U1102 pad 12: QEP2_S -> GNDH
- U1102 pad 13: QEP2_I -> Net-(U1101-Pad5)
- U1102 pad 14: QEP2_B -> /qep/QEP1_S+_H
- U1102 pad 15: QEP2_A -> /qep/QEP1_S+_H
- U1102 pad 16: 3V3 -> 5VH
- U1102 pad 2: Net-(C1112-Pad2) -> /qep/QEP1_A+_H
- U1102 pad 3: Net-(C1111-Pad2) -> Net-(U1101-Pad2)
- U1102 pad 4: Net-(C1110-Pad2) -> 5VH
- U1102 pad 5: Net-(C1109-Pad2) -> Net-(U1101-Pad3)
- U1102 pad 6: Net-(R1111-Pad1) -> /qep/QEP1_B+_H
- U1102 pad 7: Net-(R1112-Pad1) -> /qep/QEP1_B-_H
- U1102 pad 9: GND -> /qep/QEP1_I-_H
- U1801 pad 6: Net-(C1805-Pad1) -> Net-(U1801-Pad6)
- U1802 pad 6: Net-(C1808-Pad1) -> Net-(U1802-Pad6)
- U301 pad A15: QEP2_OUT1 -> Net-(U301-PadA15)
- U301 pad A17: Net-(U301-PadA17) -> DIR2
- U301 pad B15: QEP2_OUT2 -> Net-(U301-PadB15)
- U301 pad B18: Net-(U301-PadB18) -> STEP2
- U301 pad B19: Net-(U301-PadB19) -> STEP1
- U301 pad C15: QEP1_OUT1 -> Net-(U301-PadC15)
- U301 pad C18: Net-(U301-PadC18) -> DIR1
- U301 pad D15: QEP1_OUT2 -> Net-(U301-PadD15)
Routing:
- net /lem/LemB_All_1: track 0.00 -> 34.1 mm
- net /lem/LemB_All_6: track 0.00 -> 25.2 mm
- net /lem/LemB_All_5: track 0.00 -> 20.1 mm
- net /lem/LemB_All_4: track 0.00 -> 14.2 mm
- net /lem/LemB_All_3: track 0.00 -> 6.89 mm
Other:
- net class High_Current added: clearance 0.4, trace_width 2, via_dia 2, via_drill 1.5
- rule trace_min: 0.2 -> 0.152
- rule via_min_drill: 0.3 -> 0.25

Commit message: changed 200mils connector to 150mils 'cause space constraints
I've decided to change 200 mils input connector for encat, rs485 and so
for 150mis 'cose it doesn't deliver so much current and I'd save some
space in the board. I've added the step/dir differential interface that
I've fotgot, and also add differential input to all signals of
incremental encoder interface A/B/I/S .. now lets rock
Parts:
- removed J602: Conn_01x02, Connector_PinHeader_2.54mm:PinHeader_1x02_P2.54mm_Vertical_SMD_Pin1Left
- J1001, J1901: footprint Connector_Phoenix_MC:PhoenixContact_MC_1,5_6-G-3.81_1x06_P3.81mm_Horizontal -> servo:tblock02x6_3.81
- J1101: footprint Connector_Phoenix_MC:PhoenixContact_MCV_1,5_10-G-3.81_1x10_P3.81mm_Vertical -> servo:tblock02x10_3.81
- J1201: footprint Connector_Phoenix_MC:PhoenixContact_MC_1,5_4-G-3.81_1x04_P3.81mm_Horizontal -> servo:tblock02x4_3.81
- J201: moved to F.Cu
- J601: value Conn_02x05_Counter_Clockwise -> dbg_conn; footprint Connector_IDC:IDC-Header_2x05_P2.54mm_Horizontal -> Connector_PinSocket_2.54mm:PinSocket_2x06_P2.54mm_Horizontal
- JP1202: value Jumper_3_Bridged12 -> jumper
- R1201, R1203: value 1k -> 10k
- R1205: value 120e -> 1k
- moved U1104 97.3 mm to (110.3, 173.6), turned to 90 degrees
- moved U1901 87.3 mm to (126.3, 173.6), turned to 270 degrees
- moved U1103 85.2 mm to (125.4, 184.5), turned to 90 degrees
- moved U1904 81.8 mm to (145.4, 185.1), turned to 90 degrees
- moved U1905 80.3 mm to (155.4, 185.1), turned to 90 degrees
- moved U1908 72.7 mm to (142.3, 173.6), turned to 270 degrees
- moved U1101 72.2 mm to (94.2, 173.6)
- moved J601 71.7 mm to (225.6, 200.7), turned to 90 degrees
- moved J1901 52.2 mm to (151.4, 204.8)
- moved U1102 22.1 mm to (107.9, 184.5)
- moved U1202 21.8 mm to (158.3, 173.6)
- moved U201 20.2 mm to (212.1, 176.5)
- moved U1201 19.0 mm to (174.0, 173.9)
- moved U401 18.7 mm to (229.9, 194.3)
- moved Y401 17.5 mm to (200.7, 163.8)
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Connections:
- net Net-(F701-Pad2) renamed /ac_in/AC_L_C
- net Net-(F702-Pad2) renamed /ac_in/AC_L_H'
- net Net-(J701-Pad3b) renamed /ac_in/AC_N
- J601 pad 10: /uc_clk_dbg/PRG_TCK -> /uc_clk_dbg/PRG_TMS
- J601 pad 6: /uc_clk_dbg/PRG_TDO -> GND
- J601 pad 7: /uc_clk_dbg/PRG_TRSTn -> DACB_DBG_OUT
- J601 pad 8: /uc_clk_dbg/PRG_TMS -> /uc_clk_dbg/PRG_TDO
- J601 pad 9: /uc_clk_dbg/PRG_TDI -> /uc_clk_dbg/PRG_TRSTn
- JP1202 pad 1: 5VH -> Earth
- JP1202 pad 2: Net-(J1201-Pad1b) -> Net-(J1201-Pad4a)
- JP1202 pad 3: 15VH -> GNDH
- R303 pad 1: DACB_DBG_OUT -> DACB_DBG
- R608 pad 1: DACB_DBG_OUT -> DACB_DBG
- R609 pad 2: Net-(J602-Pad1) -> DACB_DBG_OUT
