File: kicad/servo.kicad_pcb (KiCad board)
At the start: 6 copper layers, 180 x 155 mm, 548 parts, among them IC201 TPD4E001QDBV, IC301 TPD4E001QDBV, IC302 TPD4E001QDBV, IC303 TPD4E001QDBV, IC304 TPD4E001QDBV, IC305 TPD4E001QDBV, J1001 tblock2x6, J1101 tblock, J1201 tblock2x4, J1401 NHD-4.3-480272FT-CTXL-T, J1402 Conn_01x02, J1501 tblock2x3, J1502 tblock2x3, J1503 tblock2x3, J1504 tblock2x3, J1505 tblock2x3, J1506 tblock2x3, J1701 NHD-4.3-480272FT-CTXL-T, J1702 NHD-4.3-480272FT-CTXL-T, J1703 NHD-4.3-480272FT-CTXL-T, J1901 tblock2x6, J201 0821-1X1T-36-F, J601 dbg_conn, J701 tblock, SW1403 SW_Push, SW1404 SW_Push, U1001 am26ls32a, U1101 SI8660BD, U1102 am26ls32a, U1103 am26ls32a, U1104 SI8660BD, U1201 ISO1050, U1202 ADM2483, U1401 PAM8301, U1501 LXS6-NPS, U1502 LXS6-NPS, U1503 LXS6-NPS, U1504 LXS6-NPS, U1505 LXS6-NPS, U1506 LXS6-NPS, U1601 AMC1311B, U1602 AMC1311B, U1603 RFM-0505S, U1604 RFM-0505S, U1801 SI8661BD, U1802 SI8661BD, U1803 SN74LVC2G17DBVR, U1804 SN74LVC2G17DBVR, U1901 SI8662BD, U1904 SN75C1167DBR, U1905 SN75C1167DBR, U1908 SI8662BD, U201 DP83822, U301 TMS320F28388DZWTS, U401 CAT24C16WI, U402 DP83822, U403 DP83822, U404 rj45x2, U601 SN74ALVC244PW, U602 M25PX32-VMW, U702 R-78E3.3-1.0, U704 R-78E5.0-1.0, U705 AP2114H-1.2TRG1, U706 AP2114H-1.2TRG1, U801 SI8660BD, U802 SI8662BD, U803 SN74LVC2G17DBVR, U804 SN74LVC2G17DBVR, U805 SN74LVC2G17DBVR, U806 SN74LVC2G17DBVR, U807 SN74LVC2G17DBVR, U808 SN74LVC2G17DBVR, U809 SN74LVC2G17DBVR, U810 SN74LVC2G17DBVR, U811 SN74LVC2G17DBVR, U812 SN74LVC2G17DBVR, U813 SI8660BD, U814 SI8662BD, U901 AMC1311B, U902 AMC1311B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

Commit message: placing smmall capacitors and resistors nerar his group
Parts:
- removed R302, R303, R304, R305, R306, R307, R308, R309, R310, R311, R312, R313, R314, R315, R316, R317, R318, R319, R320, R321: 10e, Resistor_SMD:R_0603_1608Metric
- added C1101: 100nF, servo:C_0603_1608Metric, B.Cu at (120.6, 172.7)
- added C1102: 100nF, servo:C_0603_1608Metric, B.Cu at (119.4, 178.3)
- added C1103: 100nF, servo:C_0603_1608Metric, B.Cu at (122.2, 179.5)
- added C1104: 100nF, servo:C_0603_1608Metric, B.Cu at (104.2, 179.5)
- added C1105: 100nF, servo:C_0603_1608Metric, B.Cu at (99.8, 179.9)
- added C1106: 100nF, servo:C_0603_1608Metric, B.Cu at (102.2, 173.5)
- added C1203: 100nF, servo:C_0603_1608Metric, B.Cu at (168.6, 183.1)
- added C1204: 100nF, servo:C_0603_1608Metric, B.Cu at (165.8, 168.3)
- added C1813: 100pF, servo:C_0603_1608Metric, B.Cu at (92.6, 96.7)
- added C1814: 100pF, servo:C_0603_1608Metric, B.Cu at (95.0, 105.1)
- added C1815: 100pF, servo:C_0603_1608Metric, B.Cu at (89.0, 105.1)
- added C1816: 100pF, servo:C_0603_1608Metric, B.Cu at (75.0, 104.3)
- added C1817: 100pF, servo:C_0603_1608Metric, B.Cu at (81.0, 104.3)
- added C1818: 100pF, servo:C_0603_1608Metric, B.Cu at (78.2, 96.7)
- added C917: 100nF, servo:C_0603_1608Metric, B.Cu at (103.7, 103.5)
- added C918: 100nF, servo:C_0603_1608Metric, B.Cu at (103.7, 102.0)
- added R1801: 10e, Resistor_SMD:R_0603_1608Metric, B.Cu at (94.6, 108.7)
- added R1812: 10e, Resistor_SMD:R_0603_1608Metric, B.Cu at (84.9, 104.0)
- C1201, C1202, C1801, C1802, C1803, C1804, C1805, C1806, C1808, C1810, C1811, C1901, C1904, C1905, C1910, C1913, C1914, C301, C302, C303, C304, C401, C402, C404, C406, C408, C410, C412, C413, C414, C415, C416, C417, C418, C419, C420, C421, C422, C423, C424, C425, C426, C427, C428, C429, C430, C431, C432, C433, C501, C502, C503, C504, C505, C506, C507, C508, C509, C510, C511, C512, C513, C514, C515, C516, C517, C518, C519, C520, C521, C522, C523, C524, C525, C526, C527, C528, C529, C530, C531, C601, C901, C902, C903, C904, C905, C906, C907, C908, C909, C910, C911, C912, C913, C914, C915, C916, D401, JP1101, JP1201, JP1202, JP1901, R1101, R1102, R1103, R1104, R1105, R1106, R1108, R1109, R1110, R1111, R1112, R1113, R1114, R1115, R1116, R1117, R1118, R1119, R1120, R1121, R1122, R1123, R1124, R1201, R1202, R1203, R1204, R1205, R1206, R1802, R1803, R1804, R1805, R1807, R1808, R1809, R1810, R1811, R1901, R1902, R1903, R1904, R1905, R1906, R1907, R1908, R1911, R1912, R1913, R1914, R1916, R1931, R1932, R301, R401, R402, R403, R404, R405, R406, R407, R408, R409, R410, R411, R413, R414, R415, R416, R417, R418, R419, R420, R421, R422, R423, R424, R425, R426, R427, R428, R429, R430, R431, R432, R433, R434, R435, R436, R437, R438, R439, R440, R441, R442, R445, R446, R608, R901, R902, R903, R904, R905, R906, R907, R908, R909, R910, R911, R912, R913, R914, R915, R916, R917, R918, R920, R921, R922, R923: moved to B.Cu
- C217, C434: footprint servo:C_0603_1608Metric -> Capacitor_SMD:C_1206_3216Metric; moved to B.Cu
- L501, L502, L503: footprint Inductor_SMD:L_0603_1608Metric -> Inductor_SMD:L_1206_3216Metric_Pad1.42x1.75mm_HandSolder; moved to B.Cu
- U1001, U1102, U1103: footprint Package_SO:SOIC-16_3.9x9.9mm_P1.27mm -> Package_SO:SOIC-16W_5.3x10.2mm_P1.27mm; moved to B.Cu
- U1904, U1905: value SN75C1167DBR -> SN75C1168DBR; footprint Package_SO:SSOP-16_5.3x6.2mm_P0.65mm -> Package_SO:SOIC-16W_5.3x10.2mm_P1.27mm; moved to B.Cu
- U201, U402, U403: footprint Package_DFN_QFN:QFN-32-1EP_5x5mm_P0.5mm_EP3.1x3.1mm_ThermalVias -> servo:QFN-32-1EP_5x5mm_P0.5mm_EP2.9x2.9mm_ThermalVias
- moved R903 300.4 mm to (77.4, 163.1)
- moved R904 300.3 mm to (77.0, 168.7)
- moved C906 298.8 mm to (73.0, 147.5)
- moved C904 294.0 mm to (77.0, 166.7)
- moved C909 290.9 mm to (87.4, 147.5)
- moved C902 290.5 mm to (77.4, 164.7)
- moved R921 290.2 mm to (87.4, 167.1)
- moved C915 287.5 mm to (87.4, 165.1)
- moved R914 286.6 mm to (87.8, 153.5)
- moved R906 285.7 mm to (77.4, 149.9)
- moved C908 285.3 mm to (77.4, 145.9)
- moved C913 285.0 mm to (87.4, 169.1)
- moved C911 284.6 mm to (87.8, 149.9)
- moved R922 283.5 mm to (96.6, 167.1)
- moved R915 283.1 mm to (87.4, 155.1)
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Connections:
- net /sheet5F8D42BF/ENDAT1_CLK_H renamed /endat/ENDAT1_CLK_H
- net /sheet5F8D42BF/ENDAT1_CS_H renamed /endat/ENDAT1_CS_H
- net /sheet5F8D42BF/ENDAT1_MISO_H renamed /endat/ENDAT1_MISO_H
- net /sheet5F8D42BF/ENDAT1_MOSI_H renamed /endat/ENDAT1_MOSI_H
- net /sheet5F8D42BF/ENDAT2_CLK_H renamed /endat/ENDAT2_CLK_H
- net /sheet5F8D42BF/ENDAT2_CS_H renamed /endat/ENDAT2_CS_H
- net /sheet5F8D42BF/ENDAT2_MISO_H renamed /endat/ENDAT2_MISO_H
- net /sheet5F8D42BF/ENDAT2_MOSI_H renamed /endat/ENDAT2_MOSI_H
- net Net-(J1001-Pad2b) renamed /step_dir/STEP2_A+_H
- net Net-(J1001-Pad3b) renamed /step_dir/STEP2_A-_H
- net Net-(J1001-Pad4b) renamed /step_dir/STEP2_B+_H
- net Net-(J1001-Pad5b) renamed /step_dir/STEP2_B-_H
- IC301 pad 1: Net-(IC301-Pad1) -> DACB_DBG
- IC301 pad 3: Net-(IC301-Pad3) -> NTCA1_P
- IC301 pad 4: Net-(IC301-Pad4) -> NTCA1_N
- IC301 pad 6: Net-(IC301-Pad6) -> LCD_AUDIO
- IC302 pad 1: Net-(IC302-Pad1) -> NTCB1_N
- IC302 pad 3: Net-(IC302-Pad3) -> LEM_B_U
- IC302 pad 4: Net-(IC302-Pad4) -> LEM_B_V
- IC302 pad 6: Net-(IC302-Pad6) -> NTCB1_P
- IC303 pad 1: Net-(IC303-Pad1) -> VBUS_B_P
- IC303 pad 3: Net-(IC303-Pad3) -> VBUS_B_N
- IC303 pad 4: Net-(IC303-Pad4) -> NTCA2_P
- IC303 pad 6: Net-(IC303-Pad6) -> LEM_B_ALL
- IC304 pad 1: Net-(IC304-Pad1) -> NTCB2_P
- IC304 pad 3: Net-(IC304-Pad3) -> NTCB2_N
- IC304 pad 4: Net-(IC304-Pad4) -> LEM_A_U
- IC304 pad 6: Net-(IC304-Pad6) -> NTCA2_N
- IC305 pad 1: Net-(IC305-Pad1) -> LEM_A_ALL
- IC305 pad 3: Net-(IC305-Pad3) -> VBUS_A_P
- IC305 pad 4: Net-(IC305-Pad4) -> VBUS_A_N
- IC305 pad 6: Net-(IC305-Pad6) -> LEM_A_V
- J1001 pad 2a: /step_dir/QEP1_A+_H -> /step_dir/STEP1_A+_H
- J1001 pad 3a: /step_dir/QEP1_A-_H -> /step_dir/STEP1_A-_H
- J1001 pad 4a: /step_dir/QEP1_B+_H -> /step_dir/STEP1_B+_H
- J1001 pad 5a: /step_dir/QEP1_B-_H -> /step_dir/STEP1_B-_H
- J1101 pad 2b: /qep/QEP1_A+_H -> /qep/QEP2_A+_H
- J1101 pad 3a: /qep/QEP1_A+_H -> /qep/QEP1_A-_H
- J1101 pad 3b: /qep/QEP1_A+_H -> /qep/QEP2_A-_H
- J1101 pad 4b: /qep/QEP1_B+_H -> /qep/QEP2_B+_H
- J1101 pad 5b: /qep/QEP1_B-_H -> /qep/QEP2_B-_H
- J1101 pad 6b: /qep/QEP1_I+_H -> /qep/QEP2_I+_H
- J1101 pad 7b: /qep/QEP1_I-_H -> /qep/QEP2_I-_H
- J1101 pad 8b: /qep/QEP1_S+_H -> /qep/QEP2_S+_H
- J1101 pad 9a: /qep/QEP1_S+_H -> /qep/QEP1_S-_H
- J1101 pad 9b: /qep/QEP1_S+_H -> /qep/QEP2_S-_H
- J1501 pad 1: /lem/LemAV_1 -> /lem/LemAV_4
- J1501 pad 2: /lem/LemAV_2 -> /lem/LemAV_5
- J1501 pad 3: /lem/LemAV_3 -> /lem/LemAV_1
- J1501 pad 4: /lem/LemAV_4 -> /lem/LemAV_3
- J1501 pad 5: /lem/LemAV_5 -> /lem/LemAV_2
- J1502 pad 1: /lem/LemA_All_1 -> /lem/LemA_All_4
- J1502 pad 2: /lem/LemA_All_2 -> /lem/LemA_All_5
- J1502 pad 3: /lem/LemA_All_3 -> /lem/LemA_All_1
- J1502 pad 4: /lem/LemA_All_4 -> /lem/LemA_All_3
- J1502 pad 5: /lem/LemA_All_5 -> /lem/LemA_All_2
- J1503 pad 1: /lem/LemAU_1 -> /lem/LemAU_4
- J1503 pad 2: /lem/LemAU_2 -> /lem/LemAU_5
- J1503 pad 3: /lem/LemAU_3 -> /lem/LemAU_1
- J1503 pad 4: /lem/LemAU_4 -> /lem/LemAU_3
- J1503 pad 5: /lem/LemAU_5 -> /lem/LemAU_2
- J1504 pad 1: /lem/LemBU_3 -> /lem/LemBU_4
- J1504 pad 2: /lem/LemBU_2 -> /lem/LemBU_5
- J1504 pad 4: /lem/LemBU_6 -> /lem/LemBU_3
- J1504 pad 5: /lem/LemBU_5 -> /lem/LemBU_2
- J1504 pad 6: /lem/LemBU_4 -> /lem/LemBU_6
- J1505 pad 1: /lem/LemBV_3 -> /lem/LemBV_4
- J1505 pad 2: /lem/LemBV_2 -> /lem/LemBV_5
- J1505 pad 4: /lem/LemBV_6 -> /lem/LemBV_3
- J1505 pad 5: /lem/LemBV_5 -> /lem/LemBV_2
- J1505 pad 6: /lem/LemBV_4 -> /lem/LemBV_6
- J1506 pad 1: /lem/LemB_All_3 -> /lem/LemB_All_4
- J1506 pad 2: /lem/LemB_All_2 -> /lem/LemB_All_5
- J1506 pad 4: /lem/LemB_All_6 -> /lem/LemB_All_3
- J1506 pad 5: /lem/LemB_All_5 -> /lem/LemB_All_2
- J1506 pad 6: /lem/LemB_All_4 -> /lem/LemB_All_6
- R1001 pad 2: /step_dir/QEP1_A+_H -> /step_dir/STEP1_A+_H
- R1002 pad 1: /step_dir/QEP1_A+_H -> /step_dir/STEP1_A+_H
- R1002 pad 2: /step_dir/QEP1_A-_H -> /step_dir/STEP1_A-_H
- R1003 pad 1: /step_dir/QEP1_A-_H -> /step_dir/STEP1_A-_H
- R1004 pad 2: /step_dir/QEP1_B+_H -> /step_dir/STEP1_B+_H
- R1005 pad 1: /step_dir/QEP1_B+_H -> /step_dir/STEP1_B+_H
- R1005 pad 2: /step_dir/QEP1_B-_H -> /step_dir/STEP1_B-_H
- R1006 pad 1: /step_dir/QEP1_B-_H -> /step_dir/STEP1_B-_H
- R1102 pad 2: /qep/QEP1_A+_H -> /qep/QEP1_A-_H
- R1103 pad 1: /qep/QEP1_A+_H -> /qep/QEP1_A-_H
- R1111 pad 2: /qep/QEP1_S+_H -> /qep/QEP1_S-_H
- R1112 pad 1: /qep/QEP1_S+_H -> /qep/QEP1_S-_H
- R1113 pad 2: /qep/QEP1_S+_H -> /qep/QEP2_S+_H
- R1114 pad 1: /qep/QEP1_S+_H -> /qep/QEP2_S+_H
- R1114 pad 2: /qep/QEP1_S+_H -> /qep/QEP2_S-_H
- R1115 pad 1: /qep/QEP1_S+_H -> /qep/QEP2_S-_H
- R1116 pad 2: /qep/QEP1_I+_H -> /qep/QEP2_I+_H
- R1117 pad 1: /qep/QEP1_I+_H -> /qep/QEP2_I+_H
- R1117 pad 2: /qep/QEP1_I-_H -> /qep/QEP2_I-_H
- R1118 pad 1: /qep/QEP1_I-_H -> /qep/QEP2_I-_H
- R1119 pad 2: /qep/QEP1_B+_H -> /qep/QEP2_B+_H
- R1120 pad 1: /qep/QEP1_B+_H -> /qep/QEP2_B+_H
- R1120 pad 2: /qep/QEP1_B-_H -> /qep/QEP2_B-_H
- R1121 pad 1: /qep/QEP1_B-_H -> /qep/QEP2_B-_H
- R1122 pad 2: /qep/QEP1_A+_H -> /qep/QEP2_A+_H
- R1123 pad 1: /qep/QEP1_A+_H -> /qep/QEP2_A+_H
- R1123 pad 2: /qep/QEP1_A+_H -> /qep/QEP2_A-_H
- R1124 pad 1: /qep/QEP1_A+_H -> /qep/QEP2_A-_H
- R427 pad 1: 3V3 -> ECAT_MDIO
- R427 pad 2: ECAT_MDIO -> 3V3
- R428 pad 1: 3V3 -> ECAT_MDIO
- R428 pad 2: ECAT_MDIO -> 3V3
- R429 pad 1: /ethercat/P0_TD_P -> 3V3
- R429 pad 2: 3V3 -> /ethercat/P0_TD_P
- R430 pad 1: /ethercat/P1_TD_P -> 3V3
- R430 pad 2: 3V3 -> /ethercat/P1_TD_P
- R431 pad 1: /ethercat/P0_TD_N -> 3V3
- R431 pad 2: 3V3 -> /ethercat/P0_TD_N
- R432 pad 1: /ethercat/P1_TD_N -> 3V3
- R432 pad 2: 3V3 -> /ethercat/P1_TD_N
- R435 pad 1: /ethercat/P0_RD_P -> 3V3
- R435 pad 2: 3V3 -> /ethercat/P0_RD_P
- R437 pad 1: /ethercat/P0_RD_N -> 3V3
- R437 pad 2: 3V3 -> /ethercat/P0_RD_N
- R438 pad 1: /ethercat/P1_RD_P -> 3V3
- R438 pad 2: 3V3 -> /ethercat/P1_RD_P
- R440 pad 1: /ethercat/P1_RD_N -> 3V3
- R440 pad 2: 3V3 -> /ethercat/P1_RD_N
- U1001 pad 1: /step_dir/QEP1_A-_H -> /step_dir/STEP1_B-_H
- U1001 pad 2: /step_dir/QEP1_A+_H -> /step_dir/STEP1_B+_H
- U1001 pad 6: /step_dir/QEP1_B+_H -> /step_dir/STEP1_A+_H
- U1001 pad 7: /step_dir/QEP1_B-_H -> /step_dir/STEP1_A-_H
- U1102 pad 1: /qep/QEP1_A+_H -> /qep/QEP1_A-_H
- U1102 pad 15: /qep/QEP1_S+_H -> /qep/QEP1_S-_H
- U1103 pad 1: /qep/QEP1_A+_H -> /qep/QEP2_A-_H
- U1103 pad 10: /qep/QEP1_I+_H -> /qep/QEP2_I+_H
- U1103 pad 14: /qep/QEP1_S+_H -> /qep/QEP2_S+_H
- U1103 pad 15: /qep/QEP1_S+_H -> /qep/QEP2_S-_H
- U1103 pad 2: /qep/QEP1_A+_H -> /qep/QEP2_A+_H
- U1103 pad 6: /qep/QEP1_B+_H -> /qep/QEP2_B+_H
- U1103 pad 7: /qep/QEP1_B-_H -> /qep/QEP2_B-_H
- U1103 pad 9: /qep/QEP1_I-_H -> /qep/QEP2_I-_H
- U1803 pad 6: PWM4SD_A_CLK_H -> Net-(R1801-Pad1)
- U1804 pad 6: PWM4SD_B_CLK_H -> Net-(R1812-Pad1)
- U301 pad P3: Net-(IC304-Pad6) -> NTCA2_N
- U301 pad P4: Net-(IC304-Pad3) -> NTCB2_N
- U301 pad R3: Net-(IC303-Pad4) -> NTCA2_P
- U301 pad R4: Net-(IC304-Pad1) -> NTCB2_P
- U301 pad T1: Net-(IC301-Pad1) -> DACB_DBG
- U301 pad T2: Net-(IC301-Pad4) -> NTCA1_N
- U301 pad T3: Net-(IC302-Pad1) -> NTCB1_N
- U301 pad T5: Net-(IC304-Pad4) -> LEM_A_U
- U301 pad T6: Net-(IC305-Pad1) -> LEM_A_ALL
- U301 pad T7: Net-(IC305-Pad3) -> VBUS_A_P
- U301 pad U1: Net-(IC301-Pad6) -> LCD_AUDIO
- U301 pad U2: Net-(IC301-Pad3) -> NTCA1_P
- U301 pad U3: Net-(IC302-Pad6) -> NTCB1_P
- U301 pad U5: Net-(IC305-Pad6) -> LEM_A_V
- U301 pad U7: Net-(IC305-Pad4) -> VBUS_A_N
- U301 pad V2: Net-(IC302-Pad3) -> LEM_B_U
- U301 pad V3: Net-(IC303-Pad6) -> LEM_B_ALL
- U301 pad V4: Net-(IC303-Pad1) -> VBUS_B_P
- U301 pad W2: Net-(IC302-Pad4) -> LEM_B_V
- U301 pad W4: Net-(IC303-Pad3) -> VBUS_B_N
- Y402 pad 1: 3V3 -> GND
- Y402 pad 2: GND -> 3V3
- Y402 pad 3: Net-(R426-Pad1) -> 3V3
- Y402 pad 4: 3V3 -> Net-(R426-Pad1)
Routing:
- net /qep/QEP1_S-_H: track 0.00 -> 37.7 mm
- net /lem/LemBU_5: track 0.00 -> 33.1 mm
- net /lem/LemAU_1: track 0.00 -> 31.4 mm
- net /lem/LemAV_1: track 0.00 -> 31.4 mm
- net /lem/LemA_All_1: track 0.00 -> 31.4 mm
- net /lem/LemBV_1: track 0.00 -> 31.4 mm
- net /lem/LemBU_1: track 0.00 -> 31.4 mm
- net /lem/LemAU_5: track 0.00 -> 31.2 mm
- net /lem/LemAV_5: track 0.00 -> 31.0 mm
- net /step_dir/STEP1_A+_H: track 0.00 -> 30.3 mm
- net /lem/LemBV_5: track 0.00 -> 29.0 mm
- net /lem/LemA_All_5: track 0.00 -> 29.0 mm
- net GNDH: track 0.00 -> 26.7 mm, vias 0 -> 1
- net /lem/LemA_All_6: track 0.00 -> 25.7 mm
- net /lem/LemAU_4: track 0.00 -> 24.2 mm
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Other:
- net class medium_signal added: clearance 0.25, trace_width 0.25, via_dia 0.8, via_drill 0.4
- net class small_signal added: clearance 0.1238, trace_width 0.1524, via_dia 0.457, via_drill 0.3
- net class vcc added: clearance 0.4, trace_width 0.5, via_dia 1, via_drill 0.5
- rule trace_min: 0.152 -> 0.1524
- rule via_min_drill: 0.25 -> 0.2032

Commit message: keep placing
Parts:
- removed C1503, C1506, C1507, C1516, C1517, C1518: 100pF, servo:C_0603_1608Metric
- added C825: 10u, servo:C_0603_1608Metric, B.Cu at (134.2, 137.5)
- added C826: 10u, servo:C_0603_1608Metric, B.Cu at (134.2, 149.9)
- added C827: 0.1u, servo:C_0603_1608Metric, B.Cu at (123.0, 153.5)
- added C828: 0.1u, servo:C_0603_1608Metric, B.Cu at (123.0, 149.9)
- added C829: 0.1u, servo:C_0603_1608Metric, B.Cu at (123.0, 146.3)
- added C830: 0.1u, servo:C_0603_1608Metric, B.Cu at (123.0, 140.7)
- added C831: 0.1u, servo:C_0603_1608Metric, B.Cu at (123.0, 137.1)
- added C832: 0.1u, servo:C_0603_1608Metric, B.Cu at (129.0, 149.9)
- added C833: 10u, servo:C_0603_1608Metric, B.Cu at (134.2, 107.9)
- added C834: 10u, servo:C_0603_1608Metric, B.Cu at (133.8, 121.1)
- added C835: 0.1u, servo:C_0603_1608Metric, B.Cu at (129.0, 137.1)
- added C836: 0.1u, servo:C_0603_1608Metric, B.Cu at (128.6, 107.5)
- added C837: 0.1u, servo:C_0603_1608Metric, B.Cu at (129.0, 120.7)
- added C838: 0.1u, servo:C_0603_1608Metric, B.Cu at (123.0, 107.9)
- added C839: 0.1u, servo:C_0603_1608Metric, B.Cu at (123.0, 111.5)
- added C840: 0.1u, servo:C_0603_1608Metric, B.Cu at (123.0, 117.9)
- added C841: 0.1u, servo:C_0603_1608Metric, B.Cu at (123.0, 121.5)
- added C842: 0.1u, servo:C_0603_1608Metric, B.Cu at (123.0, 125.1)
- added IC306: TPD4E001QDBV, Package_TO_SOT_SMD:SOT-23-6, B.Cu at (154.6, 90.7)
- C1401, C1402, C1403, C1404, C1405, C1501, C1502, C1504, C1505, C1508, C1509, C1510, C1511, C1512, C1513, C1514, C1515, C201, C202, C203, C204, C205, C206, C207, C208, C209, C210, C211, C212, C213, C214, C215, C216, C403, C405, C407, C409, C411, C801, C802, C803, C804, C805, C806, C807, C808, C809, C810, C811, C812, C813, C814, C815, C816, C817, C818, C819, C820, C821, C822, C823, C824, R1401, R1402, R1403, R1404, R1501, R1502, R1503, R1504, R1505, R1506, R1507, R1508, R1509, R1510, R1511, R1512, R201, R202, R203, R204, R205, R206, R207, R208, R209, R212, R609: moved to B.Cu
- J1402: footprint Connector_PinHeader_2.54mm:PinHeader_1x02_P2.54mm_Vertical_SMD_Pin1Left -> Connector_Molex:Molex_KK-254_AE-6410-02A_1x02_P2.54mm_Vertical
- moved C1504 257.7 mm to (79.8, 88.7), turned to 180 degrees
- moved C1509 252.0 mm to (88.2, 91.9), turned to 270 degrees
- moved R1502 251.3 mm to (105.8, 91.1), turned to 90 degrees
- moved R1501 250.2 mm to (107.3, 91.1), turned to 90 degrees
- moved R1505 249.3 mm to (85.4, 91.9), turned to 270 degrees
- moved C1505 236.7 mm to (100.6, 88.7), turned to 180 degrees
- moved C411 233.1 mm to (189.4, 169.5)
- moved R1402 230.3 mm to (237.0, 158.2)
- moved C1501 229.5 mm to (109.0, 91.1), turned to 90 degrees
- moved C409 228.7 mm to (189.4, 170.7)
- moved C403 226.8 mm to (199.8, 171.9)
- moved C407 226.8 mm to (194.2, 173.1), turned to 90 degrees
- moved C1508 225.0 mm to (121.8, 88.3), turned to 180 degrees
- moved R1401 224.7 mm to (237.0, 154.2)
- moved C1512 221.9 mm to (183.4, 88.3), turned to 180 degrees
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Connections:
- IC301 pad 1: DACB_DBG -> NTCA1_N
- IC301 pad 3: NTCA1_P -> NTCB1_P
- IC301 pad 4: NTCA1_N -> NTCB1_N
- IC301 pad 6: LCD_AUDIO -> NTCA1_P
- IC302 pad 1: NTCB1_N -> NTCA2_N
- IC302 pad 3: LEM_B_U -> NTCB2_P
- IC302 pad 4: LEM_B_V -> NTCB2_N
- IC302 pad 6: NTCB1_P -> NTCA2_P
- IC303 pad 1: VBUS_B_P -> LEM_B_V
- IC303 pad 3: VBUS_B_N -> LEM_B_ALL
- IC303 pad 4: NTCA2_P -> Net-(IC303-Pad4)
- IC303 pad 6: LEM_B_ALL -> LEM_B_U
- IC304 pad 1: NTCB2_P -> VBUS_B_N
- IC304 pad 3: NTCB2_N -> VBUS_A_P
- IC304 pad 4: LEM_A_U -> VBUS_A_N
- IC304 pad 6: NTCA2_N -> VBUS_B_P
- IC305 pad 1: LEM_A_ALL -> DACB_DBG
- IC305 pad 3: VBUS_A_P -> Net-(IC305-Pad3)
- IC305 pad 4: VBUS_A_N -> Net-(IC305-Pad4)
- IC305 pad 6: LEM_A_V -> LCD_AUDIO
- R204 pad 1: 3V3 -> ENET_MDIO
- R204 pad 2: ENET_MDIO -> 3V3
- Y201 pad 1: 3V3 -> GND
- Y201 pad 2: GND -> 3V3
- Y201 pad 3: Net-(R203-Pad1) -> 3V3
- Y201 pad 4: 3V3 -> Net-(R203-Pad1)

Commit message: All IC placed inside board size but....
I've placed all stuff on board size even thought all are in groups I've
to move the IC to route them. Let's begin
Parts:
- removed D601, D602: blue@2mA, servo:LED_0603_1608Metric
- removed R428: 2.2k, Resistor_SMD:R_0603_1608Metric
- removed R601, R602: 680, Resistor_SMD:R_0603_1608Metric
- removed TP601: TestPoint, TestPoint:TestPoint_Loop_D2.50mm_Drill1.0mm
- added C1001: 100nF, servo:C_0603_1608Metric, B.Cu at (75.2, 178.8)
- added R1615: 1M, Resistor_SMD:R_1206_3216Metric_Pad1.42x1.75mm_HandSolder, B.Cu at (213.7, 85.6)
- added R1616: 1M, Resistor_SMD:R_1206_3216Metric_Pad1.42x1.75mm_HandSolder, B.Cu at (206.2, 85.2)
- added R1617: 1M, Resistor_SMD:R_1206_3216Metric_Pad1.42x1.75mm_HandSolder, B.Cu at (213.7, 80.5)
- added R1618: 1M, Resistor_SMD:R_1206_3216Metric_Pad1.42x1.75mm_HandSolder, B.Cu at (213.7, 78.0)
- added R211: 2.2k, Resistor_SMD:R_0603_1608Metric, B.Cu at (208.8, 180.6)
- added R213: 470, Resistor_SMD:R_0603_1608Metric, B.Cu at (210.3, 180.6)
- added R302: 1k(dnp), Resistor_SMD:R_0603_1608Metric, B.Cu at (148.2, 120.5)
- C1601, C1602, C1603, C1604, C1605, C1606, C1607, C1608, C1609, C1610, C1807, C1809, C1812, C602, C603, C702, C703, C704, C706, C707, C708, C710, C711, C712, C713, C714, JP1001, JP701, JP702, R1001, R1002, R1003, R1004, R1005, R1006, R1007, R1008, R1009, R1010, R1011, R1012, R1107, R1601, R1602, R1603, R1604, R1605, R1606, R1607, R1608, R1609, R1610, R1806, R1915, R210, R412, R603, R606, R607, R610, R701, R704, R705, R706, R919: moved to B.Cu
- D401, U705, U706: moved to F.Cu
- F701, F702: footprint servo:Fuse_1206_3216Metric -> servo:fuse_3912; moved to B.Cu
- L1601, L1602, L1603, L1604: footprint Inductor_SMD:L_0603_1608Metric -> Inductor_SMD:L_1206_3216Metric_Pad1.42x1.75mm_HandSolder; moved to B.Cu
- R1611, R1612, R1613, R1614: footprint Resistor_SMD:R_0603_1608Metric -> Resistor_SMD:R_1206_3216Metric_Pad1.42x1.75mm_HandSolder; moved to B.Cu
- R203, R423, R426: value 0e(dnp) -> 0e
- R604, R605: footprint Resistor_SMD:R_0603_1608Metric -> Resistor_SMD:R_0805_2012Metric_Pad1.15x1.40mm_HandSolder; moved to B.Cu
- Y201, Y401, Y402: value ~ -> dnp
- moved R1006 339.5 mm to (85.3, 199.9)
- moved R1008 331.5 mm to (85.3, 197.3)
- moved R1001 330.0 mm to (85.3, 201.2)
- moved JP1001 325.9 mm to (72.6, 198.6), turned to 90 degrees
- moved R1011 325.3 mm to (76.4, 199.9)
- moved R1005 324.7 mm to (76.4, 196.1)
- moved R1012 322.0 mm to (81.5, 196.1)
- moved R1002 320.5 mm to (90.4, 197.3)
- moved R1003 320.2 mm to (90.4, 198.6)
- moved R1010 320.1 mm to (79.0, 201.2)
- moved R1007 319.2 mm to (79.0, 197.3)
- moved R1004 318.5 mm to (89.6, 201.2)
- moved R1009 316.1 mm to (79.3, 198.7)
- moved R1613 285.7 mm to (206.2, 82.5)
- moved C1807 282.1 mm to (73.3, 112.4), turned to 270 degrees
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Connections:
- net 1 renamed 1V2C
- net ECAT_MDC renamed ECAT_MDCLK
- net ENET_MDC renamed ENET_MDCLK
- net Net-(C301-Pad1) renamed /uc_adc/adc_refh
- D401 pad 1: ECAT_LED0 -> ECAT_LED_RUN
- D402 pad 1: ECAT_LED1 -> ECAT_LED_ERR
- R1612 pad 1: Net-(R1606-Pad2) -> Net-(R1605-Pad2)
- R1612 pad 2: Net-(R1612-Pad2) -> Net-(R1611-Pad2)
- R1614 pad 1: Net-(R1612-Pad2) -> Net-(R1606-Pad2)
- R1614 pad 2: VBUS_B_P_H -> Net-(R1614-Pad2)
- R412 pad 1: Net-(R412-Pad1) -> 3V3
- R412 pad 2: 3V3 -> Net-(R412-Pad2)
- R413 pad 1: Net-(R413-Pad1) -> 3V3
- R413 pad 2: 3V3 -> Net-(R413-Pad2)
- R414 pad 1: Net-(R414-Pad1) -> 3V3
- R414 pad 2: 3V3 -> Net-(R414-Pad2)
- R415 pad 1: ECAT0_RX_ER -> 3V3
- R415 pad 2: 3V3 -> ECAT0_RX_ER
- R416 pad 1: ECAT1_RX_ER -> 3V3
- R416 pad 2: 3V3 -> ECAT1_RX_ER
- R427 pad 1: ECAT_MDIO -> 3V3
- R427 pad 2: 3V3 -> ECAT_MDIO
- U201 pad 24: Net-(U201-Pad24) -> Net-(J201-Pad16)
- U301 pad D18: ECAT_LED1 -> ECAT_LED_RUN
- U301 pad E11: IN_3V3C -> 1V2
- U301 pad E17: ECAT_LED0 -> ECAT_LED_ERR
- U301 pad E9: IN_3V3C -> 1V2
- U301 pad F11: IN_3V3C -> 1V2
- U301 pad F9: IN_3V3C -> 1V2
- U301 pad G14: IN_3V3C -> 1V2
- U301 pad G15: IN_3V3C -> 1V2
- U301 pad J14: IN_3V3C -> 1V2
- U301 pad J15: IN_3V3C -> 1V2
- U301 pad K5: IN_3V3C -> 1V2
- U301 pad K6: IN_3V3C -> 1V2
- U301 pad P10: IN_3V3C -> 1V2
- U301 pad P13: IN_3V3C -> 1V2
- U301 pad R10: IN_3V3C -> 1V2
- U301 pad R13: IN_3V3C -> 1V2
- U402 pad 27: Net-(R413-Pad1) -> Net-(R413-Pad2)
- U403 pad 27: Net-(R414-Pad1) -> Net-(R414-Pad2)
- U403 pad 29: Net-(R412-Pad1) -> Net-(R412-Pad2)
