File: kicad/endat.sch (KiCad schematic (older format))
At the start: 30 parts, among them J1001 Screw_Terminal_01x07, J1002 Screw_Terminal_01x07, U1001 ADM2483, U1002 ADM2483, U1003 ADM2483, U1004 ADM2483

Commit message: begin PCB!! it's amess but IT IS
Parts:
- C1001, C1002, C1003, C1004, C1005, C1006, C1007, C1008: footprint (none) -> Capacitor_SMD:C_0603_1608Metric
- R1001, R1002, R1003, R1004, R1005, R1006, R1007, R1008, R1009, R1010, R1011, R1012, R1013, R1014, R1015, R1016: footprint (none) -> Resistor_SMD:R_0603_1608Metric
Changed lines of the file:
@@
 F 0 "C1007" V 12547 2791 60  0000 R CNN
 F 1 "100nF" V 12653 2791 60  0000 R CNN
-F 2 "" H 12550 2900 60  0000 C CNN
+F 2 "Capacitor_SMD:C_0603_1608Metric" H 12550 2900 60  0000 C CNN
 F 3 "" H 12550 2900 60  0000 C CNN
 	1    12550 2900
@@
 F 0 "R1010" V 10247 3650 60  0000 L CNN
 F 1 "120e" V 10353 3650 60  0000 L CNN
-F 2 "" H 10300 3600 60  0000 C CNN
+F 2 "Resistor_SMD:R_0603_1608Metric" H 10300 3600 60  0000 C CNN
 F 3 "" H 10300 3600 60  0000 C CNN
 	1    10300 3600
@@
 F 0 "R1011" V 10247 4050 60  0000 L CNN
 F 1 "100k" V 10353 4050 60  0000 L CNN
-F 2 "" H 10300 4000 60  0000 C CNN
+F 2 "Resistor_SMD:R_0603_1608Metric" H 10300 4000 60  0000 C CNN
 F 3 "" H 10300 4000 60  0000 C CNN
 	1    10300 4000
@@
 F 0 "R1009" V 10247 3250 60  0000 L CNN
 F 1 "100k" V 10353 3250 60  0000 L CNN
-F 2 "" H 10300 3200 60  0000 C CNN
+F 2 "Resistor_SMD:R_0603_1608Metric" H 10300 3200 60  0000 C CNN
 F 3 "" H 10300 3200 60  0000 C CNN
 	1    10300 3200
@@
 F 0 "C1005" V 10697 3010 60  0000 L CNN
 F 1 "100nF" V 10803 3010 60  0000 L CNN
-F 2 "" H 10700 2900 60  0000 C CNN
+F 2 "Capacitor_SMD:C_0603_1608Metric" H 10700 2900 60  0000 C CNN
 F 3 "" H 10700 2900 60  0000 C CNN
 	1    10700 2900
@@
 F 0 "C1008" V 12547 4841 60  0000 R CNN
 F 1 "100nF" V 12653 4841 60  0000 R CNN
-F 2 "" H 12550 4950 60  0000 C CNN
+F 2 "Capacitor_SMD:C_0603_1608Metric" H 12550 4950 60  0000 C CNN
 F 3 "" H 12550 4950 60  0000 C CNN
 	1    12550 4950
@@
 F 0 "R1013" V 10247 5700 60  0000 L CNN
 F 1 "120e" V 10353 5700 60  0000 L CNN
-F 2 "" H 10300 5650 60  0000 C CNN
+F 2 "Resistor_SMD:R_0603_1608Metric" H 10300 5650 60  0000 C CNN
 F 3 "" H 10300 5650 60  0000 C CNN
 	1    10300 5650
@@
 F 0 "R1014" V 10247 6100 60  0000 L CNN
 F 1 "100k" V 10353 6100 60  0000 L CNN
-F 2 "" H 10300 6050 60  0000 C CNN
+F 2 "Resistor_SMD:R_0603_1608Metric" H 10300 6050 60  0000 C CNN
 F 3 "" H 10300 6050 60  0000 C CNN
 	1    10300 6050
@@
 F 0 "R1012" V 10247 5300 60  0000 L CNN
 F 1 "100k" V 10353 5300 60  0000 L CNN
-F 2 "" H 10300 5250 60  0000 C CNN
+F 2 "Resistor_SMD:R_0603_1608Metric" H 10300 5250 60  0000 C CNN
 F 3 "" H 10300 5250 60  0000 C CNN
 	1    10300 5250
@@
 F 0 "C1006" V 10697 5060 60  0000 L CNN
 F 1 "100nF" V 10803 5060 60  0000 L CNN
-F 2 "" H 10700 4950 60  0000 C CNN
+F 2 "Capacitor_SMD:C_0603_1608Metric" H 10700 4950 60  0000 C CNN
 F 3 "" H 10700 4950 60  0000 C CNN
 	1    10700 4950
@@
 F 0 "C1001" V 4097 2791 60  0000 R CNN
 F 1 "100nF" V 4203 2791 60  0000 R CNN
-F 2 "" H 4100 2900 60  0000 C CNN
+F 2 "Capacitor_SMD:C_0603_1608Metric" H 4100 2900 60  0000 C CNN
 F 3 "" H 4100 2900 60  0000 C CNN
 	1    4100 2900
@@
 F 0 "R1004" V 6297 3650 60  0000 L CNN
 F 1 "120e" V 6403 3650 60  0000 L CNN
-F 2 "" H 6350 3600 60  0000 C CNN
+F 2 "Resistor_SMD:R_0603_1608Metric" H 6350 3600 60  0000 C CNN
 F 3 "" H 6350 3600 60  0000 C CNN
 	1    6350 3600
@@
 F 0 "R1005" V 6297 4050 60  0000 L CNN
 F 1 "100k" V 6403 4050 60  0000 L CNN
-F 2 "" H 6350 4000 60  0000 C CNN
+F 2 "Resistor_SMD:R_0603_1608Metric" H 6350 4000 60  0000 C CNN
 F 3 "" H 6350 4000 60  0000 C CNN
 	1    6350 4000
@@
 F 0 "R1003" V 6297 3250 60  0000 L CNN
 F 1 "100k" V 6403 3250 60  0000 L CNN
-F 2 "" H 6350 3200 60  0000 C CNN
+F 2 "Resistor_SMD:R_0603_1608Metric" H 6350 3200 60  0000 C CNN
 F 3 "" H 6350 3200 60  0000 C CNN
 	1    6350 3200
@@
 F 0 "C1003" V 5947 3010 60  0000 L CNN
 F 1 "100nF" V 6053 3010 60  0000 L CNN
-F 2 "" H 5950 2900 60  0000 C CNN
+F 2 "Capacitor_SMD:C_0603_1608Metric" H 5950 2900 60  0000 C CNN
 F 3 "" H 5950 2900 60  0000 C CNN
 	1    5950 2900
@@
 F 0 "C1002" V 4097 4841 60  0000 R CNN
 F 1 "100nF" V 4203 4841 60  0000 R CNN
-F 2 "" H 4100 4950 60  0000 C CNN
+F 2 "Capacitor_SMD:C_0603_1608Metric" H 4100 4950 60  0000 C CNN
 F 3 "" H 4100 4950 60  0000 C CNN
 	1    4100 4950
@@
 F 0 "R1007" V 6297 5700 60  0000 L CNN
 F 1 "120e" V 6403 5700 60  0000 L CNN
-F 2 "" H 6350 5650 60  0000 C CNN
+F 2 "Resistor_SMD:R_0603_1608Metric" H 6350 5650 60  0000 C CNN
 F 3 "" H 6350 5650 60  0000 C CNN
 	1    6350 5650
@@
 F 0 "R1008" V 6297 6100 60  0000 L CNN
 F 1 "100k" V 6403 6100 60  0000 L CNN
-F 2 "" H 6350 6050 60  0000 C CNN
+F 2 "Resistor_SMD:R_0603_1608Metric" H 6350 6050 60  0000 C CNN
 F 3 "" H 6350 6050 60  0000 C CNN
 	1    6350 6050
@@
 F 0 "R1006" V 6297 5300 60  0000 L CNN
 F 1 "100k" V 6403 5300 60  0000 L CNN
-F 2 "" H 6350 5250 60  0000 C CNN
+F 2 "Resistor_SMD:R_0603_1608Metric" H 6350 5250 60  0000 C CNN
 F 3 "" H 6350 5250 60  0000 C CNN
 	1    6350 5250
@@
 F 0 "C1004" V 5947 5060 60  0000 L CNN
 F 1 "100nF" V 6053 5060 60  0000 L CNN
-F 2 "" H 5950 4950 60  0000 C CNN
+F 2 "Capacitor_SMD:C_0603_1608Metric" H 5950 4950 60  0000 C CNN
 F 3 "" H 5950 4950 60  0000 C CNN
 	1    5950 4950
@@
 F 0 "R1002" H 3500 5953 60  0000 C CNN
 F 1 "0e(dnp)" H 3500 6059 60  0000 C CNN
-F 2 "" H 3500 5850 60  0000 C CNN
+F 2 "Resistor_SMD:R_0603_1608Metric" H 3500 5850 60  0000 C CNN
 F 3 "" H 3500 5850 60  0000 C CNN
 	1    3500 5850
@@
 F 0 "R1001" H 3100 5953 60  0000 C CNN
 F 1 "0e" H 3100 6059 60  0000 C CNN
-F 2 "" H 3100 5850 60  0000 C CNN
+F 2 "Resistor_SMD:R_0603_1608Metric" H 3100 5850 60  0000 C CNN
 F 3 "" H 3100 5850 60  0000 C CNN
 	1    3100 5850
@@
 F 0 "R1015" H 13650 5953 60  0000 C CNN
 F 1 "0e(dnp)" H 13650 6059 60  0000 C CNN
-F 2 "" H 13650 5850 60  0000 C CNN
+F 2 "Resistor_SMD:R_0603_1608Metric" H 13650 5850 60  0000 C CNN
 F 3 "" H 13650 5850 60  0000 C CNN
 	1    13650 5850
@@
 F 0 "R1016" H 14050 5953 60  0000 C CNN
 F 1 "0e" H 14050 6059 60  0000 C CNN
-F 2 "" H 14050 5850 60  0000 C CNN
+F 2 "Resistor_SMD:R_0603_1608Metric" H 14050 5850 60  0000 C CNN
 F 3 "" H 14050 5850 60  0000 C CNN
 	1    14050 5850

Commit message: I've passed all footprin to layout BUT...
I've passed all, first glance... I need to confirm in details a lot of
things. The objetive for these is to have an aproximation of the size
I'll need to make the board.. then I choose the final detailed footprint
Parts:
- removed J1001, J1002: Screw_Terminal_01x07, symbol Connector:Screw_Terminal_01x07
- added J1001, J1002: tblock, TerminalBlock_RND:TerminalBlock_RND_205-00291_1x06_P5.08mm_Horizontal, symbol Connector:Screw_Terminal_01x06
- added JP1001, JP1002: jumper, Jumper:SolderJumper-3_P1.3mm_Open_RoundedPad1.0x1.5mm, symbol servo:Jumper_3_Bridged12
- C1001, C1002, C1003, C1004, C1005, C1006, C1007, C1008: footprint Capacitor_SMD:C_0603_1608Metric -> servo:C_0603_1608Metric
Connections:
- wire segments 194 -> 196
Other:
- moved on the sheet: C1001, C1002, C1003

Commit message: passed all footprint, preliminarly.. and taken a pic
I've passed all 3d models, and make a pic of that, it's the first
impresion, but it need's more indeed reviews
Parts:
- J1001, J1002: footprint TerminalBlock_RND:TerminalBlock_RND_205-00291_1x06_P5.08mm_Horizontal -> Connector_Phoenix_MSTB:PhoenixContact_MSTBA_2,5_6-G-5,08_1x06_P5.08mm_Horizontal
Changed lines of the file:
@@
 F 0 "J1001" H 7830 3792 50  0000 L CNN
 F 1 "tblock" H 7830 3701 50  0000 L CNN
-F 2 "TerminalBlock_RND:TerminalBlock_RND_205-00291_1x06_P5.08mm_Horizontal" H 7750 3800 50  0001 C CNN
+F 2 "Connector_Phoenix_MSTB:PhoenixContact_MSTBA_2,5_6-G-5,08_1x06_P5.08mm_Horizontal" H 7750 3800 50  0001 C CNN
 F 3 "~" H 7750 3800 50  0001 C CNN
 	1    7750 3800
@@
 F 0 "J1002" H 8580 3792 50  0000 L CNN
 F 1 "tblock" H 8580 3701 50  0000 L CNN
-F 2 "TerminalBlock_RND:TerminalBlock_RND_205-00291_1x06_P5.08mm_Horizontal" H 8500 3800 50  0001 C CNN
+F 2 "Connector_Phoenix_MSTB:PhoenixContact_MSTBA_2,5_6-G-5,08_1x06_P5.08mm_Horizontal" H 8500 3800 50  0001 C CNN
 F 3 "~" H 8500 3800 50  0001 C CNN
 	1    8500 3800

Commit message: changing single row terminal block to double row
I've changed to double row all the connectors, RJ45 and terminal blocks,
I saves spaces and also make it more intuitive related to user
interface..lets go
Parts:
- removed J1001, J1002: tblock, Connector_Phoenix_MSTB:PhoenixContact_MSTBA_2,5_6-G-5,08_1x06_P5.08mm_Horizontal, symbol Connector:Screw_Terminal_01x06
- added J1001: tblock, servo:tblock02x06, symbol Connector_Generic:Conn_02x06_Row_Letter_Last
- renumbered C1002 to C1001, C1001 to C1002
Changed lines of the file:
@@
 $Descr A3 16535 11693
 encoding utf-8
-Sheet 10 19
+Sheet 10 18
 Title "ENDAT/BISS Interface"
 Date "2020-01-09"
@@
 2X Isolated ENDAT interface
 $Comp
-L servo:Capacitor C1001
+L servo:Capacitor C1002
 U 1 1 5FF891F6
 P 4000 2900
-F 0 "C1001" V 4028 2791 20  0000 R CNN
+F 0 "C1002" V 4028 2791 20  0000 R CNN
 F 1 "100nF" V 4071 2791 20  0000 R CNN
 F 2 "servo:C_0603_1608Metric" H 4000 2800 60  0001 C CNN
@@
 AR Path="/5DE49152/5FF8920A" Ref="#PWR?"  Part="1"
 AR Path="/5E1BAEAA/5FF8920A" Ref="#PWR?"  Part="1"
-AR Path="/5DE3DF56/5FF8920A" Ref="#PWR01006"  Part="1"
-F 0 "#PWR01006" H 5750 2550 20  0001 C CNN
+AR Path="/5DE3DF56/5FF8920A" Ref="#PWR01005"  Part="1"
+F 0 "#PWR01005" H 5750 2550 20  0001 C CNN
 F 1 "5VH" H 5755 2907 28  0000 C CNN
 F 2 "" H 5750 2750 50  0001 C CNN
@@
 AR Path="/5DE49152/5FF89213" Ref="#PWR?"  Part="1"
 AR Path="/5E1BAEAA/5FF89213" Ref="#PWR?"  Part="1"
-AR Path="/5DE3DF56/5FF89213" Ref="#PWR01010"  Part="1"
-F 0 "#PWR01010" H 6350 4050 30  0001 C CNN
+AR Path="/5DE3DF56/5FF89213" Ref="#PWR01009"  Part="1"
+F 0 "#PWR01009" H 6350 4050 30  0001 C CNN
 F 1 "GNDH" H 6350 4142 30  0000 C CNN
 F 2 "" H 6350 4300 50  0001 C CNN
@@
 AR Path="/5DE49152/5FF8923C" Ref="#PWR?"  Part="1"
 AR Path="/5E1BAEAA/5FF8923C" Ref="#PWR?"  Part="1"
-AR Path="/5DE3DF56/5FF8923C" Ref="#PWR01001"  Part="1"
-F 0 "#PWR01001" H 4017 2859 20  0000 C CNN
+AR Path="/5DE3DF56/5FF8923C" Ref="#PWR01003"  Part="1"
+F 0 "#PWR01003" H 4017 2859 20  0000 C CNN
 F 1 "3V3" H 4017 2807 30  0000 C CNN
 F 2 "" H 4000 2650 70  0000 C CNN
@@
 Wire Wire Line
 	6350 2800 6350 3000
-Wire Wire Line
-	6350 3800 7550 3800
-Wire Wire Line
-	6750 3700 7550 3700
-$Comp
-L servo:Capacitor C1002
+$Comp
+L servo:Capacitor C1001
 U 1 1 5FF89288
 P 3950 5200
-F 0 "C1002" V 3978 5091 20  0000 R CNN
+F 0 "C1001" V 3978 5091 20  0000 R CNN
 F 1 "100nF" V 4021 5091 20  0000 R CNN
 F 2 "servo:C_0603_1608Metric" H 3950 5100 60  0001 C CNN
@@
 AR Path="/5DE49152/5FF8929C" Ref="#PWR?"  Part="1"
 AR Path="/5E1BAEAA/5FF8929C" Ref="#PWR?"  Part="1"
-AR Path="/5DE3DF56/5FF8929C" Ref="#PWR01007"  Part="1"
-F 0 "#PWR01007" H 5750 4500 20  0001 C CNN
+AR Path="/5DE3DF56/5FF8929C" Ref="#PWR01006"  Part="1"
+F 0 "#PWR01006" H 5750 4500 20  0001 C CNN
 F 1 "5VH" H 5755 4857 28  0000 C CNN
 F 2 "" H 5750 4700 50  0001 C CNN
@@
 AR Path="/5DE49152/5FF892A5" Ref="#PWR?"  Part="1"
 AR Path="/5E1BAEAA/5FF892A5" Ref="#PWR?"  Part="1"
-AR Path="/5DE3DF56/5FF892A5" Ref="#PWR01011"  Part="1"
-F 0 "#PWR01011" H 6350 6100 30  0001 C CNN
+AR Path="/5DE3DF56/5FF892A5" Ref="#PWR01010"  Part="1"
+F 0 "#PWR01010" H 6350 6100 30  0001 C CNN
 F 1 "GNDH" H 6350 6192 30  0000 C CNN
 F 2 "" H 6350 6350 50  0001 C CNN
@@
 AR Path="/5DE49152/5FF892CE" Ref="#PWR?"  Part="1"
 AR Path="/5E1BAEAA/5FF892CE" Ref="#PWR?"  Part="1"
-AR Path="/5DE3DF56/5FF892CE" Ref="#PWR01003"  Part="1"
-F 0 "#PWR01003" H 3850 5050 20  0001 C CNN
+AR Path="/5DE3DF56/5FF892CE" Ref="#PWR01001"  Part="1"
+F 0 "#PWR01001" H 3850 5050 20  0001 C CNN
 F 1 "3V3" H 3950 5100 28  0000 C CNN
 F 2 "" H 3950 4950 50  0001 C CNN
@@
 Wire Wire Line
 	6750 5450 6750 3900
-Wire Wire Line
-	6750 3900 7550 3900
-Wire Wire Line
-	7550 4000 6900 4000
 Wire Wire Line
 	6900 4000 6900 5850
@@
 AR Path="/5DE49152/5FF89280" Ref="#PWR?"  Part="1"
 AR Path="/5E1BAEAA/5FF89280" Ref="#PWR?"  Part="1"
-AR Path="/5DE3DF56/5FF89280" Ref="#PWR01013"  Part="1"
-F 0 "#PWR01013" H 6950 3150 20  0001 C CNN
+AR Path="/5DE3DF56/5FF89280" Ref="#PWR01011"  Part="1"
+F 0 "#PWR01011" H 6950 3150 20  0001 C CNN
 F 1 "5VH" H 6955 3507 28  0000 C CNN
 F 2 "" H 6950 3350 50  0001 C CNN
@@
 	1    0    0    -1
 $EndComp
-Wire Wire Line
-	7550 4100 7450 4100
 Wire Wire Line
 	7450 4150 7450 4100
@@
 AR Path="/5DE49152/5FF8930B" Ref="#PWR?"  Part="1"
 AR Path="/5E1BAEAA/5FF8930B" Ref="#PWR?"  Part="1"
-AR Path="/5DE3DF56/5FF8930B" Ref="#PWR01014"  Part="1"
-F 0 "#PWR01014" H 7450 3900 30  0001 C CNN
+AR Path="/5DE3DF56/5FF8930B" Ref="#PWR01012"  Part="1"
+F 0 "#PWR01012" H 7450 3900 30  0001 C CNN
 F 1 "GNDH" H 7450 3992 30  0000 C CNN
 F 2 "" H 7450 4150 50  0001 C CNN
@@
 AR Path="/5DE49152/5FF89267" Ref="#PWR?"  Part="1"
 AR Path="/5E1BAEAA/5FF89267" Ref="#PWR?"  Part="1"
-AR Path="/5DE3DF56/5FF89267" Ref="#PWR01008"  Part="1"
-F 0 "#PWR01008" H 5950 2950 30  0001 C CNN
+AR Path="/5DE3DF56/5FF89267" Ref="#PWR01007"  Part="1"
+F 0 "#PWR01007" H 5950 2950 30  0001 C CNN
 F 1 "GNDH" H 5950 3042 30  0000 C CNN
 F 2 "" H 5950 3200 50  0001 C CNN
@@
 	4000 3150 4000 3100
 $Comp
-L servo:GND #PWR01002
+L servo:GND #PWR01004
 U 1 1 5FF891FD
 P 4000 3150
-F 0 "#PWR01002" H 4000 2900 30  0001 C CNN
+F 0 "#PWR01004" H 4000 2900 30  0001 C CNN
 F 1 "GND" H 4000 2992 30  0000 C CNN
 F 2 "" H 4000 3150 50  0001 C CNN
@@
 $EndComp
 $Comp
-L servo:GND #PWR01004
+L servo:GND #PWR01002
 U 1 1 5FF8928F
 P 3950 5400
-F 0 "#PWR01004" H 3950 5150 30  0001 C CNN
+F 0 "#PWR01002" H 3950 5150 30  0001 C CNN
 F 1 "GND" H 3950 5242 30  0000 C CNN
 F 2 "" H 3950 5400 50  0001 C CNN
@@
 AR Path="/5DE49152/5FF892F7" Ref="#PWR?"  Part="1"
 AR Path="/5E1BAEAA/5FF892F7" Ref="#PWR?"  Part="1"
-AR Path="/5DE3DF56/5FF892F7" Ref="#PWR01009"  Part="1"
-F 0 "#PWR01009" H 5950 4900 30  0001 C CNN
+AR Path="/5DE3DF56/5FF892F7" Ref="#PWR01008"  Part="1"
+F 0 "#PWR01008" H 5950 4900 30  0001 C CNN
 F 1 "GNDH" H 5950 4992 30  0000 C CNN
 F 2 "" H 5950 5150 50  0001 C CNN
@@
 P 7550 3350
 AR Path="/5E1BAEAA/616C2524" Ref="#PWR?"  Part="1"
-AR Path="/5DE3DF56/616C2524" Ref="#PWR01005"  Part="1"
-F 0 "#PWR01005" H 7550 3150 20  0001 C CNN
+AR Path="/5DE3DF56/616C2524" Ref="#PWR01013"  Part="1"
+F 0 "#PWR01013" H 7550 3150 20  0001 C CNN
 F 1 "15VH" H 7550 3507 28  0000 C CNN
 F 2 "" H 7550 3350 50  0001 C CNN
@@
 Wire Wire Line
 	7250 3600 7250 3500
-Wire Wire Line
-	7250 3600 7550 3600
-$Comp
-L Connector:Screw_Terminal_01x06 J1001
-U 1 1 6173F780
-P 7750 3800
-F 0 "J1001" H 7830 3792 50  0000 L CNN
-F 1 "tblock" H 7830 3701 50  0000 L CNN
-F 2 "Connector_Phoenix_MSTB:PhoenixContact_MSTBA_2,5_6-G-5,08_1x06_P5.08mm_Horizontal" H 7750 3800 50  0001 C CNN
-F 3 "~" H 7750 3800 50  0001 C CNN
-	1    7750 3800
-	1    0    0    -1
-$EndComp
 $Comp
 L servo:Capacitor C1007
@@
 Wire Wire Line
 	9900 2800 9900 3000
-Wire Wire Line
-	9900 3800 8700 3800
-Wire Wire Line
-	9500 3700 8700 3700
 $Comp
 L servo:Capacitor C1008
@@
 	9500 5450 9500 3900
 Wire Wire Line
-	9500 3900 8700 3900
-Wire Wire Line
-	8700 4000 9350 4000
-Wire Wire Line
 	9350 4000 9350 5850
 Wire Wire Line
@@
 $EndComp
 Wire Wire Line
-	8700 4100 8800 4100
-Wire Wire Line
 	8800 4150 8800 4100
 $Comp
@@
 P 8700 3350
 AR Path="/5E1BAEAA/617F33FB" Ref="#PWR?"  Part="1"
-AR Path="/5DE3DF56/617F33FB" Ref="#PWR01012"  Part="1"
-F 0 "#PWR01012" H 8700 3150 20  0001 C CNN
+AR Path="/5DE3DF56/617F33FB" Ref="#PWR01014"  Part="1"
+F 0 "#PWR01014" H 8700 3150 20  0001 C CNN
 F 1 "15VH" H 8700 3507 28  0000 C CNN
 F 2 "" H 8700 3350 50  0001 C CNN
@@
 Wire Wire Line
 	9000 3600 9000 3500
-Wire Wire Line
-	9000 3600 8700 3600
-$Comp
-L Connector:Screw_Terminal_01x06 J1002
-U 1 1 617F3407
-P 8500 3800
-F 0 "J1002" H 8580 3792 50  0000 L CNN
-F 1 "tblock" H 8580 3701 50  0000 L CNN
-F 2 "Connector_Phoenix_MSTB:PhoenixContact_MSTBA_2,5_6-G-5,08_1x06_P5.08mm_Horizontal" H 8500 3800 50  0001 C CNN
-F 3 "~" H 8500 3800 50  0001 C CNN
-	1    8500 3800
-	-1   0    0    -1
-$EndComp
+$Comp
+L Connector_Generic:Conn_02x06_Row_Letter_Last J1001
+U 1 1 5E215342
+P 8050 3800
+F 0 "J1001" H 8100 4217 50  0000 C CNN
+F 1 "tblock" H 8100 4126 50  0000 C CNN
+F 2 "servo:tblock02x06" H 8050 3800 50  0001 C CNN
+F 3 "~" H 8050 3800 50  0001 C CNN
+	1    8050 3800
+	1    0    0    -1
+$EndComp
+Wire Wire Line
+	7250 3600 7850 3600
+Wire Wire Line
+	6750 3700 7850 3700
+Wire Wire Line
+	6350 3800 7850 3800
+Wire Wire Line
+	6750 3900 7850 3900
+Wire Wire Line
+	6900 4000 7850 4000
+Wire Wire Line
+	7450 4100 7850 4100
+Wire Wire Line
+	8350 4100 8800 4100
+Wire Wire Line
+	8350 4000 9350 4000
+Wire Wire Line
+	8350 3900 9500 3900
+Wire Wire Line
+	8350 3800 9900 3800
+Wire Wire Line
+	8350 3700 9500 3700
+Wire Wire Line
+	8350 3600 9000 3600
 $EndSCHEMATC

Commit message: I've reducede the PCB size ADC TVS, USB host and IDC out
TVS for ADC protection, USB out 'cause it's almost free and IDC debug
out in an IDC. Better and thinner terminal block connector help in
reduce the board size.
Parts:
- removed J1001: tblock, servo:tblock02x06, symbol Connector_Generic:Conn_02x06_Row_Letter_Last
- added J1001: tblock2x6, servo:tblock02x06, symbol servo:tblock2x6
Changed lines of the file:
@@
 Wire Wire Line
 	9000 3600 9000 3500
-$Comp
-L Connector_Generic:Conn_02x06_Row_Letter_Last J1001
-U 1 1 5E215342
-P 8050 3800
-F 0 "J1001" H 8100 4217 50  0000 C CNN
-F 1 "tblock" H 8100 4126 50  0000 C CNN
-F 2 "servo:tblock02x06" H 8050 3800 50  0001 C CNN
-F 3 "~" H 8050 3800 50  0001 C CNN
-	1    8050 3800
-	1    0    0    -1
-$EndComp
 Wire Wire Line
 	7250 3600 7850 3600
@@
 Wire Wire Line
 	8350 3600 9000 3600
+$Comp
+L servo:tblock2x6 J1001
+U 1 1 5E22F1B6
+P 8050 3800
+F 0 "J1001" H 8100 4193 39  0000 C CNN
+F 1 "tblock2x6" H 8100 4118 39  0000 C CNN
+F 2 "servo:tblock02x06" H 8000 4000 50  0001 C CNN
+F 3 "../doc/datasheets/tblock2rows.pdf" H 8100 4100 50  0001 C CNN
+	1    8050 3800
+	1    0    0    -1
+$EndComp
 $EndSCHEMATC
