File: kicad/ethercat.sch (KiCad schematic (older format))
At the start: 85 parts, among them U401 CAT24C16WI, U402 DP83822, U403 DP83822, U404 rj45x2, Y401 dnp, Y402 dnp

Commit message: beginine routing... far far away
Parts:
- removed C401, C402, C416, C417: 0.01uF, servo:C_0603_1608Metric, symbol servo:Capacitor
- removed C403, C413, C415: 0.1uF, servo:C_0603_1608Metric, symbol servo:Capacitor
- removed C406, C420, C421, C424, C425, C430, C431, C432, C433: 1uF, servo:C_0603_1608Metric, symbol servo:Capacitor
- C405, C411, C412: value 1uF -> 0.1uF
Connections:
- net 3V3: now also Y402.1 (TRI-STATE), Y402.4 (VCC); no longer Y402.2 (GND), Y402.3 (OUTPUT)
- net GND: now also Y402.2 (GND); no longer Y402.1 (TRI-STATE)
- net at R426.1, U403.23 (XI): now also Y402.3 (OUTPUT); no longer Y402.4 (VCC)
Other:
- note added: "place near device\n"
- moved on the sheet: C404, C405, C407, C408, C409, C410, C411, C412, C426, C427, C428, C429
