File: kicad/ethercat.sch (KiCad schematic (older format))
At the start: 69 parts, among them U401 CAT24C16WI, U402 DP83822, U403 DP83822, U404 rj45x2, Y401 dnp, Y402 dnp

Commit message: bom bom bom...
Parts:
- C404, C414, C418, C419, C422, C423: Description (none) -> CAP CER 0.1UF 16V X7R 0603; PartNumber (none) -> CC0603KPX7R7BB104; ValueDisplayed 0.1uF -> (none); digikey (none) -> 311-1335-1-ND
- C405, C411, C412: Description (none) -> CAP CER 0.1UF 16V X7R 0603; PartNumber (none) -> CC0603KPX7R7BB104; ValueDisplayed 1uF -> (none); digikey (none) -> 311-1335-1-ND
- C407, C408, C409, C410: PartNumber (none) -> GRM188R61A106ME69D; ValueDisplayed 10uF -> (none); digikey (none) -> 490-10475-1-ND
- C426, C427, C428, C429: Description (none) -> CAP CER 1UF 10V X7R 0603; PartNumber (none) -> C0603C105K8RACTU; ValueDisplayed 1uF -> (none); digikey (none) -> 399-11133-1-ND
- C434: PartNumber (none) -> 12061C472KAT2A; ValueDisplayed 1uF -> (none); digikey (none) -> 478-1521-1-ND
- D401: value Red@2mA -> green@2mA; PartNumber (none) -> LG L29K-G2J1-24-Z; VALUE Red -> (none); digikey (none) -> LG L29K-G2J1-24-Z
- D402: value green@2mA -> red@2mA; PartNumber (none) -> LS L29K-G1H2-1-Z; VALUE Bright Green -> (none); digikey (none) -> LS L29K-G1H2-1-Z
- R401, R402, R403, R404, R405, R406, R407, R408, R409, R410, R411, R412, R413, R414, R415, R416, R427, R433, R434, R436, R439: ValueDisplayed 2.2k -> (none)
- R417, R418: ValueDisplayed 4.7k -> (none)
- R419: value 330 -> 680; ValueDisplayed 1.27k -> (none)
- R420: value 330 -> 680; ValueDisplayed 680 -> (none)
- R421, R424: ValueDisplayed 4.87k -> (none)
- R422, R423, R425, R426: ValueDisplayed 10.0k -> (none)
- R429, R430, R431, R432, R435, R437, R438, R440: ValueDisplayed 49.9 -> (none)
- R441, R442, R445, R446: ValueDisplayed 470 -> (none)
Connections:
- net ECAT0_RX_D0: now also R402.1; no longer R402.2
- net ECAT0_RX_D1: now also R404.1; no longer R404.2
- net ECAT0_RX_D2: now also R406.1; no longer R406.2
- net ECAT0_RX_D3: now also R408.1; no longer R408.2
- net ECAT0_RX_DV: now also R401.1; no longer R401.2
- net ECAT1_RX_D0: now also R405.1; no longer R405.2
- net ECAT1_RX_D1: now also R407.1; no longer R407.2
- net ECAT1_RX_D2: now also R409.1; no longer R409.2
- net ECAT1_RX_D3: now also R411.1; no longer R411.2
- net ECAT1_RX_DV: now also R403.1; no longer R403.2
- net GND: now also R401.2, R402.2, R403.2, R404.2, R405.2, R406.2, R407.2, R408.2, R409.2, R410.2, R411.2; no longer R401.1, R402.1, R403.1, R404.1, R405.1, R406.1, R407.1, R408.1, R409.1, R410.1, R411.1
- net ecat0_col: now also R410.1; no longer R410.2

Commit message: more bom...
Parts:
- C407, C408, C409, C410: Description (none) -> 10µF ±20% 10V Ceramic Capacitor X5R 0603 (1608 Metric)
- C434: Description (none) -> 4700pF ±10% 100V Ceramic Capacitor X7R 1206 (3216 Metric)
- D401: Description (none) -> LED GREEN DIFFUSED 0603 SMD
- D402: Description (none) -> LED RED DIFFUSED 0603 SMD
- R423, R426: value 0e -> 0
- U401: Description (none) -> EEPROM Memory IC 16Kb (2K x 8) I²C 400kHz 900ns 8-SOIC; PartNumber (none) -> CAT24C16WI-GT3; digikey (none) -> CAT24C16WI-GT3CT-ND; price@10 (none) -> 0.16300
- U402, U403: Description (none) -> Ethernet Interface 32-VQFN (5x5); digikey (none) -> 296-47256-1-ND; price@10 (none) -> 2.37700
- U404: value rj45x2 -> RJ45x2; Description (none) -> 2 Port RJ45 Magjack Connector Through Hole 10/100 Base-T, A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; PartNumber (none) -> 0845-2G1T-H5; digikey (none) -> 380-1123-ND; price@10 (none) -> 7.17400
Changed lines of the file:
@@
 F 3 "../doc/datasheets/dp83822i.pdf" H 6650 2850 50  0001 C CNN
 F 4 "DP83822IRHBR" V -650 1750 60  0001 C CNN "PartNumber"
+F 5 "Ethernet Interface 32-VQFN (5x5) " H 0   0   50  0001 C CNN "Description"
+F 6 "296-47256-1-ND" H 0   0   50  0001 C CNN "digikey"
+F 7 "2.37700" H 0   0   50  0001 C CNN "price@10"
 	1    6650 2850
 	1    0    0    -1
@@
 F 3 "../doc/datasheets/CAT24C01-D.PDF" H 3800 10600 60  0001 C CNN
 F 4 "CAT24C16WI-GT3" H 4200 10200 50  0001 C CNN "Fieldname"
+F 5 "EEPROM Memory IC 16Kb (2K x 8) I²C 400kHz 900ns 8-SOIC" H 0   0   50  0001 C CNN "Description"
+F 6 "CAT24C16WI-GT3" H 0   0   50  0001 C CNN "PartNumber"
+F 7 "CAT24C16WI-GT3CT-ND " H 0   0   50  0001 C CNN "digikey"
+F 8 "0.16300" H 0   0   50  0001 C CNN "price@10"
 	1    4200 10200
 	1    0    0    -1
@@
 F 4 "490-10475-1-ND" H 0   0   50  0001 C CNN "digikey"
 F 5 "GRM188R61A106ME69D " H 0   0   50  0001 C CNN "PartNumber"
+F 6 "10µF ±20% 10V Ceramic Capacitor X5R 0603 (1608 Metric) " H 0   0   50  0001 C CNN "Description"
 	1    3700 2150
 	0    -1   -1   0
@@
 F 4 "490-10475-1-ND" H 0   0   50  0001 C CNN "digikey"
 F 5 "GRM188R61A106ME69D " H 0   0   50  0001 C CNN "PartNumber"
+F 6 "10µF ±20% 10V Ceramic Capacitor X5R 0603 (1608 Metric) " H 0   0   50  0001 C CNN "Description"
 	1    3350 1850
 	0    -1   -1   0
@@
 F 4 "LS L29K-G1H2-1-Z " H 7400 10500 50  0001 C CNN "digikey"
 F 5 "LS L29K-G1H2-1-Z" H 0   0   50  0001 C CNN "PartNumber"
+F 6 "LED RED DIFFUSED 0603 SMD " H 0   0   50  0001 C CNN "Description"
 	1    7400 10500
 	-1   0    0    1
@@
 F 4 "LG L29K-G2J1-24-Z " H 7400 10250 50  0001 C CNN "digikey"
 F 5 "LG L29K-G2J1-24-Z" H 0   0   50  0001 C CNN "PartNumber"
+F 6 "LED GREEN DIFFUSED 0603 SMD " H 0   0   50  0001 C CNN "Description"
 	1    7400 10250
 	-1   0    0    1
@@
 P 8450 3350
 F 0 "R423" H 8450 3465 20  0000 C CNN
-F 1 "0e" H 8450 3422 20  0000 C CNN
+F 1 "0" H 8450 3422 20  0000 C CNN
 F 2 "servo:R_0603_1608Metric" H 7950 3250 60  0001 C CNN
 F 3 "" H 8050 3350 60  0001 C CNN
@@
 F 3 "../doc/datasheets/dp83822i.pdf" H 6800 7000 50  0001 C CNN
 F 4 "DP83822IRHBR" V -500 5900 60  0001 C CNN "PartNumber"
+F 5 "Ethernet Interface 32-VQFN (5x5) " H 0   0   50  0001 C CNN "Description"
+F 6 "296-47256-1-ND" H 0   0   50  0001 C CNN "digikey"
+F 7 "2.37700" H 0   0   50  0001 C CNN "price@10"
 	1    6800 7000
 	1    0    0    -1
@@
 F 4 "490-10475-1-ND" H 0   0   50  0001 C CNN "digikey"
 F 5 "GRM188R61A106ME69D " H 0   0   50  0001 C CNN "PartNumber"
+F 6 "10µF ±20% 10V Ceramic Capacitor X5R 0603 (1608 Metric) " H 0   0   50  0001 C CNN "Description"
 	1    3700 6300
 	0    -1   -1   0
@@
 F 4 "490-10475-1-ND" H 0   0   50  0001 C CNN "digikey"
 F 5 "GRM188R61A106ME69D " H 0   0   50  0001 C CNN "PartNumber"
+F 6 "10µF ±20% 10V Ceramic Capacitor X5R 0603 (1608 Metric) " H 0   0   50  0001 C CNN "Description"
 	1    3450 6050
 	0    -1   -1   0
@@
 P 8600 7500
 F 0 "R426" H 8600 7615 20  0000 C CNN
-F 1 "0e" H 8600 7572 20  0000 C CNN
+F 1 "0" H 8600 7572 20  0000 C CNN
 F 2 "servo:R_0603_1608Metric" H 8100 7400 60  0001 C CNN
 F 3 "" H 8200 7500 60  0001 C CNN
@@
 P 14800 4900
 F 0 "U404" H 15277 4938 39  0000 L CNN
-F 1 "rj45x2" H 15277 4863 39  0000 L CNN
+F 1 "RJ45x2" H 15277 4863 39  0000 L CNN
 F 2 "servo:rj45x2_0845-2G1T-H5" H 15300 5200 20  0001 C CNN
 F 3 "../doc/datasheets/rj45x2_dr-MAG-0845-2G1T-H5-1309698.pdf" H 15400 5300 20  0001 C CNN
+F 4 "2 Port RJ45 Magjack Connector Through Hole 10/100 Base-T, AutoMDIX " H 0   0   50  0001 C CNN "Description"
+F 5 "0845-2G1T-H5 " H 0   0   50  0001 C CNN "PartNumber"
+F 6 "380-1123-ND" H 0   0   50  0001 C CNN "digikey"
+F 7 "7.17400" H 0   0   50  0001 C CNN "price@10"
 	1    14800 4900
 	1    0    0    -1
@@
 F 4 "12061C472KAT2A" H 0   0   50  0001 C CNN "PartNumber"
 F 5 "478-1521-1-ND" H 0   0   50  0001 C CNN "digikey"
+F 6 "4700pF ±10% 100V Ceramic Capacitor X7R 1206 (3216 Metric) " H 0   0   50  0001 C CNN "Description"
 	1    14850 6500
 	0    1    1    0

Commit message: stackup
Parts:
- added JP401, JP402: jumper, servo:SolderJumper-2_P1.3mm_Open_RoundedPad1.0x1.5mm, symbol servo:jumper
- C404, C405, C411, C412, C414, C418, C419, C422, C423: price@10 (none) -> 0.05800
- C407, C408, C409, C410: price@10 (none) -> 0.15400
- C426, C427, C428, C429: price@10 (none) -> 0.06400
- C434: price@10 (none) -> 0.18700
- D401: digikey LG L29K-G2J1-24-Z -> 475-2709-1-ND; price@10 (none) -> 0.31900
- D402: digikey LS L29K-G1H2-1-Z -> 475-3124-1-ND; price@10 (none) -> 0.33900
- Y401, Y402: value dnp -> osc 25Mhz; Description (none) -> 25MHz XO (Standard) HCMOS Oscillator 3.3V Enable/Disable 4-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; PartNumber (none) -> ECS-2520S33-250-FN-TR; digikey (none) -> XC2198CT-ND; price@10 (none) -> 1.41900
Connections:
- net at R423.1, U402.23 (XI): now also JP401.1; no longer Y401.3 (OUTPUT)
- net at R426.1, U403.23 (XI): now also JP402.1; no longer Y402.3 (OUTPUT)
- new net: JP401.2, Y401.3 (OUTPUT)
- new net: JP402.2, Y402.3 (OUTPUT)

Commit message: bom copleted
Parts:
- removed R423, R426: 0, servo:R_0603_1608Metric, symbol servo:Resistor
- removed R436, R439: 0e(dnp), servo:R_0603_1608Metric, symbol servo:Resistor
- added JP403, JP404, JP405, JP406: jumper, servo:SolderJumper-2_P1.3mm_Open_RoundedPad1.0x1.5mm, symbol servo:jumper
- R401, R402, R403, R404, R405, R406, R407, R408, R409, R410, R411, R412, R413, R414, R415, R416, R427, R433, R434: Description (none) -> 2.2 kOhms ±5% 0.1W, 1/10W Chip Resistor 0603 (1608 Metric) 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; PartNumber (none) -> ERJ-3GEYJ222V; digikey (none) -> P2.2KGCT-ND; price@10 (none) -> 0.04500
- R417, R418: Description (none) -> 4.7 kOhms ±5% 0.1W, 1/10W Chip Resistor 0603 (1608 Metric) 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; PartNumber (none) -> RC0603JR-074K7L; digikey (none) -> 311-4.7KGRCT-ND; price@10 (none) -> 0.01900
- R419, R420: Description (none) -> 680 Ohms ±5% 0.1W, 1/10W Chip Resistor 0603 (1608 Metric) A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; PartNumber (none) -> RMCF0603JT680R; digikey (none) -> RMCF0603JT680RCT-ND; price@10 (none) -> 0.01400
- R421, R424: Description (none) -> 4.87 kOhms ±1% 0.1W, 1/10W Chip Resistor 0603 (1608 Metric)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; PartNumber (none) -> RMCF0603FT4K87; digikey (none) -> RMCF0603FT4K87CT-ND; price@10 (none) -> 0.01600
- R422, R425: value 10.0k -> 10k; Description (none) -> 10 kOhms ±5% 0.1W, 1/10W Chip Resistor 0603 (1608 Metric) M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; PartNumber (none) -> RC0603JR-0710KL; digikey (none) -> 311-10KGRCT-ND; price@10 (none) -> 0.01900
- R429, R430, R431, R432, R435, R437, R438, R440: Description (none) -> 49.9 Ohms ±1% 0.1W, 1/10W Chip Resistor 0603 (1608 Metric) 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; PartNumber (none) -> RC0603FR-0749R9L; digikey (none) -> 311-49.9HRCT-ND; price@10 (none) -> 0.02300
- R441, R442, R445, R446: Description (none) -> 470 Ohms ±5% 0.1W, 1/10W Chip Resistor 0603 (1608 Metric) A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; PartNumber (none) -> CRGCQ0603J470R; digikey (none) -> A130089CT-ND; price@10 (none) -> 0.02100
Connections:
- net ECAT0_RJ_LED0: now also JP405.1
- net ECAT1_RJ_LED1: now also JP406.1
- net ENET_CAT_XI: now also JP403.1, JP404.1
- net ecat1_led0: now also JP406.2
- net at R433.2, U402.17 (LED_0/AN_0/MLED): now also JP405.2
- net at JP401.1, U402.23 (XI): now also JP403.2
- net at JP402.1, U403.23 (XI): now also JP404.2
Other:
- note added: "the pullup of led_0 is mandatory, but to\n drive the led you could choose between \nPHY or uC populating/unpopulating the jumper"
- note removed: "the pullup of led_0 is mandatory, but to\n drive the led you could choose between \nPHY or uC populating/unpopulating the resistor"

Commit message: changes in footprints
Parts:
- renumbered U404 to J401
Changed lines of the file:
@@
 $EndComp
 $Comp
-L servo:rj45x2_0845-2G1T-H5 U404
+L servo:rj45x2_0845-2G1T-H5 J401
 U 1 1 5E2209F6
 P 14800 4900
-F 0 "U404" H 15277 4938 39  0000 L CNN
+F 0 "J401" H 15277 4938 39  0000 L CNN
 F 1 "RJ45x2" H 15277 4863 39  0000 L CNN
 F 2 "servo:rj45x2_0845-2G1T-H5" H 15300 5200 20  0001 C CNN

Commit message: fine imprivements
Connections:
- net Earth: now also J401.23 (shield), J401.24 (shield), J401.25 (shield), J401.26 (shield), J401.27 (shield), J401.28 (shield)
Other:
- moved on the sheet: C434
Changed lines of the file:
@@
 L servo:Earth #PWR?
 U 1 1 5E2B8CFA
-P 14600 6750
+P 14600 7450
 AR Path="/5DC3DC9E/5E2B8CFA" Ref="#PWR?"  Part="1"
 AR Path="/5DC4A59D/5E2B8CFA" Ref="#PWR0130"  Part="1"
-F 0 "#PWR0130" H 14600 6500 20  0001 C CNN
-F 1 "Earth" H 14600 6585 39  0000 C CNN
-F 2 "" H 14600 6750 50  0001 C CNN
-F 3 "~" H 14600 6750 50  0001 C CNN
-	1    14600 6750
+F 0 "#PWR0130" H 14600 7200 20  0001 C CNN
+F 1 "Earth" H 14600 7285 39  0000 C CNN
+F 2 "" H 14600 7450 50  0001 C CNN
+F 3 "~" H 14600 7450 50  0001 C CNN
+	1    14600 7450
 	1    0    0    -1
 $EndComp
@@
 L servo:Capacitor C434
 U 1 1 5E3BA4D2
-P 14850 6500
-F 0 "C434" V 14800 6450 20  0000 R CNN
-F 1 "4n7" V 14850 6450 20  0000 R CNN
-F 2 "servo:C_1206_3216Metric" H 14850 6400 60  0001 C CNN
-F 3 "" H 14850 6500 60  0000 C CNN
-F 4 "12061C472KAT2A" H 0   0   50  0001 C CNN "PartNumber"
-F 5 "478-1521-1-ND" H 0   0   50  0001 C CNN "digikey"
-F 6 "4700pF ±10% 100V Ceramic Capacitor X7R 1206 (3216 Metric) " H 0   0   50  0001 C CNN "Description"
-F 7 "0.18700" H 0   0   50  0001 C CNN "price@10"
-	1    14850 6500
+P 14850 7200
+F 0 "C434" V 14800 7150 20  0000 R CNN
+F 1 "4n7" V 14850 7150 20  0000 R CNN
+F 2 "servo:C_1206_3216Metric" H 14850 7100 60  0001 C CNN
+F 3 "" H 14850 7200 60  0000 C CNN
+F 4 "12061C472KAT2A" H 0   700 50  0001 C CNN "PartNumber"
+F 5 "478-1521-1-ND" H 0   700 50  0001 C CNN "digikey"
+F 6 "4700pF ±10% 100V Ceramic Capacitor X7R 1206 (3216 Metric) " H 0   700 50  0001 C CNN "Description"
+F 7 "0.18700" H 0   700 50  0001 C CNN "price@10"
+	1    14850 7200
 	0    1    1    0
 $EndComp
@@
 L servo:GND #GND_0102
 U 1 1 5E463A14
-P 14850 6750
-F 0 "#GND_0102" H 14855 6601 20  0001 C CNN
-F 1 "GND" H 14850 6593 30  0000 C CNN
-F 2 "" H 14850 6750 70  0000 C CNN
-F 3 "" H 14850 6750 70  0000 C CNN
-	1    14850 6750
-	1    0    0    -1
-$EndComp
-Wire Wire Line
-	14850 6750 14850 6700
-Wire Wire Line
-	14000 5600 14000 6400
-Wire Wire Line
-	14000 6400 14600 6400
+P 14850 7450
+F 0 "#GND_0102" H 14855 7301 20  0001 C CNN
+F 1 "GND" H 14850 7293 30  0000 C CNN
+F 2 "" H 14850 7450 70  0000 C CNN
+F 3 "" H 14850 7450 70  0000 C CNN
+	1    14850 7450
+	1    0    0    -1
+$EndComp
+Wire Wire Line
+	14850 7450 14850 7400
+Wire Wire Line
+	14000 5600 14000 7100
+Wire Wire Line
+	14000 7100 14100 7100
 Wire Wire Line
 	14000 4250 14000 5600
 Connection ~ 14000 5600
 Wire Wire Line
-	14600 6750 14600 6400
-Connection ~ 14600 6400
-Wire Wire Line
-	14600 6400 14850 6400
+	14600 7450 14600 7100
+Connection ~ 14600 7100
+Wire Wire Line
+	14600 7100 14850 7100
 Wire Wire Line
 	9050 950  9250 950
@@
 Wire Wire Line
 	10250 7400 10500 7400
+Wire Wire Line
+	14200 6350 14100 6350
+Wire Wire Line
+	14100 6350 14100 6450
+Wire Wire Line
+	14100 6650 14200 6650
+Wire Wire Line
+	14200 6550 14100 6550
+Connection ~ 14100 6550
+Wire Wire Line
+	14100 6550 14100 6650
+Wire Wire Line
+	14200 6450 14100 6450
+Connection ~ 14100 6450
+Wire Wire Line
+	14100 6450 14100 6550
+Wire Wire Line
+	14100 6650 14100 6750
+Connection ~ 14100 6650
+Connection ~ 14100 7100
+Wire Wire Line
+	14100 7100 14600 7100
+Wire Wire Line
+	14200 6750 14100 6750
+Connection ~ 14100 6750
+Wire Wire Line
+	14100 6750 14100 6850
+Wire Wire Line
+	14200 6850 14100 6850
+Connection ~ 14100 6850
+Wire Wire Line
+	14100 6850 14100 7100
 $EndSCHEMATC

Commit message: gerbers + pnp + bom ready
Parts:
- C404, C405, C407, C408, C409, C410, C411, C412, C414, C418, C419, C422, C423, C426, C427, C428, C429, C434, D401, D402, R401, R402, R403, R404, R405, R406, R407, R408, R409, R410, R411, R412, R413, R414, R415, R416, R417, R418, R419, R420, R421, R422, R424, R425, R427, R429, R430, R431, R432, R433, R434, R435, R437, R438, R440, R441, R442, R445, R446, Y401, Y402: bom_1 (none) -> 1; bom_2 (none) -> 1; bom_3 (none) -> 1
- J401: bom_3 (none) -> 1
- U401, U402, U403: bom_2 (none) -> 1; bom_3 (none) -> 1

Commit message: some details on gerbers, now released
Parts:
- J401, JP401, JP402, JP403, JP404, JP405, JP406: bom_1 (none) -> 0; bom_2 (none) -> 0
- U401, U402, U403: bom_1 (none) -> 0
Changed lines of the file:
@@
 F 8 "1" H 0   0   50  0001 C CNN "bom_2"
 F 9 "1" H 0   0   50  0001 C CNN "bom_3"
+F 10 "0" H 0   0   50  0001 C CNN "bom_1"
 	1    6650 2850
 	1    0    0    -1
@@
 F 7 "CAT24C16WI-GT3CT-ND " H 0   0   50  0001 C CNN "digikey"
 F 8 "0.16300" H 0   0   50  0001 C CNN "price@10"
-F 9 "" H 0   0   50  0001 C CNN "bom_1"
+F 9 "0" H 0   0   50  0001 C CNN "bom_1"
 F 10 "1" H 0   0   50  0001 C CNN "bom_2"
 F 11 "1" H 0   0   50  0001 C CNN "bom_3"
@@
 F 8 "1" H 0   0   50  0001 C CNN "bom_2"
 F 9 "1" H 0   0   50  0001 C CNN "bom_3"
+F 10 "0" H 0   0   50  0001 C CNN "bom_1"
 	1    6800 7000
 	1    0    0    -1
@@
 F 6 "380-1123-ND" H 0   0   50  0001 C CNN "digikey"
 F 7 "7.17400" H 0   0   50  0001 C CNN "price@10"
-F 8 "" H 0   0   50  0001 C CNN "bom_2"
+F 8 "0" H 0   0   50  0001 C CNN "bom_2"
 F 9 "1" H 0   0   50  0001 C CNN "bom_3"
+F 10 "0" H 0   0   50  0001 C CNN "bom_1"
 	1    14800 4900
 	1    0    0    -1
@@
 F 6 "-" H 4950 -2000 50  0001 C CNN "digikey"
 F 7 "0" H 4950 -2000 50  0001 C CNN "price@10"
-F 8 "" H 0   0   50  0001 C CNN "bom_1"
-F 9 "" H 0   0   50  0001 C CNN "bom_2"
+F 8 "0" H 0   0   50  0001 C CNN "bom_1"
+F 9 "0" H 0   0   50  0001 C CNN "bom_2"
 	1    8250 3600
 	0    1    1    0
@@
 F 6 "-" H 5100 2200 50  0001 C CNN "digikey"
 F 7 "0" H 5100 2200 50  0001 C CNN "price@10"
-F 8 "" H 0   0   50  0001 C CNN "bom_1"
-F 9 "" H 0   0   50  0001 C CNN "bom_2"
+F 8 "0" H 0   0   50  0001 C CNN "bom_1"
+F 9 "0" H 0   0   50  0001 C CNN "bom_2"
 	1    8400 7800
 	0    1    1    0
@@
 F 6 "-" H 5400 1900 50  0001 C CNN "digikey"
 F 7 "0" H 5400 1900 50  0001 C CNN "price@10"
-F 8 "" H 0   0   50  0001 C CNN "bom_1"
-F 9 "" H 0   0   50  0001 C CNN "bom_2"
+F 8 "0" H 0   0   50  0001 C CNN "bom_1"
+F 9 "0" H 0   0   50  0001 C CNN "bom_2"
 	1    8700 7500
 	-1   0    0    1
@@
 F 6 "-" H 5250 -2250 50  0001 C CNN "digikey"
 F 7 "0" H 5250 -2250 50  0001 C CNN "price@10"
-F 8 "" H 0   0   50  0001 C CNN "bom_1"
-F 9 "" H 0   0   50  0001 C CNN "bom_2"
+F 8 "0" H 0   0   50  0001 C CNN "bom_1"
+F 9 "0" H 0   0   50  0001 C CNN "bom_2"
 	1    8550 3350
 	-1   0    0    1
@@
 F 6 "-" H 7150 -2350 50  0001 C CNN "digikey"
 F 7 "0" H 7150 -2350 50  0001 C CNN "price@10"
-F 8 "" H 0   0   50  0001 C CNN "bom_1"
-F 9 "" H 0   0   50  0001 C CNN "bom_2"
+F 8 "0" H 0   0   50  0001 C CNN "bom_1"
+F 9 "0" H 0   0   50  0001 C CNN "bom_2"
 	1    10450 3250
 	-1   0    0    1
@@
 F 6 "-" H 7300 1800 50  0001 C CNN "digikey"
 F 7 "0" H 7300 1800 50  0001 C CNN "price@10"
-F 8 "" H 0   0   50  0001 C CNN "bom_1"
-F 9 "" H 0   0   50  0001 C CNN "bom_2"
+F 8 "0" H 0   0   50  0001 C CNN "bom_1"
+F 9 "0" H 0   0   50  0001 C CNN "bom_2"
 	1    10600 7400
 	-1   0    0    1
