File: kicad/ethernet.sch (KiCad schematic (older format))
At the start: 26 parts, among them IC201 TPD4E001QDBV, J201 0821-1X1T-36-F, U201 DP83822, Y201 dnp

Commit message: added sloted holes everyware
Parts:
- Y201: footprint Oscillator:Oscillator_SMD_SeikoEpson_SG210-4Pin_2.5x2.0mm -> servo:Crystal_SMD_2520-4Pin_2.5x2.0mm
Changed lines of the file:
@@
 F 0 "Y201" H 9250 5643 39  0000 C CNN
 F 1 "dnp" H 9250 5568 39  0000 C CNN
-F 2 "Oscillator:Oscillator_SMD_SeikoEpson_SG210-4Pin_2.5x2.0mm" H 9300 5300 60  0001 C CNN
+F 2 "servo:Crystal_SMD_2520-4Pin_2.5x2.0mm" H 9300 5300 60  0001 C CNN
 F 3 "../doc/datasheets//ECS-2520S.pdf" H 9150 5900 60  0001 C CNN
 	1    9250 5350

Commit message: serigrafia...
Parts:
- R201, R202, R203, R204, R205, R206, R207, R208, R209, R211, R212, R213: footprint Resistor_SMD:R_0603_1608Metric -> servo:R_0603_1608Metric
- R210: footprint Resistor_SMD:R_1206_3216Metric_Pad1.42x1.75mm_HandSolder -> servo:R_1206_3216Metric_Pad1.42x1.75mm_HandSolder
Changed lines of the file:
@@
 F 0 "R204" H 9350 4115 20  0000 C CNN
 F 1 "2.2k" H 9350 4072 20  0000 C CNN
-F 2 "Resistor_SMD:R_0603_1608Metric" H 8850 3900 60  0001 C CNN
+F 2 "servo:R_0603_1608Metric" H 8850 3900 60  0001 C CNN
 F 3 "" H 8950 4000 60  0001 C CNN
 F 4 "2.2k" V -150 2900 60  0001 C CNN "ValueDisplayed"
@@
 F 0 "R201" H 8850 3515 20  0000 C CNN
 F 1 "4.87k" H 8850 3472 20  0000 C CNN
-F 2 "Resistor_SMD:R_0603_1608Metric" H 8350 3300 60  0001 C CNN
+F 2 "servo:R_0603_1608Metric" H 8350 3300 60  0001 C CNN
 F 3 "" H 8450 3400 60  0001 C CNN
 F 4 "4.87k" V -150 2900 60  0001 C CNN "ValueDisplayed"
@@
 F 0 "R202" H 8750 4150 20  0000 C CNN
 F 1 "10.0k" H 9000 4150 20  0000 C CNN
-F 2 "Resistor_SMD:R_0603_1608Metric" H 8350 4000 60  0001 C CNN
+F 2 "servo:R_0603_1608Metric" H 8350 4000 60  0001 C CNN
 F 3 "" H 8450 4100 60  0001 C CNN
 F 4 "10.0k" V -150 2900 60  0001 C CNN "ValueDisplayed"
@@
 F 0 "R205" V 9528 2150 20  0000 L CNN
 F 1 "49.9" V 9571 2150 20  0000 L CNN
-F 2 "Resistor_SMD:R_0603_1608Metric" H 9050 2000 60  0001 C CNN
+F 2 "servo:R_0603_1608Metric" H 9050 2000 60  0001 C CNN
 F 3 "" H 9150 2100 60  0001 C CNN
 F 4 "49.9" V -750 3500 60  0001 C CNN "ValueDisplayed"
@@
 F 0 "R206" V 9728 2150 20  0000 L CNN
 F 1 "49.9" V 9771 2150 20  0000 L CNN
-F 2 "Resistor_SMD:R_0603_1608Metric" H 9250 2000 60  0001 C CNN
+F 2 "servo:R_0603_1608Metric" H 9250 2000 60  0001 C CNN
 F 3 "" H 9350 2100 60  0001 C CNN
 F 4 "49.9" V -550 3300 60  0001 C CNN "ValueDisplayed"
@@
 F 0 "R207" V 10778 2150 20  0000 R CNN
 F 1 "49.9" V 10821 2150 20  0000 R CNN
-F 2 "Resistor_SMD:R_0603_1608Metric" H 10300 2100 60  0001 C CNN
+F 2 "servo:R_0603_1608Metric" H 10300 2100 60  0001 C CNN
 F 3 "" H 10400 2200 60  0001 C CNN
 F 4 "49.9" V 0   1600 60  0001 C CNN "ValueDisplayed"
@@
 F 0 "R209" V 10928 2250 20  0000 L CNN
 F 1 "49.9" V 10971 2250 20  0000 L CNN
-F 2 "Resistor_SMD:R_0603_1608Metric" H 10450 2100 60  0001 C CNN
+F 2 "servo:R_0603_1608Metric" H 10450 2100 60  0001 C CNN
 F 3 "" H 10550 2200 60  0001 C CNN
 F 4 "49.9" V 150 1400 60  0001 C CNN "ValueDisplayed"
@@
 F 0 "R208" V 10828 4050 20  0000 L CNN
 F 1 "2.2k" V 10871 4050 20  0000 L CNN
-F 2 "Resistor_SMD:R_0603_1608Metric" H 10350 3900 60  0001 C CNN
+F 2 "servo:R_0603_1608Metric" H 10350 3900 60  0001 C CNN
 F 3 "" H 10450 4000 60  0001 C CNN
 F 4 "2.2k" V -450 1800 60  0001 C CNN "ValueDisplayed"
@@
 F 0 "R203" H 8950 4615 20  0000 C CNN
 F 1 "0e" H 8950 4572 20  0000 C CNN
-F 2 "Resistor_SMD:R_0603_1608Metric" H 8450 4400 60  0001 C CNN
+F 2 "servo:R_0603_1608Metric" H 8450 4400 60  0001 C CNN
 F 3 "" H 8550 4500 60  0001 C CNN
 F 4 "10.0k" V -50 3300 60  0001 C CNN "ValueDisplayed"
@@
 F 0 "R212" V 13428 2050 20  0000 L CNN
 F 1 "470" V 13471 2050 20  0000 L CNN
-F 2 "Resistor_SMD:R_0603_1608Metric" H 12950 1900 60  0001 C CNN
+F 2 "servo:R_0603_1608Metric" H 12950 1900 60  0001 C CNN
 F 3 "" H 13050 2000 60  0001 C CNN
 F 4 "470" V 3850 -2500 60  0001 C CNN "ValueDisplayed"
@@
 F 0 "R210" H 8500 8465 20  0000 C CNN
 F 1 "1oe" H 8500 8422 20  0000 C CNN
-F 2 "Resistor_SMD:R_1206_3216Metric_Pad1.42x1.75mm_HandSolder" H 8000 8250 60  0001 C CNN
+F 2 "servo:R_1206_3216Metric_Pad1.42x1.75mm_HandSolder" H 8000 8250 60  0001 C CNN
 F 3 "" H 8100 8350 60  0001 C CNN
 F 4 "10.0k" V -500 7150 60  0001 C CNN "ValueDisplayed"
@@
 F 0 "R211" V 11028 4050 20  0000 L CNN
 F 1 "2.2k" V 11071 4050 20  0000 L CNN
-F 2 "Resistor_SMD:R_0603_1608Metric" H 10550 3900 60  0001 C CNN
+F 2 "servo:R_0603_1608Metric" H 10550 3900 60  0001 C CNN
 F 3 "" H 10650 4000 60  0001 C CNN
 F 4 "2.2k" V -250 1800 60  0001 C CNN "ValueDisplayed"
@@
 F 0 "R213" V 13278 2050 20  0000 L CNN
 F 1 "470" V 13321 2050 20  0000 L CNN
-F 2 "Resistor_SMD:R_0603_1608Metric" H 12800 1900 60  0001 C CNN
+F 2 "servo:R_0603_1608Metric" H 12800 1900 60  0001 C CNN
 F 3 "" H 12900 2000 60  0001 C CNN
 F 4 "470" V 3700 -2500 60  0001 C CNN "ValueDisplayed"

Commit message: more serigraphy and now begin with planes
Parts:
- C217: footprint Capacitor_SMD:C_1206_3216Metric -> servo:C_1206_3216Metric
- IC201: footprint Package_TO_SOT_SMD:SOT-23-6 -> servo:SOT-23-6
Changed lines of the file:
@@
 F 0 "C217" V 15350 4400 20  0000 R CNN
 F 1 "4n7" V 15400 4400 20  0000 R CNN
-F 2 "Capacitor_SMD:C_1206_3216Metric" H 15400 4350 60  0001 C CNN
+F 2 "servo:C_1206_3216Metric" H 15400 4350 60  0001 C CNN
 F 3 "" H 15400 4450 60  0000 C CNN
 F 4 "1uF" V 3300 4950 60  0001 C CNN "ValueDisplayed"
@@
 F 0 "IC201" H 7800 8643 39  0000 C CNN
 F 1 "TPD4E001QDBV" H 7800 8568 39  0000 C CNN
-F 2 "Package_TO_SOT_SMD:SOT-23-6" H 7800 8350 60  0001 C CNN
+F 2 "servo:SOT-23-6" H 7800 8350 60  0001 C CNN
 F 3 "../doc/datasheets/tpd4e001-q1.pdf" H 7850 8650 60  0001 C CNN
 	1    7800 8350

Commit message: bom bom bom...
Parts:
- C202, C207, C209, C211: Description (none) -> CAP CER 0.1UF 16V X7R 0603; PartNumber (none) -> CC0603KPX7R7BB104; ValueDisplayed 0.1uF -> (none); digikey (none) -> 311-1335-1-ND
- C204, C205: PartNumber (none) -> GRM188R61A106ME69D; ValueDisplayed 10uF -> (none); digikey (none) -> 490-10475-1-ND
- C214, C216: Description (none) -> CAP CER 1UF 10V X7R 0603; PartNumber (none) -> C0603C105K8RACTU; ValueDisplayed 0.1uF -> (none); digikey (none) -> 399-11133-1-ND
- C217: PartNumber (none) -> 12061C472KAT2A; ValueDisplayed 1uF -> (none); digikey (none) -> 478-1521-1-ND
- R201: ValueDisplayed 4.87k -> (none)
- R202, R203: ValueDisplayed 10.0k -> (none)
- R204, R208, R211: ValueDisplayed 2.2k -> (none)
- R205, R206, R207, R209: ValueDisplayed 49.9 -> (none)
- R210: value 1oe -> 10e; ValueDisplayed 10.0k -> (none)
- R212, R213: ValueDisplayed 470 -> (none)
Changed lines of the file:
@@
 F 2 "servo:C_0603_1608Metric" H 10000 2100 60  0001 C CNN
 F 3 "" H 10000 2200 60  0000 C CNN
-F 4 "0.1uF" V -400 3000 60  0001 C CNN "ValueDisplayed"
+F 4 "311-1335-1-ND" H 0   0   50  0001 C CNN "digikey"
+F 5 "CAP CER 0.1UF 16V X7R 0603 " H 0   0   50  0001 C CNN "Description"
+F 6 "CC0603KPX7R7BB104" H 0   0   50  0001 C CNN "PartNumber"
 	1    10000 2200
 	0    -1   -1   0
@@
 F 2 "servo:R_0603_1608Metric" H 8850 3900 60  0001 C CNN
 F 3 "" H 8950 4000 60  0001 C CNN
-F 4 "2.2k" V -150 2900 60  0001 C CNN "ValueDisplayed"
 	1    9350 4000
 	1    0    0    -1
@@
 F 2 "servo:C_0603_1608Metric" H 12150 3750 60  0001 C CNN
 F 3 "" H 12150 3850 60  0000 C CNN
-F 4 "0.1uF" V 50  4150 60  0001 C CNN "ValueDisplayed"
+F 4 "CAP CER 1UF 10V X7R 0603" H 0   0   50  0001 C CNN "Description"
+F 5 "" H 0   0   50  0001 C CNN "Mfr part number"
+F 6 "399-11133-1-ND" H 0   0   50  0001 C CNN "digikey"
+F 7 "C0603C105K8RACTU" H 0   0   50  0001 C CNN "PartNumber"
 	1    12150 3850
 	0    1    1    0
@@
 F 2 "servo:C_0603_1608Metric" H 12450 3750 60  0001 C CNN
 F 3 "" H 12450 3850 60  0000 C CNN
-F 4 "0.1uF" V 350 3150 60  0001 C CNN "ValueDisplayed"
+F 4 "" V 350 3150 60  0001 C CNN "ValueDisplayed"
+F 5 "CAP CER 1UF 10V X7R 0603" H 0   0   50  0001 C CNN "Description"
+F 6 "" H 0   0   50  0001 C CNN "Mfr part number"
+F 7 "399-11133-1-ND" H 0   0   50  0001 C CNN "digikey"
+F 8 "C0603C105K8RACTU" H 0   0   50  0001 C CNN "PartNumber"
 	1    12450 3850
 	0    1    1    0
@@
 U 1 1 63C68164
 P 11250 2250
-F 0 "C211" V 11322 2360 20  0000 L CNN
-F 1 "0.1uF" V 11279 2360 20  0000 L CNN
+F 0 "C211" V 11322 2140 20  0000 R CNN
+F 1 "0.1uF" V 11279 2140 20  0000 R CNN
 F 2 "servo:C_0603_1608Metric" H 11250 2150 60  0001 C CNN
 F 3 "" H 11250 2250 60  0000 C CNN
-F 4 "0.1uF" V 350 850 60  0001 C CNN "ValueDisplayed"
+F 4 "CAP CER 0.1UF 16V X7R 0603 " H 11250 2250 50  0001 C CNN "Description"
+F 5 "311-1335-1-ND" H 0   0   50  0001 C CNN "digikey"
+F 6 "CC0603KPX7R7BB104" H 0   0   50  0001 C CNN "PartNumber"
 	1    11250 2250
 	0    -1   -1   0
@@
 F 2 "servo:C_0603_1608Metric" H 4750 3200 60  0001 C CNN
 F 3 "" H 4750 3300 60  0000 C CNN
-F 4 "0.1uF" V 450 4300 60  0001 C CNN "ValueDisplayed"
+F 4 "311-1335-1-ND" H 0   0   50  0001 C CNN "digikey"
+F 5 "CAP CER 0.1UF 16V X7R 0603 " H 0   0   50  0001 C CNN "Description"
+F 6 "CC0603KPX7R7BB104" H 0   0   50  0001 C CNN "PartNumber"
 	1    4750 3300
 	0    -1   -1   0
@@
 F 2 "servo:C_0603_1608Metric" H 3900 2900 60  0001 C CNN
 F 3 "" H 3900 3000 60  0000 C CNN
-F 4 "0.1uF" V -2700 4000 60  0001 C CNN "ValueDisplayed"
+F 4 "311-1335-1-ND" H 0   0   50  0001 C CNN "digikey"
+F 5 "CAP CER 0.1UF 16V X7R 0603 " H 0   0   50  0001 C CNN "Description"
+F 6 "CC0603KPX7R7BB104" H 0   0   50  0001 C CNN "PartNumber"
 	1    3900 3000
 	0    1    1    0
@@
 F 2 "servo:R_0603_1608Metric" H 8350 3300 60  0001 C CNN
 F 3 "" H 8450 3400 60  0001 C CNN
-F 4 "4.87k" V -150 2900 60  0001 C CNN "ValueDisplayed"
 	1    8850 3400
 	1    0    0    -1
@@
 F 2 "servo:R_0603_1608Metric" H 8350 4000 60  0001 C CNN
 F 3 "" H 8450 4100 60  0001 C CNN
-F 4 "10.0k" V -150 2900 60  0001 C CNN "ValueDisplayed"
 	1    8850 4100
 	1    0    0    -1
@@
 F 2 "servo:R_0603_1608Metric" H 9050 2000 60  0001 C CNN
 F 3 "" H 9150 2100 60  0001 C CNN
-F 4 "49.9" V -750 3500 60  0001 C CNN "ValueDisplayed"
 	1    9550 2100
 	0    1    1    0
@@
 F 2 "servo:R_0603_1608Metric" H 9250 2000 60  0001 C CNN
 F 3 "" H 9350 2100 60  0001 C CNN
-F 4 "49.9" V -550 3300 60  0001 C CNN "ValueDisplayed"
 	1    9750 2100
 	0    1    1    0
@@
 F 2 "servo:R_0603_1608Metric" H 10300 2100 60  0001 C CNN
 F 3 "" H 10400 2200 60  0001 C CNN
-F 4 "49.9" V 0   1600 60  0001 C CNN "ValueDisplayed"
 	1    10800 2200
 	0    1    1    0
@@
 F 2 "servo:R_0603_1608Metric" H 10450 2100 60  0001 C CNN
 F 3 "" H 10550 2200 60  0001 C CNN
-F 4 "49.9" V 150 1400 60  0001 C CNN "ValueDisplayed"
 	1    10950 2200
 	0    1    1    0
@@
 F 2 "servo:C_0603_1608Metric" H 4450 3200 60  0001 C CNN
 F 3 "" H 4450 3300 60  0000 C CNN
-F 4 "10uF" V 950 4300 60  0001 C CNN "ValueDisplayed"
+F 4 "490-10475-1-ND" H 0   0   50  0001 C CNN "digikey"
+F 5 "GRM188R61A106ME69D " H 0   0   50  0001 C CNN "PartNumber"
 	1    4450 3300
 	0    -1   -1   0
@@
 F 2 "servo:C_0603_1608Metric" H 4150 3000 60  0001 C CNN
 F 3 "" H 4150 3100 60  0000 C CNN
-F 4 "10uF" V -3250 4100 60  0001 C CNN "ValueDisplayed"
+F 4 "490-10475-1-ND" H 0   0   50  0001 C CNN "digikey"
+F 5 "GRM188R61A106ME69D " H 0   0   50  0001 C CNN "PartNumber"
 	1    4150 3100
 	0    -1   -1   0
@@
 F 2 "servo:R_0603_1608Metric" H 10350 3900 60  0001 C CNN
 F 3 "" H 10450 4000 60  0001 C CNN
-F 4 "2.2k" V -450 1800 60  0001 C CNN "ValueDisplayed"
 	1    10850 4000
 	0    1    1    0
@@
 F 2 "servo:R_0603_1608Metric" H 8450 4400 60  0001 C CNN
 F 3 "" H 8550 4500 60  0001 C CNN
-F 4 "10.0k" V -50 3300 60  0001 C CNN "ValueDisplayed"
 	1    8950 4500
 	1    0    0    -1
@@
 F 2 "servo:R_0603_1608Metric" H 12950 1900 60  0001 C CNN
 F 3 "" H 13050 2000 60  0001 C CNN
-F 4 "470" V 3850 -2500 60  0001 C CNN "ValueDisplayed"
 	1    13450 2000
 	0    1    1    0
@@
 F 2 "servo:C_1206_3216Metric" H 15400 4350 60  0001 C CNN
 F 3 "" H 15400 4450 60  0000 C CNN
-F 4 "1uF" V 3300 4950 60  0001 C CNN "ValueDisplayed"
+F 4 "12061C472KAT2A" H 0   0   50  0001 C CNN "PartNumber"
+F 5 "478-1521-1-ND" H 0   0   50  0001 C CNN "digikey"
 	1    15400 4450
 	0    1    1    0
@@
 P 8500 8350
 F 0 "R210" H 8500 8465 20  0000 C CNN
-F 1 "1oe" H 8500 8422 20  0000 C CNN
+F 1 "10e" H 8500 8422 20  0000 C CNN
 F 2 "servo:R_1206_3216Metric_Pad1.42x1.75mm_HandSolder" H 8000 8250 60  0001 C CNN
 F 3 "" H 8100 8350 60  0001 C CNN
-F 4 "10.0k" V -500 7150 60  0001 C CNN "ValueDisplayed"
 	1    8500 8350
 	1    0    0    -1
@@
 F 2 "servo:R_0603_1608Metric" H 10550 3900 60  0001 C CNN
 F 3 "" H 10650 4000 60  0001 C CNN
-F 4 "2.2k" V -250 1800 60  0001 C CNN "ValueDisplayed"
 	1    11050 4000
 	0    1    1    0
@@
 F 2 "servo:R_0603_1608Metric" H 12800 1900 60  0001 C CNN
 F 3 "" H 12900 2000 60  0001 C CNN
-F 4 "470" V 3700 -2500 60  0001 C CNN "ValueDisplayed"
 	1    13300 2000
 	0    1    1    0

Commit message: more bom...
Parts:
- C204, C205: Description (none) -> 10µF ±20% 10V Ceramic Capacitor X5R 0603 (1608 Metric)
- C217: Description (none) -> 4700pF ±10% 100V Ceramic Capacitor X7R 1206 (3216 Metric)
- IC201: Description (none) -> TVS DIODE 5.5V 16V SOT23-6; PartNumber (none) -> TPD4E001QDBVRQ1; digikey (none) -> 296-39344-1-ND
- J201: value 0821-1X1T-36-F -> RJ45 USB; Description (none) -> 1 Port RJ45 with USB A Magjack Connector Through Hole 10/10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; PartNumber (none) -> 0821-1X1T-36-F; digikey (none) -> 0821-1X1T-36-F
- R203: value 0e -> 0
- R210: value 10e -> 10
- U201: Description (none) -> Ethernet Interface 32-VQFN (5x5); digikey (none) -> 296-47256-1-ND; price@10 (none) -> 2.37700
Changed lines of the file:
@@
 F 3 "../doc/datasheets/dp83822i.pdf" H 7150 4000 50  0001 C CNN
 F 4 "DP83822IRHBR" V -150 2900 60  0001 C CNN "PartNumber"
+F 5 "Ethernet Interface 32-VQFN (5x5) " H 0   0   50  0001 C CNN "Description"
+F 6 "296-47256-1-ND" H 0   0   50  0001 C CNN "digikey"
+F 7 "2.37700" H 0   0   50  0001 C CNN "price@10"
 	1    7150 4000
 	1    0    0    -1
@@
 F 4 "490-10475-1-ND" H 0   0   50  0001 C CNN "digikey"
 F 5 "GRM188R61A106ME69D " H 0   0   50  0001 C CNN "PartNumber"
+F 6 "10µF ±20% 10V Ceramic Capacitor X5R 0603 (1608 Metric) " H 0   0   50  0001 C CNN "Description"
 	1    4450 3300
 	0    -1   -1   0
@@
 F 4 "490-10475-1-ND" H 0   0   50  0001 C CNN "digikey"
 F 5 "GRM188R61A106ME69D " H 0   0   50  0001 C CNN "PartNumber"
+F 6 "10µF ±20% 10V Ceramic Capacitor X5R 0603 (1608 Metric) " H 0   0   50  0001 C CNN "Description"
 	1    4150 3100
 	0    -1   -1   0
@@
 P 8950 4500
 F 0 "R203" H 8950 4615 20  0000 C CNN
-F 1 "0e" H 8950 4572 20  0000 C CNN
+F 1 "0" H 8950 4572 20  0000 C CNN
 F 2 "servo:R_0603_1608Metric" H 8450 4400 60  0001 C CNN
 F 3 "" H 8550 4500 60  0001 C CNN
@@
 F 4 "12061C472KAT2A" H 0   0   50  0001 C CNN "PartNumber"
 F 5 "478-1521-1-ND" H 0   0   50  0001 C CNN "digikey"
+F 6 "4700pF ±10% 100V Ceramic Capacitor X7R 1206 (3216 Metric) " H 0   0   50  0001 C CNN "Description"
 	1    15400 4450
 	0    1    1    0
@@
 F 2 "servo:SOT-23-6" H 7800 8350 60  0001 C CNN
 F 3 "../doc/datasheets/tpd4e001-q1.pdf" H 7850 8650 60  0001 C CNN
+F 4 "TVS DIODE 5.5V 16V SOT23-6 " H 0   0   50  0001 C CNN "Description"
+F 5 "TPD4E001QDBVRQ1" H 0   0   50  0001 C CNN "PartNumber"
+F 6 " 296-39344-1-ND" H 0   0   50  0001 C CNN "digikey"
 	1    7800 8350
 	1    0    0    -1
@@
 P 8500 8350
 F 0 "R210" H 8500 8465 20  0000 C CNN
-F 1 "10e" H 8500 8422 20  0000 C CNN
+F 1 "10" H 8500 8422 20  0000 C CNN
 F 2 "servo:R_1206_3216Metric_Pad1.42x1.75mm_HandSolder" H 8000 8250 60  0001 C CNN
 F 3 "" H 8100 8350 60  0001 C CNN
@@
 P 14150 3300
 F 0 "J201" H 14400 4565 50  0000 C CNN
-F 1 "0821-1X1T-36-F" H 14400 4474 50  0000 C CNN
+F 1 "RJ45 USB" H 14400 4474 50  0000 C CNN
 F 2 "servo:BEL_0821-1X1T-36-F" H 14000 4650 50  0001 L BNN
 F 3 "../doc/datasheets/dr-MAG-0821-1X1T-36-F.pdf" H 14150 4550 50  0001 L BNN
+F 4 "1 Port RJ45 with USB A Magjack Connector Through Hole 10/100 Base-T, AutoMDIX " H 0   0   50  0001 C CNN "Description"
+F 5 "0821-1X1T-36-F " H 0   0   50  0001 C CNN "PartNumber"
+F 6 "0821-1X1T-36-F " H 0   0   50  0001 C CNN "digikey"
 	1    14150 3300
 	1    0    0    -1

Commit message: stackup
Parts:
- added JP201: jumper, servo:SolderJumper-2_P1.3mm_Open_RoundedPad1.0x1.5mm, symbol servo:jumper
- C202, C207, C209, C211: price@10 (none) -> 0.05800
- C204, C205: price@10 (none) -> 0.15400
- C214, C216: price@10 (none) -> 0.06400
- C217: price@10 (none) -> 0.18700
- IC201: digikey 296-39344-1-ND -> 296-39344-1-ND; price@10 (none) -> 0.56800
- J201: digikey 0821-1X1T-36-F -> 507-1424-ND; price@10 (none) -> 4.89600
- Y201: value dnp -> osc 25Mhz; Description (none) -> 25MHz XO (Standard) HCMOS Oscillator 3.3V Enable/Disable 4-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; PartNumber (none) -> ECS-2520S33-250-FN-TR; digikey (none) -> XC2198CT-ND; price@10 (none) -> 1.41900
Connections:
- net clk_xi: now also JP201.1; no longer Y201.3 (OUTPUT)
- new net: JP201.2, Y201.3 (OUTPUT)
Changed lines of the file:
@@
 F 5 "CAP CER 0.1UF 16V X7R 0603 " H 0   0   50  0001 C CNN "Description"
 F 6 "CC0603KPX7R7BB104" H 0   0   50  0001 C CNN "PartNumber"
+F 7 "0.05800" H 0   0   50  0001 C CNN "price@10"
 	1    10000 2200
 	0    -1   -1   0
@@
 F 3 "" H 12150 3850 60  0000 C CNN
 F 4 "CAP CER 1UF 10V X7R 0603" H 0   0   50  0001 C CNN "Description"
-F 5 "" H 0   0   50  0001 C CNN "Mfr part number"
-F 6 "399-11133-1-ND" H 0   0   50  0001 C CNN "digikey"
-F 7 "C0603C105K8RACTU" H 0   0   50  0001 C CNN "PartNumber"
+F 5 "399-11133-1-ND" H 0   0   50  0001 C CNN "digikey"
+F 6 "C0603C105K8RACTU" H 0   0   50  0001 C CNN "PartNumber"
+F 7 "0.06400" H 0   0   50  0001 C CNN "price@10"
 	1    12150 3850
 	0    1    1    0
@@
 F 2 "servo:C_0603_1608Metric" H 12450 3750 60  0001 C CNN
 F 3 "" H 12450 3850 60  0000 C CNN
-F 4 "" V 350 3150 60  0001 C CNN "ValueDisplayed"
-F 5 "CAP CER 1UF 10V X7R 0603" H 0   0   50  0001 C CNN "Description"
-F 6 "" H 0   0   50  0001 C CNN "Mfr part number"
-F 7 "399-11133-1-ND" H 0   0   50  0001 C CNN "digikey"
-F 8 "C0603C105K8RACTU" H 0   0   50  0001 C CNN "PartNumber"
+F 4 "CAP CER 1UF 10V X7R 0603" H 0   0   50  0001 C CNN "Description"
+F 5 "399-11133-1-ND" H 0   0   50  0001 C CNN "digikey"
+F 6 "C0603C105K8RACTU" H 0   0   50  0001 C CNN "PartNumber"
+F 7 "0.06400" H 0   0   50  0001 C CNN "price@10"
 	1    12450 3850
 	0    1    1    0
@@
 F 5 "311-1335-1-ND" H 0   0   50  0001 C CNN "digikey"
 F 6 "CC0603KPX7R7BB104" H 0   0   50  0001 C CNN "PartNumber"
+F 7 "0.05800" H 0   0   50  0001 C CNN "price@10"
 	1    11250 2250
 	0    -1   -1   0
@@
 F 5 "CAP CER 0.1UF 16V X7R 0603 " H 0   0   50  0001 C CNN "Description"
 F 6 "CC0603KPX7R7BB104" H 0   0   50  0001 C CNN "PartNumber"
+F 7 "0.05800" H 0   0   50  0001 C CNN "price@10"
 	1    4750 3300
 	0    -1   -1   0
@@
 F 5 "CAP CER 0.1UF 16V X7R 0603 " H 0   0   50  0001 C CNN "Description"
 F 6 "CC0603KPX7R7BB104" H 0   0   50  0001 C CNN "PartNumber"
+F 7 "0.05800" H 0   0   50  0001 C CNN "price@10"
 	1    3900 3000
 	0    1    1    0
@@
 F 5 "GRM188R61A106ME69D " H 0   0   50  0001 C CNN "PartNumber"
 F 6 "10µF ±20% 10V Ceramic Capacitor X5R 0603 (1608 Metric) " H 0   0   50  0001 C CNN "Description"
+F 7 "0.15400" H 0   0   50  0001 C CNN "price@10"
 	1    4450 3300
 	0    -1   -1   0
@@
 F 5 "GRM188R61A106ME69D " H 0   0   50  0001 C CNN "PartNumber"
 F 6 "10µF ±20% 10V Ceramic Capacitor X5R 0603 (1608 Metric) " H 0   0   50  0001 C CNN "Description"
+F 7 "0.15400" H 0   0   50  0001 C CNN "price@10"
 	1    4150 3100
 	0    -1   -1   0
@@
 AR Path="/5DC4A59D/63C6828B" Ref="Y?"  Part="1"
 F 0 "Y201" H 9250 5643 39  0000 C CNN
-F 1 "dnp" H 9250 5568 39  0000 C CNN
+F 1 "osc 25Mhz" H 9250 5568 39  0000 C CNN
 F 2 "servo:Crystal_SMD_2520-4Pin_2.5x2.0mm" H 9300 5300 60  0001 C CNN
 F 3 "../doc/datasheets//ECS-2520S.pdf" H 9150 5900 60  0001 C CNN
+F 4 "25MHz XO (Standard) HCMOS Oscillator 3.3V Enable/Disable 4-SMD, No Lead " H 0   0   50  0001 C CNN "Description"
+F 5 "ECS-2520S33-250-FN-TR" H 0   0   50  0001 C CNN "PartNumber"
+F 6 "XC2198CT-ND " H 0   0   50  0001 C CNN "digikey"
+F 7 "1.41900" H 0   0   50  0001 C CNN "price@10"
 	1    9250 5350
 	-1   0    0    -1
@@
 	8550 4500 8750 4500
 Wire Wire Line
-	8750 4500 8750 5250
-Wire Wire Line
 	8750 5250 9000 5250
-Connection ~ 8750 4500
 $Comp
 L servo:GND #GND_0204
@@
 F 5 "478-1521-1-ND" H 0   0   50  0001 C CNN "digikey"
 F 6 "4700pF ±10% 100V Ceramic Capacitor X7R 1206 (3216 Metric) " H 0   0   50  0001 C CNN "Description"
+F 7 "0.18700" H 0   0   50  0001 C CNN "price@10"
 	1    15400 4450
 	0    1    1    0
@@
 F 4 "TVS DIODE 5.5V 16V SOT23-6 " H 0   0   50  0001 C CNN "Description"
 F 5 "TPD4E001QDBVRQ1" H 0   0   50  0001 C CNN "PartNumber"
-F 6 " 296-39344-1-ND" H 0   0   50  0001 C CNN "digikey"
+F 6 "296-39344-1-ND" H 0   0   50  0001 C CNN "digikey"
+F 7 "0.56800" H 0   0   50  0001 C CNN "price@10"
 	1    7800 8350
 	1    0    0    -1
@@
 F 4 "1 Port RJ45 with USB A Magjack Connector Through Hole 10/100 Base-T, AutoMDIX " H 0   0   50  0001 C CNN "Description"
 F 5 "0821-1X1T-36-F " H 0   0   50  0001 C CNN "PartNumber"
-F 6 "0821-1X1T-36-F " H 0   0   50  0001 C CNN "digikey"
+F 6 "507-1424-ND " H 0   0   50  0001 C CNN "digikey"
+F 7 "4.89600" H 0   0   50  0001 C CNN "price@10"
 	1    14150 3300
 	1    0    0    -1
@@
 Wire Wire Line
 	4600 3500 4750 3500
+$Comp
+L servo:jumper JP?
+U 1 1 5EBCD9AF
+P 8750 4700
+AR Path="/5DD76B18/5EBCD9AF" Ref="JP?"  Part="1"
+AR Path="/5DC4A59D/5EBCD9AF" Ref="JP?"  Part="1"
+AR Path="/5DC3DC9E/5EBCD9AF" Ref="JP201"  Part="1"
+F 0 "JP201" V 8712 4748 39  0000 L CNN
+F 1 "jumper" V 8787 4748 39  0000 L CNN
+F 2 "servo:SolderJumper-2_P1.3mm_Open_RoundedPad1.0x1.5mm" H 8650 4680 50  0001 C CNN
+F 3 "~" H 8750 4780 50  0001 C CNN
+F 4 "jumper smd bridge using tin" H 5450 -900 50  0001 C CNN "Description"
+F 5 "-" H 5450 -900 50  0001 C CNN "PartNumber"
+F 6 "-" H 5450 -900 50  0001 C CNN "digikey"
+F 7 "0" H 5450 -900 50  0001 C CNN "price@10"
+	1    8750 4700
+	0    1    1    0
+$EndComp
+Wire Wire Line
+	8750 4600 8750 4500
+Connection ~ 8750 4500
+Wire Wire Line
+	8750 4800 8750 5250
 $EndSCHEMATC
