File: kicad/ethernet.sch (KiCad schematic (older format))
At the start: 27 parts, among them IC201 TPD4E001QDBV, J201 RJ45 USB, U201 DP83822, Y201 osc 25Mhz

Commit message: bom copleted
Parts:
- removed R203: 0, servo:R_0603_1608Metric, symbol servo:Resistor
- added JP202: jumper, servo:SolderJumper-2_P1.3mm_Open_RoundedPad1.0x1.5mm, symbol servo:jumper
- R201: Description (none) -> 4.87 kOhms ±1% 0.1W, 1/10W Chip Resistor 0603 (1608 Metric)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; PartNumber (none) -> RMCF0603FT4K87; digikey (none) -> RMCF0603FT4K87CT-ND; price@10 (none) -> 0.01600
- R202: value 10.0k -> 10k; Description (none) -> 10 kOhms ±5% 0.1W, 1/10W Chip Resistor 0603 (1608 Metric) M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; PartNumber (none) -> RC0603JR-0710KL; digikey (none) -> 311-10KGRCT-ND; price@10 (none) -> 0.01900
- R204, R208, R211: Description (none) -> 2.2 kOhms ±5% 0.1W, 1/10W Chip Resistor 0603 (1608 Metric) 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; PartNumber (none) -> ERJ-3GEYJ222V; digikey (none) -> P2.2KGCT-ND; price@10 (none) -> 0.04500
- R205, R206, R207, R209: Description (none) -> 49.9 Ohms ±1% 0.1W, 1/10W Chip Resistor 0603 (1608 Metric) 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; PartNumber (none) -> RC0603FR-0749R9L; digikey (none) -> 311-49.9HRCT-ND; price@10 (none) -> 0.02300
- R210: Description (none) -> 10 Ohms ±5% 0.1W, 1/10W Chip Resistor 0603 (1608 Metric) Au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; PartNumber (none) -> CRGCQ0603J10R; digikey (none) -> A130079CT-ND; price@10 (none) -> 0.02100
- R212, R213: Description (none) -> 470 Ohms ±5% 0.1W, 1/10W Chip Resistor 0603 (1608 Metric) A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; PartNumber (none) -> CRGCQ0603J470R; digikey (none) -> A130089CT-ND; price@10 (none) -> 0.02100
Connections:
- net ENET_CAT_XI: now also JP202.1
- net clk_xi: now also JP202.2
Changed lines of the file:
@@
 F 2 "servo:R_0603_1608Metric" H 8850 3900 60  0001 C CNN
 F 3 "" H 8950 4000 60  0001 C CNN
+F 4 "2.2 kOhms ±5% 0.1W, 1/10W Chip Resistor 0603 (1608 Metric) Automotive AEC-Q200 Thick Film " H 0   0   50  0001 C CNN "Description"
+F 5 "ERJ-3GEYJ222V" H 0   0   50  0001 C CNN "PartNumber"
+F 6 "P2.2KGCT-ND " H 0   0   50  0001 C CNN "digikey"
+F 7 "0.04500" H 0   0   50  0001 C CNN "price@10"
 	1    9350 4000
 	1    0    0    -1
@@
 F 2 "servo:R_0603_1608Metric" H 8350 3300 60  0001 C CNN
 F 3 "" H 8450 3400 60  0001 C CNN
+F 4 "4.87 kOhms ±1% 0.1W, 1/10W Chip Resistor 0603 (1608 Metric) Automotive AEC-Q200 Thick Film" H 0   0   50  0001 C CNN "Description"
+F 5 "RMCF0603FT4K87" H 0   0   50  0001 C CNN "PartNumber"
+F 6 " RMCF0603FT4K87CT-ND" H 0   0   50  0001 C CNN "digikey"
+F 7 "0.01600" H 0   0   50  0001 C CNN "price@10"
 	1    8850 3400
 	1    0    0    -1
@@
 P 8850 4100
 F 0 "R202" H 8750 4150 20  0000 C CNN
-F 1 "10.0k" H 9000 4150 20  0000 C CNN
+F 1 "10k" H 9000 4150 20  0000 C CNN
 F 2 "servo:R_0603_1608Metric" H 8350 4000 60  0001 C CNN
 F 3 "" H 8450 4100 60  0001 C CNN
+F 4 "10 kOhms ±5% 0.1W, 1/10W Chip Resistor 0603 (1608 Metric) Moisture Resistant Thick Film " H 0   0   50  0001 C CNN "Description"
+F 5 "RC0603JR-0710KL" H 0   0   50  0001 C CNN "PartNumber"
+F 6 "311-10KGRCT-ND" H 0   0   50  0001 C CNN "digikey"
+F 7 "0.01900" H 0   0   50  0001 C CNN "price@10"
 	1    8850 4100
 	1    0    0    -1
@@
 F 2 "servo:R_0603_1608Metric" H 9050 2000 60  0001 C CNN
 F 3 "" H 9150 2100 60  0001 C CNN
+F 4 "49.9 Ohms ±1% 0.1W, 1/10W Chip Resistor 0603 (1608 Metric) Moisture Resistant Thick Film " H 0   0   50  0001 C CNN "Description"
+F 5 "RC0603FR-0749R9L" H 0   0   50  0001 C CNN "PartNumber"
+F 6 "311-49.9HRCT-ND" H 0   0   50  0001 C CNN "digikey"
+F 7 "0.02300" H 0   0   50  0001 C CNN "price@10"
 	1    9550 2100
 	0    1    1    0
@@
 F 2 "servo:R_0603_1608Metric" H 9250 2000 60  0001 C CNN
 F 3 "" H 9350 2100 60  0001 C CNN
+F 4 "49.9 Ohms ±1% 0.1W, 1/10W Chip Resistor 0603 (1608 Metric) Moisture Resistant Thick Film " H 0   0   50  0001 C CNN "Description"
+F 5 "RC0603FR-0749R9L" H 0   0   50  0001 C CNN "PartNumber"
+F 6 "311-49.9HRCT-ND" H 0   0   50  0001 C CNN "digikey"
+F 7 "0.02300" H 0   0   50  0001 C CNN "price@10"
 	1    9750 2100
 	0    1    1    0
@@
 F 2 "servo:R_0603_1608Metric" H 10300 2100 60  0001 C CNN
 F 3 "" H 10400 2200 60  0001 C CNN
+F 4 "49.9 Ohms ±1% 0.1W, 1/10W Chip Resistor 0603 (1608 Metric) Moisture Resistant Thick Film " H 0   0   50  0001 C CNN "Description"
+F 5 "RC0603FR-0749R9L" H 0   0   50  0001 C CNN "PartNumber"
+F 6 "311-49.9HRCT-ND" H 0   0   50  0001 C CNN "digikey"
+F 7 "0.02300" H 0   0   50  0001 C CNN "price@10"
 	1    10800 2200
 	0    1    1    0
@@
 F 2 "servo:R_0603_1608Metric" H 10450 2100 60  0001 C CNN
 F 3 "" H 10550 2200 60  0001 C CNN
+F 4 "49.9 Ohms ±1% 0.1W, 1/10W Chip Resistor 0603 (1608 Metric) Moisture Resistant Thick Film " H 0   0   50  0001 C CNN "Description"
+F 5 "RC0603FR-0749R9L" H 0   0   50  0001 C CNN "PartNumber"
+F 6 "311-49.9HRCT-ND" H 0   0   50  0001 C CNN "digikey"
+F 7 "0.02300" H 0   0   50  0001 C CNN "price@10"
 	1    10950 2200
 	0    1    1    0
@@
 F 2 "servo:R_0603_1608Metric" H 10350 3900 60  0001 C CNN
 F 3 "" H 10450 4000 60  0001 C CNN
+F 4 "2.2 kOhms ±5% 0.1W, 1/10W Chip Resistor 0603 (1608 Metric) Automotive AEC-Q200 Thick Film " H 0   0   50  0001 C CNN "Description"
+F 5 "ERJ-3GEYJ222V" H 0   0   50  0001 C CNN "PartNumber"
+F 6 "P2.2KGCT-ND " H 0   0   50  0001 C CNN "digikey"
+F 7 "0.04500" H 0   0   50  0001 C CNN "price@10"
 	1    10850 4000
 	0    1    1    0
@@
 Text GLabel 9550 4500 2    50   Input ~ 0
 ENET_CAT_XI
-$Comp
-L servo:Resistor R203
-U 1 1 63C68282
-P 8950 4500
-F 0 "R203" H 8950 4615 20  0000 C CNN
-F 1 "0" H 8950 4572 20  0000 C CNN
-F 2 "servo:R_0603_1608Metric" H 8450 4400 60  0001 C CNN
-F 3 "" H 8550 4500 60  0001 C CNN
-	1    8950 4500
-	1    0    0    -1
-$EndComp
-Wire Wire Line
-	9550 4500 9150 4500
+Wire Wire Line
+	9550 4500 9250 4500
 Text Notes 6700 1800 0    197  ~ 39
 EtherNET
@@
 F 2 "servo:R_0603_1608Metric" H 12950 1900 60  0001 C CNN
 F 3 "" H 13050 2000 60  0001 C CNN
+F 4 "470 Ohms ±5% 0.1W, 1/10W Chip Resistor 0603 (1608 Metric) Automotive AEC-Q200, Moisture Resistant Thick Film " H 0   0   50  0001 C CNN "Description"
+F 5 "CRGCQ0603J470R" H 0   0   50  0001 C CNN "PartNumber"
+F 6 "A130089CT-ND" H 0   0   50  0001 C CNN "digikey"
+F 7 "0.02100" H 0   0   50  0001 C CNN "price@10"
 	1    13450 2000
 	0    1    1    0
@@
 F 2 "servo:R_1206_3216Metric_Pad1.42x1.75mm_HandSolder" H 8000 8250 60  0001 C CNN
 F 3 "" H 8100 8350 60  0001 C CNN
+F 4 " 10 Ohms ±5% 0.1W, 1/10W Chip Resistor 0603 (1608 Metric) Automotive AEC-Q200, Moisture Resistant Thick Film " H 0   0   50  0001 C CNN "Description"
+F 5 "CRGCQ0603J10R" H 0   0   50  0001 C CNN "PartNumber"
+F 6 "A130079CT-ND" H 0   0   50  0001 C CNN "digikey"
+F 7 "0.02100" H 0   0   50  0001 C CNN "price@10"
 	1    8500 8350
 	1    0    0    -1
@@
 F 2 "servo:R_0603_1608Metric" H 10550 3900 60  0001 C CNN
 F 3 "" H 10650 4000 60  0001 C CNN
+F 4 "2.2 kOhms ±5% 0.1W, 1/10W Chip Resistor 0603 (1608 Metric) Automotive AEC-Q200 Thick Film " H 0   0   50  0001 C CNN "Description"
+F 5 "ERJ-3GEYJ222V" H 0   0   50  0001 C CNN "PartNumber"
+F 6 "P2.2KGCT-ND " H 0   0   50  0001 C CNN "digikey"
+F 7 "0.04500" H 0   0   50  0001 C CNN "price@10"
 	1    11050 4000
 	0    1    1    0
@@
 F 2 "servo:R_0603_1608Metric" H 12800 1900 60  0001 C CNN
 F 3 "" H 12900 2000 60  0001 C CNN
+F 4 "470 Ohms ±5% 0.1W, 1/10W Chip Resistor 0603 (1608 Metric) Automotive AEC-Q200, Moisture Resistant Thick Film " H 0   0   50  0001 C CNN "Description"
+F 5 "CRGCQ0603J470R" H 0   0   50  0001 C CNN "PartNumber"
+F 6 "A130089CT-ND" H 0   0   50  0001 C CNN "digikey"
+F 7 "0.02100" H 0   0   50  0001 C CNN "price@10"
 	1    13300 2000
 	0    1    1    0
@@
 Wire Wire Line
 	8750 4600 8750 4500
+Wire Wire Line
+	8750 4800 8750 5250
+$Comp
+L servo:jumper JP?
+U 1 1 5E57DF30
+P 9150 4500
+AR Path="/5DD76B18/5E57DF30" Ref="JP?"  Part="1"
+AR Path="/5DC4A59D/5E57DF30" Ref="JP?"  Part="1"
+AR Path="/5DC3DC9E/5E57DF30" Ref="JP202"  Part="1"
+F 0 "JP202" H 9150 4585 39  0000 C CNN
+F 1 "jumper" H 9150 4660 39  0000 C CNN
+F 2 "servo:SolderJumper-2_P1.3mm_Open_RoundedPad1.0x1.5mm" H 9050 4480 50  0001 C CNN
+F 3 "~" H 9150 4580 50  0001 C CNN
+F 4 "jumper smd bridge using tin" H 5850 -1100 50  0001 C CNN "Description"
+F 5 "-" H 5850 -1100 50  0001 C CNN "PartNumber"
+F 6 "-" H 5850 -1100 50  0001 C CNN "digikey"
+F 7 "0" H 5850 -1100 50  0001 C CNN "price@10"
+	1    9150 4500
+	-1   0    0    1
+$EndComp
+Wire Wire Line
+	9050 4500 8750 4500
 Connection ~ 8750 4500
-Wire Wire Line
-	8750 4800 8750 5250
 $EndSCHEMATC
