File: kicad/qep.sch (KiCad schematic (older format))
At the start: 35 parts, among them J1101 tblock, U1101 SI8660BD, U1102 am26ls32a, U1103 am26ls32a, U1104 SI8660BD

Commit message: serigrafia...
Parts:
- R1101, R1102, R1103, R1104, R1105, R1106, R1107, R1108, R1109, R1110, R1111, R1112, R1113, R1114, R1115, R1116, R1117, R1118, R1119, R1120, R1121, R1122, R1123, R1124: footprint Resistor_SMD:R_0603_1608Metric -> servo:R_0603_1608Metric
- U1102, U1103: footprint Package_SO:SOIC-16W_5.3x10.2mm_P1.27mm -> servo:SOIC-16W_5.3x10.2mm_P1.27mm
Changed lines of the file:
@@
 F 0 "R1122" H 7359 2272 20  0000 L CNN
 F 1 "10k" H 7359 2229 20  0000 L CNN
-F 2 "Resistor_SMD:R_0603_1608Metric" H 7300 2250 50  0001 C CNN
+F 2 "servo:R_0603_1608Metric" H 7300 2250 50  0001 C CNN
 F 3 "~" H 7300 2250 50  0001 C CNN
 	1    7300 2250
@@
 F 0 "R1123" H 7359 2472 20  0000 L CNN
 F 1 "1k" H 7359 2429 20  0000 L CNN
-F 2 "Resistor_SMD:R_0603_1608Metric" H 7300 2450 50  0001 C CNN
+F 2 "servo:R_0603_1608Metric" H 7300 2450 50  0001 C CNN
 F 3 "~" H 7300 2450 50  0001 C CNN
 	1    7300 2450
@@
 F 0 "R1124" H 7359 2672 20  0000 L CNN
 F 1 "10k" H 7359 2629 20  0000 L CNN
-F 2 "Resistor_SMD:R_0603_1608Metric" H 7300 2650 50  0001 C CNN
+F 2 "servo:R_0603_1608Metric" H 7300 2650 50  0001 C CNN
 F 3 "~" H 7300 2650 50  0001 C CNN
 	1    7300 2650
@@
 F 0 "R1119" H 7109 2272 20  0000 L CNN
 F 1 "10k" H 7109 2229 20  0000 L CNN
-F 2 "Resistor_SMD:R_0603_1608Metric" H 7050 2250 50  0001 C CNN
+F 2 "servo:R_0603_1608Metric" H 7050 2250 50  0001 C CNN
 F 3 "~" H 7050 2250 50  0001 C CNN
 	1    7050 2250
@@
 F 0 "R1120" H 7109 2472 20  0000 L CNN
 F 1 "1k" H 7109 2429 20  0000 L CNN
-F 2 "Resistor_SMD:R_0603_1608Metric" H 7050 2450 50  0001 C CNN
+F 2 "servo:R_0603_1608Metric" H 7050 2450 50  0001 C CNN
 F 3 "~" H 7050 2450 50  0001 C CNN
 	1    7050 2450
@@
 F 0 "R1121" H 7109 2672 20  0000 L CNN
 F 1 "10k" H 7109 2629 20  0000 L CNN
-F 2 "Resistor_SMD:R_0603_1608Metric" H 7050 2650 50  0001 C CNN
+F 2 "servo:R_0603_1608Metric" H 7050 2650 50  0001 C CNN
 F 3 "~" H 7050 2650 50  0001 C CNN
 	1    7050 2650
@@
 F 0 "R1116" H 6859 2272 20  0000 L CNN
 F 1 "10k" H 6859 2229 20  0000 L CNN
-F 2 "Resistor_SMD:R_0603_1608Metric" H 6800 2250 50  0001 C CNN
+F 2 "servo:R_0603_1608Metric" H 6800 2250 50  0001 C CNN
 F 3 "~" H 6800 2250 50  0001 C CNN
 	1    6800 2250
@@
 F 0 "R1117" H 6859 2472 20  0000 L CNN
 F 1 "1k" H 6859 2429 20  0000 L CNN
-F 2 "Resistor_SMD:R_0603_1608Metric" H 6800 2450 50  0001 C CNN
+F 2 "servo:R_0603_1608Metric" H 6800 2450 50  0001 C CNN
 F 3 "~" H 6800 2450 50  0001 C CNN
 	1    6800 2450
@@
 F 0 "R1118" H 6859 2672 20  0000 L CNN
 F 1 "10k" H 6859 2629 20  0000 L CNN
-F 2 "Resistor_SMD:R_0603_1608Metric" H 6800 2650 50  0001 C CNN
+F 2 "servo:R_0603_1608Metric" H 6800 2650 50  0001 C CNN
 F 3 "~" H 6800 2650 50  0001 C CNN
 	1    6800 2650
@@
 F 0 "R1113" H 6609 2272 20  0000 L CNN
 F 1 "10k" H 6609 2229 20  0000 L CNN
-F 2 "Resistor_SMD:R_0603_1608Metric" H 6550 2250 50  0001 C CNN
+F 2 "servo:R_0603_1608Metric" H 6550 2250 50  0001 C CNN
 F 3 "~" H 6550 2250 50  0001 C CNN
 	1    6550 2250
@@
 F 0 "R1114" H 6609 2472 20  0000 L CNN
 F 1 "1k" H 6609 2429 20  0000 L CNN
-F 2 "Resistor_SMD:R_0603_1608Metric" H 6550 2450 50  0001 C CNN
+F 2 "servo:R_0603_1608Metric" H 6550 2450 50  0001 C CNN
 F 3 "~" H 6550 2450 50  0001 C CNN
 	1    6550 2450
@@
 F 0 "R1115" H 6609 2672 20  0000 L CNN
 F 1 "10k" H 6609 2629 20  0000 L CNN
-F 2 "Resistor_SMD:R_0603_1608Metric" H 6550 2650 50  0001 C CNN
+F 2 "servo:R_0603_1608Metric" H 6550 2650 50  0001 C CNN
 F 3 "~" H 6550 2650 50  0001 C CNN
 	1    6550 2650
@@
 F 0 "U1103" H 7950 5150 39  0000 C CNN
 F 1 "am26ls32a" H 7900 5050 39  0000 C CNN
-F 2 "Package_SO:SOIC-16W_5.3x10.2mm_P1.27mm" H 9100 3150 50  0001 C CNN
+F 2 "servo:SOIC-16W_5.3x10.2mm_P1.27mm" H 9100 3150 50  0001 C CNN
 F 3 "../doc/datasheets/am26ls32a.pdf" H 8100 3700 50  0001 C CNN
 	1    8100 4100
@@
 F 0 "R1101" H 4459 2272 20  0000 L CNN
 F 1 "10k" H 4459 2229 20  0000 L CNN
-F 2 "Resistor_SMD:R_0603_1608Metric" H 4400 2250 50  0001 C CNN
+F 2 "servo:R_0603_1608Metric" H 4400 2250 50  0001 C CNN
 F 3 "~" H 4400 2250 50  0001 C CNN
 	1    4400 2250
@@
 F 0 "R1102" H 4459 2472 20  0000 L CNN
 F 1 "1k" H 4459 2429 20  0000 L CNN
-F 2 "Resistor_SMD:R_0603_1608Metric" H 4400 2450 50  0001 C CNN
+F 2 "servo:R_0603_1608Metric" H 4400 2450 50  0001 C CNN
 F 3 "~" H 4400 2450 50  0001 C CNN
 	1    4400 2450
@@
 F 0 "R1103" H 4459 2672 20  0000 L CNN
 F 1 "10k" H 4459 2629 20  0000 L CNN
-F 2 "Resistor_SMD:R_0603_1608Metric" H 4400 2650 50  0001 C CNN
+F 2 "servo:R_0603_1608Metric" H 4400 2650 50  0001 C CNN
 F 3 "~" H 4400 2650 50  0001 C CNN
 	1    4400 2650
@@
 F 0 "R1104" H 4709 2272 20  0000 L CNN
 F 1 "10k" H 4709 2229 20  0000 L CNN
-F 2 "Resistor_SMD:R_0603_1608Metric" H 4650 2250 50  0001 C CNN
+F 2 "servo:R_0603_1608Metric" H 4650 2250 50  0001 C CNN
 F 3 "~" H 4650 2250 50  0001 C CNN
 	1    4650 2250
@@
 F 0 "R1105" H 4709 2472 20  0000 L CNN
 F 1 "1k" H 4709 2429 20  0000 L CNN
-F 2 "Resistor_SMD:R_0603_1608Metric" H 4650 2450 50  0001 C CNN
+F 2 "servo:R_0603_1608Metric" H 4650 2450 50  0001 C CNN
 F 3 "~" H 4650 2450 50  0001 C CNN
 	1    4650 2450
@@
 F 0 "R1106" H 4709 2672 20  0000 L CNN
 F 1 "10k" H 4709 2629 20  0000 L CNN
-F 2 "Resistor_SMD:R_0603_1608Metric" H 4650 2650 50  0001 C CNN
+F 2 "servo:R_0603_1608Metric" H 4650 2650 50  0001 C CNN
 F 3 "~" H 4650 2650 50  0001 C CNN
 	1    4650 2650
@@
 F 0 "R1107" H 4959 2272 20  0000 L CNN
 F 1 "10k" H 4959 2229 20  0000 L CNN
-F 2 "Resistor_SMD:R_0603_1608Metric" H 4900 2250 50  0001 C CNN
+F 2 "servo:R_0603_1608Metric" H 4900 2250 50  0001 C CNN
 F 3 "~" H 4900 2250 50  0001 C CNN
 	1    4900 2250
@@
 F 0 "R1108" H 4959 2472 20  0000 L CNN
 F 1 "1k" H 4959 2429 20  0000 L CNN
-F 2 "Resistor_SMD:R_0603_1608Metric" H 4900 2450 50  0001 C CNN
+F 2 "servo:R_0603_1608Metric" H 4900 2450 50  0001 C CNN
 F 3 "~" H 4900 2450 50  0001 C CNN
 	1    4900 2450
@@
 F 0 "R1109" H 4959 2672 20  0000 L CNN
 F 1 "10k" H 4959 2629 20  0000 L CNN
-F 2 "Resistor_SMD:R_0603_1608Metric" H 4900 2650 50  0001 C CNN
+F 2 "servo:R_0603_1608Metric" H 4900 2650 50  0001 C CNN
 F 3 "~" H 4900 2650 50  0001 C CNN
 	1    4900 2650
@@
 F 0 "R1110" H 5209 2272 20  0000 L CNN
 F 1 "10k" H 5209 2229 20  0000 L CNN
-F 2 "Resistor_SMD:R_0603_1608Metric" H 5150 2250 50  0001 C CNN
+F 2 "servo:R_0603_1608Metric" H 5150 2250 50  0001 C CNN
 F 3 "~" H 5150 2250 50  0001 C CNN
 	1    5150 2250
@@
 F 0 "R1111" H 5209 2472 20  0000 L CNN
 F 1 "1k" H 5209 2429 20  0000 L CNN
-F 2 "Resistor_SMD:R_0603_1608Metric" H 5150 2450 50  0001 C CNN
+F 2 "servo:R_0603_1608Metric" H 5150 2450 50  0001 C CNN
 F 3 "~" H 5150 2450 50  0001 C CNN
 	1    5150 2450
@@
 F 0 "R1112" H 5209 2672 20  0000 L CNN
 F 1 "10k" H 5209 2629 20  0000 L CNN
-F 2 "Resistor_SMD:R_0603_1608Metric" H 5150 2650 50  0001 C CNN
+F 2 "servo:R_0603_1608Metric" H 5150 2650 50  0001 C CNN
 F 3 "~" H 5150 2650 50  0001 C CNN
 	1    5150 2650
@@
 F 0 "U1102" H 3450 5150 39  0000 C CNN
 F 1 "am26ls32a" H 3400 5050 39  0000 C CNN
-F 2 "Package_SO:SOIC-16W_5.3x10.2mm_P1.27mm" H 4600 3150 50  0001 C CNN
+F 2 "servo:SOIC-16W_5.3x10.2mm_P1.27mm" H 4600 3150 50  0001 C CNN
 F 3 "../doc/datasheets/am26ls32a.pdf" H 3600 3700 50  0001 C CNN
 	1    3600 4100
