File: kicad/qep.sch (KiCad schematic (older format))
At the start: 35 parts, among them J1101 tblock 2x10 3.81, U1101 SI8660BD, U1102 AM26LS32A, U1103 AM26LS32A, U1104 SI8660BD

Commit message: fine imprivements
Parts:
- R1102, R1105, R1108, R1111, R1114, R1117, R1120, R1123: value 1k -> 10k; Description 1 kOhms ±5% 0.1W, 1/10W Chip Resistor 0603 (1608 Metric) Mo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 -> 10 kOhms ±5% 0.1W, 1/10W Chip Resistor 0603 (1608 Metric) M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; PartNumber RC0603JR-071KL -> RC0603JR-0710KL; digikey 311-1.0KGRCT-ND -> 311-10KGRCT-ND
Other:
- note added: "for final release, remove pull-up \nand pull-down from bus, and \nreplace 10k to 120 as the Z"
Changed lines of the file:
@@
 U 1 1 6027FD06
 P 5800 3750
-F 0 "J1101" H 5850 4367 50  0000 C CNN
-F 1 "tblock 2x10 3.81" H 5850 4276 50  0000 C CNN
+F 0 "J1101" H 5850 4295 20  0000 C CNN
+F 1 "tblock 2x10 3.81" H 5850 4252 20  0000 C CNN
 F 2 "servo:tblock02x10_3.81" H 5800 3750 50  0001 C CNN
 F 3 "~" H 5800 3750 50  0001 C CNN
@@
 P 7300 2450
 F 0 "R1123" H 7359 2472 20  0000 L CNN
-F 1 "1k" H 7359 2429 20  0000 L CNN
+F 1 "10k" H 7359 2429 20  0000 L CNN
 F 2 "servo:R_0603_1608Metric" H 7300 2450 50  0001 C CNN
 F 3 "~" H 7300 2450 50  0001 C CNN
-F 4 "1 kOhms ±5% 0.1W, 1/10W Chip Resistor 0603 (1608 Metric) Moisture Resistant Thick Film " H 0   0   50  0001 C CNN "Description"
-F 5 "RC0603JR-071KL" H 0   0   50  0001 C CNN "PartNumber"
-F 6 "311-1.0KGRCT-ND" H 0   0   50  0001 C CNN "digikey"
+F 4 "10 kOhms ±5% 0.1W, 1/10W Chip Resistor 0603 (1608 Metric) Moisture Resistant Thick Film " H 0   0   50  0001 C CNN "Description"
+F 5 "RC0603JR-0710KL" H 0   0   50  0001 C CNN "PartNumber"
+F 6 "311-10KGRCT-ND" H 0   0   50  0001 C CNN "digikey"
 F 7 "0.01900" H 0   0   50  0001 C CNN "price@10"
 	1    7300 2450
@@
 P 7050 2450
 F 0 "R1120" H 7109 2472 20  0000 L CNN
-F 1 "1k" H 7109 2429 20  0000 L CNN
+F 1 "10k" H 7109 2429 20  0000 L CNN
 F 2 "servo:R_0603_1608Metric" H 7050 2450 50  0001 C CNN
 F 3 "~" H 7050 2450 50  0001 C CNN
-F 4 "1 kOhms ±5% 0.1W, 1/10W Chip Resistor 0603 (1608 Metric) Moisture Resistant Thick Film " H 0   0   50  0001 C CNN "Description"
-F 5 "RC0603JR-071KL" H 0   0   50  0001 C CNN "PartNumber"
-F 6 "311-1.0KGRCT-ND" H 0   0   50  0001 C CNN "digikey"
+F 4 "10 kOhms ±5% 0.1W, 1/10W Chip Resistor 0603 (1608 Metric) Moisture Resistant Thick Film " H 0   0   50  0001 C CNN "Description"
+F 5 "RC0603JR-0710KL" H 0   0   50  0001 C CNN "PartNumber"
+F 6 "311-10KGRCT-ND" H 0   0   50  0001 C CNN "digikey"
 F 7 "0.01900" H 0   0   50  0001 C CNN "price@10"
 	1    7050 2450
@@
 Wire Wire Line
 	7600 4500 8100 4500
-Text Notes 9200 3800 2    20   ~ 0
+Text Notes 7650 3850 2    20   ~ 0
 optional one to hi \nor/and one to low
 Text Label 6500 3350 2    20   ~ 0
@@
 P 6800 2450
 F 0 "R1117" H 6859 2472 20  0000 L CNN
-F 1 "1k" H 6859 2429 20  0000 L CNN
+F 1 "10k" H 6859 2429 20  0000 L CNN
 F 2 "servo:R_0603_1608Metric" H 6800 2450 50  0001 C CNN
 F 3 "~" H 6800 2450 50  0001 C CNN
-F 4 "1 kOhms ±5% 0.1W, 1/10W Chip Resistor 0603 (1608 Metric) Moisture Resistant Thick Film " H 0   0   50  0001 C CNN "Description"
-F 5 "RC0603JR-071KL" H 0   0   50  0001 C CNN "PartNumber"
-F 6 "311-1.0KGRCT-ND" H 0   0   50  0001 C CNN "digikey"
+F 4 "10 kOhms ±5% 0.1W, 1/10W Chip Resistor 0603 (1608 Metric) Moisture Resistant Thick Film " H 0   0   50  0001 C CNN "Description"
+F 5 "RC0603JR-0710KL" H 0   0   50  0001 C CNN "PartNumber"
+F 6 "311-10KGRCT-ND" H 0   0   50  0001 C CNN "digikey"
 F 7 "0.01900" H 0   0   50  0001 C CNN "price@10"
 	1    6800 2450
@@
 P 6550 2450
 F 0 "R1114" H 6609 2472 20  0000 L CNN
-F 1 "1k" H 6609 2429 20  0000 L CNN
+F 1 "10k" H 6609 2429 20  0000 L CNN
 F 2 "servo:R_0603_1608Metric" H 6550 2450 50  0001 C CNN
 F 3 "~" H 6550 2450 50  0001 C CNN
-F 4 "1 kOhms ±5% 0.1W, 1/10W Chip Resistor 0603 (1608 Metric) Moisture Resistant Thick Film " H 0   0   50  0001 C CNN "Description"
-F 5 "RC0603JR-071KL" H 0   0   50  0001 C CNN "PartNumber"
-F 6 "311-1.0KGRCT-ND" H 0   0   50  0001 C CNN "digikey"
+F 4 "10 kOhms ±5% 0.1W, 1/10W Chip Resistor 0603 (1608 Metric) Moisture Resistant Thick Film " H 0   0   50  0001 C CNN "Description"
+F 5 "RC0603JR-0710KL" H 0   0   50  0001 C CNN "PartNumber"
+F 6 "311-10KGRCT-ND" H 0   0   50  0001 C CNN "digikey"
 F 7 "0.01900" H 0   0   50  0001 C CNN "price@10"
 	1    6550 2450
@@
 P 4400 2450
 F 0 "R1102" H 4459 2472 20  0000 L CNN
-F 1 "1k" H 4459 2429 20  0000 L CNN
+F 1 "10k" H 4459 2429 20  0000 L CNN
 F 2 "servo:R_0603_1608Metric" H 4400 2450 50  0001 C CNN
 F 3 "~" H 4400 2450 50  0001 C CNN
-F 4 "1 kOhms ±5% 0.1W, 1/10W Chip Resistor 0603 (1608 Metric) Moisture Resistant Thick Film " H 0   0   50  0001 C CNN "Description"
-F 5 "RC0603JR-071KL" H 0   0   50  0001 C CNN "PartNumber"
-F 6 "311-1.0KGRCT-ND" H 0   0   50  0001 C CNN "digikey"
+F 4 "10 kOhms ±5% 0.1W, 1/10W Chip Resistor 0603 (1608 Metric) Moisture Resistant Thick Film " H 0   0   50  0001 C CNN "Description"
+F 5 "RC0603JR-0710KL" H 0   0   50  0001 C CNN "PartNumber"
+F 6 "311-10KGRCT-ND" H 0   0   50  0001 C CNN "digikey"
 F 7 "0.01900" H 0   0   50  0001 C CNN "price@10"
 	1    4400 2450
@@
 P 4650 2450
 F 0 "R1105" H 4709 2472 20  0000 L CNN
-F 1 "1k" H 4709 2429 20  0000 L CNN
+F 1 "10k" H 4709 2429 20  0000 L CNN
 F 2 "servo:R_0603_1608Metric" H 4650 2450 50  0001 C CNN
 F 3 "~" H 4650 2450 50  0001 C CNN
-F 4 "1 kOhms ±5% 0.1W, 1/10W Chip Resistor 0603 (1608 Metric) Moisture Resistant Thick Film " H 0   0   50  0001 C CNN "Description"
-F 5 "RC0603JR-071KL" H 0   0   50  0001 C CNN "PartNumber"
-F 6 "311-1.0KGRCT-ND" H 0   0   50  0001 C CNN "digikey"
+F 4 "10 kOhms ±5% 0.1W, 1/10W Chip Resistor 0603 (1608 Metric) Moisture Resistant Thick Film " H 0   0   50  0001 C CNN "Description"
+F 5 "RC0603JR-0710KL" H 0   0   50  0001 C CNN "PartNumber"
+F 6 "311-10KGRCT-ND" H 0   0   50  0001 C CNN "digikey"
 F 7 "0.01900" H 0   0   50  0001 C CNN "price@10"
 	1    4650 2450
@@
 Wire Wire Line
 	4100 4500 3600 4500
-Text Notes 2500 3800 0    20   ~ 0
+Text Notes 4000 3850 0    20   ~ 0
 optional one to hi \nor/and one to low
 Text Label 5200 3350 0    20   ~ 0
@@
 P 4900 2450
 F 0 "R1108" H 4959 2472 20  0000 L CNN
-F 1 "1k" H 4959 2429 20  0000 L CNN
+F 1 "10k" H 4959 2429 20  0000 L CNN
 F 2 "servo:R_0603_1608Metric" H 4900 2450 50  0001 C CNN
 F 3 "~" H 4900 2450 50  0001 C CNN
-F 4 "1 kOhms ±5% 0.1W, 1/10W Chip Resistor 0603 (1608 Metric) Moisture Resistant Thick Film " H 0   0   50  0001 C CNN "Description"
-F 5 "RC0603JR-071KL" H 0   0   50  0001 C CNN "PartNumber"
-F 6 "311-1.0KGRCT-ND" H 0   0   50  0001 C CNN "digikey"
+F 4 "10 kOhms ±5% 0.1W, 1/10W Chip Resistor 0603 (1608 Metric) Moisture Resistant Thick Film " H 0   0   50  0001 C CNN "Description"
+F 5 "RC0603JR-0710KL" H 0   0   50  0001 C CNN "PartNumber"
+F 6 "311-10KGRCT-ND" H 0   0   50  0001 C CNN "digikey"
 F 7 "0.01900" H 0   0   50  0001 C CNN "price@10"
 	1    4900 2450
@@
 P 5150 2450
 F 0 "R1111" H 5209 2472 20  0000 L CNN
-F 1 "1k" H 5209 2429 20  0000 L CNN
+F 1 "10k" H 5209 2429 20  0000 L CNN
 F 2 "servo:R_0603_1608Metric" H 5150 2450 50  0001 C CNN
 F 3 "~" H 5150 2450 50  0001 C CNN
-F 4 "1 kOhms ±5% 0.1W, 1/10W Chip Resistor 0603 (1608 Metric) Moisture Resistant Thick Film " H 0   0   50  0001 C CNN "Description"
-F 5 "RC0603JR-071KL" H 0   0   50  0001 C CNN "PartNumber"
-F 6 "311-1.0KGRCT-ND" H 0   0   50  0001 C CNN "digikey"
+F 4 "10 kOhms ±5% 0.1W, 1/10W Chip Resistor 0603 (1608 Metric) Moisture Resistant Thick Film " H 0   0   50  0001 C CNN "Description"
+F 5 "RC0603JR-0710KL" H 0   0   50  0001 C CNN "PartNumber"
+F 6 "311-10KGRCT-ND" H 0   0   50  0001 C CNN "digikey"
 F 7 "0.01900" H 0   0   50  0001 C CNN "price@10"
 	1    5150 2450
@@
 	5200 3850 5600 3850
 Wire Wire Line
-	3250 2500 3250 2550
+	3250 2500 3250 2750
 Wire Wire Line
 	3250 2200 3250 2150
@@
 $EndComp
 Wire Wire Line
-	2950 2500 2950 2550
+	2950 2500 2950 2750
 Wire Wire Line
 	2950 2200 2950 2150
@@
 	2750 2150 2750 3400
 Wire Wire Line
-	2950 2550 3250 2550
+	2950 2750 3250 2750
 Wire Wire Line
 	4400 2750 3250 2750
-Wire Wire Line
-	3250 2750 3250 2550
-Connection ~ 3250 2550
+Connection ~ 3250 2750
 Wire Wire Line
 	7300 2750 8450 2750
@@
 Text Notes 3250 4650 0    20   ~ 0
 I've chossen so16w but the landpattern is compatible\n with soic16 also 'cause soic has more available \npieces and are cheaper
+Text Notes 5650 2400 0    20   ~ 0
+for final release, remove pull-up \nand pull-down from bus, and \nreplace 10k to 120 as the Z
 $EndSCHEMATC

Commit message: gerbers + pnp + bom ready
Parts:
- C1101, C1102, C1103, C1104, C1105, C1106, R1101, R1102, R1103, R1104, R1105, R1106, R1107, R1108, R1109, R1110, R1111, R1112, R1113, R1114, R1115, R1116, R1117, R1118, R1119, R1120, R1121, R1122, R1123, R1124: bom_1 (none) -> 1; bom_2 (none) -> 1; bom_3 (none) -> 1
- J1101: bom_3 (none) -> 1
- U1101, U1102, U1103, U1104: bom_2 (none) -> 1; bom_3 (none) -> 1
Changed lines of the file:
@@
 F 6 "277-6029-ND" H 0   0   50  0001 C CNN "digikey"
 F 7 "12.49300" H 0   0   50  0001 C CNN "price@10"
+F 8 "1" H 0   0   50  0001 C CNN "bom_3"
 	1    5800 3750
 	1    0    0    -1
@@
 F 6 "311-10KGRCT-ND" H 0   0   50  0001 C CNN "digikey"
 F 7 "0.01900" H 0   0   50  0001 C CNN "price@10"
+F 8 "1" H 0   0   50  0001 C CNN "bom_1"
+F 9 "1" H 0   0   50  0001 C CNN "bom_2"
+F 10 "1" H 0   0   50  0001 C CNN "bom_3"
 	1    7300 2250
 	-1   0    0    -1
@@
 F 6 "311-10KGRCT-ND" H 0   0   50  0001 C CNN "digikey"
 F 7 "0.01900" H 0   0   50  0001 C CNN "price@10"
+F 8 "1" H 0   0   50  0001 C CNN "bom_1"
+F 9 "1" H 0   0   50  0001 C CNN "bom_2"
+F 10 "1" H 0   0   50  0001 C CNN "bom_3"
 	1    7300 2450
 	-1   0    0    -1
@@
 F 6 "311-10KGRCT-ND" H 0   0   50  0001 C CNN "digikey"
 F 7 "0.01900" H 0   0   50  0001 C CNN "price@10"
+F 8 "1" H 0   0   50  0001 C CNN "bom_1"
+F 9 "1" H 0   0   50  0001 C CNN "bom_2"
+F 10 "1" H 0   0   50  0001 C CNN "bom_3"
 	1    7300 2650
 	-1   0    0    -1
@@
 F 6 "311-10KGRCT-ND" H 0   0   50  0001 C CNN "digikey"
 F 7 "0.01900" H 0   0   50  0001 C CNN "price@10"
+F 8 "1" H 0   0   50  0001 C CNN "bom_1"
+F 9 "1" H 0   0   50  0001 C CNN "bom_2"
+F 10 "1" H 0   0   50  0001 C CNN "bom_3"
 	1    7050 2250
 	-1   0    0    -1
@@
 F 6 "311-10KGRCT-ND" H 0   0   50  0001 C CNN "digikey"
 F 7 "0.01900" H 0   0   50  0001 C CNN "price@10"
+F 8 "1" H 0   0   50  0001 C CNN "bom_1"
+F 9 "1" H 0   0   50  0001 C CNN "bom_2"
+F 10 "1" H 0   0   50  0001 C CNN "bom_3"
 	1    7050 2450
 	-1   0    0    -1
@@
 F 6 "311-10KGRCT-ND" H 0   0   50  0001 C CNN "digikey"
 F 7 "0.01900" H 0   0   50  0001 C CNN "price@10"
+F 8 "1" H 0   0   50  0001 C CNN "bom_1"
+F 9 "1" H 0   0   50  0001 C CNN "bom_2"
+F 10 "1" H 0   0   50  0001 C CNN "bom_3"
 	1    7050 2650
 	-1   0    0    -1
@@
 F 6 " 336-4786-1-ND" H 0   0   50  0001 C CNN "digikey"
 F 7 "2.75000" H 0   0   50  0001 C CNN "price@10"
+F 8 "" H 0   0   50  0001 C CNN "bom_1"
+F 9 "1" H 0   0   50  0001 C CNN "bom_2"
+F 10 "1" H 0   0   50  0001 C CNN "bom_3"
 	1    9750 3700
 	1    0    0    -1
@@
 F 6 "311-10KGRCT-ND" H 0   0   50  0001 C CNN "digikey"
 F 7 "0.01900" H 0   0   50  0001 C CNN "price@10"
+F 8 "1" H 0   0   50  0001 C CNN "bom_1"
+F 9 "1" H 0   0   50  0001 C CNN "bom_2"
+F 10 "1" H 0   0   50  0001 C CNN "bom_3"
 	1    6800 2250
 	-1   0    0    -1
@@
 F 6 "311-10KGRCT-ND" H 0   0   50  0001 C CNN "digikey"
 F 7 "0.01900" H 0   0   50  0001 C CNN "price@10"
+F 8 "1" H 0   0   50  0001 C CNN "bom_1"
+F 9 "1" H 0   0   50  0001 C CNN "bom_2"
+F 10 "1" H 0   0   50  0001 C CNN "bom_3"
 	1    6800 2450
 	-1   0    0    -1
@@
 F 6 "311-10KGRCT-ND" H 0   0   50  0001 C CNN "digikey"
 F 7 "0.01900" H 0   0   50  0001 C CNN "price@10"
+F 8 "1" H 0   0   50  0001 C CNN "bom_1"
+F 9 "1" H 0   0   50  0001 C CNN "bom_2"
+F 10 "1" H 0   0   50  0001 C CNN "bom_3"
 	1    6800 2650
 	-1   0    0    -1
@@
 F 6 "311-10KGRCT-ND" H 0   0   50  0001 C CNN "digikey"
 F 7 "0.01900" H 0   0   50  0001 C CNN "price@10"
+F 8 "1" H 0   0   50  0001 C CNN "bom_1"
+F 9 "1" H 0   0   50  0001 C CNN "bom_2"
+F 10 "1" H 0   0   50  0001 C CNN "bom_3"
 	1    6550 2250
 	-1   0    0    -1
@@
 F 6 "311-10KGRCT-ND" H 0   0   50  0001 C CNN "digikey"
 F 7 "0.01900" H 0   0   50  0001 C CNN "price@10"
+F 8 "1" H 0   0   50  0001 C CNN "bom_1"
+F 9 "1" H 0   0   50  0001 C CNN "bom_2"
+F 10 "1" H 0   0   50  0001 C CNN "bom_3"
 	1    6550 2450
 	-1   0    0    -1
@@
 F 6 "311-10KGRCT-ND" H 0   0   50  0001 C CNN "digikey"
 F 7 "0.01900" H 0   0   50  0001 C CNN "price@10"
+F 8 "1" H 0   0   50  0001 C CNN "bom_1"
+F 9 "1" H 0   0   50  0001 C CNN "bom_2"
+F 10 "1" H 0   0   50  0001 C CNN "bom_3"
 	1    6550 2650
 	-1   0    0    -1
@@
 F 6 "296-1011-1-ND" H 0   0   50  0001 C CNN "digikey"
 F 7 "0.57800" H 0   0   50  0001 C CNN "price@10"
+F 8 "1" H 0   0   50  0001 C CNN "bom_2"
+F 9 "1" H 0   0   50  0001 C CNN "bom_3"
 	1    8100 4100
 	1    0    0    -1
@@
 F 6 "311-10KGRCT-ND" H 0   0   50  0001 C CNN "digikey"
 F 7 "0.01900" H 0   0   50  0001 C CNN "price@10"
+F 8 "1" H 0   0   50  0001 C CNN "bom_1"
+F 9 "1" H 0   0   50  0001 C CNN "bom_2"
+F 10 "1" H 0   0   50  0001 C CNN "bom_3"
 	1    4400 2250
 	1    0    0    -1
@@
 F 6 "311-10KGRCT-ND" H 0   0   50  0001 C CNN "digikey"
 F 7 "0.01900" H 0   0   50  0001 C CNN "price@10"
+F 8 "1" H 0   0   50  0001 C CNN "bom_1"
+F 9 "1" H 0   0   50  0001 C CNN "bom_2"
+F 10 "1" H 0   0   50  0001 C CNN "bom_3"
 	1    4400 2450
 	1    0    0    -1
@@
 F 6 "311-10KGRCT-ND" H 0   0   50  0001 C CNN "digikey"
 F 7 "0.01900" H 0   0   50  0001 C CNN "price@10"
+F 8 "1" H 0   0   50  0001 C CNN "bom_1"
+F 9 "1" H 0   0   50  0001 C CNN "bom_2"
+F 10 "1" H 0   0   50  0001 C CNN "bom_3"
 	1    4400 2650
 	1    0    0    -1
@@
 F 6 "311-10KGRCT-ND" H 0   0   50  0001 C CNN "digikey"
 F 7 "0.01900" H 0   0   50  0001 C CNN "price@10"
+F 8 "1" H 0   0   50  0001 C CNN "bom_1"
+F 9 "1" H 0   0   50  0001 C CNN "bom_2"
+F 10 "1" H 0   0   50  0001 C CNN "bom_3"
 	1    4650 2250
 	1    0    0    -1
@@
 F 6 "311-10KGRCT-ND" H 0   0   50  0001 C CNN "digikey"
 F 7 "0.01900" H 0   0   50  0001 C CNN "price@10"
+F 8 "1" H 0   0   50  0001 C CNN "bom_1"
+F 9 "1" H 0   0   50  0001 C CNN "bom_2"
+F 10 "1" H 0   0   50  0001 C CNN "bom_3"
 	1    4650 2450
 	1    0    0    -1
@@
 F 6 "311-10KGRCT-ND" H 0   0   50  0001 C CNN "digikey"
 F 7 "0.01900" H 0   0   50  0001 C CNN "price@10"
+F 8 "1" H 0   0   50  0001 C CNN "bom_1"
+F 9 "1" H 0   0   50  0001 C CNN "bom_2"
+F 10 "1" H 0   0   50  0001 C CNN "bom_3"
 	1    4650 2650
 	1    0    0    -1
@@
 F 6 " 336-4786-1-ND" H 0   0   50  0001 C CNN "digikey"
 F 7 "2.75000" H 0   0   50  0001 C CNN "price@10"
+F 8 "" H 0   0   50  0001 C CNN "bom_1"
+F 9 "1" H 0   0   50  0001 C CNN "bom_2"
+F 10 "1" H 0   0   50  0001 C CNN "bom_3"
 	1    1950 3700
 	-1   0    0    -1
@@
 F 6 "311-10KGRCT-ND" H 0   0   50  0001 C CNN "digikey"
 F 7 "0.01900" H 0   0   50  0001 C CNN "price@10"
+F 8 "1" H 0   0   50  0001 C CNN "bom_1"
+F 9 "1" H 0   0   50  0001 C CNN "bom_2"
+F 10 "1" H 0   0   50  0001 C CNN "bom_3"
 	1    4900 2250
 	1    0    0    -1
@@
 F 6 "311-10KGRCT-ND" H 0   0   50  0001 C CNN "digikey"
 F 7 "0.01900" H 0   0   50  0001 C CNN "price@10"
+F 8 "1" H 0   0   50  0001 C CNN "bom_1"
+F 9 "1" H 0   0   50  0001 C CNN "bom_2"
+F 10 "1" H 0   0   50  0001 C CNN "bom_3"
 	1    4900 2450
 	1    0    0    -1
@@
 F 6 "311-10KGRCT-ND" H 0   0   50  0001 C CNN "digikey"
 F 7 "0.01900" H 0   0   50  0001 C CNN "price@10"
+F 8 "1" H 0   0   50  0001 C CNN "bom_1"
+F 9 "1" H 0   0   50  0001 C CNN "bom_2"
+F 10 "1" H 0   0   50  0001 C CNN "bom_3"
 	1    4900 2650
 	1    0    0    -1
@@
 F 6 "311-10KGRCT-ND" H 0   0   50  0001 C CNN "digikey"
 F 7 "0.01900" H 0   0   50  0001 C CNN "price@10"
+F 8 "1" H 0   0   50  0001 C CNN "bom_1"
+F 9 "1" H 0   0   50  0001 C CNN "bom_2"
+F 10 "1" H 0   0   50  0001 C CNN "bom_3"
 	1    5150 2250
 	1    0    0    -1
@@
 F 6 "311-10KGRCT-ND" H 0   0   50  0001 C CNN "digikey"
 F 7 "0.01900" H 0   0   50  0001 C CNN "price@10"
+F 8 "1" H 0   0   50  0001 C CNN "bom_1"
+F 9 "1" H 0   0   50  0001 C CNN "bom_2"
+F 10 "1" H 0   0   50  0001 C CNN "bom_3"
 	1    5150 2450
 	1    0    0    -1
@@
 F 6 "311-10KGRCT-ND" H 0   0   50  0001 C CNN "digikey"
 F 7 "0.01900" H 0   0   50  0001 C CNN "price@10"
+F 8 "1" H 0   0   50  0001 C CNN "bom_1"
+F 9 "1" H 0   0   50  0001 C CNN "bom_2"
+F 10 "1" H 0   0   50  0001 C CNN "bom_3"
 	1    5150 2650
 	1    0    0    -1
@@
 F 6 "296-1011-1-ND" H 0   0   50  0001 C CNN "digikey"
 F 7 "0.57800" H 0   0   50  0001 C CNN "price@10"
+F 8 "1" H 0   0   50  0001 C CNN "bom_2"
+F 9 "1" H 0   0   50  0001 C CNN "bom_3"
 	1    3600 4100
 	-1   0    0    -1
@@
 F 6 "CAP CER 0.1UF 16V X7R 0603 " H 0   0   50  0001 C CNN "Description"
 F 7 "0.05800" H 0   0   50  0001 C CNN "price@10"
+F 8 "1" H 0   0   50  0001 C CNN "bom_1"
+F 9 "1" H 0   0   50  0001 C CNN "bom_2"
+F 10 "1" H 0   0   50  0001 C CNN "bom_3"
 	1    3250 2300
 	0    1    1    0
@@
 F 6 "CAP CER 0.1UF 16V X7R 0603 " H 0   0   50  0001 C CNN "Description"
 F 7 "0.05800" H 0   0   50  0001 C CNN "price@10"
+F 8 "1" H 0   0   50  0001 C CNN "bom_1"
+F 9 "1" H 0   0   50  0001 C CNN "bom_2"
+F 10 "1" H 0   0   50  0001 C CNN "bom_3"
 	1    2950 2300
 	0    1    1    0
@@
 F 6 "CAP CER 0.1UF 16V X7R 0603 " H 0   0   50  0001 C CNN "Description"
 F 7 "0.05800" H 0   0   50  0001 C CNN "price@10"
+F 8 "1" H 0   0   50  0001 C CNN "bom_1"
+F 9 "1" H 0   0   50  0001 C CNN "bom_2"
+F 10 "1" H 0   0   50  0001 C CNN "bom_3"
 	1    8750 2300
 	0    1    1    0
@@
 F 6 "CAP CER 0.1UF 16V X7R 0603 " H 0   0   50  0001 C CNN "Description"
 F 7 "0.05800" H 0   0   50  0001 C CNN "price@10"
+F 8 "1" H 0   0   50  0001 C CNN "bom_1"
+F 9 "1" H 0   0   50  0001 C CNN "bom_2"
+F 10 "1" H 0   0   50  0001 C CNN "bom_3"
 	1    8450 2300
 	0    1    1    0
@@
 F 6 "CAP CER 0.1UF 16V X7R 0603 " H 0   0   50  0001 C CNN "Description"
 F 7 "0.05800" H 0   0   50  0001 C CNN "price@10"
+F 8 "1" H 0   0   50  0001 C CNN "bom_1"
+F 9 "1" H 0   0   50  0001 C CNN "bom_2"
+F 10 "1" H 0   0   50  0001 C CNN "bom_3"
 	1    10900 3000
 	0    1    1    0
@@
 F 6 "CAP CER 0.1UF 16V X7R 0603 " H 0   0   50  0001 C CNN "Description"
 F 7 "0.05800" H 0   0   50  0001 C CNN "price@10"
+F 8 "1" H 0   0   50  0001 C CNN "bom_1"
+F 9 "1" H 0   0   50  0001 C CNN "bom_2"
+F 10 "1" H 0   0   50  0001 C CNN "bom_3"
 	1    850  2950
 	0    1    1    0
