File: kicad/temp.sch (KiCad schematic (older format))
At the start: 46 parts, among them U901 AMC1311B, U902 AMC1311B, U903 ADM2483, U904 AMC1311B, U905 AMC1311B

Commit message: bom bom bom...
Parts:
- C903, C904, C905, C906, C907, C908, C909, C910, C911, C912, C913, C914, C917, C918: value 100nF -> 0.1uF; PartNumber (none) -> CC0603KPX7R7BB104; digikey (none) -> 311-1335-1-ND
Changed lines of the file:
@@
 AR Path="/5DE49152/5E5095C3" Ref="C905"  Part="1"
 F 0 "C905" V 8478 5096 20  0000 L BNN
-F 1 "100nF" V 8521 5143 20  0000 C CNN
+F 1 "0.1uF" V 8521 5143 20  0000 C CNN
 F 2 "servo:C_0603_1608Metric" H 8450 5200 60  0001 C CNN
 F 3 "" H 8450 5300 60  0000 C CNN
+F 4 "CC0603KPX7R7BB104" H 0   0   50  0001 C CNN "PartNumber"
+F 5 "311-1335-1-ND" H 0   0   50  0001 C CNN "digikey"
 	1    8450 5300
 	0    1    1    0
@@
 AR Path="/5DE49152/5E5095E8" Ref="C907"  Part="1"
 F 0 "C907" V 8728 5410 20  0000 L BNN
-F 1 "100nF" V 8771 5450 20  0000 C CNN
+F 1 "0.1uF" V 8771 5450 20  0000 C CNN
 F 2 "servo:C_0603_1608Metric" H 8700 5200 60  0001 C CNN
 F 3 "" H 8700 5300 60  0000 C CNN
+F 4 "CC0603KPX7R7BB104" H 0   0   50  0001 C CNN "PartNumber"
+F 5 "311-1335-1-ND" H 0   0   50  0001 C CNN "digikey"
 	1    8700 5300
 	0    1    1    0
@@
 AR Path="/5DE49152/5E5095E1" Ref="C903"  Part="1"
 F 0 "C903" V 6978 4610 20  0000 L BNN
-F 1 "100nF" V 7021 4657 20  0000 C CNN
+F 1 "0.1uF" V 7021 4657 20  0000 C CNN
 F 2 "servo:C_0603_1608Metric" H 6950 4400 60  0001 C CNN
 F 3 "" H 6950 4500 60  0000 C CNN
+F 4 "CC0603KPX7R7BB104" H 0   0   50  0001 C CNN "PartNumber"
+F 5 "311-1335-1-ND" H 0   0   50  0001 C CNN "digikey"
 	1    6950 4500
 	0    1    1    0
@@
 AR Path="/5DE49152/5FE9D175" Ref="C911"  Part="1"
 F 0 "C911" V 11278 5096 20  0000 L BNN
-F 1 "100nF" V 11321 5143 20  0000 C CNN
+F 1 "0.1uF" V 11321 5143 20  0000 C CNN
 F 2 "servo:C_0603_1608Metric" H 11250 5200 60  0001 C CNN
 F 3 "" H 11250 5300 60  0000 C CNN
+F 4 "CC0603KPX7R7BB104" H 0   0   50  0001 C CNN "PartNumber"
+F 5 "311-1335-1-ND" H 0   0   50  0001 C CNN "digikey"
 	1    11250 5300
 	0    -1   1    0
@@
 AR Path="/5DE49152/5FE9D191" Ref="C909"  Part="1"
 F 0 "C909" V 11028 5410 20  0000 L BNN
-F 1 "100nF" V 11071 5450 20  0000 C CNN
+F 1 "0.1uF" V 11071 5450 20  0000 C CNN
 F 2 "servo:C_0603_1608Metric" H 11000 5200 60  0001 C CNN
 F 3 "" H 11000 5300 60  0000 C CNN
+F 4 "CC0603KPX7R7BB104" H 0   0   50  0001 C CNN "PartNumber"
+F 5 "311-1335-1-ND" H 0   0   50  0001 C CNN "digikey"
 	1    11000 5300
 	0    -1   1    0
@@
 AR Path="/5DE49152/5FE9D1F6" Ref="C913"  Part="1"
 F 0 "C913" V 12778 4390 20  0000 R CNN
-F 1 "100nF" V 12821 4390 20  0000 R CNN
+F 1 "0.1uF" V 12821 4390 20  0000 R CNN
 F 2 "servo:C_0603_1608Metric" H 12750 4400 60  0001 C CNN
 F 3 "" H 12750 4500 60  0000 C CNN
+F 4 "CC0603KPX7R7BB104" H 0   0   50  0001 C CNN "PartNumber"
+F 5 "311-1335-1-ND" H 0   0   50  0001 C CNN "digikey"
 	1    12750 4500
 	0    -1   1    0
@@
 AR Path="/5DE49152/5E1BD4FE" Ref="C906"  Part="1"
 F 0 "C906" V 8478 6746 20  0000 L BNN
-F 1 "100nF" V 8521 6793 20  0000 C CNN
+F 1 "0.1uF" V 8521 6793 20  0000 C CNN
 F 2 "servo:C_0603_1608Metric" H 8450 6850 60  0001 C CNN
 F 3 "" H 8450 6950 60  0000 C CNN
+F 4 "CC0603KPX7R7BB104" H 0   0   50  0001 C CNN "PartNumber"
+F 5 "311-1335-1-ND" H 0   0   50  0001 C CNN "digikey"
 	1    8450 6950
 	0    1    1    0
@@
 AR Path="/5DE49152/5E1BD51A" Ref="C908"  Part="1"
 F 0 "C908" V 8728 7060 20  0000 L BNN
-F 1 "100nF" V 8771 7100 20  0000 C CNN
+F 1 "0.1uF" V 8771 7100 20  0000 C CNN
 F 2 "servo:C_0603_1608Metric" H 8700 6850 60  0001 C CNN
 F 3 "" H 8700 6950 60  0000 C CNN
+F 4 "CC0603KPX7R7BB104" H 0   0   50  0001 C CNN "PartNumber"
+F 5 "311-1335-1-ND" H 0   0   50  0001 C CNN "digikey"
 	1    8700 6950
 	0    1    1    0
@@
 AR Path="/5DE49152/5E1BD570" Ref="C904"  Part="1"
 F 0 "C904" V 6978 6260 20  0000 L BNN
-F 1 "100nF" V 7021 6307 20  0000 C CNN
+F 1 "0.1uF" V 7021 6307 20  0000 C CNN
 F 2 "servo:C_0603_1608Metric" H 6950 6050 60  0001 C CNN
 F 3 "" H 6950 6150 60  0000 C CNN
+F 4 "CC0603KPX7R7BB104" H 0   0   50  0001 C CNN "PartNumber"
+F 5 "311-1335-1-ND" H 0   0   50  0001 C CNN "digikey"
 	1    6950 6150
 	0    1    1    0
@@
 AR Path="/5DE49152/5E1BD594" Ref="C912"  Part="1"
 F 0 "C912" V 11278 6746 20  0000 L BNN
-F 1 "100nF" V 11321 6793 20  0000 C CNN
+F 1 "0.1uF" V 11321 6793 20  0000 C CNN
 F 2 "servo:C_0603_1608Metric" H 11250 6850 60  0001 C CNN
 F 3 "" H 11250 6950 60  0000 C CNN
+F 4 "CC0603KPX7R7BB104" H 0   0   50  0001 C CNN "PartNumber"
+F 5 "311-1335-1-ND" H 0   0   50  0001 C CNN "digikey"
 	1    11250 6950
 	0    -1   1    0
@@
 AR Path="/5DE49152/5E1BD5B0" Ref="C910"  Part="1"
 F 0 "C910" V 11028 7060 20  0000 L BNN
-F 1 "100nF" V 11071 7100 20  0000 C CNN
+F 1 "0.1uF" V 11071 7100 20  0000 C CNN
 F 2 "servo:C_0603_1608Metric" H 11000 6850 60  0001 C CNN
 F 3 "" H 11000 6950 60  0000 C CNN
+F 4 "CC0603KPX7R7BB104" H 0   0   50  0001 C CNN "PartNumber"
+F 5 "311-1335-1-ND" H 0   0   50  0001 C CNN "digikey"
 	1    11000 6950
 	0    -1   1    0
@@
 AR Path="/5DE49152/5E1BD605" Ref="C914"  Part="1"
 F 0 "C914" V 12778 6260 20  0000 L BNN
-F 1 "100nF" V 12821 6307 20  0000 C CNN
+F 1 "0.1uF" V 12821 6307 20  0000 C CNN
 F 2 "servo:C_0603_1608Metric" H 12750 6050 60  0001 C CNN
 F 3 "" H 12750 6150 60  0000 C CNN
+F 4 "CC0603KPX7R7BB104" H 0   0   50  0001 C CNN "PartNumber"
+F 5 "311-1335-1-ND" H 0   0   50  0001 C CNN "digikey"
 	1    12750 6150
 	0    -1   1    0
@@
 AR Path="/5DE49152/5E31D563" Ref="C918"  Part="1"
 F 0 "C918" V 10128 2096 20  0000 L BNN
-F 1 "100nF" V 10171 2143 20  0000 C CNN
+F 1 "0.1uF" V 10171 2143 20  0000 C CNN
 F 2 "servo:C_0603_1608Metric" H 10100 2200 60  0001 C CNN
 F 3 "" H 10100 2300 60  0000 C CNN
+F 4 "CC0603KPX7R7BB104" H 0   0   50  0001 C CNN "PartNumber"
+F 5 "311-1335-1-ND" H 0   0   50  0001 C CNN "digikey"
 	1    10100 2300
 	0    1    1    0
@@
 AR Path="/5DE49152/5E33EC9B" Ref="C917"  Part="1"
 F 0 "C917" V 6778 2046 20  0000 L BNN
-F 1 "100nF" V 6821 2093 20  0000 C CNN
+F 1 "0.1uF" V 6821 2093 20  0000 C CNN
 F 2 "servo:C_0603_1608Metric" H 6750 2150 60  0001 C CNN
 F 3 "" H 6750 2250 60  0000 C CNN
+F 4 "CC0603KPX7R7BB104" H 0   0   50  0001 C CNN "PartNumber"
+F 5 "311-1335-1-ND" H 0   0   50  0001 C CNN "digikey"
 	1    6750 2250
 	0    1    1    0
