File: kicad/temp.sch (KiCad schematic (older format))
At the start: 46 parts, among them U901 AMC1311B, U902 AMC1311B, U903 ADM2483, U904 AMC1311B, U905 AMC1311B

Commit message: more bom...
Parts:
- C901, C902, C915, C916: Description (none) -> CAP CER 1000PF 16V X7R 0603; PartNumber (none) -> 0603B102K160CT; digikey (none) -> 1292-1378-1-ND
- C903, C904, C905, C906, C907, C908, C909, C910, C911, C912, C913, C914, C917, C918: Description (none) -> CAP CER 0.1UF 16V X7R 0603
- R905, R906, R918, R919: value 12e -> 12
- R908: value 120e NP -> 120(dnp)
Changed lines of the file:
@@
 AR Path="/5DE49152/5E096250" Ref="R908"  Part="1"
 F 0 "R908" V 8978 2850 20  0000 L BNN
-F 1 "120e NP" V 9021 2916 20  0000 C CNN
+F 1 "120(dnp)" V 9021 2916 20  0000 C CNN
 F 2 "servo:R_0603_1608Metric" H 8500 2700 60  0001 C CNN
 F 3 "" H 8600 2800 60  0001 C CNN
@@
 F 4 "CC0603KPX7R7BB104" H 0   0   50  0001 C CNN "PartNumber"
 F 5 "311-1335-1-ND" H 0   0   50  0001 C CNN "digikey"
+F 6 "CAP CER 0.1UF 16V X7R 0603 " H 0   0   50  0001 C CNN "Description"
 	1    8450 5300
 	0    1    1    0
@@
 F 4 "CC0603KPX7R7BB104" H 0   0   50  0001 C CNN "PartNumber"
 F 5 "311-1335-1-ND" H 0   0   50  0001 C CNN "digikey"
+F 6 "CAP CER 0.1UF 16V X7R 0603 " H 0   0   50  0001 C CNN "Description"
 	1    8700 5300
 	0    1    1    0
@@
 AR Path="/5DE49152/5E5095EF" Ref="R905"  Part="1"
 F 0 "R905" H 8910 5165 20  0000 L BNN
-F 1 "12e" H 8950 5122 20  0000 C CNN
+F 1 "12" H 8950 5122 20  0000 C CNN
 F 2 "servo:R_0603_1608Metric" H 8450 4950 60  0001 C CNN
 F 3 "" H 8550 5050 60  0001 C CNN
@@
 F 2 "servo:C_0603_1608Metric" H 6200 4650 60  0001 C CNN
 F 3 "" H 6200 4750 60  0000 C CNN
+F 4 "CAP CER 1000PF 16V X7R 0603 " H 0   0   50  0001 C CNN "Description"
+F 5 "0603B102K160CT" H 0   0   50  0001 C CNN "PartNumber"
+F 6 "1292-1378-1-ND " H 0   0   50  0001 C CNN "digikey"
 	1    6200 4750
 	0    1    1    0
@@
 F 4 "CC0603KPX7R7BB104" H 0   0   50  0001 C CNN "PartNumber"
 F 5 "311-1335-1-ND" H 0   0   50  0001 C CNN "digikey"
+F 6 "CAP CER 0.1UF 16V X7R 0603 " H 0   0   50  0001 C CNN "Description"
 	1    6950 4500
 	0    1    1    0
@@
 F 4 "CC0603KPX7R7BB104" H 0   0   50  0001 C CNN "PartNumber"
 F 5 "311-1335-1-ND" H 0   0   50  0001 C CNN "digikey"
+F 6 "CAP CER 0.1UF 16V X7R 0603 " H 0   0   50  0001 C CNN "Description"
 	1    11250 5300
 	0    -1   1    0
@@
 F 4 "CC0603KPX7R7BB104" H 0   0   50  0001 C CNN "PartNumber"
 F 5 "311-1335-1-ND" H 0   0   50  0001 C CNN "digikey"
+F 6 "CAP CER 0.1UF 16V X7R 0603 " H 0   0   50  0001 C CNN "Description"
 	1    11000 5300
 	0    -1   1    0
@@
 AR Path="/5DE49152/5FE9D198" Ref="R918"  Part="1"
 F 0 "R918" H 10710 5165 20  0000 L BNN
-F 1 "12e" H 10750 5122 20  0000 C CNN
+F 1 "12" H 10750 5122 20  0000 C CNN
 F 2 "servo:R_0603_1608Metric" H 10250 4950 60  0001 C CNN
 F 3 "" H 10350 5050 60  0001 C CNN
@@
 F 2 "servo:C_0603_1608Metric" H 13500 4650 60  0001 C CNN
 F 3 "" H 13500 4750 60  0000 C CNN
+F 4 "CAP CER 1000PF 16V X7R 0603 " H 0   0   50  0001 C CNN "Description"
+F 5 "0603B102K160CT" H 0   0   50  0001 C CNN "PartNumber"
+F 6 "1292-1378-1-ND " H 0   0   50  0001 C CNN "digikey"
 	1    13500 4750
 	0    -1   1    0
@@
 F 4 "CC0603KPX7R7BB104" H 0   0   50  0001 C CNN "PartNumber"
 F 5 "311-1335-1-ND" H 0   0   50  0001 C CNN "digikey"
+F 6 "CAP CER 0.1UF 16V X7R 0603 " H 0   0   50  0001 C CNN "Description"
 	1    12750 4500
 	0    -1   1    0
@@
 F 4 "CC0603KPX7R7BB104" H 0   0   50  0001 C CNN "PartNumber"
 F 5 "311-1335-1-ND" H 0   0   50  0001 C CNN "digikey"
+F 6 "CAP CER 0.1UF 16V X7R 0603 " H 0   0   50  0001 C CNN "Description"
 	1    8450 6950
 	0    1    1    0
@@
 F 4 "CC0603KPX7R7BB104" H 0   0   50  0001 C CNN "PartNumber"
 F 5 "311-1335-1-ND" H 0   0   50  0001 C CNN "digikey"
+F 6 "CAP CER 0.1UF 16V X7R 0603 " H 0   0   50  0001 C CNN "Description"
 	1    8700 6950
 	0    1    1    0
@@
 AR Path="/5DE49152/5E1BD521" Ref="R906"  Part="1"
 F 0 "R906" H 8910 6815 20  0000 L BNN
-F 1 "12e" H 8950 6772 20  0000 C CNN
+F 1 "12" H 8950 6772 20  0000 C CNN
 F 2 "servo:R_0603_1608Metric" H 8450 6600 60  0001 C CNN
 F 3 "" H 8550 6700 60  0001 C CNN
@@
 F 2 "servo:C_0603_1608Metric" H 6200 6300 60  0001 C CNN
 F 3 "" H 6200 6400 60  0000 C CNN
+F 4 "CAP CER 1000PF 16V X7R 0603 " H 0   0   50  0001 C CNN "Description"
+F 5 "0603B102K160CT" H 0   0   50  0001 C CNN "PartNumber"
+F 6 "1292-1378-1-ND " H 0   0   50  0001 C CNN "digikey"
 	1    6200 6400
 	0    1    1    0
@@
 F 4 "CC0603KPX7R7BB104" H 0   0   50  0001 C CNN "PartNumber"
 F 5 "311-1335-1-ND" H 0   0   50  0001 C CNN "digikey"
+F 6 "CAP CER 0.1UF 16V X7R 0603 " H 0   0   50  0001 C CNN "Description"
 	1    6950 6150
 	0    1    1    0
@@
 F 4 "CC0603KPX7R7BB104" H 0   0   50  0001 C CNN "PartNumber"
 F 5 "311-1335-1-ND" H 0   0   50  0001 C CNN "digikey"
+F 6 "CAP CER 0.1UF 16V X7R 0603 " H 0   0   50  0001 C CNN "Description"
 	1    11250 6950
 	0    -1   1    0
@@
 F 4 "CC0603KPX7R7BB104" H 0   0   50  0001 C CNN "PartNumber"
 F 5 "311-1335-1-ND" H 0   0   50  0001 C CNN "digikey"
+F 6 "CAP CER 0.1UF 16V X7R 0603 " H 0   0   50  0001 C CNN "Description"
 	1    11000 6950
 	0    -1   1    0
@@
 AR Path="/5DE49152/5E1BD5B7" Ref="R919"  Part="1"
 F 0 "R919" H 10710 6815 20  0000 L BNN
-F 1 "12e" H 10750 6772 20  0000 C CNN
+F 1 "12" H 10750 6772 20  0000 C CNN
 F 2 "servo:R_0603_1608Metric" H 10250 6600 60  0001 C CNN
 F 3 "" H 10350 6700 60  0001 C CNN
@@
 F 2 "servo:C_0603_1608Metric" H 13500 6300 60  0001 C CNN
 F 3 "" H 13500 6400 60  0000 C CNN
+F 4 "CAP CER 1000PF 16V X7R 0603 " H 0   0   50  0001 C CNN "Description"
+F 5 "0603B102K160CT" H 0   0   50  0001 C CNN "PartNumber"
+F 6 "1292-1378-1-ND " H 0   0   50  0001 C CNN "digikey"
 	1    13500 6400
 	0    -1   1    0
@@
 F 4 "CC0603KPX7R7BB104" H 0   0   50  0001 C CNN "PartNumber"
 F 5 "311-1335-1-ND" H 0   0   50  0001 C CNN "digikey"
+F 6 "CAP CER 0.1UF 16V X7R 0603 " H 0   0   50  0001 C CNN "Description"
 	1    12750 6150
 	0    -1   1    0
@@
 F 4 "CC0603KPX7R7BB104" H 0   0   50  0001 C CNN "PartNumber"
 F 5 "311-1335-1-ND" H 0   0   50  0001 C CNN "digikey"
+F 6 "CAP CER 0.1UF 16V X7R 0603 " H 0   0   50  0001 C CNN "Description"
 	1    10100 2300
 	0    1    1    0
@@
 F 4 "CC0603KPX7R7BB104" H 0   0   50  0001 C CNN "PartNumber"
 F 5 "311-1335-1-ND" H 0   0   50  0001 C CNN "digikey"
+F 6 "CAP CER 0.1UF 16V X7R 0603 " H 0   0   50  0001 C CNN "Description"
 	1    6750 2250
 	0    1    1    0

Commit message: stackup
Parts:
- C901, C902, C915, C916: price@10 (none) -> 0.04100
- C903, C904, C905, C906, C907, C908, C909, C910, C911, C912, C913, C914, C917, C918: price@10 (none) -> 0.05800
- U901, U902, U904, U905: Description (none) -> Isolation IC 8-SOIC; PartNumber (none) -> AMC1311BDWV; digikey (none) -> 296-47610-ND; price@10 (none) -> 7.24300
- U903: Description (none) -> RS422, RS485 Digital Isolator 2500Vrms 3 Channel 500kbps 25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; PartNumber (none) -> ADM2483BRWZ; digikey (none) -> ADM2483BRWZ-ND; price@10 (none) -> 5.59000
Changed lines of the file:
@@
 F 2 "servo:SOIC-16W_7.5x10.3mm_P1.27mm" H 7850 2150 50  0001 C CNN
 F 3 "../doc/datasheets/adm2483.pdf" H 7100 2750 50  0001 C CNN
+F 4 "RS422, RS485 Digital Isolator 2500Vrms 3 Channel 500kbps 25kV/µs CMTI 16-SOIC (0.295\", 7.50mm Width) " H 0   0   50  0001 C CNN "Description"
+F 5 "ADM2483BRWZ" H 0   0   50  0001 C CNN "PartNumber"
+F 6 "ADM2483BRWZ-ND" H 0   0   50  0001 C CNN "digikey"
+F 7 "5.59000" H 0   0   50  0001 C CNN "price@10"
 	1    7850 2850
 	1    0    0    -1
@@
 AR Path="/605BEC04/5E5095C3" Ref="C?"  Part="1"
 AR Path="/5DE49152/5E5095C3" Ref="C905"  Part="1"
-F 0 "C905" V 8478 5096 20  0000 L BNN
-F 1 "0.1uF" V 8521 5143 20  0000 C CNN
+F 0 "C905" V 8478 5410 20  0000 L CNN
+F 1 "0.1uF" V 8521 5410 20  0000 L CNN
 F 2 "servo:C_0603_1608Metric" H 8450 5200 60  0001 C CNN
 F 3 "" H 8450 5300 60  0000 C CNN
@@
 F 5 "311-1335-1-ND" H 0   0   50  0001 C CNN "digikey"
 F 6 "CAP CER 0.1UF 16V X7R 0603 " H 0   0   50  0001 C CNN "Description"
+F 7 "0.05800" H 0   0   50  0001 C CNN "price@10"
 	1    8450 5300
 	0    1    1    0
@@
 F 5 "311-1335-1-ND" H 0   0   50  0001 C CNN "digikey"
 F 6 "CAP CER 0.1UF 16V X7R 0603 " H 0   0   50  0001 C CNN "Description"
+F 7 "0.05800" H 0   0   50  0001 C CNN "price@10"
 	1    8700 5300
 	0    1    1    0
@@
 F 2 "servo:SSO-8_7.6x5.9mm_P1.27mm_Clearance9.1mm" H 7750 3700 50  0001 C CIN
 F 3 "../doc/datasheets/amc1311.pdf" H 7650 4200 50  0001 C CNN
+F 4 "Isolation IC 8-SOIC " H 0   0   50  0001 C CNN "Description"
+F 5 "AMC1311BDWV" H 0   0   50  0001 C CNN "PartNumber"
+F 6 "296-47610-ND" H 0   0   50  0001 C CNN "digikey"
+F 7 "7.24300" H 0   0   50  0001 C CNN "price@10"
 	1    7700 4700
 	-1   0    0    -1
@@
 F 5 "0603B102K160CT" H 0   0   50  0001 C CNN "PartNumber"
 F 6 "1292-1378-1-ND " H 0   0   50  0001 C CNN "digikey"
+F 7 "0.04100" H 0   0   50  0001 C CNN "price@10"
 	1    6200 4750
 	0    1    1    0
@@
 F 5 "311-1335-1-ND" H 0   0   50  0001 C CNN "digikey"
 F 6 "CAP CER 0.1UF 16V X7R 0603 " H 0   0   50  0001 C CNN "Description"
+F 7 "0.05800" H 0   0   50  0001 C CNN "price@10"
 	1    6950 4500
 	0    1    1    0
@@
 F 5 "311-1335-1-ND" H 0   0   50  0001 C CNN "digikey"
 F 6 "CAP CER 0.1UF 16V X7R 0603 " H 0   0   50  0001 C CNN "Description"
+F 7 "0.05800" H 0   0   50  0001 C CNN "price@10"
 	1    11250 5300
 	0    -1   1    0
@@
 F 5 "311-1335-1-ND" H 0   0   50  0001 C CNN "digikey"
 F 6 "CAP CER 0.1UF 16V X7R 0603 " H 0   0   50  0001 C CNN "Description"
+F 7 "0.05800" H 0   0   50  0001 C CNN "price@10"
 	1    11000 5300
 	0    -1   1    0
@@
 F 2 "servo:SSO-8_7.6x5.9mm_P1.27mm_Clearance9.1mm" H 12050 3700 50  0001 C CIN
 F 3 "../doc/datasheets/amc1311.pdf" H 11950 4200 50  0001 C CNN
+F 4 "Isolation IC 8-SOIC " H 0   0   50  0001 C CNN "Description"
+F 5 "AMC1311BDWV" H 0   0   50  0001 C CNN "PartNumber"
+F 6 "296-47610-ND" H 0   0   50  0001 C CNN "digikey"
+F 7 "7.24300" H 0   0   50  0001 C CNN "price@10"
 	1    12000 4700
 	1    0    0    -1
@@
 F 5 "0603B102K160CT" H 0   0   50  0001 C CNN "PartNumber"
 F 6 "1292-1378-1-ND " H 0   0   50  0001 C CNN "digikey"
+F 7 "0.04100" H 0   0   50  0001 C CNN "price@10"
 	1    13500 4750
 	0    -1   1    0
@@
 F 5 "311-1335-1-ND" H 0   0   50  0001 C CNN "digikey"
 F 6 "CAP CER 0.1UF 16V X7R 0603 " H 0   0   50  0001 C CNN "Description"
+F 7 "0.05800" H 0   0   50  0001 C CNN "price@10"
 	1    12750 4500
 	0    -1   1    0
@@
 F 5 "311-1335-1-ND" H 0   0   50  0001 C CNN "digikey"
 F 6 "CAP CER 0.1UF 16V X7R 0603 " H 0   0   50  0001 C CNN "Description"
+F 7 "0.05800" H 0   0   50  0001 C CNN "price@10"
 	1    8450 6950
 	0    1    1    0
@@
 F 5 "311-1335-1-ND" H 0   0   50  0001 C CNN "digikey"
 F 6 "CAP CER 0.1UF 16V X7R 0603 " H 0   0   50  0001 C CNN "Description"
+F 7 "0.05800" H 0   0   50  0001 C CNN "price@10"
 	1    8700 6950
 	0    1    1    0
@@
 F 2 "servo:SSO-8_7.6x5.9mm_P1.27mm_Clearance9.1mm" H 7750 5350 50  0001 C CIN
 F 3 "../doc/datasheets/amc1311.pdf" H 7650 5850 50  0001 C CNN
+F 4 "Isolation IC 8-SOIC " H 0   0   50  0001 C CNN "Description"
+F 5 "AMC1311BDWV" H 0   0   50  0001 C CNN "PartNumber"
+F 6 "296-47610-ND" H 0   0   50  0001 C CNN "digikey"
+F 7 "7.24300" H 0   0   50  0001 C CNN "price@10"
 	1    7700 6350
 	-1   0    0    -1
@@
 F 5 "0603B102K160CT" H 0   0   50  0001 C CNN "PartNumber"
 F 6 "1292-1378-1-ND " H 0   0   50  0001 C CNN "digikey"
+F 7 "0.04100" H 0   0   50  0001 C CNN "price@10"
 	1    6200 6400
 	0    1    1    0
@@
 F 5 "311-1335-1-ND" H 0   0   50  0001 C CNN "digikey"
 F 6 "CAP CER 0.1UF 16V X7R 0603 " H 0   0   50  0001 C CNN "Description"
+F 7 "0.05800" H 0   0   50  0001 C CNN "price@10"
 	1    6950 6150
 	0    1    1    0
@@
 AR Path="/605BEC04/5E1BD594" Ref="C?"  Part="1"
 AR Path="/5DE49152/5E1BD594" Ref="C912"  Part="1"
-F 0 "C912" V 11278 6746 20  0000 L BNN
-F 1 "0.1uF" V 11321 6793 20  0000 C CNN
+F 0 "C912" V 11278 6840 20  0000 R CNN
+F 1 "0.1uF" V 11321 6840 20  0000 R CNN
 F 2 "servo:C_0603_1608Metric" H 11250 6850 60  0001 C CNN
 F 3 "" H 11250 6950 60  0000 C CNN
@@
 F 5 "311-1335-1-ND" H 0   0   50  0001 C CNN "digikey"
 F 6 "CAP CER 0.1UF 16V X7R 0603 " H 0   0   50  0001 C CNN "Description"
+F 7 "0.05800" H 0   0   50  0001 C CNN "price@10"
 	1    11250 6950
 	0    -1   1    0
@@
 AR Path="/605BEC04/5E1BD5B0" Ref="C?"  Part="1"
 AR Path="/5DE49152/5E1BD5B0" Ref="C910"  Part="1"
-F 0 "C910" V 11028 7060 20  0000 L BNN
-F 1 "0.1uF" V 11071 7100 20  0000 C CNN
+F 0 "C910" V 11028 7060 20  0000 L CNN
+F 1 "0.1uF" V 11071 7060 20  0000 L CNN
 F 2 "servo:C_0603_1608Metric" H 11000 6850 60  0001 C CNN
 F 3 "" H 11000 6950 60  0000 C CNN
@@
 F 5 "311-1335-1-ND" H 0   0   50  0001 C CNN "digikey"
 F 6 "CAP CER 0.1UF 16V X7R 0603 " H 0   0   50  0001 C CNN "Description"
+F 7 "0.05800" H 0   0   50  0001 C CNN "price@10"
 	1    11000 6950
 	0    -1   1    0
@@
 F 2 "servo:SSO-8_7.6x5.9mm_P1.27mm_Clearance9.1mm" H 12050 5350 50  0001 C CIN
 F 3 "../doc/datasheets/amc1311.pdf" H 11950 5850 50  0001 C CNN
+F 4 "Isolation IC 8-SOIC " H 0   0   50  0001 C CNN "Description"
+F 5 "AMC1311BDWV" H 0   0   50  0001 C CNN "PartNumber"
+F 6 "296-47610-ND" H 0   0   50  0001 C CNN "digikey"
+F 7 "7.24300" H 0   0   50  0001 C CNN "price@10"
 	1    12000 6350
 	1    0    0    -1
@@
 AR Path="/605BEC04/5E1BD5DD" Ref="R?"  Part="1"
 AR Path="/5DE49152/5E1BD5DD" Ref="R916"  Part="1"
-F 0 "R916" V 10428 6550 20  0000 L BNN
-F 1 "1k(dnp)" V 10471 6590 20  0000 C CNN
+F 0 "R916" V 10428 6450 20  0000 R CNN
+F 1 "1k(dnp)" V 10471 6450 20  0000 R CNN
 F 2 "servo:R_0603_1608Metric" H 9950 6400 60  0001 C CNN
 F 3 "" H 10050 6500 60  0001 C CNN
@@
 F 5 "0603B102K160CT" H 0   0   50  0001 C CNN "PartNumber"
 F 6 "1292-1378-1-ND " H 0   0   50  0001 C CNN "digikey"
+F 7 "0.04100" H 0   0   50  0001 C CNN "price@10"
 	1    13500 6400
 	0    -1   1    0
@@
 F 5 "311-1335-1-ND" H 0   0   50  0001 C CNN "digikey"
 F 6 "CAP CER 0.1UF 16V X7R 0603 " H 0   0   50  0001 C CNN "Description"
+F 7 "0.05800" H 0   0   50  0001 C CNN "price@10"
 	1    12750 6150
 	0    -1   1    0
@@
 F 5 "311-1335-1-ND" H 0   0   50  0001 C CNN "digikey"
 F 6 "CAP CER 0.1UF 16V X7R 0603 " H 0   0   50  0001 C CNN "Description"
+F 7 "0.05800" H 0   0   50  0001 C CNN "price@10"
 	1    10100 2300
 	0    1    1    0
@@
 F 5 "311-1335-1-ND" H 0   0   50  0001 C CNN "digikey"
 F 6 "CAP CER 0.1UF 16V X7R 0603 " H 0   0   50  0001 C CNN "Description"
+F 7 "0.05800" H 0   0   50  0001 C CNN "price@10"
 	1    6750 2250
 	0    1    1    0

Commit message: bom copleted
Parts:
- R901, R902, R903, R904, R907, R920, R921, R922, R923: value 2k2 -> 2.2k; Description (none) -> 2.2 kOhms ±5% 0.1W, 1/10W Chip Resistor 0603 (1608 Metric) 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; PartNumber (none) -> ERJ-3GEYJ222V; digikey (none) -> P2.2KGCT-ND; price@10 (none) -> 0.04500
- R905, R906, R918, R919: Description (none) -> 12 Ohms ±5% 0.1W, 1/10W Chip Resistor 0603 (1608 Metric) Mo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; PartNumber (none) -> RC0603JR-0712RL; digikey (none) -> 311-12GRCT-ND; price@10 (none) -> 0.01900
- R908: Description (none) -> 120 Ohms ±5% 0.1W, 1/10W Chip Resistor 0603 (1608 Metric) A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; PartNumber (none) -> RMCF0603JT120R; digikey (none) -> RMCF0603JT120RCT-ND; price@10 (none) -> 0.01400
- R909, R911, R913, R915, R917: Description (none) -> 10 kOhms ±5% 0.1W, 1/10W Chip Resistor 0603 (1608 Metric) M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; PartNumber (none) -> RC0603JR-0710KL; digikey (none) -> 311-10KGRCT-ND; price@10 (none) -> 0.01900
- R910, R912, R914, R916: Description (none) -> 1 kOhms ±5% 0.1W, 1/10W Chip Resistor 0603 (1608 Metric) Mo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; PartNumber (none) -> RC0603JR-071KL; digikey (none) -> 311-1.0KGRCT-ND; price@10 (none) -> 0.01900
