File: kicad/lem.sch (KiCad schematic (older format))
At the start: 42 parts, among them J1501 tblock2x3, J1502 tblock2x3, J1503 tblock2x3, J1504 tblock2x3, J1505 tblock2x3, J1506 tblock2x3, U1501 LXS6-NPS, U1502 LXS6-NPS, U1503 LXS6-NPS, U1504 LXS6-NPS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

Commit message: keep placing
Parts:
- removed C1503, C1506, C1507, C1516, C1517, C1518: 100pF, servo:C_0603_1608Metric, symbol servo:Capacitor
Other:
- note removed: "one near LEM, \nthe other near uC"
Changed lines of the file:
@@
 The intention of these lems is to have the capacity on the control board\n to measure all the current, without the need of the sigma delta chips\n on power board side. Why?? becouse I've study the two options\n carrefullty and I've conclude that there are very similar, and more or\n less buck per byck (a little expensive is SD) but the new generation\n LEM's I'm includin here has <0.5uSeg response time, and the SD has\n all the SD filter delay, so LEM is faster. The other advantage is that for\n same LEM I've choosen you could rearange the connection to multiply\n the preccision 1x,2x or 3x without touching nothing, and is pretty\n linear.  In the case of SD you have to change the precission shunt. or\n puts more than one, that is costly and take some board space.\nThe disadvantage of LEM is that the output is single ended, so it could\n not travel across boards, for that reason I've put them on control\n board, but is completely isolated becouse of these phisics effect. and\n also becouse of that single ended I just use one ADC channel per\n current. I't not the only option, becous if you insist and wanna use SD,\n I'eft all the SD channels available as an inputs on SD schematic page.\n\nthese LEM's version doesn't need a buffer, \nit's one already included inside LEM\n\nLXS6 is LTS and CAS pin to pin compatible, but LXS is a little better.\n I don't usa an opamp becous with the external conection I have x,2x\n and 3x amplifier option without any component\n\nI've decided to make the loop over the LEM on board and if you\n wanna change it you have to use the soldering iron..becouse the\n connetor is 2 terminal, not 6\n
-$Comp
-L servo:Capacitor C1506
-U 1 1 5E3E8DDF
-P 3900 4350
-F 0 "C1506" V 3928 4460 20  0000 L CNN
-F 1 "100pF" V 3971 4460 20  0000 L CNN
-F 2 "servo:C_0603_1608Metric" H 3900 4250 60  0001 C CNN
-F 3 "" H 3900 4350 60  0000 C CNN
-	1    3900 4350
-	0    -1   1    0
-$EndComp
 $Comp
 L servo:GND #PWR01504
@@
 $EndComp
 $Comp
-L servo:GND #PWR01512
-U 1 1 5E3E8DFA
-P 3900 4550
-F 0 "#PWR01512" H 3900 4300 30  0001 C CNN
-F 1 "GND" H 3900 4392 30  0000 C CNN
-F 2 "" H 3900 4550 50  0001 C CNN
-F 3 "" H 3900 4550 50  0001 C CNN
-	1    3900 4550
-	-1   0    0    -1
-$EndComp
-Wire Wire Line
-	3900 4250 3900 4150
-Wire Wire Line
-	3900 4150 4200 4150
-Connection ~ 3900 4150
-$Comp
 L servo:Capacitor C1509
 U 1 1 5E3E8E03
@@
 Wire Wire Line
 	3600 4150 3600 4250
-Text Notes 3850 4250 2    20   ~ 0
-one near LEM, \nthe other near uC
-Wire Wire Line
-	3900 4150 3600 4150
 Connection ~ 3600 4150
 Wire Wire Line
@@
 Connection ~ 3750 5300
 $Comp
-L servo:Capacitor C1503
-U 1 1 5E274FDC
-P 3700 6300
-F 0 "C1503" V 3728 6410 20  0000 L CNN
-F 1 "100pF" V 3771 6410 20  0000 L CNN
-F 2 "servo:C_0603_1608Metric" H 3700 6200 60  0001 C CNN
-F 3 "" H 3700 6300 60  0000 C CNN
-	1    3700 6300
-	0    -1   1    0
-$EndComp
-$Comp
 L servo:GND #PWR0103
 U 1 1 5E274FE3
@@
 $EndComp
 $Comp
-L servo:GND #PWR0104
-U 1 1 5E274FF7
-P 3700 6500
-F 0 "#PWR0104" H 3700 6250 30  0001 C CNN
-F 1 "GND" H 3700 6342 30  0000 C CNN
-F 2 "" H 3700 6500 50  0001 C CNN
-F 3 "" H 3700 6500 50  0001 C CNN
-	1    3700 6500
-	-1   0    0    -1
-$EndComp
-Wire Wire Line
-	3700 6200 3700 6100
-Wire Wire Line
-	3700 6100 4000 6100
-Connection ~ 3700 6100
-$Comp
 L servo:Capacitor C1501
 U 1 1 5E275000
@@
 Wire Wire Line
 	3400 6100 3400 6200
-Text Notes 3650 6200 2    20   ~ 0
-one near LEM, \nthe other near uC
-Wire Wire Line
-	3700 6100 3400 6100
 Connection ~ 3400 6100
 Wire Wire Line
@@
 Connection ~ 3850 7900
 $Comp
-L servo:Capacitor C1507
-U 1 1 5E276226
-P 3800 8900
-F 0 "C1507" V 3828 9010 20  0000 L CNN
-F 1 "100pF" V 3871 9010 20  0000 L CNN
-F 2 "servo:C_0603_1608Metric" H 3800 8800 60  0001 C CNN
-F 3 "" H 3800 8900 60  0000 C CNN
-	1    3800 8900
-	0    -1   1    0
-$EndComp
-$Comp
 L servo:GND #PWR0108
 U 1 1 5E27622D
@@
 $EndComp
 $Comp
-L servo:GND #PWR0109
-U 1 1 5E276241
-P 3800 9100
-F 0 "#PWR0109" H 3800 8850 30  0001 C CNN
-F 1 "GND" H 3800 8942 30  0000 C CNN
-F 2 "" H 3800 9100 50  0001 C CNN
-F 3 "" H 3800 9100 50  0001 C CNN
-	1    3800 9100
-	-1   0    0    -1
-$EndComp
-Wire Wire Line
-	3800 8800 3800 8700
-Wire Wire Line
-	3800 8700 4100 8700
-Connection ~ 3800 8700
-$Comp
 L servo:Capacitor C1502
 U 1 1 5E27624A
@@
 Wire Wire Line
 	3500 8700 3500 8800
-Text Notes 3750 8800 2    20   ~ 0
-one near LEM, \nthe other near uC
-Wire Wire Line
-	3800 8700 3500 8700
 Connection ~ 3500 8700
 Wire Wire Line
@@
 	8800 4150 8500 4150
 Connection ~ 8800 4150
-$Comp
-L servo:Capacitor C1516
-U 1 1 5E27869E
-P 9100 4350
-F 0 "C1516" V 9128 4460 20  0000 L CNN
-F 1 "100pF" V 9171 4460 20  0000 L CNN
-F 2 "servo:C_0603_1608Metric" H 9100 4250 60  0001 C CNN
-F 3 "" H 9100 4350 60  0000 C CNN
-	1    9100 4350
-	0    1    1    0
-$EndComp
-$Comp
-L servo:GND #PWR0115
-U 1 1 5E2786A5
-P 9100 4550
-F 0 "#PWR0115" H 9100 4300 30  0001 C CNN
-F 1 "GND" H 9100 4392 30  0000 C CNN
-F 2 "" H 9100 4550 50  0001 C CNN
-F 3 "" H 9100 4550 50  0001 C CNN
-	1    9100 4550
-	1    0    0    -1
-$EndComp
-Wire Wire Line
-	9100 4150 9100 4250
-Text Notes 8850 4250 0    20   ~ 0
-one near LEM, \nthe other near uC
-Wire Wire Line
-	8800 4150 9100 4150
-Connection ~ 9100 4150
-Wire Wire Line
-	9100 4150 9300 4150
 Connection ~ 8500 4150
 $Comp
@@
 	8800 6100 8500 6100
 Connection ~ 8800 6100
-$Comp
-L servo:Capacitor C1517
-U 1 1 5E2833C5
-P 9100 6300
-F 0 "C1517" V 9128 6410 20  0000 L CNN
-F 1 "100pF" V 9171 6410 20  0000 L CNN
-F 2 "servo:C_0603_1608Metric" H 9100 6200 60  0001 C CNN
-F 3 "" H 9100 6300 60  0000 C CNN
-	1    9100 6300
-	0    1    1    0
-$EndComp
-$Comp
-L servo:GND #PWR0120
-U 1 1 5E2833CC
-P 9100 6500
-F 0 "#PWR0120" H 9100 6250 30  0001 C CNN
-F 1 "GND" H 9100 6342 30  0000 C CNN
-F 2 "" H 9100 6500 50  0001 C CNN
-F 3 "" H 9100 6500 50  0001 C CNN
-	1    9100 6500
-	1    0    0    -1
-$EndComp
-Wire Wire Line
-	9100 6100 9100 6200
-Text Notes 8850 6200 0    20   ~ 0
-one near LEM, \nthe other near uC
-Wire Wire Line
-	8800 6100 9100 6100
-Connection ~ 9100 6100
-Wire Wire Line
-	9100 6100 9300 6100
 Connection ~ 8500 6100
 $Comp
@@
 	8800 8700 8500 8700
 Connection ~ 8800 8700
-$Comp
-L servo:Capacitor C1518
-U 1 1 5E288A33
-P 9100 8900
-F 0 "C1518" V 9128 9010 20  0000 L CNN
-F 1 "100pF" V 9171 9010 20  0000 L CNN
-F 2 "servo:C_0603_1608Metric" H 9100 8800 60  0001 C CNN
-F 3 "" H 9100 8900 60  0000 C CNN
-	1    9100 8900
-	0    1    1    0
-$EndComp
-$Comp
-L servo:GND #PWR0125
-U 1 1 5E288A3A
-P 9100 9100
-F 0 "#PWR0125" H 9100 8850 30  0001 C CNN
-F 1 "GND" H 9100 8942 30  0000 C CNN
-F 2 "" H 9100 9100 50  0001 C CNN
-F 3 "" H 9100 9100 50  0001 C CNN
-	1    9100 9100
-	1    0    0    -1
-$EndComp
-Wire Wire Line
-	9100 8700 9100 8800
-Text Notes 8850 8800 0    20   ~ 0
-one near LEM, \nthe other near uC
-Wire Wire Line
-	8800 8700 9100 8700
-Connection ~ 9100 8700
-Wire Wire Line
-	9100 8700 9300 8700
 Connection ~ 8500 8700
 $Comp
@@
 Wire Wire Line
 	7150 3100 7150 3400
+Wire Wire Line
+	3400 6100 4000 6100
+Wire Wire Line
+	3600 4150 4200 4150
+Wire Wire Line
+	8800 4150 9300 4150
+Wire Wire Line
+	8800 6100 9300 6100
+Wire Wire Line
+	8800 8700 9300 8700
+Wire Wire Line
+	3500 8700 4100 8700
 $EndSCHEMATC

Commit message: touting....
Parts:
- U1501, U1502, U1503, U1504, U1505, U1506: footprint servo:LEM_LTSR-NP -> servo:LEM_LXS-NP
Changed lines of the file:
@@
 F 0 "U1503" H 4350 4150 39  0000 L CNN
 F 1 "LXS6-NPS" H 4300 4050 39  0000 L CNN
-F 2 "servo:LEM_LTSR-NP" H 4850 2850 50  0001 C CNN
+F 2 "servo:LEM_LXS-NP" H 4850 2850 50  0001 C CNN
 F 3 "../doc/datasheets/lem_lxs_series.pdf" H 4850 3000 50  0001 C CNN
 	1    4850 3650
@@
 F 0 "U1501" H 4150 6100 39  0000 L CNN
 F 1 "LXS6-NPS" H 4100 6000 39  0000 L CNN
-F 2 "servo:LEM_LTSR-NP" H 4650 4800 50  0001 C CNN
+F 2 "servo:LEM_LXS-NP" H 4650 4800 50  0001 C CNN
 F 3 "../doc/datasheets/lem_lxs_series.pdf" H 4650 4950 50  0001 C CNN
 	1    4650 5600
@@
 F 0 "U1504" H 7350 4150 39  0000 L CNN
 F 1 "LXS6-NPS" H 7300 4050 39  0000 L CNN
-F 2 "servo:LEM_LTSR-NP" H 7850 2850 50  0001 C CNN
+F 2 "servo:LEM_LXS-NP" H 7850 2850 50  0001 C CNN
 F 3 "../doc/datasheets/lem_lxs_series.pdf" H 7850 3000 50  0001 C CNN
 	1    7850 3650
@@
 F 0 "U1505" H 7350 6100 39  0000 L CNN
 F 1 "LXS6-NPS" H 7300 6000 39  0000 L CNN
-F 2 "servo:LEM_LTSR-NP" H 7850 4800 50  0001 C CNN
+F 2 "servo:LEM_LXS-NP" H 7850 4800 50  0001 C CNN
 F 3 "../doc/datasheets/lem_lxs_series.pdf" H 7850 4950 50  0001 C CNN
 	1    7850 5600
@@
 F 0 "U1506" H 7350 8700 39  0000 L CNN
 F 1 "LXS6-NPS" H 7300 8600 39  0000 L CNN
-F 2 "servo:LEM_LTSR-NP" H 7850 7400 50  0001 C CNN
+F 2 "servo:LEM_LXS-NP" H 7850 7400 50  0001 C CNN
 F 3 "../doc/datasheets/lem_lxs_series.pdf" H 7850 7550 50  0001 C CNN
 	1    7850 8200
@@
 F 0 "U1502" H 4250 8700 39  0000 L CNN
 F 1 "LXS6-NPS" H 4200 8600 39  0000 L CNN
-F 2 "servo:LEM_LTSR-NP" H 4750 7400 50  0001 C CNN
+F 2 "servo:LEM_LXS-NP" H 4750 7400 50  0001 C CNN
 F 3 "../doc/datasheets/lem_lxs_series.pdf" H 4750 7550 50  0001 C CNN
 	1    4750 8200

Commit message: serigrafia...
Parts:
- R1501, R1502, R1503, R1504, R1505, R1506, R1507, R1508, R1509, R1510, R1511, R1512: footprint Resistor_SMD:R_0603_1608Metric -> servo:R_0603_1608Metric
Changed lines of the file:
@@
 F 0 "R1506" V 4178 4400 20  0000 L CNN
 F 1 "3.3k" V 4221 4400 20  0000 L CNN
-F 2 "Resistor_SMD:R_0603_1608Metric" H 3700 4250 60  0001 C CNN
+F 2 "servo:R_0603_1608Metric" H 3700 4250 60  0001 C CNN
 F 3 "" H 3800 4350 60  0001 C CNN
 	1    4200 4350
@@
 F 0 "R1505" V 4178 4000 20  0000 L CNN
 F 1 "5k" V 4221 4000 20  0000 L CNN
-F 2 "Resistor_SMD:R_0603_1608Metric" H 3700 3850 60  0001 C CNN
+F 2 "servo:R_0603_1608Metric" H 3700 3850 60  0001 C CNN
 F 3 "" H 3800 3950 60  0001 C CNN
 	1    4200 3950
@@
 F 0 "R1502" V 3978 6350 20  0000 L CNN
 F 1 "3.3k" V 4021 6350 20  0000 L CNN
-F 2 "Resistor_SMD:R_0603_1608Metric" H 3500 6200 60  0001 C CNN
+F 2 "servo:R_0603_1608Metric" H 3500 6200 60  0001 C CNN
 F 3 "" H 3600 6300 60  0001 C CNN
 	1    4000 6300
@@
 F 0 "R1501" V 3978 5950 20  0000 L CNN
 F 1 "5k" V 4021 5950 20  0000 L CNN
-F 2 "Resistor_SMD:R_0603_1608Metric" H 3500 5800 60  0001 C CNN
+F 2 "servo:R_0603_1608Metric" H 3500 5800 60  0001 C CNN
 F 3 "" H 3600 5900 60  0001 C CNN
 	1    4000 5900
@@
 F 0 "R1504" V 4078 8950 20  0000 L CNN
 F 1 "3.3k" V 4121 8950 20  0000 L CNN
-F 2 "Resistor_SMD:R_0603_1608Metric" H 3600 8800 60  0001 C CNN
+F 2 "servo:R_0603_1608Metric" H 3600 8800 60  0001 C CNN
 F 3 "" H 3700 8900 60  0001 C CNN
 	1    4100 8900
@@
 F 0 "R1503" V 4078 8550 20  0000 L CNN
 F 1 "5k" V 4121 8550 20  0000 L CNN
-F 2 "Resistor_SMD:R_0603_1608Metric" H 3600 8400 60  0001 C CNN
+F 2 "servo:R_0603_1608Metric" H 3600 8400 60  0001 C CNN
 F 3 "" H 3700 8500 60  0001 C CNN
 	1    4100 8500
@@
 F 0 "R1508" V 8478 4400 20  0000 L CNN
 F 1 "3.3k" V 8521 4400 20  0000 L CNN
-F 2 "Resistor_SMD:R_0603_1608Metric" H 8000 4250 60  0001 C CNN
+F 2 "servo:R_0603_1608Metric" H 8000 4250 60  0001 C CNN
 F 3 "" H 8100 4350 60  0001 C CNN
 	1    8500 4350
@@
 F 0 "R1507" V 8478 4000 20  0000 L CNN
 F 1 "5k" V 8521 4000 20  0000 L CNN
-F 2 "Resistor_SMD:R_0603_1608Metric" H 8000 3850 60  0001 C CNN
+F 2 "servo:R_0603_1608Metric" H 8000 3850 60  0001 C CNN
 F 3 "" H 8100 3950 60  0001 C CNN
 	1    8500 3950
@@
 F 0 "R1510" V 8478 6350 20  0000 L CNN
 F 1 "3.3k" V 8521 6350 20  0000 L CNN
-F 2 "Resistor_SMD:R_0603_1608Metric" H 8000 6200 60  0001 C CNN
+F 2 "servo:R_0603_1608Metric" H 8000 6200 60  0001 C CNN
 F 3 "" H 8100 6300 60  0001 C CNN
 	1    8500 6300
@@
 F 0 "R1509" V 8478 5950 20  0000 L CNN
 F 1 "5k" V 8521 5950 20  0000 L CNN
-F 2 "Resistor_SMD:R_0603_1608Metric" H 8000 5800 60  0001 C CNN
+F 2 "servo:R_0603_1608Metric" H 8000 5800 60  0001 C CNN
 F 3 "" H 8100 5900 60  0001 C CNN
 	1    8500 5900
@@
 F 0 "R1512" V 8478 8950 20  0000 L CNN
 F 1 "3.3k" V 8521 8950 20  0000 L CNN
-F 2 "Resistor_SMD:R_0603_1608Metric" H 8000 8800 60  0001 C CNN
+F 2 "servo:R_0603_1608Metric" H 8000 8800 60  0001 C CNN
 F 3 "" H 8100 8900 60  0001 C CNN
 	1    8500 8900
@@
 F 0 "R1511" V 8478 8550 20  0000 L CNN
 F 1 "5k" V 8521 8550 20  0000 L CNN
-F 2 "Resistor_SMD:R_0603_1608Metric" H 8000 8400 60  0001 C CNN
+F 2 "servo:R_0603_1608Metric" H 8000 8400 60  0001 C CNN
 F 3 "" H 8100 8500 60  0001 C CNN
 	1    8500 8500

Commit message: bom bom bom...
Parts:
- C1504, C1505, C1508, C1510, C1511, C1512: value 100nF -> 0.1uF; PartNumber (none) -> CC0603KPX7R7BB104; digikey (none) -> 311-1335-1-ND
Changed lines of the file:
@@
 P 3950 3450
 F 0 "C1504" V 3978 3560 20  0000 L CNN
-F 1 "100nF" V 4021 3560 20  0000 L CNN
+F 1 "0.1uF" V 4021 3560 20  0000 L CNN
 F 2 "servo:C_0603_1608Metric" H 3950 3350 60  0001 C CNN
 F 3 "" H 3950 3450 60  0000 C CNN
+F 4 "CC0603KPX7R7BB104" H 0   0   50  0001 C CNN "PartNumber"
+F 5 "311-1335-1-ND" H 0   0   50  0001 C CNN "digikey"
 	1    3950 3450
 	0    -1   1    0
@@
 P 3750 5400
 F 0 "C1505" V 3778 5510 20  0000 L CNN
-F 1 "100nF" V 3821 5510 20  0000 L CNN
+F 1 "0.1uF" V 3821 5510 20  0000 L CNN
 F 2 "servo:C_0603_1608Metric" H 3750 5300 60  0001 C CNN
 F 3 "" H 3750 5400 60  0000 C CNN
+F 4 "CC0603KPX7R7BB104" H 0   0   50  0001 C CNN "PartNumber"
+F 5 "311-1335-1-ND" H 0   0   50  0001 C CNN "digikey"
 	1    3750 5400
 	0    -1   1    0
@@
 P 3850 8000
 F 0 "C1508" V 3878 8110 20  0000 L CNN
-F 1 "100nF" V 3921 8110 20  0000 L CNN
+F 1 "0.1uF" V 3921 8110 20  0000 L CNN
 F 2 "servo:C_0603_1608Metric" H 3850 7900 60  0001 C CNN
 F 3 "" H 3850 8000 60  0000 C CNN
+F 4 "CC0603KPX7R7BB104" H 0   0   50  0001 C CNN "PartNumber"
+F 5 "311-1335-1-ND" H 0   0   50  0001 C CNN "digikey"
 	1    3850 8000
 	0    -1   1    0
@@
 P 8750 3450
 F 0 "C1510" V 8778 3560 20  0000 L CNN
-F 1 "100nF" V 8821 3560 20  0000 L CNN
+F 1 "0.1uF" V 8821 3560 20  0000 L CNN
 F 2 "servo:C_0603_1608Metric" H 8750 3350 60  0001 C CNN
 F 3 "" H 8750 3450 60  0000 C CNN
+F 4 "CC0603KPX7R7BB104" H 0   0   50  0001 C CNN "PartNumber"
+F 5 "311-1335-1-ND" H 0   0   50  0001 C CNN "digikey"
 	1    8750 3450
 	0    1    1    0
@@
 P 8750 5400
 F 0 "C1511" V 8778 5510 20  0000 L CNN
-F 1 "100nF" V 8821 5510 20  0000 L CNN
+F 1 "0.1uF" V 8821 5510 20  0000 L CNN
 F 2 "servo:C_0603_1608Metric" H 8750 5300 60  0001 C CNN
 F 3 "" H 8750 5400 60  0000 C CNN
+F 4 "CC0603KPX7R7BB104" H 0   0   50  0001 C CNN "PartNumber"
+F 5 "311-1335-1-ND" H 0   0   50  0001 C CNN "digikey"
 	1    8750 5400
 	0    1    1    0
@@
 P 8750 8000
 F 0 "C1512" V 8778 8110 20  0000 L CNN
-F 1 "100nF" V 8821 8110 20  0000 L CNN
+F 1 "0.1uF" V 8821 8110 20  0000 L CNN
 F 2 "servo:C_0603_1608Metric" H 8750 7900 60  0001 C CNN
 F 3 "" H 8750 8000 60  0000 C CNN
+F 4 "CC0603KPX7R7BB104" H 0   0   50  0001 C CNN "PartNumber"
+F 5 "311-1335-1-ND" H 0   0   50  0001 C CNN "digikey"
 	1    8750 8000
 	0    1    1    0
