File: kicad/lem.sch (KiCad schematic (older format))
At the start: 36 parts, among them J1501 tblock2x3, J1502 tblock2x3, J1503 tblock2x3, J1504 tblock2x3, J1505 tblock2x3, J1506 tblock2x3, U1501 LXS6-NPS, U1502 LXS6-NPS, U1503 LXS6-NPS, U1504 LXS6-NPS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

Commit message: more bom...
Parts:
- C1501, C1502, C1509, C1513, C1514, C1515: value 100pF -> 1nF; Description (none) -> CAP CER 1000PF 16V X7R 0603; PartNumber (none) -> 0603B102K160CT; digikey (none) -> 1292-1378-1-ND
- C1504, C1505, C1508, C1510, C1511, C1512: Description (none) -> CAP CER 0.1UF 16V X7R 0603
- J1501, J1502, J1503, J1504, J1505, J1506: value tblock2x3 -> tblock 2x3 5.08; Description (none) -> 6 Position Terminal Block Header, Male Pins, Shrouded (4 Si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; PartNumber (none) -> 1762376; digikey (none) -> 277-1400-ND; price@10 (none) -> 3.95500
Changed lines of the file:
@@
 F 4 "CC0603KPX7R7BB104" H 0   0   50  0001 C CNN "PartNumber"
 F 5 "311-1335-1-ND" H 0   0   50  0001 C CNN "digikey"
+F 6 "CAP CER 0.1UF 16V X7R 0603 " H 0   0   50  0001 C CNN "Description"
 	1    3950 3450
 	0    -1   1    0
@@
 P 3600 4350
 F 0 "C1509" V 3628 4460 20  0000 L CNN
-F 1 "100pF" V 3671 4460 20  0000 L CNN
+F 1 "1nF" V 3671 4460 20  0000 L CNN
 F 2 "servo:C_0603_1608Metric" H 3600 4250 60  0001 C CNN
 F 3 "" H 3600 4350 60  0000 C CNN
+F 4 "CAP CER 1000PF 16V X7R 0603 " H 0   0   50  0001 C CNN "Description"
+F 5 "0603B102K160CT" H 0   0   50  0001 C CNN "PartNumber"
+F 6 "1292-1378-1-ND " H 0   0   50  0001 C CNN "digikey"
 	1    3600 4350
 	0    -1   1    0
@@
 F 4 "CC0603KPX7R7BB104" H 0   0   50  0001 C CNN "PartNumber"
 F 5 "311-1335-1-ND" H 0   0   50  0001 C CNN "digikey"
+F 6 "CAP CER 0.1UF 16V X7R 0603 " H 0   0   50  0001 C CNN "Description"
 	1    3750 5400
 	0    -1   1    0
@@
 P 3400 6300
 F 0 "C1501" V 3428 6410 20  0000 L CNN
-F 1 "100pF" V 3471 6410 20  0000 L CNN
+F 1 "1nF" V 3471 6410 20  0000 L CNN
 F 2 "servo:C_0603_1608Metric" H 3400 6200 60  0001 C CNN
 F 3 "" H 3400 6300 60  0000 C CNN
+F 4 "CAP CER 1000PF 16V X7R 0603 " H 0   0   50  0001 C CNN "Description"
+F 5 "0603B102K160CT" H 0   0   50  0001 C CNN "PartNumber"
+F 6 "1292-1378-1-ND " H 0   0   50  0001 C CNN "digikey"
 	1    3400 6300
 	0    -1   1    0
@@
 F 4 "CC0603KPX7R7BB104" H 0   0   50  0001 C CNN "PartNumber"
 F 5 "311-1335-1-ND" H 0   0   50  0001 C CNN "digikey"
+F 6 "CAP CER 0.1UF 16V X7R 0603 " H 0   0   50  0001 C CNN "Description"
 	1    3850 8000
 	0    -1   1    0
@@
 P 3500 8900
 F 0 "C1502" V 3528 9010 20  0000 L CNN
-F 1 "100pF" V 3571 9010 20  0000 L CNN
+F 1 "1nF" V 3571 9010 20  0000 L CNN
 F 2 "servo:C_0603_1608Metric" H 3500 8800 60  0001 C CNN
 F 3 "" H 3500 8900 60  0000 C CNN
+F 4 "CAP CER 1000PF 16V X7R 0603 " H 0   0   50  0001 C CNN "Description"
+F 5 "0603B102K160CT" H 0   0   50  0001 C CNN "PartNumber"
+F 6 "1292-1378-1-ND " H 0   0   50  0001 C CNN "digikey"
 	1    3500 8900
 	0    -1   1    0
@@
 F 4 "CC0603KPX7R7BB104" H 0   0   50  0001 C CNN "PartNumber"
 F 5 "311-1335-1-ND" H 0   0   50  0001 C CNN "digikey"
+F 6 "CAP CER 0.1UF 16V X7R 0603 " H 0   0   50  0001 C CNN "Description"
 	1    8750 3450
 	0    1    1    0
@@
 P 8800 4350
 F 0 "C1513" V 8828 4460 20  0000 L CNN
-F 1 "100pF" V 8871 4460 20  0000 L CNN
+F 1 "1nF" V 8871 4460 20  0000 L CNN
 F 2 "servo:C_0603_1608Metric" H 8800 4250 60  0001 C CNN
 F 3 "" H 8800 4350 60  0000 C CNN
+F 4 "CAP CER 1000PF 16V X7R 0603 " H 0   0   50  0001 C CNN "Description"
+F 5 "0603B102K160CT" H 0   0   50  0001 C CNN "PartNumber"
+F 6 "1292-1378-1-ND " H 0   0   50  0001 C CNN "digikey"
 	1    8800 4350
 	0    1    1    0
@@
 F 4 "CC0603KPX7R7BB104" H 0   0   50  0001 C CNN "PartNumber"
 F 5 "311-1335-1-ND" H 0   0   50  0001 C CNN "digikey"
+F 6 "CAP CER 0.1UF 16V X7R 0603 " H 0   0   50  0001 C CNN "Description"
 	1    8750 5400
 	0    1    1    0
@@
 P 8800 6300
 F 0 "C1514" V 8828 6410 20  0000 L CNN
-F 1 "100pF" V 8871 6410 20  0000 L CNN
+F 1 "1nF" V 8871 6410 20  0000 L CNN
 F 2 "servo:C_0603_1608Metric" H 8800 6200 60  0001 C CNN
 F 3 "" H 8800 6300 60  0000 C CNN
+F 4 "CAP CER 1000PF 16V X7R 0603 " H 0   0   50  0001 C CNN "Description"
+F 5 "0603B102K160CT" H 0   0   50  0001 C CNN "PartNumber"
+F 6 "1292-1378-1-ND " H 0   0   50  0001 C CNN "digikey"
 	1    8800 6300
 	0    1    1    0
@@
 F 4 "CC0603KPX7R7BB104" H 0   0   50  0001 C CNN "PartNumber"
 F 5 "311-1335-1-ND" H 0   0   50  0001 C CNN "digikey"
+F 6 "CAP CER 0.1UF 16V X7R 0603 " H 0   0   50  0001 C CNN "Description"
 	1    8750 8000
 	0    1    1    0
@@
 P 8800 8900
 F 0 "C1515" V 8828 9010 20  0000 L CNN
-F 1 "100pF" V 8871 9010 20  0000 L CNN
+F 1 "1nF" V 8871 9010 20  0000 L CNN
 F 2 "servo:C_0603_1608Metric" H 8800 8800 60  0001 C CNN
 F 3 "" H 8800 8900 60  0000 C CNN
+F 4 "CAP CER 1000PF 16V X7R 0603 " H 0   0   50  0001 C CNN "Description"
+F 5 "0603B102K160CT" H 0   0   50  0001 C CNN "PartNumber"
+F 6 "1292-1378-1-ND " H 0   0   50  0001 C CNN "digikey"
 	1    8800 8900
 	0    1    1    0
@@
 P 5450 3700
 F 0 "J1503" V 5462 3880 39  0000 L CNN
-F 1 "tblock2x3" V 5537 3880 39  0000 L CNN
+F 1 "tblock 2x3 5.08" V 5537 3880 39  0000 L CNN
 F 2 "servo:tblock02x03" H 5400 3800 50  0001 C CNN
 F 3 "../doc/dfatasheets/tblock2rows.pdf" H 5500 3900 50  0001 C CNN
+F 4 "6 Position Terminal Block Header, Male Pins, Shrouded (4 Side) 0.200\" (5.08mm) 90°, Right Angle Through Hole " H 0   0   50  0001 C CNN "Description"
+F 5 "1762376 " H 0   0   50  0001 C CNN "PartNumber"
+F 6 " 277-1400-ND " H 0   0   50  0001 C CNN "digikey"
+F 7 "3.95500" H 0   0   50  0001 C CNN "price@10"
 	1    5450 3700
 	0    -1   -1   0
@@
 P 7250 3700
 F 0 "J1504" V 7262 3880 39  0000 L CNN
-F 1 "tblock2x3" V 7337 3880 39  0000 L CNN
+F 1 "tblock 2x3 5.08" V 7337 3880 39  0000 L CNN
 F 2 "servo:tblock02x03" H 7200 3800 50  0001 C CNN
 F 3 "../doc/dfatasheets/tblock2rows.pdf" H 7300 3900 50  0001 C CNN
+F 4 "6 Position Terminal Block Header, Male Pins, Shrouded (4 Side) 0.200\" (5.08mm) 90°, Right Angle Through Hole " H 0   0   50  0001 C CNN "Description"
+F 5 "1762376 " H 0   0   50  0001 C CNN "PartNumber"
+F 6 " 277-1400-ND " H 0   0   50  0001 C CNN "digikey"
+F 7 "3.95500" H 0   0   50  0001 C CNN "price@10"
 	1    7250 3700
 	0    1    -1   0
@@
 P 5250 5650
 F 0 "J1501" V 5338 5462 39  0000 R CNN
-F 1 "tblock2x3" V 5263 5462 39  0000 R CNN
+F 1 "tblock 2x3 5.08" V 5263 5462 39  0000 R CNN
 F 2 "servo:tblock02x03" H 5200 5750 50  0001 C CNN
 F 3 "../doc/dfatasheets/tblock2rows.pdf" H 5300 5850 50  0001 C CNN
+F 4 "6 Position Terminal Block Header, Male Pins, Shrouded (4 Side) 0.200\" (5.08mm) 90°, Right Angle Through Hole " H 0   0   50  0001 C CNN "Description"
+F 5 "1762376 " H 0   0   50  0001 C CNN "PartNumber"
+F 6 " 277-1400-ND " H 0   0   50  0001 C CNN "digikey"
+F 7 "3.95500" H 0   0   50  0001 C CNN "price@10"
 	1    5250 5650
 	0    -1   -1   0
@@
 P 7250 5650
 F 0 "J1505" V 7262 5830 39  0000 L CNN
-F 1 "tblock2x3" V 7337 5830 39  0000 L CNN
+F 1 "tblock 2x3 5.08" V 7337 5830 39  0000 L CNN
 F 2 "servo:tblock02x03" H 7200 5750 50  0001 C CNN
 F 3 "../doc/dfatasheets/tblock2rows.pdf" H 7300 5850 50  0001 C CNN
+F 4 "6 Position Terminal Block Header, Male Pins, Shrouded (4 Side) 0.200\" (5.08mm) 90°, Right Angle Through Hole " H 0   0   50  0001 C CNN "Description"
+F 5 "1762376 " H 0   0   50  0001 C CNN "PartNumber"
+F 6 " 277-1400-ND " H 0   0   50  0001 C CNN "digikey"
+F 7 "3.95500" H 0   0   50  0001 C CNN "price@10"
 	1    7250 5650
 	0    1    -1   0
@@
 P 5350 8250
 F 0 "J1502" V 5362 8430 39  0000 L CNN
-F 1 "tblock2x3" V 5437 8430 39  0000 L CNN
+F 1 "tblock 2x3 5.08" V 5437 8430 39  0000 L CNN
 F 2 "servo:tblock02x03" H 5300 8350 50  0001 C CNN
 F 3 "../doc/dfatasheets/tblock2rows.pdf" H 5400 8450 50  0001 C CNN
+F 4 "6 Position Terminal Block Header, Male Pins, Shrouded (4 Side) 0.200\" (5.08mm) 90°, Right Angle Through Hole " H 0   0   50  0001 C CNN "Description"
+F 5 "1762376 " H 0   0   50  0001 C CNN "PartNumber"
+F 6 " 277-1400-ND " H 0   0   50  0001 C CNN "digikey"
+F 7 "3.95500" H 0   0   50  0001 C CNN "price@10"
 	1    5350 8250
 	0    -1   -1   0
@@
 P 7250 8250
 F 0 "J1506" V 7262 8430 39  0000 L CNN
-F 1 "tblock2x3" V 7337 8430 39  0000 L CNN
+F 1 "tblock 2x3 5.08" V 7337 8430 39  0000 L CNN
 F 2 "servo:tblock02x03" H 7200 8350 50  0001 C CNN
 F 3 "../doc/datasheets/tblock2rows.pdf" H 7300 8450 50  0001 C CNN
+F 4 "6 Position Terminal Block Header, Male Pins, Shrouded (4 Side) 0.200\" (5.08mm) 90°, Right Angle Through Hole " H 0   0   50  0001 C CNN "Description"
+F 5 "1762376 " H 0   0   50  0001 C CNN "PartNumber"
+F 6 " 277-1400-ND " H 0   0   50  0001 C CNN "digikey"
+F 7 "3.95500" H 0   0   50  0001 C CNN "price@10"
 	1    7250 8250
 	0    1    -1   0
