File: kicad/symbols.sch (KiCad schematic (older format))
At the start: 70 parts

Commit message: bom bom bom...
Parts:
- H1309, H1310, H1311, H1312, H1313, H1314, H1315, H1316, H1317, H1318, H1319, H1320, H1321, H1322, H1323, H1324, H1325, H1326, H1327, H1328, H1329, H1330, H1331, H1332, H1333, H1334, H1335, H1336, H1337, H1338, H1339, H1340, H1341, H1342, H1343, H1344, H1357, H1358: footprint servo:slot2 -> servo:slot
Changed lines of the file:
@@
 F 0 "H1309" H 4350 4596 50  0000 L CNN
 F 1 "Slot" H 4350 4505 50  0000 L CNN
-F 2 "servo:slot2" H 4250 4550 50  0001 C CNN
+F 2 "servo:slot" H 4250 4550 50  0001 C CNN
 F 3 "~" H 4250 4550 50  0001 C CNN
 	1    4250 4550
@@
 F 0 "H1310" H 4750 4596 50  0000 L CNN
 F 1 "Slot" H 4750 4505 50  0000 L CNN
-F 2 "servo:slot2" H 4650 4550 50  0001 C CNN
+F 2 "servo:slot" H 4650 4550 50  0001 C CNN
 F 3 "~" H 4650 4550 50  0001 C CNN
 	1    4650 4550
@@
 F 0 "H1311" H 5150 4596 50  0000 L CNN
 F 1 "Slot" H 5150 4505 50  0000 L CNN
-F 2 "servo:slot2" H 5050 4550 50  0001 C CNN
+F 2 "servo:slot" H 5050 4550 50  0001 C CNN
 F 3 "~" H 5050 4550 50  0001 C CNN
 	1    5050 4550
@@
 F 0 "H1312" H 5550 4596 50  0000 L CNN
 F 1 "Slot" H 5550 4505 50  0000 L CNN
-F 2 "servo:slot2" H 5450 4550 50  0001 C CNN
+F 2 "servo:slot" H 5450 4550 50  0001 C CNN
 F 3 "~" H 5450 4550 50  0001 C CNN
 	1    5450 4550
@@
 F 0 "H1313" H 4350 4946 50  0000 L CNN
 F 1 "Slot" H 4350 4855 50  0000 L CNN
-F 2 "servo:slot2" H 4250 4900 50  0001 C CNN
+F 2 "servo:slot" H 4250 4900 50  0001 C CNN
 F 3 "~" H 4250 4900 50  0001 C CNN
 	1    4250 4900
@@
 F 0 "H1319" H 4750 4946 50  0000 L CNN
 F 1 "Slot" H 4750 4855 50  0000 L CNN
-F 2 "servo:slot2" H 4650 4900 50  0001 C CNN
+F 2 "servo:slot" H 4650 4900 50  0001 C CNN
 F 3 "~" H 4650 4900 50  0001 C CNN
 	1    4650 4900
@@
 F 0 "H1325" H 5150 4946 50  0000 L CNN
 F 1 "Slot" H 5150 4855 50  0000 L CNN
-F 2 "servo:slot2" H 5050 4900 50  0001 C CNN
+F 2 "servo:slot" H 5050 4900 50  0001 C CNN
 F 3 "~" H 5050 4900 50  0001 C CNN
 	1    5050 4900
@@
 F 0 "H1331" H 5550 4946 50  0000 L CNN
 F 1 "Slot" H 5550 4855 50  0000 L CNN
-F 2 "servo:slot2" H 5450 4900 50  0001 C CNN
+F 2 "servo:slot" H 5450 4900 50  0001 C CNN
 F 3 "~" H 5450 4900 50  0001 C CNN
 	1    5450 4900
@@
 F 0 "H1314" H 4350 5246 50  0000 L CNN
 F 1 "Slot" H 4350 5155 50  0000 L CNN
-F 2 "servo:slot2" H 4250 5200 50  0001 C CNN
+F 2 "servo:slot" H 4250 5200 50  0001 C CNN
 F 3 "~" H 4250 5200 50  0001 C CNN
 	1    4250 5200
@@
 F 0 "H1320" H 4750 5246 50  0000 L CNN
 F 1 "Slot" H 4750 5155 50  0000 L CNN
-F 2 "servo:slot2" H 4650 5200 50  0001 C CNN
+F 2 "servo:slot" H 4650 5200 50  0001 C CNN
 F 3 "~" H 4650 5200 50  0001 C CNN
 	1    4650 5200
@@
 F 0 "H1326" H 5150 5246 50  0000 L CNN
 F 1 "Slot" H 5150 5155 50  0000 L CNN
-F 2 "servo:slot2" H 5050 5200 50  0001 C CNN
+F 2 "servo:slot" H 5050 5200 50  0001 C CNN
 F 3 "~" H 5050 5200 50  0001 C CNN
 	1    5050 5200
@@
 F 0 "H1332" H 5550 5246 50  0000 L CNN
 F 1 "Slot" H 5550 5155 50  0000 L CNN
-F 2 "servo:slot2" H 5450 5200 50  0001 C CNN
+F 2 "servo:slot" H 5450 5200 50  0001 C CNN
 F 3 "~" H 5450 5200 50  0001 C CNN
 	1    5450 5200
@@
 F 0 "H1315" H 4350 5596 50  0000 L CNN
 F 1 "Slot" H 4350 5505 50  0000 L CNN
-F 2 "servo:slot2" H 4250 5550 50  0001 C CNN
+F 2 "servo:slot" H 4250 5550 50  0001 C CNN
 F 3 "~" H 4250 5550 50  0001 C CNN
 	1    4250 5550
@@
 F 0 "H1321" H 4750 5596 50  0000 L CNN
 F 1 "Slot" H 4750 5505 50  0000 L CNN
-F 2 "servo:slot2" H 4650 5550 50  0001 C CNN
+F 2 "servo:slot" H 4650 5550 50  0001 C CNN
 F 3 "~" H 4650 5550 50  0001 C CNN
 	1    4650 5550
@@
 F 0 "H1327" H 5150 5596 50  0000 L CNN
 F 1 "Slot" H 5150 5505 50  0000 L CNN
-F 2 "servo:slot2" H 5050 5550 50  0001 C CNN
+F 2 "servo:slot" H 5050 5550 50  0001 C CNN
 F 3 "~" H 5050 5550 50  0001 C CNN
 	1    5050 5550
@@
 F 0 "H1333" H 5550 5596 50  0000 L CNN
 F 1 "Slot" H 5550 5505 50  0000 L CNN
-F 2 "servo:slot2" H 5450 5550 50  0001 C CNN
+F 2 "servo:slot" H 5450 5550 50  0001 C CNN
 F 3 "~" H 5450 5550 50  0001 C CNN
 	1    5450 5550
@@
 F 0 "H1316" H 4350 5946 50  0000 L CNN
 F 1 "Slot" H 4350 5855 50  0000 L CNN
-F 2 "servo:slot2" H 4250 5900 50  0001 C CNN
+F 2 "servo:slot" H 4250 5900 50  0001 C CNN
 F 3 "~" H 4250 5900 50  0001 C CNN
 	1    4250 5900
@@
 F 0 "H1322" H 4750 5946 50  0000 L CNN
 F 1 "Slot" H 4750 5855 50  0000 L CNN
-F 2 "servo:slot2" H 4650 5900 50  0001 C CNN
+F 2 "servo:slot" H 4650 5900 50  0001 C CNN
 F 3 "~" H 4650 5900 50  0001 C CNN
 	1    4650 5900
@@
 F 0 "H1328" H 5150 5946 50  0000 L CNN
 F 1 "Slot" H 5150 5855 50  0000 L CNN
-F 2 "servo:slot2" H 5050 5900 50  0001 C CNN
+F 2 "servo:slot" H 5050 5900 50  0001 C CNN
 F 3 "~" H 5050 5900 50  0001 C CNN
 	1    5050 5900
@@
 F 0 "H1334" H 5550 5946 50  0000 L CNN
 F 1 "Slot" H 5550 5855 50  0000 L CNN
-F 2 "servo:slot2" H 5450 5900 50  0001 C CNN
+F 2 "servo:slot" H 5450 5900 50  0001 C CNN
 F 3 "~" H 5450 5900 50  0001 C CNN
 	1    5450 5900
@@
 F 0 "H1317" H 4350 6246 50  0000 L CNN
 F 1 "Slot" H 4350 6155 50  0000 L CNN
-F 2 "servo:slot2" H 4250 6200 50  0001 C CNN
+F 2 "servo:slot" H 4250 6200 50  0001 C CNN
 F 3 "~" H 4250 6200 50  0001 C CNN
 	1    4250 6200
@@
 F 0 "H1323" H 4750 6246 50  0000 L CNN
 F 1 "Slot" H 4750 6155 50  0000 L CNN
-F 2 "servo:slot2" H 4650 6200 50  0001 C CNN
+F 2 "servo:slot" H 4650 6200 50  0001 C CNN
 F 3 "~" H 4650 6200 50  0001 C CNN
 	1    4650 6200
@@
 F 0 "H1329" H 5150 6246 50  0000 L CNN
 F 1 "Slot" H 5150 6155 50  0000 L CNN
-F 2 "servo:slot2" H 5050 6200 50  0001 C CNN
+F 2 "servo:slot" H 5050 6200 50  0001 C CNN
 F 3 "~" H 5050 6200 50  0001 C CNN
 	1    5050 6200
@@
 F 0 "H1335" H 5550 6246 50  0000 L CNN
 F 1 "Slot" H 5550 6155 50  0000 L CNN
-F 2 "servo:slot2" H 5450 6200 50  0001 C CNN
+F 2 "servo:slot" H 5450 6200 50  0001 C CNN
 F 3 "~" H 5450 6200 50  0001 C CNN
 	1    5450 6200
@@
 F 0 "H1318" H 4350 6596 50  0000 L CNN
 F 1 "Slot" H 4350 6505 50  0000 L CNN
-F 2 "servo:slot2" H 4250 6550 50  0001 C CNN
+F 2 "servo:slot" H 4250 6550 50  0001 C CNN
 F 3 "~" H 4250 6550 50  0001 C CNN
 	1    4250 6550
@@
 F 0 "H1324" H 4750 6596 50  0000 L CNN
 F 1 "Slot" H 4750 6505 50  0000 L CNN
-F 2 "servo:slot2" H 4650 6550 50  0001 C CNN
+F 2 "servo:slot" H 4650 6550 50  0001 C CNN
 F 3 "~" H 4650 6550 50  0001 C CNN
 	1    4650 6550
@@
 F 0 "H1330" H 5150 6596 50  0000 L CNN
 F 1 "Slot" H 5150 6505 50  0000 L CNN
-F 2 "servo:slot2" H 5050 6550 50  0001 C CNN
+F 2 "servo:slot" H 5050 6550 50  0001 C CNN
 F 3 "~" H 5050 6550 50  0001 C CNN
 	1    5050 6550
@@
 F 0 "H1336" H 5550 6596 50  0000 L CNN
 F 1 "Slot" H 5550 6505 50  0000 L CNN
-F 2 "servo:slot2" H 5450 6550 50  0001 C CNN
+F 2 "servo:slot" H 5450 6550 50  0001 C CNN
 F 3 "~" H 5450 6550 50  0001 C CNN
 	1    5450 6550
@@
 F 0 "H1337" H 4350 6946 50  0000 L CNN
 F 1 "Slot" H 4350 6855 50  0000 L CNN
-F 2 "servo:slot2" H 4250 6900 50  0001 C CNN
+F 2 "servo:slot" H 4250 6900 50  0001 C CNN
 F 3 "~" H 4250 6900 50  0001 C CNN
 	1    4250 6900
@@
 F 0 "H1339" H 4750 6946 50  0000 L CNN
 F 1 "Slot" H 4750 6855 50  0000 L CNN
-F 2 "servo:slot2" H 4650 6900 50  0001 C CNN
+F 2 "servo:slot" H 4650 6900 50  0001 C CNN
 F 3 "~" H 4650 6900 50  0001 C CNN
 	1    4650 6900
@@
 F 0 "H1341" H 5150 6946 50  0000 L CNN
 F 1 "Slot" H 5150 6855 50  0000 L CNN
-F 2 "servo:slot2" H 5050 6900 50  0001 C CNN
+F 2 "servo:slot" H 5050 6900 50  0001 C CNN
 F 3 "~" H 5050 6900 50  0001 C CNN
 	1    5050 6900
@@
 F 0 "H1343" H 5550 6946 50  0000 L CNN
 F 1 "Slot" H 5550 6855 50  0000 L CNN
-F 2 "servo:slot2" H 5450 6900 50  0001 C CNN
+F 2 "servo:slot" H 5450 6900 50  0001 C CNN
 F 3 "~" H 5450 6900 50  0001 C CNN
 	1    5450 6900
@@
 F 0 "H1338" H 4350 7346 50  0000 L CNN
 F 1 "Slot" H 4350 7255 50  0000 L CNN
-F 2 "servo:slot2" H 4250 7300 50  0001 C CNN
+F 2 "servo:slot" H 4250 7300 50  0001 C CNN
 F 3 "~" H 4250 7300 50  0001 C CNN
 	1    4250 7300
@@
 F 0 "H1340" H 4750 7346 50  0000 L CNN
 F 1 "Slot" H 4750 7255 50  0000 L CNN
-F 2 "servo:slot2" H 4650 7300 50  0001 C CNN
+F 2 "servo:slot" H 4650 7300 50  0001 C CNN
 F 3 "~" H 4650 7300 50  0001 C CNN
 	1    4650 7300
@@
 F 0 "H1342" H 5150 7346 50  0000 L CNN
 F 1 "Slot" H 5150 7255 50  0000 L CNN
-F 2 "servo:slot2" H 5050 7300 50  0001 C CNN
+F 2 "servo:slot" H 5050 7300 50  0001 C CNN
 F 3 "~" H 5050 7300 50  0001 C CNN
 	1    5050 7300
@@
 F 0 "H1344" H 5550 7346 50  0000 L CNN
 F 1 "Slot" H 5550 7255 50  0000 L CNN
-F 2 "servo:slot2" H 5450 7300 50  0001 C CNN
+F 2 "servo:slot" H 5450 7300 50  0001 C CNN
 F 3 "~" H 5450 7300 50  0001 C CNN
 	1    5450 7300
@@
 F 0 "H1357" H 5550 7646 50  0000 L CNN
 F 1 "Slot" H 5550 7555 50  0000 L CNN
-F 2 "servo:slot2" H 5450 7600 50  0001 C CNN
+F 2 "servo:slot" H 5450 7600 50  0001 C CNN
 F 3 "~" H 5450 7600 50  0001 C CNN
 	1    5450 7600
@@
 F 0 "H1358" H 5150 7646 50  0000 L CNN
 F 1 "Slot" H 5150 7555 50  0000 L CNN
-F 2 "servo:slot2" H 5050 7600 50  0001 C CNN
+F 2 "servo:slot" H 5050 7600 50  0001 C CNN
 F 3 "~" H 5050 7600 50  0001 C CNN
 	1    5050 7600

Commit message: more bom...
Parts:
- H1301, H1302, H1303, H1304, H1305, H1306, H1307, H1308: Description (none) -> fiducials
- H1309, H1310, H1311, H1312, H1313, H1314, H1315, H1316, H1317, H1318, H1319, H1320, H1321, H1322, H1323, H1324, H1325, H1326, H1327, H1328, H1329, H1330, H1331, H1332, H1333, H1334, H1335, H1336, H1337, H1338, H1339, H1340, H1341, H1342, H1343, H1344, H1345, H1346, H1347, H1348, H1349, H1350, H1351, H1352, H1353, H1354, H1355, H1356, H1357, H1358: Description (none) -> slots for isolation
- LOGO1301: Description (none) -> logo open hard; PartNumber (none) -> -; price@10 (none) -> 0
- N1301: Description (none) -> case housing; PartNumber (none) -> -; price@10 (none) -> 0
- logo1301: Description (none) -> logo nanocut; PartNumber (none) -> -; price@10 (none) -> 0
- logo1302: Description (none) -> logo pslavkin; PartNumber (none) -> -; price@10 (none) -> 0
- logo1303: Description (none) -> logo recycler; PartNumber (none) -> -; price@10 (none) -> 0
- logo1304: Description (none) -> logo gnu; PartNumber (none) -> -; price@10 (none) -> 0
- logo1305: Description (none) -> ,logo neurona; PartNumber (none) -> -; price@10 (none) -> 0
- ref1301: Description (none) -> logo kicad; PartNumber (none) -> -; price@10 (none) -> 0
- ref1302, ref1303, ref1304, ref1305: Description (none) -> logo high voltage; PartNumber (none) -> -; price@10 (none) -> 0
