File: kicad/vbus_meas.sch (KiCad schematic (older format))
At the start: 36 parts, among them U1601 AMC1311B, U1602 AMC1311B, U1603 RFM-0505S, U1604 RFM-0505S

Commit message: serigrafia...
Parts:
- L1601, L1602, L1603, L1604: footprint Inductor_SMD:L_1206_3216Metric_Pad1.42x1.75mm_HandSolder -> servo:L_1206_3216Metric_Pad1.42x1.75mm_HandSolder
- R1601, R1602, R1603, R1604, R1605, R1606, R1607, R1608, R1609, R1610: footprint Resistor_SMD:R_0603_1608Metric -> servo:R_0603_1608Metric
- R1611, R1612, R1613, R1614, R1615, R1616, R1617, R1618: footprint Resistor_SMD:R_1206_3216Metric_Pad1.42x1.75mm_HandSolder -> servo:R_1206_3216Metric_Pad1.42x1.75mm_HandSolder
- U1601, U1602: footprint Package_SO:SSO-8_6.8x5.9mm_P1.27mm_Clearance8mm -> servo:SSO-8_6.8x5.9mm_P1.27mm_Clearance8mm
Changed lines of the file:
@@
 F 0 "U1601" H 7250 3317 50  0000 C CNN
 F 1 "AMC1311B" H 7250 3226 50  0000 C CNN
-F 2 "Package_SO:SSO-8_6.8x5.9mm_P1.27mm_Clearance8mm" H 7300 1950 50  0001 C CIN
+F 2 "servo:SSO-8_6.8x5.9mm_P1.27mm_Clearance8mm" H 7300 1950 50  0001 C CIN
 F 3 "../doc/datasheets/amc1311.pdf" H 7200 2450 50  0001 C CNN
 	1    7250 2950
@@
 F 0 "R1607" V 8778 3150 20  0000 L CNN
 F 1 "1k" V 8821 3150 20  0000 L CNN
-F 2 "Resistor_SMD:R_0603_1608Metric" H 8300 3000 60  0001 C CNN
+F 2 "servo:R_0603_1608Metric" H 8300 3000 60  0001 C CNN
 F 3 "" H 8400 3100 60  0001 C CNN
 	1    8800 3100
@@
 F 0 "R1611" H 9100 3415 20  0000 C CNN
 F 1 "1M" H 9100 3372 20  0000 C CNN
-F 2 "Resistor_SMD:R_1206_3216Metric_Pad1.42x1.75mm_HandSolder" H 8600 3200 60  0001 C CNN
+F 2 "servo:R_1206_3216Metric_Pad1.42x1.75mm_HandSolder" H 8600 3200 60  0001 C CNN
 F 3 "" H 8700 3300 60  0001 C CNN
 	1    9100 3300
@@
 F 0 "R1608" V 8778 3800 20  0000 L CNN
 F 1 "1k" V 8821 3800 20  0000 L CNN
-F 2 "Resistor_SMD:R_0603_1608Metric" H 8300 3650 60  0001 C CNN
+F 2 "servo:R_0603_1608Metric" H 8300 3650 60  0001 C CNN
 F 3 "" H 8400 3750 60  0001 C CNN
 	1    8800 3750
@@
 F 0 "R1605" H 8500 3415 20  0000 C CNN
 F 1 "12e" H 8500 3372 20  0000 C CNN
-F 2 "Resistor_SMD:R_0603_1608Metric" H 8000 3200 60  0001 C CNN
+F 2 "servo:R_0603_1608Metric" H 8000 3200 60  0001 C CNN
 F 3 "" H 8100 3300 60  0001 C CNN
 	1    8500 3300
@@
 F 0 "L1601" V 8594 2500 20  0000 C CNN
 F 1 "L_Small" V 8637 2500 20  0000 C CNN
-F 2 "Inductor_SMD:L_1206_3216Metric_Pad1.42x1.75mm_HandSolder" H 8630 2440 50  0001 C CNN
+F 2 "servo:L_1206_3216Metric_Pad1.42x1.75mm_HandSolder" H 8630 2440 50  0001 C CNN
 F 3 "~" H 8730 2540 50  0001 C CNN
 	1    8700 2500
@@
 F 0 "L1603" H 10398 2222 20  0000 L CNN
 F 1 "L_Small" H 10398 2179 20  0000 L CNN
-F 2 "Inductor_SMD:L_1206_3216Metric_Pad1.42x1.75mm_HandSolder" H 10280 2140 50  0001 C CNN
+F 2 "servo:L_1206_3216Metric_Pad1.42x1.75mm_HandSolder" H 10280 2140 50  0001 C CNN
 F 3 "~" H 10380 2240 50  0001 C CNN
 	1    10350 2200
@@
 F 0 "R1601" H 5900 2965 20  0000 C CNN
 F 1 "12e" H 5900 2922 20  0000 C CNN
-F 2 "Resistor_SMD:R_0603_1608Metric" H 5400 2750 60  0001 C CNN
+F 2 "servo:R_0603_1608Metric" H 5400 2750 60  0001 C CNN
 F 3 "" H 5500 2850 60  0001 C CNN
 	1    5900 2850
@@
 F 0 "R1602" H 5900 3365 20  0000 C CNN
 F 1 "12e" H 5900 3322 20  0000 C CNN
-F 2 "Resistor_SMD:R_0603_1608Metric" H 5400 3150 60  0001 C CNN
+F 2 "servo:R_0603_1608Metric" H 5400 3150 60  0001 C CNN
 F 3 "" H 5500 3250 60  0001 C CNN
 	1    5900 3250
@@
 F 0 "U1602" H 7350 5617 50  0000 C CNN
 F 1 "AMC1311B" H 7350 5526 50  0000 C CNN
-F 2 "Package_SO:SSO-8_6.8x5.9mm_P1.27mm_Clearance8mm" H 7400 4250 50  0001 C CIN
+F 2 "servo:SSO-8_6.8x5.9mm_P1.27mm_Clearance8mm" H 7400 4250 50  0001 C CIN
 F 3 "../doc/datasheets/amc1311.pdf" H 7300 4750 50  0001 C CNN
 	1    7350 5250
@@
 F 0 "R1609" V 8878 5450 20  0000 L CNN
 F 1 "1k" V 8921 5450 20  0000 L CNN
-F 2 "Resistor_SMD:R_0603_1608Metric" H 8400 5300 60  0001 C CNN
+F 2 "servo:R_0603_1608Metric" H 8400 5300 60  0001 C CNN
 F 3 "" H 8500 5400 60  0001 C CNN
 	1    8900 5400
@@
 F 0 "R1610" V 8878 6100 20  0000 L CNN
 F 1 "1k" V 8921 6100 20  0000 L CNN
-F 2 "Resistor_SMD:R_0603_1608Metric" H 8400 5950 60  0001 C CNN
+F 2 "servo:R_0603_1608Metric" H 8400 5950 60  0001 C CNN
 F 3 "" H 8500 6050 60  0001 C CNN
 	1    8900 6050
@@
 F 0 "R1606" H 8600 5715 20  0000 C CNN
 F 1 "12e" H 8600 5672 20  0000 C CNN
-F 2 "Resistor_SMD:R_0603_1608Metric" H 8100 5500 60  0001 C CNN
+F 2 "servo:R_0603_1608Metric" H 8100 5500 60  0001 C CNN
 F 3 "" H 8200 5600 60  0001 C CNN
 	1    8600 5600
@@
 F 0 "L1602" V 8694 4800 20  0000 C CNN
 F 1 "L_Small" V 8737 4800 20  0000 C CNN
-F 2 "Inductor_SMD:L_1206_3216Metric_Pad1.42x1.75mm_HandSolder" H 8730 4740 50  0001 C CNN
+F 2 "servo:L_1206_3216Metric_Pad1.42x1.75mm_HandSolder" H 8730 4740 50  0001 C CNN
 F 3 "~" H 8830 4840 50  0001 C CNN
 	1    8800 4800
@@
 F 0 "L1604" H 10498 4522 20  0000 L CNN
 F 1 "L_Small" H 10498 4479 20  0000 L CNN
-F 2 "Inductor_SMD:L_1206_3216Metric_Pad1.42x1.75mm_HandSolder" H 10380 4440 50  0001 C CNN
+F 2 "servo:L_1206_3216Metric_Pad1.42x1.75mm_HandSolder" H 10380 4440 50  0001 C CNN
 F 3 "~" H 10480 4540 50  0001 C CNN
 	1    10450 4500
@@
 F 0 "R1603" H 6000 5265 20  0000 C CNN
 F 1 "12e" H 6000 5222 20  0000 C CNN
-F 2 "Resistor_SMD:R_0603_1608Metric" H 5500 5050 60  0001 C CNN
+F 2 "servo:R_0603_1608Metric" H 5500 5050 60  0001 C CNN
 F 3 "" H 5600 5150 60  0001 C CNN
 	1    6000 5150
@@
 F 0 "R1604" H 6000 5665 20  0000 C CNN
 F 1 "12e" H 6000 5622 20  0000 C CNN
-F 2 "Resistor_SMD:R_0603_1608Metric" H 5500 5450 60  0001 C CNN
+F 2 "servo:R_0603_1608Metric" H 5500 5450 60  0001 C CNN
 F 3 "" H 5600 5550 60  0001 C CNN
 	1    6000 5550
@@
 F 0 "R1613" H 9500 3415 20  0000 C CNN
 F 1 "1M" H 9500 3372 20  0000 C CNN
-F 2 "Resistor_SMD:R_1206_3216Metric_Pad1.42x1.75mm_HandSolder" H 9000 3200 60  0001 C CNN
+F 2 "servo:R_1206_3216Metric_Pad1.42x1.75mm_HandSolder" H 9000 3200 60  0001 C CNN
 F 3 "" H 9100 3300 60  0001 C CNN
 	1    9500 3300
@@
 F 0 "R1612" H 9100 3565 20  0000 C CNN
 F 1 "1M" H 9100 3522 20  0000 C CNN
-F 2 "Resistor_SMD:R_1206_3216Metric_Pad1.42x1.75mm_HandSolder" H 8600 3350 60  0001 C CNN
+F 2 "servo:R_1206_3216Metric_Pad1.42x1.75mm_HandSolder" H 8600 3350 60  0001 C CNN
 F 3 "" H 8700 3450 60  0001 C CNN
 	1    9100 3450
@@
 F 0 "R1616" H 9500 3565 20  0000 C CNN
 F 1 "1M" H 9500 3522 20  0000 C CNN
-F 2 "Resistor_SMD:R_1206_3216Metric_Pad1.42x1.75mm_HandSolder" H 9000 3350 60  0001 C CNN
+F 2 "servo:R_1206_3216Metric_Pad1.42x1.75mm_HandSolder" H 9000 3350 60  0001 C CNN
 F 3 "" H 9100 3450 60  0001 C CNN
 	1    9500 3450
@@
 F 0 "R1614" H 9200 5715 20  0000 C CNN
 F 1 "1M" H 9200 5672 20  0000 C CNN
-F 2 "Resistor_SMD:R_1206_3216Metric_Pad1.42x1.75mm_HandSolder" H 8700 5500 60  0001 C CNN
+F 2 "servo:R_1206_3216Metric_Pad1.42x1.75mm_HandSolder" H 8700 5500 60  0001 C CNN
 F 3 "" H 8800 5600 60  0001 C CNN
 	1    9200 5600
@@
 F 0 "R1617" H 9600 5715 20  0000 C CNN
 F 1 "1M" H 9600 5672 20  0000 C CNN
-F 2 "Resistor_SMD:R_1206_3216Metric_Pad1.42x1.75mm_HandSolder" H 9100 5500 60  0001 C CNN
+F 2 "servo:R_1206_3216Metric_Pad1.42x1.75mm_HandSolder" H 9100 5500 60  0001 C CNN
 F 3 "" H 9200 5600 60  0001 C CNN
 	1    9600 5600
@@
 F 0 "R1615" H 9200 5865 20  0000 C CNN
 F 1 "1M" H 9200 5822 20  0000 C CNN
-F 2 "Resistor_SMD:R_1206_3216Metric_Pad1.42x1.75mm_HandSolder" H 8700 5650 60  0001 C CNN
+F 2 "servo:R_1206_3216Metric_Pad1.42x1.75mm_HandSolder" H 8700 5650 60  0001 C CNN
 F 3 "" H 8800 5750 60  0001 C CNN
 	1    9200 5750
@@
 F 0 "R1618" H 9600 5865 20  0000 C CNN
 F 1 "1M" H 9600 5822 20  0000 C CNN
-F 2 "Resistor_SMD:R_1206_3216Metric_Pad1.42x1.75mm_HandSolder" H 9100 5650 60  0001 C CNN
+F 2 "servo:R_1206_3216Metric_Pad1.42x1.75mm_HandSolder" H 9100 5650 60  0001 C CNN
 F 3 "" H 9200 5750 60  0001 C CNN
 	1    9600 5750

Commit message: serigraphi, improve of nets. change of soic 8 footprint
Parts:
- U1601, U1602: footprint servo:SSO-8_6.8x5.9mm_P1.27mm_Clearance8mm -> servo:SSO-8_7.6x5.9mm_P1.27mm_Clearance9.1mm
Changed lines of the file:
@@
 F 0 "U1601" H 7250 3317 50  0000 C CNN
 F 1 "AMC1311B" H 7250 3226 50  0000 C CNN
-F 2 "servo:SSO-8_6.8x5.9mm_P1.27mm_Clearance8mm" H 7300 1950 50  0001 C CIN
+F 2 "servo:SSO-8_7.6x5.9mm_P1.27mm_Clearance9.1mm" H 7300 1950 50  0001 C CIN
 F 3 "../doc/datasheets/amc1311.pdf" H 7200 2450 50  0001 C CNN
 	1    7250 2950
@@
 F 0 "U1602" H 7350 5617 50  0000 C CNN
 F 1 "AMC1311B" H 7350 5526 50  0000 C CNN
-F 2 "servo:SSO-8_6.8x5.9mm_P1.27mm_Clearance8mm" H 7400 4250 50  0001 C CIN
+F 2 "servo:SSO-8_7.6x5.9mm_P1.27mm_Clearance9.1mm" H 7400 4250 50  0001 C CIN
 F 3 "../doc/datasheets/amc1311.pdf" H 7300 4750 50  0001 C CNN
 	1    7350 5250

Commit message: bom bom bom...
Parts:
- C1601, C1602, C1603, C1604, C1607, C1608, C1609, C1610: value 100nF -> 0.1uF; PartNumber (none) -> CC0603KPX7R7BB104; digikey (none) -> 311-1335-1-ND
Changed lines of the file:
@@
 AR Path="/5DE49152/5E1AD37E" Ref="C?"  Part="1"
 F 0 "C1607" V 8478 2710 20  0000 L CNN
-F 1 "100nF" V 8521 2710 20  0000 L CNN
+F 1 "0.1uF" V 8521 2710 20  0000 L CNN
 F 2 "servo:C_0603_1608Metric" H 8450 2500 60  0001 C CNN
 F 3 "" H 8450 2600 60  0000 C CNN
+F 4 "CC0603KPX7R7BB104" H 0   0   50  0001 C CNN "PartNumber"
+F 5 "311-1335-1-ND" H 0   0   50  0001 C CNN "digikey"
 	1    8450 2600
 	0    1    1    0
@@
 AR Path="/5DE49152/5E1AD39C" Ref="C?"  Part="1"
 F 0 "C1603" V 6528 2860 20  0000 L CNN
-F 1 "100nF" V 6571 2860 20  0000 L CNN
+F 1 "0.1uF" V 6571 2860 20  0000 L CNN
 F 2 "servo:C_0603_1608Metric" H 6500 2650 60  0001 C CNN
 F 3 "" H 6500 2750 60  0000 C CNN
+F 4 "CC0603KPX7R7BB104" H 0   0   50  0001 C CNN "PartNumber"
+F 5 "311-1335-1-ND" H 0   0   50  0001 C CNN "digikey"
 	1    6500 2750
 	0    1    1    0
@@
 AR Path="/5DE49152/5E1AD366" Ref="C?"  Part="1"
 F 0 "C1609" V 10378 2560 20  0000 L CNN
-F 1 "100nF" V 10421 2560 20  0000 L CNN
+F 1 "0.1uF" V 10421 2560 20  0000 L CNN
 F 2 "servo:C_0603_1608Metric" H 10350 2350 60  0001 C CNN
 F 3 "" H 10350 2450 60  0000 C CNN
+F 4 "CC0603KPX7R7BB104" H 0   0   50  0001 C CNN "PartNumber"
+F 5 "311-1335-1-ND" H 0   0   50  0001 C CNN "digikey"
 	1    10350 2450
 	0    1    1    0
@@
 AR Path="/5DE49152/5E19AFC3" Ref="C?"  Part="1"
 F 0 "C1601" V 5628 3110 20  0000 L CNN
-F 1 "100nF" V 5671 3110 20  0000 L CNN
+F 1 "0.1uF" V 5671 3110 20  0000 L CNN
 F 2 "servo:C_0603_1608Metric" H 5600 2900 60  0001 C CNN
 F 3 "" H 5600 3000 60  0000 C CNN
+F 4 "CC0603KPX7R7BB104" H 0   0   50  0001 C CNN "PartNumber"
+F 5 "311-1335-1-ND" H 0   0   50  0001 C CNN "digikey"
 	1    5600 3000
 	0    1    1    0
@@
 AR Path="/5DE49152/5E1B9A69" Ref="C?"  Part="1"
 F 0 "C1608" V 8578 5010 20  0000 L CNN
-F 1 "100nF" V 8621 5010 20  0000 L CNN
+F 1 "0.1uF" V 8621 5010 20  0000 L CNN
 F 2 "servo:C_0603_1608Metric" H 8550 4800 60  0001 C CNN
 F 3 "" H 8550 4900 60  0000 C CNN
+F 4 "CC0603KPX7R7BB104" H 0   0   50  0001 C CNN "PartNumber"
+F 5 "311-1335-1-ND" H 0   0   50  0001 C CNN "digikey"
 	1    8550 4900
 	0    1    1    0
@@
 AR Path="/5DE49152/5E1B9A7E" Ref="C?"  Part="1"
 F 0 "C1604" V 6628 5160 20  0000 L CNN
-F 1 "100nF" V 6671 5160 20  0000 L CNN
+F 1 "0.1uF" V 6671 5160 20  0000 L CNN
 F 2 "servo:C_0603_1608Metric" H 6600 4950 60  0001 C CNN
 F 3 "" H 6600 5050 60  0000 C CNN
+F 4 "CC0603KPX7R7BB104" H 0   0   50  0001 C CNN "PartNumber"
+F 5 "311-1335-1-ND" H 0   0   50  0001 C CNN "digikey"
 	1    6600 5050
 	0    1    1    0
@@
 AR Path="/5DE49152/5E1B9B0D" Ref="C?"  Part="1"
 F 0 "C1610" V 10478 4860 20  0000 L CNN
-F 1 "100nF" V 10521 4860 20  0000 L CNN
+F 1 "0.1uF" V 10521 4860 20  0000 L CNN
 F 2 "servo:C_0603_1608Metric" H 10450 4650 60  0001 C CNN
 F 3 "" H 10450 4750 60  0000 C CNN
+F 4 "CC0603KPX7R7BB104" H 0   0   50  0001 C CNN "PartNumber"
+F 5 "311-1335-1-ND" H 0   0   50  0001 C CNN "digikey"
 	1    10450 4750
 	0    1    1    0
@@
 AR Path="/5DE49152/5E1B9B2E" Ref="C?"  Part="1"
 F 0 "C1602" V 5728 5410 20  0000 L CNN
-F 1 "100nF" V 5771 5410 20  0000 L CNN
+F 1 "0.1uF" V 5771 5410 20  0000 L CNN
 F 2 "servo:C_0603_1608Metric" H 5700 5200 60  0001 C CNN
 F 3 "" H 5700 5300 60  0000 C CNN
+F 4 "CC0603KPX7R7BB104" H 0   0   50  0001 C CNN "PartNumber"
+F 5 "311-1335-1-ND" H 0   0   50  0001 C CNN "digikey"
 	1    5700 5300
 	0    1    1    0

Commit message: more bom...
Parts:
- C1601, C1602, C1603, C1604, C1607, C1608, C1609, C1610: Description (none) -> CAP CER 0.1UF 16V X7R 0603
- C1605, C1606: value 330p -> 0.1uF
- L1601, L1602, L1603, L1604: value L_Small -> 50 ohm@100Mhz; Description (none) -> 50 Ohms @ 100MHz 1 Power Line Ferrite Bead 1206 (3216 Metri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; PartNumber (none) -> PE-1206PFB500ST; digikey (none) -> 553-2403-1-ND; price@10 (none) -> 0.14900
- R1601, R1602, R1603, R1604: value 12e -> 12
- R1605, R1606: value 12e -> 100
- R1607, R1609: value 1k -> 1k(dnp)
- R1608, R1610: value 1k -> 3k3
- R1611, R1612, R1613, R1614, R1615, R1616, R1617, R1618: value 1M -> 2M2
Other:
- note added: "No more than 600V"
- note added: "No more than 600v"
Changed lines of the file:
@@
 F 4 "CC0603KPX7R7BB104" H 0   0   50  0001 C CNN "PartNumber"
 F 5 "311-1335-1-ND" H 0   0   50  0001 C CNN "digikey"
+F 6 "CAP CER 0.1UF 16V X7R 0603 " H 0   0   50  0001 C CNN "Description"
 	1    8450 2600
 	0    1    1    0
@@
 F 4 "CC0603KPX7R7BB104" H 0   0   50  0001 C CNN "PartNumber"
 F 5 "311-1335-1-ND" H 0   0   50  0001 C CNN "digikey"
+F 6 "CAP CER 0.1UF 16V X7R 0603 " H 0   0   50  0001 C CNN "Description"
 	1    6500 2750
 	0    1    1    0
@@
 AR Path="/5DE49152/5E1AD3A3" Ref="C?"  Part="1"
 F 0 "C1605" V 8278 3591 20  0000 R CNN
-F 1 "330p" V 8321 3591 20  0000 R CNN
+F 1 "0.1uF" V 8321 3591 20  0000 R CNN
 F 2 "servo:C_0603_1608Metric" H 8250 3600 60  0001 C CNN
 F 3 "" H 8250 3700 60  0000 C CNN
@@
 AR Path="/5DE49152/5E1AD42C" Ref="R?"  Part="1"
 F 0 "R1607" V 8778 3150 20  0000 L CNN
-F 1 "1k" V 8821 3150 20  0000 L CNN
+F 1 "1k(dnp)" V 8821 3150 20  0000 L CNN
 F 2 "servo:R_0603_1608Metric" H 8300 3000 60  0001 C CNN
 F 3 "" H 8400 3100 60  0001 C CNN
@@
 AR Path="/5DE49152/5E1AD417" Ref="R?"  Part="1"
 F 0 "R1611" H 9100 3415 20  0000 C CNN
-F 1 "1M" H 9100 3372 20  0000 C CNN
+F 1 "2M2" H 9100 3372 20  0000 C CNN
 F 2 "servo:R_1206_3216Metric_Pad1.42x1.75mm_HandSolder" H 8600 3200 60  0001 C CNN
 F 3 "" H 8700 3300 60  0001 C CNN
@@
 AR Path="/5DE49152/5E1AD395" Ref="R?"  Part="1"
 F 0 "R1608" V 8778 3800 20  0000 L CNN
-F 1 "1k" V 8821 3800 20  0000 L CNN
+F 1 "3k3" V 8821 3800 20  0000 L CNN
 F 2 "servo:R_0603_1608Metric" H 8300 3650 60  0001 C CNN
 F 3 "" H 8400 3750 60  0001 C CNN
@@
 AR Path="/5DE49152/5E1AD3AA" Ref="R?"  Part="1"
 F 0 "R1605" H 8500 3415 20  0000 C CNN
-F 1 "12e" H 8500 3372 20  0000 C CNN
+F 1 "100" H 8500 3372 20  0000 C CNN
 F 2 "servo:R_0603_1608Metric" H 8000 3200 60  0001 C CNN
 F 3 "" H 8100 3300 60  0001 C CNN
@@
 AR Path="/605BEC04/5E1AD3C1" Ref="L1601"  Part="1"
 F 0 "L1601" V 8594 2500 20  0000 C CNN
-F 1 "L_Small" V 8637 2500 20  0000 C CNN
+F 1 "50 ohm@100Mhz" V 8637 2500 20  0000 C CNN
 F 2 "servo:L_1206_3216Metric_Pad1.42x1.75mm_HandSolder" H 8630 2440 50  0001 C CNN
 F 3 "~" H 8730 2540 50  0001 C CNN
+F 4 "50 Ohms @ 100MHz 1 Power Line Ferrite Bead 1206 (3216 Metric) 3A 30mOhm " H 0   0   50  0001 C CNN "Description"
+F 5 "PE-1206PFB500ST" H 0   0   50  0001 C CNN "PartNumber"
+F 6 "553-2403-1-ND" H 0   0   50  0001 C CNN "digikey"
+F 7 "0.14900" H 0   0   50  0001 C CNN "price@10"
 	1    8700 2500
 	0    1    1    0
@@
 AR Path="/605BEC04/5E1AD3CB" Ref="L1603"  Part="1"
 F 0 "L1603" H 10398 2222 20  0000 L CNN
-F 1 "L_Small" H 10398 2179 20  0000 L CNN
+F 1 "50 ohm@100Mhz" H 10398 2179 20  0000 L CNN
 F 2 "servo:L_1206_3216Metric_Pad1.42x1.75mm_HandSolder" H 10280 2140 50  0001 C CNN
 F 3 "~" H 10380 2240 50  0001 C CNN
+F 4 "50 Ohms @ 100MHz 1 Power Line Ferrite Bead 1206 (3216 Metric) 3A 30mOhm " H 0   0   50  0001 C CNN "Description"
+F 5 "PE-1206PFB500ST" H 0   0   50  0001 C CNN "PartNumber"
+F 6 "553-2403-1-ND" H 0   0   50  0001 C CNN "digikey"
+F 7 "0.14900" H 0   0   50  0001 C CNN "price@10"
 	1    10350 2200
 	1    0    0    -1
@@
 F 4 "CC0603KPX7R7BB104" H 0   0   50  0001 C CNN "PartNumber"
 F 5 "311-1335-1-ND" H 0   0   50  0001 C CNN "digikey"
+F 6 "CAP CER 0.1UF 16V X7R 0603 " H 0   0   50  0001 C CNN "Description"
 	1    10350 2450
 	0    1    1    0
@@
 F 4 "CC0603KPX7R7BB104" H 0   0   50  0001 C CNN "PartNumber"
 F 5 "311-1335-1-ND" H 0   0   50  0001 C CNN "digikey"
+F 6 "CAP CER 0.1UF 16V X7R 0603 " H 0   0   50  0001 C CNN "Description"
 	1    5600 3000
 	0    1    1    0
@@
 AR Path="/5DE49152/5E19B1CF" Ref="R?"  Part="1"
 F 0 "R1601" H 5900 2965 20  0000 C CNN
-F 1 "12e" H 5900 2922 20  0000 C CNN
+F 1 "12" H 5900 2922 20  0000 C CNN
 F 2 "servo:R_0603_1608Metric" H 5400 2750 60  0001 C CNN
 F 3 "" H 5500 2850 60  0001 C CNN
@@
 AR Path="/5DE49152/5E19B35E" Ref="R?"  Part="1"
 F 0 "R1602" H 5900 3365 20  0000 C CNN
-F 1 "12e" H 5900 3322 20  0000 C CNN
+F 1 "12" H 5900 3322 20  0000 C CNN
 F 2 "servo:R_0603_1608Metric" H 5400 3150 60  0001 C CNN
 F 3 "" H 5500 3250 60  0001 C CNN
@@
 F 4 "CC0603KPX7R7BB104" H 0   0   50  0001 C CNN "PartNumber"
 F 5 "311-1335-1-ND" H 0   0   50  0001 C CNN "digikey"
+F 6 "CAP CER 0.1UF 16V X7R 0603 " H 0   0   50  0001 C CNN "Description"
 	1    8550 4900
 	0    1    1    0
@@
 F 4 "CC0603KPX7R7BB104" H 0   0   50  0001 C CNN "PartNumber"
 F 5 "311-1335-1-ND" H 0   0   50  0001 C CNN "digikey"
+F 6 "CAP CER 0.1UF 16V X7R 0603 " H 0   0   50  0001 C CNN "Description"
 	1    6600 5050
 	0    1    1    0
@@
 AR Path="/5DE49152/5E1B9A85" Ref="C?"  Part="1"
 F 0 "C1606" V 8378 5891 20  0000 R CNN
-F 1 "330p" V 8421 5891 20  0000 R CNN
+F 1 "0.1uF" V 8421 5891 20  0000 R CNN
 F 2 "servo:C_0603_1608Metric" H 8350 5900 60  0001 C CNN
 F 3 "" H 8350 6000 60  0000 C CNN
@@
 AR Path="/5DE49152/5E1B9AAE" Ref="R?"  Part="1"
 F 0 "R1609" V 8878 5450 20  0000 L CNN
-F 1 "1k" V 8921 5450 20  0000 L CNN
+F 1 "1k(dnp)" V 8921 5450 20  0000 L CNN
 F 2 "servo:R_0603_1608Metric" H 8400 5300 60  0001 C CNN
 F 3 "" H 8500 5400 60  0001 C CNN
@@
 AR Path="/5DE49152/5E1B9AD0" Ref="R?"  Part="1"
 F 0 "R1610" V 8878 6100 20  0000 L CNN
-F 1 "1k" V 8921 6100 20  0000 L CNN
+F 1 "3k3" V 8921 6100 20  0000 L CNN
 F 2 "servo:R_0603_1608Metric" H 8400 5950 60  0001 C CNN
 F 3 "" H 8500 6050 60  0001 C CNN
@@
 AR Path="/5DE49152/5E1B9AD7" Ref="R?"  Part="1"
 F 0 "R1606" H 8600 5715 20  0000 C CNN
-F 1 "12e" H 8600 5672 20  0000 C CNN
+F 1 "100" H 8600 5672 20  0000 C CNN
 F 2 "servo:R_0603_1608Metric" H 8100 5500 60  0001 C CNN
 F 3 "" H 8200 5600 60  0001 C CNN
@@
 AR Path="/605BEC04/5E1B9AEA" Ref="L1602"  Part="1"
 F 0 "L1602" V 8694 4800 20  0000 C CNN
-F 1 "L_Small" V 8737 4800 20  0000 C CNN
+F 1 "50 ohm@100Mhz" V 8737 4800 20  0000 C CNN
 F 2 "servo:L_1206_3216Metric_Pad1.42x1.75mm_HandSolder" H 8730 4740 50  0001 C CNN
 F 3 "~" H 8830 4840 50  0001 C CNN
+F 4 "50 Ohms @ 100MHz 1 Power Line Ferrite Bead 1206 (3216 Metric) 3A 30mOhm " H 0   0   50  0001 C CNN "Description"
+F 5 "PE-1206PFB500ST" H 0   0   50  0001 C CNN "PartNumber"
+F 6 "553-2403-1-ND" H 0   0   50  0001 C CNN "digikey"
+F 7 "0.14900" H 0   0   50  0001 C CNN "price@10"
 	1    8800 4800
 	0    1    1    0
@@
 AR Path="/605BEC04/5E1B9AF3" Ref="L1604"  Part="1"
 F 0 "L1604" H 10498 4522 20  0000 L CNN
-F 1 "L_Small" H 10498 4479 20  0000 L CNN
+F 1 "50 ohm@100Mhz" H 10498 4479 20  0000 L CNN
 F 2 "servo:L_1206_3216Metric_Pad1.42x1.75mm_HandSolder" H 10380 4440 50  0001 C CNN
 F 3 "~" H 10480 4540 50  0001 C CNN
+F 4 "50 Ohms @ 100MHz 1 Power Line Ferrite Bead 1206 (3216 Metric) 3A 30mOhm " H 0   0   50  0001 C CNN "Description"
+F 5 "PE-1206PFB500ST" H 0   0   50  0001 C CNN "PartNumber"
+F 6 "553-2403-1-ND" H 0   0   50  0001 C CNN "digikey"
+F 7 "0.14900" H 0   0   50  0001 C CNN "price@10"
 	1    10450 4500
 	1    0    0    -1
@@
 F 4 "CC0603KPX7R7BB104" H 0   0   50  0001 C CNN "PartNumber"
 F 5 "311-1335-1-ND" H 0   0   50  0001 C CNN "digikey"
+F 6 "CAP CER 0.1UF 16V X7R 0603 " H 0   0   50  0001 C CNN "Description"
 	1    10450 4750
 	0    1    1    0
@@
 F 4 "CC0603KPX7R7BB104" H 0   0   50  0001 C CNN "PartNumber"
 F 5 "311-1335-1-ND" H 0   0   50  0001 C CNN "digikey"
+F 6 "CAP CER 0.1UF 16V X7R 0603 " H 0   0   50  0001 C CNN "Description"
 	1    5700 5300
 	0    1    1    0
@@
 AR Path="/5DE49152/5E1B9B35" Ref="R?"  Part="1"
 F 0 "R1603" H 6000 5265 20  0000 C CNN
-F 1 "12e" H 6000 5222 20  0000 C CNN
+F 1 "12" H 6000 5222 20  0000 C CNN
 F 2 "servo:R_0603_1608Metric" H 5500 5050 60  0001 C CNN
 F 3 "" H 5600 5150 60  0001 C CNN
@@
 AR Path="/5DE49152/5E1B9B3C" Ref="R?"  Part="1"
 F 0 "R1604" H 6000 5665 20  0000 C CNN
-F 1 "12e" H 6000 5622 20  0000 C CNN
+F 1 "12" H 6000 5622 20  0000 C CNN
 F 2 "servo:R_0603_1608Metric" H 5500 5450 60  0001 C CNN
 F 3 "" H 5600 5550 60  0001 C CNN
@@
 AR Path="/5DE49152/5E26C457" Ref="R?"  Part="1"
 F 0 "R1613" H 9500 3415 20  0000 C CNN
-F 1 "1M" H 9500 3372 20  0000 C CNN
+F 1 "2M2" H 9500 3372 20  0000 C CNN
 F 2 "servo:R_1206_3216Metric_Pad1.42x1.75mm_HandSolder" H 9000 3200 60  0001 C CNN
 F 3 "" H 9100 3300 60  0001 C CNN
@@
 AR Path="/5DE49152/5E256879" Ref="R?"  Part="1"
 F 0 "R1612" H 9100 3565 20  0000 C CNN
-F 1 "1M" H 9100 3522 20  0000 C CNN
+F 1 "2M2" H 9100 3522 20  0000 C CNN
 F 2 "servo:R_1206_3216Metric_Pad1.42x1.75mm_HandSolder" H 8600 3350 60  0001 C CNN
 F 3 "" H 8700 3450 60  0001 C CNN
@@
 AR Path="/5DE49152/5E256880" Ref="R?"  Part="1"
 F 0 "R1616" H 9500 3565 20  0000 C CNN
-F 1 "1M" H 9500 3522 20  0000 C CNN
+F 1 "2M2" H 9500 3522 20  0000 C CNN
 F 2 "servo:R_1206_3216Metric_Pad1.42x1.75mm_HandSolder" H 9000 3350 60  0001 C CNN
 F 3 "" H 9100 3450 60  0001 C CNN
@@
 AR Path="/5DE49152/5E2642A2" Ref="R?"  Part="1"
 F 0 "R1614" H 9200 5715 20  0000 C CNN
-F 1 "1M" H 9200 5672 20  0000 C CNN
+F 1 "2M2" H 9200 5672 20  0000 C CNN
 F 2 "servo:R_1206_3216Metric_Pad1.42x1.75mm_HandSolder" H 8700 5500 60  0001 C CNN
 F 3 "" H 8800 5600 60  0001 C CNN
@@
 AR Path="/5DE49152/5E2642A9" Ref="R?"  Part="1"
 F 0 "R1617" H 9600 5715 20  0000 C CNN
-F 1 "1M" H 9600 5672 20  0000 C CNN
+F 1 "2M2" H 9600 5672 20  0000 C CNN
 F 2 "servo:R_1206_3216Metric_Pad1.42x1.75mm_HandSolder" H 9100 5500 60  0001 C CNN
 F 3 "" H 9200 5600 60  0001 C CNN
@@
 AR Path="/5DE49152/5E2642B0" Ref="R?"  Part="1"
 F 0 "R1615" H 9200 5865 20  0000 C CNN
-F 1 "1M" H 9200 5822 20  0000 C CNN
+F 1 "2M2" H 9200 5822 20  0000 C CNN
 F 2 "servo:R_1206_3216Metric_Pad1.42x1.75mm_HandSolder" H 8700 5650 60  0001 C CNN
 F 3 "" H 8800 5750 60  0001 C CNN
@@
 AR Path="/5DE49152/5E2642B7" Ref="R?"  Part="1"
 F 0 "R1618" H 9600 5865 20  0000 C CNN
-F 1 "1M" H 9600 5822 20  0000 C CNN
+F 1 "2M2" H 9600 5822 20  0000 C CNN
 F 2 "servo:R_1206_3216Metric_Pad1.42x1.75mm_HandSolder" H 9100 5650 60  0001 C CNN
 F 3 "" H 9200 5750 60  0001 C CNN
@@
 	10850 2700 10350 2700
 Connection ~ 10850 5000
+Text Notes 10050 3700 0    20   ~ 0
+No more than 600v
+Text Notes 10050 6000 0    20   ~ 0
+No more than 600V
 $EndSCHEMATC
