File: kicad/uc_clk_dbg.sch (KiCad schematic (older format))
At the start: 17 parts, among them J601 pinHeader, U301 TMS320F28388DZWTS, U602 M25PX32-VMW

Commit message: added sloted holes everyware
Parts:
- Y601: footprint Oscillator:Oscillator_SMD_SeikoEpson_SG210-4Pin_2.5x2.0mm -> servo:Crystal_SMD_2520-4Pin_2.5x2.0mm
Changed lines of the file:
@@
 F 0 "Y601" H 13900 2367 60  0000 C CNN
 F 1 "~" H 13900 2600 50  0001 C CNN
-F 2 "Oscillator:Oscillator_SMD_SeikoEpson_SG210-4Pin_2.5x2.0mm" H 13900 2600 50  0001 C CNN
+F 2 "servo:Crystal_SMD_2520-4Pin_2.5x2.0mm" H 13900 2600 50  0001 C CNN
 F 3 "../doc/datasheets//ECS-2520S.pdf" H 13900 2600 50  0001 C CNN
 	1    13900 2600

Commit message: serigrafia...
Parts:
- R603, R606, R607, R608, R609, R610: footprint Resistor_SMD:R_0603_1608Metric -> servo:R_0603_1608Metric
- R604, R605: footprint Resistor_SMD:R_0805_2012Metric_Pad1.15x1.40mm_HandSolder -> servo:R_0805_2012Metric_Pad1.15x1.40mm_HandSolder
- Y601: value ~ -> 26mhz
Changed lines of the file:
@@
 F 0 "R610" V 13945 3300 60  0000 R CNN
 F 1 "2.2k" V 13847 3300 50  0000 R CNN
-F 2 "Resistor_SMD:R_0603_1608Metric" H 13900 3350 50  0001 C CNN
+F 2 "servo:R_0603_1608Metric" H 13900 3350 50  0001 C CNN
 F 3 "" H 13900 3350 50  0001 C CNN
 F 4 "2.2k" V 11100 1150 60  0001 C CNN "ValueDisplayed"
@@
 F 0 "R604" V 6278 7600 20  0000 L CNN
 F 1 "56k" V 6321 7600 20  0000 L CNN
-F 2 "Resistor_SMD:R_0805_2012Metric_Pad1.15x1.40mm_HandSolder" H 5800 7450 60  0001 C CNN
+F 2 "servo:R_0805_2012Metric_Pad1.15x1.40mm_HandSolder" H 5800 7450 60  0001 C CNN
 F 3 "" H 5900 7550 60  0001 C CNN
 F 4 "56k" V -7900 4050 60  0001 C CNN "ValueDisplayed"
@@
 F 0 "R605" V 6578 7600 20  0000 L CNN
 F 1 "56k" V 6621 7600 20  0000 L CNN
-F 2 "Resistor_SMD:R_0805_2012Metric_Pad1.15x1.40mm_HandSolder" H 6100 7450 60  0001 C CNN
+F 2 "servo:R_0805_2012Metric_Pad1.15x1.40mm_HandSolder" H 6100 7450 60  0001 C CNN
 F 3 "" H 6200 7550 60  0001 C CNN
 F 4 "56k" V -7900 4050 60  0001 C CNN "ValueDisplayed"
@@
 F 0 "R607" V 10095 3150 60  0000 R CNN
 F 1 "2.2k" V 9997 3150 50  0000 R CNN
-F 2 "Resistor_SMD:R_0603_1608Metric" H 10050 3200 50  0001 C CNN
+F 2 "servo:R_0603_1608Metric" H 10050 3200 50  0001 C CNN
 F 3 "" H 10050 3200 50  0001 C CNN
 F 4 "2.2k" V 9950 2500 60  0001 C CNN "ValueDisplayed"
@@
 P 13900 2600
 F 0 "Y601" H 13900 2367 60  0000 C CNN
-F 1 "~" H 13900 2600 50  0001 C CNN
+F 1 "26mhz" H 13900 2600 50  0001 C CNN
 F 2 "servo:Crystal_SMD_2520-4Pin_2.5x2.0mm" H 13900 2600 50  0001 C CNN
 F 3 "../doc/datasheets//ECS-2520S.pdf" H 13900 2600 50  0001 C CNN
@@
 F 0 "R606" V 8325 3750 20  0000 R CNN
 F 1 "1.0k" V 8282 3750 20  0000 R CNN
-F 2 "Resistor_SMD:R_0603_1608Metric" H 7750 3700 60  0001 C CNN
+F 2 "servo:R_0603_1608Metric" H 7750 3700 60  0001 C CNN
 F 3 "" H 7850 3800 60  0001 C CNN
 	1    8250 3800
@@
 F 0 "R603" V 4347 3650 60  0000 L CNN
 F 1 "1.0k" H 4400 3600 50  0001 C CNN
-F 2 "Resistor_SMD:R_0603_1608Metric" H 4400 3600 50  0001 C CNN
+F 2 "servo:R_0603_1608Metric" H 4400 3600 50  0001 C CNN
 F 3 "" H 4400 3600 50  0001 C CNN
 F 4 "1.0k" V 4453 3650 60  0000 L CNN "ValueDisplayed"
@@
 F 0 "R608" H 10100 7465 20  0000 C CNN
 F 1 "680" H 10100 7422 20  0000 C CNN
-F 2 "Resistor_SMD:R_0603_1608Metric" H 9600 7250 60  0001 C CNN
+F 2 "servo:R_0603_1608Metric" H 9600 7250 60  0001 C CNN
 F 3 "" H 9700 7350 60  0001 C CNN
 F 4 "680" V 1100 8150 60  0001 C CNN "ValueDisplayed"
@@
 F 0 "R609" H 10500 7465 20  0000 C CNN
 F 1 "680" H 10500 7422 20  0000 C CNN
-F 2 "Resistor_SMD:R_0603_1608Metric" H 10000 7250 60  0001 C CNN
+F 2 "servo:R_0603_1608Metric" H 10000 7250 60  0001 C CNN
 F 3 "" H 10100 7350 60  0001 C CNN
 F 4 "680" V 1500 8150 60  0001 C CNN "ValueDisplayed"

Commit message: serigraphi, improve of nets. change of soic 8 footprint
Parts:
- U602: footprint Package_SO:SOIJ-8_5.3x5.3mm_P1.27mm -> servo:SOIJ-8_5.3x5.3mm_P1.27mm
Changed lines of the file:
@@
 F 0 "U602" H 14491 8046 50  0000 L CNN
 F 1 "M25PX32-VMW" H 14491 7955 50  0000 L CNN
-F 2 "Package_SO:SOIJ-8_5.3x5.3mm_P1.27mm" H 14500 8050 50  0001 C CNN
+F 2 "servo:SOIJ-8_5.3x5.3mm_P1.27mm" H 14500 8050 50  0001 C CNN
 F 3 "../doc/datasheets/m25px32.pdf" H 14000 7900 50  0001 C CNN
 	1    13850 8000

Commit message: bom bom bom...
Parts:
- C601: value 1nF -> 10nF
- C602: value 0.01uF -> 0.1uF; Description (none) -> CAP CER 0.1UF 16V X7R 0603; PartNumber (none) -> CC0603KPX7R7BB104; ValueDisplayed 0.01uF -> (none); digikey (none) -> 311-1335-1-ND
- C603: Description (none) -> CAP CER 0.1UF 16V X7R 0603; PartNumber (none) -> CC0603KPX7R7BB104; ValueDisplayed 0.1uF -> (none); digikey (none) -> 311-1335-1-ND
- D603: value green -> blue@5mA; PartNumber (none) -> LB Q39G-L2OO-35-1; VALUE green@2mA -> (none); digikey (none) -> LB Q39G-L2OO-35-1
- D604: value blue -> blue@5mA; PartNumber (none) -> LB Q39G-L2OO-35-1; VALUE blue@2mA -> (none); digikey (none) -> LB Q39G-L2OO-35-1
- R603: value 1.0k -> 560; ValueDisplayed 1.0k -> (none)
- R604, R605: ValueDisplayed 56k -> (none)
- R606: value 1.0k -> 560
- R607, R610: ValueDisplayed 2.2k -> (none)
- R608, R609: value 680 -> 100e; ValueDisplayed 680 -> (none)
Connections:
- net 3V3uC: now also R610.1; no longer R610.2
- net GND: now also R607.2; no longer R607.1
- net MCU_TRSTn: now also R607.1; no longer R607.2
- net MCU_XRSn: now also R610.2; no longer R610.1
- no-connect marks 8 -> 7
Changed lines of the file:
@@
 U 1 1 5DB38F69
 P 13900 3350
-F 0 "R610" V 13945 3300 60  0000 R CNN
-F 1 "2.2k" V 13847 3300 50  0000 R CNN
-F 2 "servo:R_0603_1608Metric" H 13900 3350 50  0001 C CNN
-F 3 "" H 13900 3350 50  0001 C CNN
-F 4 "2.2k" V 11100 1150 60  0001 C CNN "ValueDisplayed"
+F 0 "R610" V 13878 3400 20  0000 L CNN
+F 1 "2.2k" V 13921 3400 20  0000 L CNN
+F 2 "servo:R_0603_1608Metric" H 13400 3250 60  0001 C CNN
+F 3 "" H 13500 3350 60  0001 C CNN
 	1    13900 3350
-	0    -1   -1   0
+	0    1    1    0
 $EndComp
 $Comp
@@
 U 1 1 5DB38F68
 P 13900 3800
-F 0 "C602" V 13995 3909 60  0000 L CNN
-F 1 "0.01uF" V 13897 3909 50  0000 L CNN
-F 2 "servo:C_0603_1608Metric" H 13900 3800 50  0001 C CNN
-F 3 "" H 13900 3800 50  0001 C CNN
-F 4 "0.01uF" V 11100 900 60  0001 C CNN "ValueDisplayed"
+F 0 "C602" V 13972 3690 20  0000 R CNN
+F 1 "0.1uF" V 13929 3690 20  0000 R CNN
+F 2 "servo:C_0603_1608Metric" H 13900 3700 60  0001 C CNN
+F 3 "" H 13900 3800 60  0000 C CNN
+F 4 "311-1335-1-ND" H 0   0   50  0001 C CNN "digikey"
+F 5 "CAP CER 0.1UF 16V X7R 0603 " H 0   0   50  0001 C CNN "Description"
+F 6 "" H 0   0   50  0001 C CNN "Mfr part number"
+F 7 "CC0603KPX7R7BB104" H 0   0   50  0001 C CNN "PartNumber"
 	1    13900 3800
 	0    -1   -1   0
@@
 F 2 "servo:R_0805_2012Metric_Pad1.15x1.40mm_HandSolder" H 5800 7450 60  0001 C CNN
 F 3 "" H 5900 7550 60  0001 C CNN
-F 4 "56k" V -7900 4050 60  0001 C CNN "ValueDisplayed"
 	1    6300 7550
 	0    1    1    0
@@
 F 2 "servo:R_0805_2012Metric_Pad1.15x1.40mm_HandSolder" H 6100 7450 60  0001 C CNN
 F 3 "" H 6200 7550 60  0001 C CNN
-F 4 "56k" V -7900 4050 60  0001 C CNN "ValueDisplayed"
 	1    6600 7550
 	0    1    1    0
@@
 U 1 1 5DB38F5A
 P 10050 3200
-F 0 "R607" V 10095 3150 60  0000 R CNN
-F 1 "2.2k" V 9997 3150 50  0000 R CNN
-F 2 "servo:R_0603_1608Metric" H 10050 3200 50  0001 C CNN
-F 3 "" H 10050 3200 50  0001 C CNN
-F 4 "2.2k" V 9950 2500 60  0001 C CNN "ValueDisplayed"
+F 0 "R607" V 10028 3250 20  0000 L CNN
+F 1 "2.2k" V 10071 3250 20  0000 L CNN
+F 2 "servo:R_0603_1608Metric" H 9550 3100 60  0001 C CNN
+F 3 "" H 9650 3200 60  0001 C CNN
 	1    10050 3200
-	0    -1   -1   0
+	0    1    1    0
 $EndComp
 $Comp
@@
 Wire Wire Line
 	6450 7100 6450 7200
-Connection ~ 13900 3600
 Wire Wire Line
 	13000 3300 12650 3300
@@
 AR Path="/5DD4DF4C/5DE66EAC" Ref="R606"  Part="1"
 F 0 "R606" V 8325 3750 20  0000 R CNN
-F 1 "1.0k" V 8282 3750 20  0000 R CNN
+F 1 "560" V 8282 3750 20  0000 R CNN
 F 2 "servo:R_0603_1608Metric" H 7750 3700 60  0001 C CNN
 F 3 "" H 7850 3800 60  0001 C CNN
@@
 AR Path="/5DD4DF4C/5DE66EBC" Ref="D603"  Part="1"
 F 0 "D603" V 4385 3172 20  0000 R CNN
-F 1 "green" V 4425 3172 16  0000 R CNN
+F 1 "blue@5mA" V 4425 3172 16  0000 R CNN
 F 2 "servo:LED_0603_1608Metric" H 4200 3050 60  0001 C CNN
-F 3 "" H 4200 3050 60  0001 C CNN
-F 4 "green@2mA" V 4465 3172 20  0000 R CNN "VALUE"
+F 3 "../doc/datasheets/LB_Q39G_v1.4_9-1-15.pdf" H 4200 3050 60  0001 C CNN
+F 4 "LB Q39G-L2OO-35-1" H 4400 3250 50  0001 C CNN "digikey"
+F 5 "LB Q39G-L2OO-35-1" H 0   0   50  0001 C CNN "PartNumber"
 	1    4400 3250
 	0    1    1    0
@@
 AR Path="/5DD4DF4C/5DE66EC4" Ref="D604"  Part="1"
 F 0 "D604" V 8235 3580 20  0000 L CNN
-F 1 "blue" V 8275 3580 16  0000 L CNN
+F 1 "blue@5mA" V 8275 3580 16  0000 L CNN
 F 2 "servo:LED_0603_1608Metric" H 8050 3250 60  0001 C CNN
-F 3 "" H 8050 3250 60  0001 C CNN
-F 4 "blue@2mA" V 8315 3580 20  0000 L CNN "VALUE"
+F 3 "../doc/datasheets/LB_Q39G_v1.4_9-1-15.pdf" H 8050 3250 60  0001 C CNN
+F 4 "LB Q39G-L2OO-35-1" H 8250 3450 50  0001 C CNN "digikey"
+F 5 "LB Q39G-L2OO-35-1" H 0   0   50  0001 C CNN "PartNumber"
 	1    8250 3450
 	0    1    1    0
@@
 AR Path="/5DCD812E/5DE66EB4" Ref="R?"  Part="1"
 AR Path="/5DD4DF4C/5DE66EB4" Ref="R603"  Part="1"
-F 0 "R603" V 4347 3650 60  0000 L CNN
-F 1 "1.0k" H 4400 3600 50  0001 C CNN
-F 2 "servo:R_0603_1608Metric" H 4400 3600 50  0001 C CNN
-F 3 "" H 4400 3600 50  0001 C CNN
-F 4 "1.0k" V 4453 3650 60  0000 L CNN "ValueDisplayed"
+F 0 "R603" V 4378 3650 20  0000 L CNN
+F 1 "560" V 4421 3650 20  0000 L CNN
+F 2 "servo:R_0603_1608Metric" H 3900 3500 60  0001 C CNN
+F 3 "" H 4000 3600 60  0001 C CNN
 	1    4400 3600
 	0    1    1    0
@@
 AR Path="/5DC4A59D/5ECD3F89" Ref="C?"  Part="1"
 AR Path="/5DD4DF4C/5ECD3F89" Ref="C603"  Part="1"
-F 0 "C603" H 14350 7350 20  0000 L BNN
-F 1 "0.1uF" H 14350 7400 20  0000 C CNN
+F 0 "C603" V 14328 7360 20  0000 L CNN
+F 1 "0.1uF" V 14371 7360 20  0000 L CNN
 F 2 "servo:C_0603_1608Metric" H 14300 7150 60  0001 C CNN
 F 3 "" H 14300 7250 60  0000 C CNN
-F 4 "0.1uF" V 11700 7650 60  0001 C CNN "ValueDisplayed"
+F 4 "311-1335-1-ND" H 0   0   50  0001 C CNN "digikey"
+F 5 "CAP CER 0.1UF 16V X7R 0603 " H 0   0   50  0001 C CNN "Description"
+F 6 "" H 0   0   50  0001 C CNN "Mfr part number"
+F 7 "CC0603KPX7R7BB104" H 0   0   50  0001 C CNN "PartNumber"
 	1    14300 7250
 	0    1    1    0
@@
 Wire Wire Line
 	2750 2500 3100 2500
-$Comp
-L servo:GND #PWR_0602
-U 1 1 5EEC9C34
-P 6300 4350
-F 0 "#PWR_0602" H 6305 4201 20  0001 C CNN
-F 1 "GND" H 6300 4192 30  0000 C CNN
-F 2 "" H 6300 4350 70  0000 C CNN
-F 3 "" H 6300 4350 70  0000 C CNN
-	1    6300 4350
-	1    0    0    -1
-$EndComp
-Wire Wire Line
-	7700 2800 10050 2800
-$Comp
-L servo:GND #PWR_0604
-U 1 1 5EF4D354
-P 7250 3600
-F 0 "#PWR_0604" H 7255 3451 20  0001 C CNN
-F 1 "GND" H 7250 3442 30  0000 C CNN
-F 2 "" H 7250 3600 70  0000 C CNN
-F 3 "" H 7250 3600 70  0000 C CNN
-	1    7250 3600
-	1    0    0    -1
-$EndComp
 Wire Wire Line
 	7950 2600 10650 2600
@@
 AR Path="/5E72D841/5E228777" Ref="R?"  Part="1"
 F 0 "R608" H 10100 7465 20  0000 C CNN
-F 1 "680" H 10100 7422 20  0000 C CNN
+F 1 "100e" H 10100 7422 20  0000 C CNN
 F 2 "servo:R_0603_1608Metric" H 9600 7250 60  0001 C CNN
 F 3 "" H 9700 7350 60  0001 C CNN
-F 4 "680" V 1100 8150 60  0001 C CNN "ValueDisplayed"
 	1    10100 7350
 	1    0    0    -1
@@
 AR Path="/5DD4DF4C/5E22877E" Ref="C601"  Part="1"
 F 0 "C601" V 10328 7660 20  0000 L CNN
-F 1 "1nF" V 10371 7660 20  0000 L CNN
+F 1 "10nF" V 10371 7660 20  0000 L CNN
 F 2 "servo:C_0603_1608Metric" H 10300 7450 60  0001 C CNN
 F 3 "" H 10300 7550 60  0000 C CNN
@@
 AR Path="/5E72D841/5E228785" Ref="R?"  Part="1"
 F 0 "R609" H 10500 7465 20  0000 C CNN
-F 1 "680" H 10500 7422 20  0000 C CNN
+F 1 "100e" H 10500 7422 20  0000 C CNN
 F 2 "servo:R_0603_1608Metric" H 10000 7250 60  0001 C CNN
 F 3 "" H 10100 7350 60  0001 C CNN
-F 4 "680" V 1500 8150 60  0001 C CNN "ValueDisplayed"
 	1    10500 7350
 	1    0    0    -1
@@
 PRG_SCI_TX
 Wire Wire Line
-	5250 2500 5250 2600
-Wire Wire Line
-	5000 2800 5000 2600
-Wire Wire Line
-	3600 2500 5250 2500
-Wire Wire Line
-	3600 2600 5000 2600
-Wire Wire Line
-	4900 2700 4900 3000
+	4900 2700 4900 2800
 Wire Wire Line
 	3600 2700 4900 2700
 Wire Wire Line
-	4700 2800 4700 3400
-Wire Wire Line
 	3600 2800 4700 2800
 Wire Wire Line
-	7500 2500 7500 2600
-Wire Wire Line
-	7500 2500 10650 2500
-Wire Wire Line
-	7550 2700 7550 2800
-Wire Wire Line
-	7550 2700 10650 2700
-Wire Wire Line
-	7700 2800 7700 3000
-Wire Wire Line
-	7950 2600 7950 3400
+	7950 2600 7950 2900
 Wire Wire Line
 	8250 3300 8250 3350
@@
 Wire Wire Line
 	13100 8100 13100 7400
-Wire Wire Line
-	7100 3600 7250 3600
 NoConn ~ 12650 3100
 NoConn ~ 12650 2700
@@
 	3600 2400 10650 2400
 Wire Wire Line
-	5250 2600 7500 2600
-Wire Wire Line
-	4700 3400 7950 3400
-Wire Wire Line
-	4900 3000 7700 3000
-Wire Wire Line
-	5000 2800 7550 2800
-Wire Wire Line
 	4400 3800 7450 3800
-NoConn ~ 5500 3600
 Wire Wire Line
 	2800 4000 8250 4000
@@
 	1    0    0    -1
 $EndComp
+Wire Wire Line
+	3600 2500 10650 2500
+Wire Wire Line
+	5350 2700 5350 2600
+Wire Wire Line
+	3600 2600 5350 2600
+Wire Wire Line
+	5350 2700 10650 2700
+Wire Wire Line
+	4900 2800 10050 2800
+Wire Wire Line
+	7950 2900 4700 2900
+Wire Wire Line
+	4700 2800 4700 2900
+Connection ~ 13900 3600
 $EndSCHEMATC

Commit message: more bom...
Parts:
- C601: value 10nF -> 0.1uF; Description (none) -> CAP CER 0.1UF 16V X7R 0603; PartNumber (none) -> CC0603KPX7R7BB104; digikey (none) -> 311-1335-1-ND
- D603, D604: Description (none) -> LED BLUE DIFFUSED 0603 SMD
- J601: value pinHeader -> pin header 2x6 2.54; Description (none) -> Connector Header Surface Mount 12 position 0.100\" (2.54mm); PartNumber (none) -> GBC06DABN-M30; digikey (none) -> S2351E-06-ND; price@10 (none) -> 1.10200
- U301: Description (none) -> 32-bit MCU with connectivity manager, 2x C28x+CLA CPU, 1.5 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; price@10 (none) -> 14.96
Changed lines of the file:
@@
 F 3 "../doc/datasheets/tms320f28388d_datasheet.pdf" H 11650 2800 50  0001 C CNN
 F 4 "TMS320F28388DZWTS" V 10250 2600 60  0001 C CNN "PartNumber"
+F 5 "32-bit MCU with connectivity manager, 2x C28x+CLA CPU, 1.5 MB flash, FPU64, CLB, Ethernet, EtherCAT" H 0   0   50  0001 C CNN "Description"
+F 6 "14.96" H 0   0   50  0001 C CNN "price@10"
 	3    11650 2800
 	1    0    0    -1
@@
 F 4 "LB Q39G-L2OO-35-1" H 4400 3250 50  0001 C CNN "digikey"
 F 5 "LB Q39G-L2OO-35-1" H 0   0   50  0001 C CNN "PartNumber"
+F 6 "LED BLUE DIFFUSED 0603 SMD " H 0   0   50  0001 C CNN "Description"
 	1    4400 3250
 	0    1    1    0
@@
 F 4 "LB Q39G-L2OO-35-1" H 8250 3450 50  0001 C CNN "digikey"
 F 5 "LB Q39G-L2OO-35-1" H 0   0   50  0001 C CNN "PartNumber"
+F 6 "LED BLUE DIFFUSED 0603 SMD " H 0   0   50  0001 C CNN "Description"
 	1    8250 3450
 	0    1    1    0
@@
 AR Path="/5DD4DF4C/5E22877E" Ref="C601"  Part="1"
 F 0 "C601" V 10328 7660 20  0000 L CNN
-F 1 "10nF" V 10371 7660 20  0000 L CNN
+F 1 "0.1uF" V 10371 7660 20  0000 L CNN
 F 2 "servo:C_0603_1608Metric" H 10300 7450 60  0001 C CNN
 F 3 "" H 10300 7550 60  0000 C CNN
+F 4 "CAP CER 0.1UF 16V X7R 0603 " H 0   0   50  0001 C CNN "Description"
+F 5 "CC0603KPX7R7BB104" H 0   0   50  0001 C CNN "PartNumber"
+F 6 "311-1335-1-ND" H 0   0   50  0001 C CNN "digikey"
 	1    10300 7550
 	0    1    1    0
@@
 P 3300 2600
 F 0 "J601" H 3350 3017 50  0000 C CNN
-F 1 "pinHeader" H 3350 2926 50  0000 C CNN
+F 1 "pin header 2x6 2.54" H 3350 2926 50  0000 C CNN
 F 2 "servo:PinSocket_2x06_P2.54mm_Vertical_SMD" H 3300 2600 50  0001 C CNN
 F 3 "~" H 3300 2600 50  0001 C CNN
+F 4 "Connector Header Surface Mount 12 position 0.100\" (2.54mm) " H 0   0   50  0001 C CNN "Description"
+F 5 "GBC06DABN-M30" H 0   0   50  0001 C CNN "PartNumber"
+F 6 "S2351E-06-ND" H 0   0   50  0001 C CNN "digikey"
+F 7 "1.10200" H 0   0   50  0001 C CNN "price@10"
 	1    3300 2600
 	1    0    0    -1

Commit message: stackup
Parts:
- C601, C602, C603: price@10 (none) -> 0.05800
- D603, D604: digikey LB Q39G-L2OO-35-1 -> 475-2816-1-ND; price@10 (none) -> 0.40100
- U602: value M25PX32-VMW -> SST26VF032B-104V/SM (M25PX32-VMW); Description (none) -> FLASH Memory IC 32Mb (4M x 8) SPI - Quad I/O 104MHz 8-SOIJ; PartNumber (none) -> SST26VF032B-104V/SM; digikey (none) -> SST26VF032B-104V/SM-ND; price@10 (none) -> 1.67000
- Y601: value 26mhz -> osc 25Mhz; Description (none) -> 25MHz XO (Standard) HCMOS Oscillator 3.3V Enable/Disable 4-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; PartNumber (none) -> ECS-2520S33-250-FN-TR; digikey (none) -> XC2198CT-ND; price@10 (none) -> 1.41900
Changed lines of the file:
@@
 F 4 "311-1335-1-ND" H 0   0   50  0001 C CNN "digikey"
 F 5 "CAP CER 0.1UF 16V X7R 0603 " H 0   0   50  0001 C CNN "Description"
-F 6 "" H 0   0   50  0001 C CNN "Mfr part number"
-F 7 "CC0603KPX7R7BB104" H 0   0   50  0001 C CNN "PartNumber"
+F 6 "CC0603KPX7R7BB104" H 0   0   50  0001 C CNN "PartNumber"
+F 7 "0.05800" H 0   0   50  0001 C CNN "price@10"
 	1    13900 3800
 	0    -1   -1   0
@@
 P 13900 2600
 F 0 "Y601" H 13900 2367 60  0000 C CNN
-F 1 "26mhz" H 13900 2600 50  0001 C CNN
+F 1 "osc 25Mhz" H 13900 2600 50  0001 C CNN
 F 2 "servo:Crystal_SMD_2520-4Pin_2.5x2.0mm" H 13900 2600 50  0001 C CNN
 F 3 "../doc/datasheets//ECS-2520S.pdf" H 13900 2600 50  0001 C CNN
+F 4 "25MHz XO (Standard) HCMOS Oscillator 3.3V Enable/Disable 4-SMD, No Lead " H 0   0   50  0001 C CNN "Description"
+F 5 "ECS-2520S33-250-FN-TR" H 0   0   50  0001 C CNN "PartNumber"
+F 6 "XC2198CT-ND " H 0   0   50  0001 C CNN "digikey"
+F 7 "1.41900" H 0   0   50  0001 C CNN "price@10"
 	1    13900 2600
 	-1   0    0    -1
@@
 F 2 "servo:LED_0603_1608Metric" H 4200 3050 60  0001 C CNN
 F 3 "../doc/datasheets/LB_Q39G_v1.4_9-1-15.pdf" H 4200 3050 60  0001 C CNN
-F 4 "LB Q39G-L2OO-35-1" H 4400 3250 50  0001 C CNN "digikey"
+F 4 "475-2816-1-ND" H 4400 3250 50  0001 C CNN "digikey"
 F 5 "LB Q39G-L2OO-35-1" H 0   0   50  0001 C CNN "PartNumber"
 F 6 "LED BLUE DIFFUSED 0603 SMD " H 0   0   50  0001 C CNN "Description"
+F 7 "0.40100" H 0   0   50  0001 C CNN "price@10"
 	1    4400 3250
 	0    1    1    0
@@
 F 2 "servo:LED_0603_1608Metric" H 8050 3250 60  0001 C CNN
 F 3 "../doc/datasheets/LB_Q39G_v1.4_9-1-15.pdf" H 8050 3250 60  0001 C CNN
-F 4 "LB Q39G-L2OO-35-1" H 8250 3450 50  0001 C CNN "digikey"
+F 4 "475-2816-1-ND" H 8250 3450 50  0001 C CNN "digikey"
 F 5 "LB Q39G-L2OO-35-1" H 0   0   50  0001 C CNN "PartNumber"
 F 6 "LED BLUE DIFFUSED 0603 SMD " H 0   0   50  0001 C CNN "Description"
+F 7 "0.40100" H 0   0   50  0001 C CNN "price@10"
 	1    8250 3450
 	0    1    1    0
@@
 F 4 "311-1335-1-ND" H 0   0   50  0001 C CNN "digikey"
 F 5 "CAP CER 0.1UF 16V X7R 0603 " H 0   0   50  0001 C CNN "Description"
-F 6 "" H 0   0   50  0001 C CNN "Mfr part number"
-F 7 "CC0603KPX7R7BB104" H 0   0   50  0001 C CNN "PartNumber"
+F 6 "CC0603KPX7R7BB104" H 0   0   50  0001 C CNN "PartNumber"
+F 7 "0.05800" H 0   0   50  0001 C CNN "price@10"
 	1    14300 7250
 	0    1    1    0
@@
 U 1 1 5ECE67BA
 P 13850 8000
-F 0 "U602" H 14491 8046 50  0000 L CNN
-F 1 "M25PX32-VMW" H 14491 7955 50  0000 L CNN
+F 0 "U602" H 14491 8046 39  0000 L CNN
+F 1 "SST26VF032B-104V/SM (M25PX32-VMW)" H 14491 7955 39  0000 L CNN
 F 2 "servo:SOIJ-8_5.3x5.3mm_P1.27mm" H 14500 8050 50  0001 C CNN
-F 3 "../doc/datasheets/m25px32.pdf" H 14000 7900 50  0001 C CNN
+F 3 "../doc/datasheets/SST26VF032B_nor_flash.pdf" H 14000 7900 50  0001 C CNN
+F 4 "FLASH Memory IC 32Mb (4M x 8) SPI - Quad I/O 104MHz 8-SOIJ" H 0   0   50  0001 C CNN "Description"
+F 5 "SST26VF032B-104V/SM" H 0   0   50  0001 C CNN "PartNumber"
+F 6 "SST26VF032B-104V/SM-ND " H 0   0   50  0001 C CNN "digikey"
+F 7 "1.67000" H 0   0   50  0001 C CNN "price@10"
 	1    13850 8000
 	1    0    0    -1
@@
 F 5 "CC0603KPX7R7BB104" H 0   0   50  0001 C CNN "PartNumber"
 F 6 "311-1335-1-ND" H 0   0   50  0001 C CNN "digikey"
+F 7 "0.05800" H 0   0   50  0001 C CNN "price@10"
 	1    10300 7550
 	0    1    1    0
