File: kicad/can_485.sch (KiCad schematic (older format))
At the start: 15 parts, among them J1201 tblock2x4, U1201 ISO1050, U1202 ADM2483

Commit message: added sloted holes everyware
Parts:
- removed JP1201: jumper, servo:SolderJumper-2_P1.3mm_Open_RoundedPad1.0x1.5mm, symbol servo:jumper
- removed JP1202: jumper, Jumper:SolderJumper-3_P1.3mm_Open_RoundedPad1.0x1.5mm, symbol servo:Jumper_3_Bridged12
Connections:
- net labels added: 5VI, GNDI
- net labels removed: 5VH, CAN_5VH, CAN_GND, Earth, GNDH
- wire segments 82 -> 91
Other:
- moved on the sheet: C1203

Commit message: serigrafia...
Parts:
- R1201, R1202, R1203, R1204, R1205, R1206: footprint Resistor_SMD:R_0603_1608Metric -> servo:R_0603_1608Metric
Changed lines of the file:
@@
 F 0 "R1201" H 7359 3272 20  0000 L CNN
 F 1 "10k" H 7359 3229 20  0000 L CNN
-F 2 "Resistor_SMD:R_0603_1608Metric" H 7300 3250 50  0001 C CNN
+F 2 "servo:R_0603_1608Metric" H 7300 3250 50  0001 C CNN
 F 3 "~" H 7300 3250 50  0001 C CNN
 	1    7300 3250
@@
 F 0 "R1202" H 7359 3472 20  0000 L CNN
 F 1 "1k" H 7359 3429 20  0000 L CNN
-F 2 "Resistor_SMD:R_0603_1608Metric" H 7300 3450 50  0001 C CNN
+F 2 "servo:R_0603_1608Metric" H 7300 3450 50  0001 C CNN
 F 3 "~" H 7300 3450 50  0001 C CNN
 	1    7300 3450
@@
 F 0 "R1203" H 7359 3672 20  0000 L CNN
 F 1 "10k" H 7359 3629 20  0000 L CNN
-F 2 "Resistor_SMD:R_0603_1608Metric" H 7300 3650 50  0001 C CNN
+F 2 "servo:R_0603_1608Metric" H 7300 3650 50  0001 C CNN
 F 3 "~" H 7300 3650 50  0001 C CNN
 	1    7300 3650
@@
 F 0 "R1204" H 9259 3322 20  0000 L CNN
 F 1 "10k" H 9259 3279 20  0000 L CNN
-F 2 "Resistor_SMD:R_0603_1608Metric" H 9200 3300 50  0001 C CNN
+F 2 "servo:R_0603_1608Metric" H 9200 3300 50  0001 C CNN
 F 3 "~" H 9200 3300 50  0001 C CNN
 	1    9200 3300
@@
 F 0 "R1205" H 9259 3522 20  0000 L CNN
 F 1 "1k" H 9259 3479 20  0000 L CNN
-F 2 "Resistor_SMD:R_0603_1608Metric" H 9200 3500 50  0001 C CNN
+F 2 "servo:R_0603_1608Metric" H 9200 3500 50  0001 C CNN
 F 3 "~" H 9200 3500 50  0001 C CNN
 	1    9200 3500
@@
 F 0 "R1206" H 9259 3722 20  0000 L CNN
 F 1 "10k" H 9259 3679 20  0000 L CNN
-F 2 "Resistor_SMD:R_0603_1608Metric" H 9200 3700 50  0001 C CNN
+F 2 "servo:R_0603_1608Metric" H 9200 3700 50  0001 C CNN
 F 3 "~" H 9200 3700 50  0001 C CNN
 	1    9200 3700

Commit message: serigraphi, improve of nets. change of soic 8 footprint
Parts:
- U1201: footprint Package_SO:SSO-8_6.7x9.8mm_P2.54mm_Clearance8mm -> servo:SSO-8_6.7x9.8mm_P2.54mm_Clearance8mm
- U1202: footprint Package_SO:SOIC-16W_7.5x10.3mm_P1.27mm -> servo:SOIC-16W_7.5x10.3mm_P1.27mm
Changed lines of the file:
@@
 F 0 "U1201" H 5750 4400 50  0000 C CNN
 F 1 "ISO1050" H 5750 4300 50  0000 C CNN
-F 2 "Package_SO:SSO-8_6.7x9.8mm_P2.54mm_Clearance8mm" H 5700 2950 50  0001 C CNN
+F 2 "servo:SSO-8_6.7x9.8mm_P2.54mm_Clearance8mm" H 5700 2950 50  0001 C CNN
 F 3 "../doc/datasheets/iso1050.pdf" H 5850 4450 50  0001 C CNN
 	1    5800 3650
@@
 F 0 "U1202" H 10500 4117 50  0000 C CNN
 F 1 "ADM2483" H 10500 4026 50  0000 C CNN
-F 2 "Package_SO:SOIC-16W_7.5x10.3mm_P1.27mm" H 10500 2800 50  0001 C CNN
+F 2 "servo:SOIC-16W_7.5x10.3mm_P1.27mm" H 10500 2800 50  0001 C CNN
 F 3 "../doc/datasheets/adm2483.pdf" H 9750 3400 50  0001 C CNN
 	1    10500 3500

Commit message: bom bom bom...
Parts:
- C1201, C1202, C1203, C1204: value 100nF -> 0.1uF; PartNumber (none) -> CC0603KPX7R7BB104; digikey (none) -> 311-1335-1-ND
Changed lines of the file:
@@
 AR Path="/5E21534F/5E21DD6E" Ref="C1202"  Part="1"
 F 0 "C1202" V 6828 3210 20  0000 L CNN
-F 1 "100nF" V 6871 3210 20  0000 L CNN
+F 1 "0.1uF" V 6871 3210 20  0000 L CNN
 F 2 "servo:C_0603_1608Metric" H 6800 3000 60  0001 C CNN
 F 3 "" H 6800 3100 60  0000 C CNN
+F 4 "CC0603KPX7R7BB104" H 0   0   50  0001 C CNN "PartNumber"
+F 5 "311-1335-1-ND" H 0   0   50  0001 C CNN "digikey"
 	1    6800 3100
 	0    1    1    0
@@
 AR Path="/5E21534F/5E21DD7B" Ref="C1201"  Part="1"
 F 0 "C1201" V 4828 3210 20  0000 L CNN
-F 1 "100nF" V 4871 3210 20  0000 L CNN
+F 1 "0.1uF" V 4871 3210 20  0000 L CNN
 F 2 "servo:C_0603_1608Metric" H 4800 3000 60  0001 C CNN
 F 3 "" H 4800 3100 60  0000 C CNN
+F 4 "CC0603KPX7R7BB104" H 0   0   50  0001 C CNN "PartNumber"
+F 5 "311-1335-1-ND" H 0   0   50  0001 C CNN "digikey"
 	1    4800 3100
 	0    1    1    0
@@
 AR Path="/5E21534F/5E4BC98A" Ref="C1203"  Part="1"
 F 0 "C1203" V 9478 3010 20  0000 L CNN
-F 1 "100nF" V 9521 3010 20  0000 L CNN
+F 1 "0.1uF" V 9521 3010 20  0000 L CNN
 F 2 "servo:C_0603_1608Metric" H 9450 2800 60  0001 C CNN
 F 3 "" H 9450 2900 60  0000 C CNN
+F 4 "CC0603KPX7R7BB104" H 0   0   50  0001 C CNN "PartNumber"
+F 5 "311-1335-1-ND" H 0   0   50  0001 C CNN "digikey"
 	1    9450 2900
 	0    1    1    0
@@
 AR Path="/5E21534F/5E4C0B93" Ref="C1204"  Part="1"
 F 0 "C1204" V 11678 3110 20  0000 L CNN
-F 1 "100nF" V 11721 3110 20  0000 L CNN
+F 1 "0.1uF" V 11721 3110 20  0000 L CNN
 F 2 "servo:C_0603_1608Metric" H 11650 2900 60  0001 C CNN
 F 3 "" H 11650 3000 60  0000 C CNN
+F 4 "CC0603KPX7R7BB104" H 0   0   50  0001 C CNN "PartNumber"
+F 5 "311-1335-1-ND" H 0   0   50  0001 C CNN "digikey"
 	1    11650 3000
 	0    1    1    0

Commit message: more bom...
Parts:
- C1201, C1202, C1203, C1204: Description (none) -> CAP CER 0.1UF 16V X7R 0603
- J1201: value tblock2x4 -> tblock 2x4 3.81; Description (none) -> 8 Position Terminal Block Header, Male Pins, Shrouded (4 Si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; PartNumber (none) -> 1843091; digikey (none) -> 277-6025-ND; price@10 (none) -> 5.01100
Changed lines of the file:
@@
 F 4 "CC0603KPX7R7BB104" H 0   0   50  0001 C CNN "PartNumber"
 F 5 "311-1335-1-ND" H 0   0   50  0001 C CNN "digikey"
+F 6 "CAP CER 0.1UF 16V X7R 0603 " H 0   0   50  0001 C CNN "Description"
 	1    6800 3100
 	0    1    1    0
@@
 F 4 "CC0603KPX7R7BB104" H 0   0   50  0001 C CNN "PartNumber"
 F 5 "311-1335-1-ND" H 0   0   50  0001 C CNN "digikey"
+F 6 "CAP CER 0.1UF 16V X7R 0603 " H 0   0   50  0001 C CNN "Description"
 	1    4800 3100
 	0    1    1    0
@@
 P 8050 3400
 F 0 "J1201" H 8100 3693 39  0000 C CNN
-F 1 "tblock2x4" H 8100 3618 39  0000 C CNN
+F 1 "tblock 2x4 3.81" H 8100 3618 39  0000 C CNN
 F 2 "servo:tblock02x4_3.81" H 8000 3500 50  0001 C CNN
 F 3 "../doc/datsheets/tblock2xrows.pdf" H 8100 3600 50  0001 C CNN
+F 4 "8 Position Terminal Block Header, Male Pins, Shrouded (4 Side) 0.150\" (3.81mm) 90°, Right Angle Through Hole" H 0   0   50  0001 C CNN "Description"
+F 5 "1843091" H 0   0   50  0001 C CNN "PartNumber"
+F 6 "277-6025-ND" H 0   0   50  0001 C CNN "digikey"
+F 7 "5.01100" H 0   0   50  0001 C CNN "price@10"
 	1    8050 3400
 	1    0    0    -1
@@
 F 4 "CC0603KPX7R7BB104" H 0   0   50  0001 C CNN "PartNumber"
 F 5 "311-1335-1-ND" H 0   0   50  0001 C CNN "digikey"
+F 6 "CAP CER 0.1UF 16V X7R 0603 " H 0   0   50  0001 C CNN "Description"
 	1    9450 2900
 	0    1    1    0
@@
 F 4 "CC0603KPX7R7BB104" H 0   0   50  0001 C CNN "PartNumber"
 F 5 "311-1335-1-ND" H 0   0   50  0001 C CNN "digikey"
+F 6 "CAP CER 0.1UF 16V X7R 0603 " H 0   0   50  0001 C CNN "Description"
 	1    11650 3000
 	0    1    1    0

Commit message: stackup
Parts:
- C1201, C1202, C1203, C1204: price@10 (none) -> 0.05800
- U1201: Description (none) -> 1/1 Transceiver Half CANbus 8-SOP; PartNumber (none) -> ISO1050DUB; digikey (none) -> 296-33295-5-ND; price@10 (none) -> 5.27900
- U1202: Description (none) -> RS422, RS485 Digital Isolator 2500Vrms 3 Channel 500kbps 25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; PartNumber (none) -> ADM2483BRWZ; digikey (none) -> ADM2483BRWZ-ND; price@10 (none) -> 5.59000
Changed lines of the file:
@@
 F 2 "servo:SSO-8_6.7x9.8mm_P2.54mm_Clearance8mm" H 5700 2950 50  0001 C CNN
 F 3 "../doc/datasheets/iso1050.pdf" H 5850 4450 50  0001 C CNN
+F 4 "1/1 Transceiver Half CANbus 8-SOP " H 0   0   50  0001 C CNN "Description"
+F 5 "ISO1050DUB" H 0   0   50  0001 C CNN "PartNumber"
+F 6 "296-33295-5-ND" H 0   0   50  0001 C CNN "digikey"
+F 7 "5.27900" H 0   0   50  0001 C CNN "price@10"
 	1    5800 3650
 	1    0    0    -1
@@
 F 5 "311-1335-1-ND" H 0   0   50  0001 C CNN "digikey"
 F 6 "CAP CER 0.1UF 16V X7R 0603 " H 0   0   50  0001 C CNN "Description"
+F 7 "0.05800" H 0   0   50  0001 C CNN "price@10"
 	1    6800 3100
 	0    1    1    0
@@
 F 5 "311-1335-1-ND" H 0   0   50  0001 C CNN "digikey"
 F 6 "CAP CER 0.1UF 16V X7R 0603 " H 0   0   50  0001 C CNN "Description"
+F 7 "0.05800" H 0   0   50  0001 C CNN "price@10"
 	1    4800 3100
 	0    1    1    0
@@
 F 2 "servo:SOIC-16W_7.5x10.3mm_P1.27mm" H 10500 2800 50  0001 C CNN
 F 3 "../doc/datasheets/adm2483.pdf" H 9750 3400 50  0001 C CNN
+F 4 "RS422, RS485 Digital Isolator 2500Vrms 3 Channel 500kbps 25kV/µs CMTI 16-SOIC (0.295\", 7.50mm Width) " H 0   0   50  0001 C CNN "Description"
+F 5 "ADM2483BRWZ" H 0   0   50  0001 C CNN "PartNumber"
+F 6 "ADM2483BRWZ-ND" H 0   0   50  0001 C CNN "digikey"
+F 7 "5.59000" H 0   0   50  0001 C CNN "price@10"
 	1    10500 3500
 	-1   0    0    -1
@@
 F 5 "311-1335-1-ND" H 0   0   50  0001 C CNN "digikey"
 F 6 "CAP CER 0.1UF 16V X7R 0603 " H 0   0   50  0001 C CNN "Description"
+F 7 "0.05800" H 0   0   50  0001 C CNN "price@10"
 	1    9450 2900
 	0    1    1    0
@@
 F 5 "311-1335-1-ND" H 0   0   50  0001 C CNN "digikey"
 F 6 "CAP CER 0.1UF 16V X7R 0603 " H 0   0   50  0001 C CNN "Description"
+F 7 "0.05800" H 0   0   50  0001 C CNN "price@10"
 	1    11650 3000
 	0    1    1    0

Commit message: bom copleted
Parts:
- R1201, R1203, R1204, R1206: Description (none) -> 10 kOhms ±5% 0.1W, 1/10W Chip Resistor 0603 (1608 Metric) M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; PartNumber (none) -> RC0603JR-0710KL; digikey (none) -> 311-10KGRCT-ND; price@10 (none) -> 0.01900
- R1202, R1205: Description (none) -> 1 kOhms ±5% 0.1W, 1/10W Chip Resistor 0603 (1608 Metric) Mo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; PartNumber (none) -> RC0603JR-071KL; digikey (none) -> 311-1.0KGRCT-ND; price@10 (none) -> 0.01900
Changed lines of the file:
@@
 F 2 "servo:R_0603_1608Metric" H 7300 3250 50  0001 C CNN
 F 3 "~" H 7300 3250 50  0001 C CNN
+F 4 "10 kOhms ±5% 0.1W, 1/10W Chip Resistor 0603 (1608 Metric) Moisture Resistant Thick Film " H 0   0   50  0001 C CNN "Description"
+F 5 "RC0603JR-0710KL" H 0   0   50  0001 C CNN "PartNumber"
+F 6 "311-10KGRCT-ND" H 0   0   50  0001 C CNN "digikey"
+F 7 "0.01900" H 0   0   50  0001 C CNN "price@10"
 	1    7300 3250
 	1    0    0    -1
@@
 F 2 "servo:R_0603_1608Metric" H 7300 3450 50  0001 C CNN
 F 3 "~" H 7300 3450 50  0001 C CNN
+F 4 "1 kOhms ±5% 0.1W, 1/10W Chip Resistor 0603 (1608 Metric) Moisture Resistant Thick Film " H 0   0   50  0001 C CNN "Description"
+F 5 "RC0603JR-071KL" H 0   0   50  0001 C CNN "PartNumber"
+F 6 "311-1.0KGRCT-ND" H 0   0   50  0001 C CNN "digikey"
+F 7 "0.01900" H 0   0   50  0001 C CNN "price@10"
 	1    7300 3450
 	1    0    0    -1
@@
 F 2 "servo:R_0603_1608Metric" H 7300 3650 50  0001 C CNN
 F 3 "~" H 7300 3650 50  0001 C CNN
+F 4 "10 kOhms ±5% 0.1W, 1/10W Chip Resistor 0603 (1608 Metric) Moisture Resistant Thick Film " H 0   0   50  0001 C CNN "Description"
+F 5 "RC0603JR-0710KL" H 0   0   50  0001 C CNN "PartNumber"
+F 6 "311-10KGRCT-ND" H 0   0   50  0001 C CNN "digikey"
+F 7 "0.01900" H 0   0   50  0001 C CNN "price@10"
 	1    7300 3650
 	1    0    0    -1
@@
 F 2 "servo:R_0603_1608Metric" H 9200 3300 50  0001 C CNN
 F 3 "~" H 9200 3300 50  0001 C CNN
+F 4 "10 kOhms ±5% 0.1W, 1/10W Chip Resistor 0603 (1608 Metric) Moisture Resistant Thick Film " H 0   0   50  0001 C CNN "Description"
+F 5 "RC0603JR-0710KL" H 0   0   50  0001 C CNN "PartNumber"
+F 6 "311-10KGRCT-ND" H 0   0   50  0001 C CNN "digikey"
+F 7 "0.01900" H 0   0   50  0001 C CNN "price@10"
 	1    9200 3300
 	1    0    0    -1
@@
 F 2 "servo:R_0603_1608Metric" H 9200 3500 50  0001 C CNN
 F 3 "~" H 9200 3500 50  0001 C CNN
+F 4 "1 kOhms ±5% 0.1W, 1/10W Chip Resistor 0603 (1608 Metric) Moisture Resistant Thick Film " H 0   0   50  0001 C CNN "Description"
+F 5 "RC0603JR-071KL" H 0   0   50  0001 C CNN "PartNumber"
+F 6 "311-1.0KGRCT-ND" H 0   0   50  0001 C CNN "digikey"
+F 7 "0.01900" H 0   0   50  0001 C CNN "price@10"
 	1    9200 3500
 	1    0    0    -1
@@
 F 2 "servo:R_0603_1608Metric" H 9200 3700 50  0001 C CNN
 F 3 "~" H 9200 3700 50  0001 C CNN
+F 4 "10 kOhms ±5% 0.1W, 1/10W Chip Resistor 0603 (1608 Metric) Moisture Resistant Thick Film " H 0   0   50  0001 C CNN "Description"
+F 5 "RC0603JR-0710KL" H 0   0   50  0001 C CNN "PartNumber"
+F 6 "311-10KGRCT-ND" H 0   0   50  0001 C CNN "digikey"
+F 7 "0.01900" H 0   0   50  0001 C CNN "price@10"
 	1    9200 3700
 	1    0    0    -1

Commit message: fine imprivements
Parts:
- R1202, R1205: value 1k -> 10k; Description 1 kOhms ±5% 0.1W, 1/10W Chip Resistor 0603 (1608 Metric) Mo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 -> 10 kOhms ±5% 0.1W, 1/10W Chip Resistor 0603 (1608 Metric) M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; PartNumber RC0603JR-071KL -> RC0603JR-0710KL; digikey 311-1.0KGRCT-ND -> 311-10KGRCT-ND
Other:
- note added: "for final release, remove pull-up \nand pull-down from bus, and \nreplace 10k to 120 as the Z"
Changed lines of the file:
@@
 AR Path="/5E21534F/5E47F534" Ref="R1202"  Part="1"
 F 0 "R1202" H 7359 3472 20  0000 L CNN
-F 1 "1k" H 7359 3429 20  0000 L CNN
+F 1 "10k" H 7359 3429 20  0000 L CNN
 F 2 "servo:R_0603_1608Metric" H 7300 3450 50  0001 C CNN
 F 3 "~" H 7300 3450 50  0001 C CNN
-F 4 "1 kOhms ±5% 0.1W, 1/10W Chip Resistor 0603 (1608 Metric) Moisture Resistant Thick Film " H 0   0   50  0001 C CNN "Description"
-F 5 "RC0603JR-071KL" H 0   0   50  0001 C CNN "PartNumber"
-F 6 "311-1.0KGRCT-ND" H 0   0   50  0001 C CNN "digikey"
+F 4 "10 kOhms ±5% 0.1W, 1/10W Chip Resistor 0603 (1608 Metric) Moisture Resistant Thick Film " H 0   0   50  0001 C CNN "Description"
+F 5 "RC0603JR-0710KL" H 0   0   50  0001 C CNN "PartNumber"
+F 6 "311-10KGRCT-ND" H 0   0   50  0001 C CNN "digikey"
 F 7 "0.01900" H 0   0   50  0001 C CNN "price@10"
 	1    7300 3450
@@
 AR Path="/5E21534F/5E496E84" Ref="R1205"  Part="1"
 F 0 "R1205" H 9259 3522 20  0000 L CNN
-F 1 "1k" H 9259 3479 20  0000 L CNN
+F 1 "10k" H 9259 3479 20  0000 L CNN
 F 2 "servo:R_0603_1608Metric" H 9200 3500 50  0001 C CNN
 F 3 "~" H 9200 3500 50  0001 C CNN
-F 4 "1 kOhms ±5% 0.1W, 1/10W Chip Resistor 0603 (1608 Metric) Moisture Resistant Thick Film " H 0   0   50  0001 C CNN "Description"
-F 5 "RC0603JR-071KL" H 0   0   50  0001 C CNN "PartNumber"
-F 6 "311-1.0KGRCT-ND" H 0   0   50  0001 C CNN "digikey"
+F 4 "10 kOhms ±5% 0.1W, 1/10W Chip Resistor 0603 (1608 Metric) Moisture Resistant Thick Film " H 0   0   50  0001 C CNN "Description"
+F 5 "RC0603JR-0710KL" H 0   0   50  0001 C CNN "PartNumber"
+F 6 "311-10KGRCT-ND" H 0   0   50  0001 C CNN "digikey"
 F 7 "0.01900" H 0   0   50  0001 C CNN "price@10"
 	1    9200 3500
@@
 AR Path="/5E21534F/5E4C0C89" Ref="#PWR_0102"  Part="1"
 F 0 "#PWR_0102" H 11655 3051 20  0001 C CNN
-F 1 "GND" H 11650 3042 30  0000 C CNN
+F 1 "GND" H 11650 3050 30  0000 C CNN
 F 2 "" H 11650 3200 70  0000 C CNN
 F 3 "" H 11650 3200 70  0000 C CNN
@@
 Wire Wire Line
 	9450 4100 9200 4100
+Text Notes 7900 2700 0    20   ~ 0
+for final release, remove pull-up \nand pull-down from bus, and \nreplace 10k to 120 as the Z
 $EndSCHEMATC
