File: kicad/uc_power.sch (KiCad schematic (older format))
At the start: 29 parts, among them U301 TMS320F28388DZWTS

Commit message: improving tracks under uC
Parts:
- L501, L502, L503: footprint Inductor_SMD:L_1206_3216Metric_Pad1.42x1.75mm_HandSolder -> servo:L_1206_3216Metric_Pad1.42x1.75mm_HandSolder
Changed lines of the file:
@@
 F 0 "L502" H 12000 4679 60  0000 C CNN
 F 1 "60 ohm" H 12000 4573 60  0000 C CNN
-F 2 "Inductor_SMD:L_1206_3216Metric_Pad1.42x1.75mm_HandSolder" H 11920 4310 60  0001 C CNN
+F 2 "servo:L_1206_3216Metric_Pad1.42x1.75mm_HandSolder" H 11920 4310 60  0001 C CNN
 F 3 "" H 11920 4310 60  0000 C CNN
 	1    12000 4450
@@
 F 0 "L501" H 11920 2990 60  0000 L BNN
 F 1 "60 ohm" H 11920 2810 60  0000 L BNN
-F 2 "Inductor_SMD:L_1206_3216Metric_Pad1.42x1.75mm_HandSolder" H 11920 2810 60  0001 C CNN
+F 2 "servo:L_1206_3216Metric_Pad1.42x1.75mm_HandSolder" H 11920 2810 60  0001 C CNN
 F 3 "" H 11920 2810 60  0000 C CNN
 	1    12000 2950
@@
 F 0 "L503" H 11920 5990 60  0000 L BNN
 F 1 "220 ohm" H 11920 5810 60  0000 L BNN
-F 2 "Inductor_SMD:L_1206_3216Metric_Pad1.42x1.75mm_HandSolder" H 11920 5810 60  0001 C CNN
+F 2 "servo:L_1206_3216Metric_Pad1.42x1.75mm_HandSolder" H 11920 5810 60  0001 C CNN
 F 3 "" H 11920 5810 60  0000 C CNN
 	1    12000 5950

Commit message: bom bom bom...
Parts:
- C501, C502, C503, C504, C505, C506, C507, C511, C512, C514, C515, C516, C517, C518, C519, C520, C521, C523, C524, C525: Description (none) -> CAP CER 0.1UF 16V X7R 0603; PartNumber (none) -> CC0603KPX7R7BB104; ValueDisplayed 0.1uF -> (none); digikey (none) -> 311-1335-1-ND
- C526, C530: PartNumber (none) -> GRM188R61A106ME69D; ValueDisplayed 10uF -> (none); digikey (none) -> 490-10475-1-ND
- C528, C529, C531: ValueDisplayed 2.2uF -> (none)

Commit message: more bom...
Parts:
- C526, C530: Description (none) -> 10µF ±20% 10V Ceramic Capacitor X5R 0603 (1608 Metric)
- C528, C529, C531: Description (none) -> CAP CER 2.2UF 16V X6S 0603; PartNumber (none) -> GRT188C81C225KE13D; digikey (none) -> 490-12287-2-ND
- L501, L502: value 60 ohm -> 50 ohm@100Mhz; Description (none) -> 50 Ohms @ 100MHz 1 Power Line Ferrite Bead 1206 (3216 Metri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; PartNumber (none) -> PE-1206PFB500ST; digikey (none) -> 553-2403-1-ND; price@10 (none) -> 0.14900
- L503: value 220 ohm -> 120 ohm@100mHz; Description (none) -> 120 Ohms @ 100MHz 1 Power Line Ferrite Bead 1206 (3216 Metr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; PartNumber (none) -> PE-1206PFB121ST; digikey (none) -> 553-2402-1-ND; price@10 (none) -> 0.14900
- U301: Description (none) -> 32-bit MCU with connectivity manager, 2x C28x+CLA CPU, 1.5 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; price@10 (none) -> 14.96
Changed lines of the file:
@@
 F 3 "../doc/datasheets/tms320f28388d_datasheet.pdf" H 6300 4300 50  0001 C CNN
 F 4 "TMS320F28388DZWTS" H 4700 -1800 60  0001 C CNN "PartNumber"
+F 5 "32-bit MCU with connectivity manager, 2x C28x+CLA CPU, 1.5 MB flash, FPU64, CLB, Ethernet, EtherCAT" H 0   0   50  0001 C CNN "Description"
+F 6 "14.96" H 0   0   50  0001 C CNN "price@10"
 	4    6300 4300
 	1    0    0    -1
@@
 U 1 1 5DF0B53E
 P 12000 4450
-F 0 "L502" H 12000 4679 60  0000 C CNN
-F 1 "60 ohm" H 12000 4573 60  0000 C CNN
-F 2 "servo:L_1206_3216Metric_Pad1.42x1.75mm_HandSolder" H 11920 4310 60  0001 C CNN
-F 3 "" H 11920 4310 60  0000 C CNN
+F 0 "L502" H 11950 4550 20  0000 L BNN
+F 1 "50 ohm@100Mhz" H 12050 4350 20  0000 C CNN
+F 2 "servo:L_1206_3216Metric_Pad1.42x1.75mm_HandSolder" H 11850 4450 60  0001 C CNN
+F 3 "" H 11950 4550 60  0001 C CNN
+F 4 "50 Ohms @ 100MHz 1 Power Line Ferrite Bead 1206 (3216 Metric) 3A 30mOhm " H 0   0   50  0001 C CNN "Description"
+F 5 "PE-1206PFB500ST" H 0   0   50  0001 C CNN "PartNumber"
+F 6 "553-2403-1-ND" H 0   0   50  0001 C CNN "digikey"
+F 7 "0.14900" H 0   0   50  0001 C CNN "price@10"
 	1    12000 4450
 	1    0    0    -1
@@
 U 1 1 5DF0B545
 P 12000 2950
-F 0 "L501" H 11920 2990 60  0000 L BNN
-F 1 "60 ohm" H 11920 2810 60  0000 L BNN
-F 2 "servo:L_1206_3216Metric_Pad1.42x1.75mm_HandSolder" H 11920 2810 60  0001 C CNN
-F 3 "" H 11920 2810 60  0000 C CNN
+F 0 "L501" H 11950 3050 20  0000 L BNN
+F 1 "50 ohm@100Mhz" H 12000 2850 20  0000 C CNN
+F 2 "servo:L_1206_3216Metric_Pad1.42x1.75mm_HandSolder" H 11850 2950 60  0001 C CNN
+F 3 "" H 11950 3050 60  0001 C CNN
+F 4 "50 Ohms @ 100MHz 1 Power Line Ferrite Bead 1206 (3216 Metric) 3A 30mOhm " H 0   0   50  0001 C CNN "Description"
+F 5 "PE-1206PFB500ST" H 0   0   50  0001 C CNN "PartNumber"
+F 6 "553-2403-1-ND" H 0   0   50  0001 C CNN "digikey"
+F 7 "0.14900" H 0   0   50  0001 C CNN "price@10"
 	1    12000 2950
 	1    0    0    -1
@@
 P 12000 5950
 F 0 "L503" H 11920 5990 60  0000 L BNN
-F 1 "220 ohm" H 11920 5810 60  0000 L BNN
+F 1 "120 ohm@100mHz" H 11920 5810 60  0000 L BNN
 F 2 "servo:L_1206_3216Metric_Pad1.42x1.75mm_HandSolder" H 11920 5810 60  0001 C CNN
 F 3 "" H 11920 5810 60  0000 C CNN
+F 4 "120 Ohms @ 100MHz 1 Power Line Ferrite Bead 1206 (3216 Metric) 3A 30mOhm " H 0   0   50  0001 C CNN "Description"
+F 5 "PE-1206PFB121ST" H 0   0   50  0001 C CNN "PartNumber"
+F 6 "553-2402-1-ND" H 0   0   50  0001 C CNN "digikey"
+F 7 "0.14900" H 0   0   50  0001 C CNN "price@10"
 	1    12000 5950
 	1    0    0    -1
@@
 F 4 "490-10475-1-ND" H 0   0   50  0001 C CNN "digikey"
 F 5 "GRM188R61A106ME69D " H 0   0   50  0001 C CNN "PartNumber"
+F 6 "10µF ±20% 10V Ceramic Capacitor X5R 0603 (1608 Metric) " H 0   0   50  0001 C CNN "Description"
 	1    12350 6250
 	0    -1   -1   0
@@
 F 2 "servo:C_0603_1608Metric" H 12400 3150 60  0001 C CNN
 F 3 "" H 12400 3250 60  0000 C CNN
+F 4 "CAP CER 2.2UF 16V X6S 0603 " H 0   0   50  0001 C CNN "Description"
+F 5 "GRT188C81C225KE13D" H 0   0   50  0001 C CNN "PartNumber"
+F 6 "490-12287-2-ND" H 0   0   50  0001 C CNN "digikey"
 	1    12400 3250
 	0    1    1    0
@@
 F 2 "servo:C_0603_1608Metric" H 12350 4650 60  0001 C CNN
 F 3 "" H 12350 4750 60  0000 C CNN
+F 4 "CAP CER 2.2UF 16V X6S 0603 " H 0   0   50  0001 C CNN "Description"
+F 5 "GRT188C81C225KE13D" H 0   0   50  0001 C CNN "PartNumber"
+F 6 "490-12287-2-ND" H 0   0   50  0001 C CNN "digikey"
 	1    12350 4750
 	0    1    1    0
@@
 F 2 "servo:C_0603_1608Metric" H 11650 4650 60  0001 C CNN
 F 3 "" H 11650 4750 60  0000 C CNN
+F 4 "CAP CER 2.2UF 16V X6S 0603 " H 0   0   50  0001 C CNN "Description"
+F 5 "GRT188C81C225KE13D" H 0   0   50  0001 C CNN "PartNumber"
+F 6 "490-12287-2-ND" H 0   0   50  0001 C CNN "digikey"
 	1    11650 4750
 	0    1    1    0
@@
 F 3 "../doc/datasheets/tms320f28388d_datasheet.pdf" H 3550 4750 50  0001 C CNN
 F 4 "TMS320F28388DZWTS" H 1950 4250 60  0001 C CNN "PartNumber"
+F 5 "32-bit MCU with connectivity manager, 2x C28x+CLA CPU, 1.5 MB flash, FPU64, CLB, Ethernet, EtherCAT" H 0   0   50  0001 C CNN "Description"
+F 6 "14.96" H 0   0   50  0001 C CNN "price@10"
 	5    3550 4750
 	1    0    0    -1
@@
 F 4 "490-10475-1-ND" H 0   0   50  0001 C CNN "digikey"
 F 5 "GRM188R61A106ME69D " H 0   0   50  0001 C CNN "PartNumber"
+F 6 "10µF ±20% 10V Ceramic Capacitor X5R 0603 (1608 Metric) " H 0   0   50  0001 C CNN "Description"
 	1    11600 6150
 	0    1    1    0

Commit message: stackup
Parts:
- C501, C502, C503, C504, C505, C506, C507, C511, C512, C514, C515, C516, C517, C518, C519, C520, C521, C523, C524, C525: price@10 (none) -> 0.05800
- C526, C530: price@10 (none) -> 0.15400
- C528, C529, C531: digikey 490-12287-2-ND -> 490-12287-1-ND; price@10 (none) -> 0.35500

Commit message: gerbers + pnp + bom ready
Parts:
- removed C528: 2.2uF, servo:C_0603_1608Metric, symbol servo:Capacitor
- added C508: 2.2uF, servo:C_0603_1608Metric, symbol servo:Capacitor
- added JP501, JP502, JP503: jumper, servo:SolderJumper-2_P1.3mm_Open_RoundedPad1.0x1.5mm, symbol servo:jumper
- C501, C502, C503, C504, C505, C506, C507, C511, C512, C514, C515, C516, C517, C518, C519, C520, C521, C523, C524, C525, C526, C529, C530, C531, L501, L502, L503, U301: bom_1 (none) -> 1; bom_2 (none) -> 1; bom_3 (none) -> 1
Connections:
- net labels added: 1V2uC_in, 3V3A_in, 3V3uC_in
- wire segments 259 -> 264
Other:
- moved on the sheet: C526, C530, L503

Commit message: some details on gerbers, now released
Parts:
- JP501, JP502, JP503: bom_1 (none) -> 0; bom_2 (none) -> 0
Changed lines of the file:
@@
 F 6 "-" H 8250 -2650 50  0001 C CNN "digikey"
 F 7 "0" H 8250 -2650 50  0001 C CNN "price@10"
-F 8 "" H 0   0   50  0001 C CNN "bom_1"
-F 9 "" H 0   0   50  0001 C CNN "bom_2"
+F 8 "0" H 0   0   50  0001 C CNN "bom_1"
+F 9 "0" H 0   0   50  0001 C CNN "bom_2"
 	1    11550 2950
 	1    0    0    -1
@@
 F 6 "-" H 8200 -1150 50  0001 C CNN "digikey"
 F 7 "0" H 8200 -1150 50  0001 C CNN "price@10"
-F 8 "" H 0   0   50  0001 C CNN "bom_1"
-F 9 "" H 0   0   50  0001 C CNN "bom_2"
+F 8 "0" H 0   0   50  0001 C CNN "bom_1"
+F 9 "0" H 0   0   50  0001 C CNN "bom_2"
 	1    11500 4450
 	1    0    0    -1
@@
 F 6 "-" H 8350 400 50  0001 C CNN "digikey"
 F 7 "0" H 8350 400 50  0001 C CNN "price@10"
-F 8 "" H 0   0   50  0001 C CNN "bom_1"
-F 9 "" H 0   0   50  0001 C CNN "bom_2"
+F 8 "0" H 0   0   50  0001 C CNN "bom_1"
+F 9 "0" H 0   0   50  0001 C CNN "bom_2"
 	1    11650 6000
 	1    0    0    -1
